Commit message: add tether

File: tether_description/urdf/tether_fragment.urdf (robot description, URDF)
Before this commit: robot tether_fragment, 4 links, 3 joints
Links:
- added link small_link1, mass 1.0
- added link small_link2, mass 1.0
Joints:
- removed joint Joint3
- added joint Joint_pitch: type continuous, parent small_link1, child small_link2, origin xyz=0 0 0.001, axis 0 1 0
- added joint Joint_roll: type continuous, parent tether_fragment2, child small_link1, origin xyz=0 0 0.1, axis 1 0 0
- added joint Joint_yaw: type continuous, parent small_link2, child tether_fragment3, origin xyz=0 0 0.001, axis 0 0 1
