Commit message: clean up

File: tether_description/urdf/tether.urdf.xacro (robot description, xacro)
@@ -1,4 +1,5 @@
 <?xml version="1.0" encoding="utf-8"?>
 <robot name="tether" xmlns:xacro="http://ros.org/wiki/xacro">
+    <xacro:include filename="$(find world_description)/urdf/common_properties.xacro"/>
     <xacro:include filename="$(find tether_description)/urdf/tether.xacro"/>
     <xacro:tether />

File: tether_description/urdf/tether.xacro (robot description, xacro)
@@ -1,7 +1,6 @@
 <?xml version="1.0"?>
 <robot xmlns:xacro="http://ros.org/wiki/xacro">
-    <xacro:include filename="$(find world_description)/urdf/common_properties.xacro"/>
     <!--tether model-->
-    <xacro:macro name="tether"><!--tether fragment param--><!--small link inatial--><!--link number--><!--tether world joint--><!--tether_cylinder_joint--><!-- main-->
+    <xacro:macro name="tether"><!--tether fragment param--><!--small link inatial--><!--link number--><!--tether_cylinder_joint--><!-- main-->
         <link name="tether_fragment_0">
             <visual>
@@ -10,19 +9,11 @@
                     <cylinder length="0.03" radius="0.001"/>
                 </geometry>
-                <material name="black"/>
-            </visual>
-            <inertial>
-                <mass value="0.0005"/>
-                <inertia ixx="3.7625e-08" iyy="3.7625e-08" izz="2.5e-10" ixy="0.0" ixz="0.0" iyz="0.0"/>
-            </inertial>
-        </link>
-                <!--link between world and tether-->
-        <link name="world"/>
-        <!--world joint-->
-        <joint name="joint_world" type="fixed">
-            <parent link="world"/>
-            <child link="tether_fragment_0"/>
-            <origin rpy="0 0 0" xyz="0 0 0.015"/>
-        </joint>
+                <!--material name="black"/-->
+            </visual>
+            <inertial>
+                <mass value="0.0001"/>
+                <inertia ixx="7.525e-09" iyy="7.525e-09" izz="5e-11" ixy="0.0" ixz="0.0" iyz="0.0"/>
+            </inertial>
+        </link>
         <link name="tether_fragment_1">
             <visual>
@@ -31,9 +22,9 @@
                     <cylinder length="0.03" radius="0.001"/>
                 </geometry>
-                <material name="black"/>
-            </visual>
-            <inertial>
-                <mass value="0.0005"/>
-                <inertia ixx="3.7625e-08" iyy="3.7625e-08" izz="2.5e-10" ixy="0.0" ixz="0.0" iyz="0.0"/>
+                <!--material name="black"/-->
+            </visual>
+            <inertial>
+                <mass value="0.0001"/>
+                <inertia ixx="7.525e-09" iyy="7.525e-09" izz="5e-11" ixy="0.0" ixz="0.0" iyz="0.0"/>
             </inertial>
         </link>
@@ -41,12 +32,12 @@
         <link name="small_link_1_1">
             <inertial>
-                <mass value="0.0005"/>
-                <inertia ixx="0.0005" iyy="0.0005" izz="0.0005" ixy="0.0" ixz="0.0" iyz="0.0"/>
+                <mass value="1e-05"/>
+                <inertia ixx="1e-05" iyy="1e-05" izz="1e-05" ixy="0.0" ixz="0.0" iyz="0.0"/>
             </inertial>
         </link>
         <link name="small_link_2_1">
             <inertial>
-                <mass value="0.0005"/>
-                <inertia ixx="0.0005" iyy="0.0005" izz="0.0005" ixy="0.0" ixz="0.0" iyz="0.0"/>
+                <mass value="1e-05"/>
+                <inertia ixx="1e-05" iyy="1e-05" izz="1e-05" ixy="0.0" ixz="0.0" iyz="0.0"/>
             </inertial>
         </link>
@@ -74,9 +65,9 @@
                     <cylinder length="0.03" radius="0.001"/>
                 </geometry>
-                <material name="black"/>
-            </visual>
-            <inertial>
-                <mass value="0.0005"/>
-                <inertia ixx="3.7625e-08" iyy="3.7625e-08" izz="2.5e-10" ixy="0.0" ixz="0.0" iyz="0.0"/>
+                <!--material name="black"/-->
+            </visual>
+            <inertial>
+                <mass value="0.0001"/>
+                <inertia ixx="7.525e-09" iyy="7.525e-09" izz="5e-11" ixy="0.0" ixz="0.0" iyz="0.0"/>
             </inertial>
         </link>
@@ -84,12 +75,12 @@
         <link name="small_link_1_2">
             <inertial>
-                <mass value="0.0005"/>
-                <inertia ixx="0.0005" iyy="0.0005" izz="0.0005" ixy="0.0" ixz="0.0" iyz="0.0"/>
+                <mass value="1e-05"/>
+                <inertia ixx="1e-05" iyy="1e-05" izz="1e-05" ixy="0.0" ixz="0.0" iyz="0.0"/>
             </inertial>
         </link>
         <link name="small_link_2_2">
             <inertial>
-                <mass value="0.0005"/>
-                <inertia ixx="0.0005" iyy="0.0005" izz="0.0005" ixy="0.0" ixz="0.0" iyz="0.0"/>
+                <mass value="1e-05"/>
+                <inertia ixx="1e-05" iyy="1e-05" izz="1e-05" ixy="0.0" ixz="0.0" iyz="0.0"/>
             </inertial>
         </link>
@@ -117,9 +108,9 @@
                     <cylinder length="0.03" radius="0.001"/>
                 </geometry>
-                <material name="black"/>
-            </visual>
-            <inertial>
-                <mass value="0.0005"/>
-                <inertia ixx="3.7625e-08" iyy="3.7625e-08" izz="2.5e-10" ixy="0.0" ixz="0.0" iyz="0.0"/>
+                <!--material name="black"/-->
+            </visual>
+            <inertial>
+                <mass value="0.0001"/>
+                <inertia ixx="7.525e-09" iyy="7.525e-09" izz="5e-11" ixy="0.0" ixz="0.0" iyz="0.0"/>
             </inertial>
         </link>
@@ -127,12 +118,12 @@
         <link name="small_link_1_3">
             <inertial>
-                <mass value="0.0005"/>
-                <inertia ixx="0.0005" iyy="0.0005" izz="0.0005" ixy="0.0" ixz="0.0" iyz="0.0"/>
+                <mass value="1e-05"/>
+                <inertia ixx="1e-05" iyy="1e-05" izz="1e-05" ixy="0.0" ixz="0.0" iyz="0.0"/>
             </inertial>
         </link>
         <link name="small_link_2_3">
             <inertial>
-                <mass value="0.0005"/>
-                <inertia ixx="0.0005" iyy="0.0005" izz="0.0005" ixy="0.0" ixz="0.0" iyz="0.0"/>
+                <mass value="1e-05"/>
+                <inertia ixx="1e-05" iyy="1e-05" izz="1e-05" ixy="0.0" ixz="0.0" iyz="0.0"/>
             </inertial>
         </link>
@@ -160,9 +151,9 @@
                     <cylinder length="0.03" radius="0.001"/>
                 </geometry>
-                <material name="black"/>
-            </visual>
-            <inertial>
-                <mass value="0.0005"/>
-                <inertia ixx="3.7625e-08" iyy="3.7625e-08" izz="2.5e-10" ixy="0.0" ixz="0.0" iyz="0.0"/>
+                <!--material name="black"/-->
+            </visual>
+            <inertial>
+                <mass value="0.0001"/>
+                <inertia ixx="7.525e-09" iyy="7.525e-09" izz="5e-11" ixy="0.0" ixz="0.0" iyz="0.0"/>
             </inertial>
         </link>
@@ -170,12 +161,12 @@
         <link name="small_link_1_4">
             <inertial>
-                <mass value="0.0005"/>
-                <inertia ixx="0.0005" iyy="0.0005" izz="0.0005" ixy="0.0" ixz="0.0" iyz="0.0"/>
+                <mass value="1e-05"/>
+                <inertia ixx="1e-05" iyy="1e-05" izz="1e-05" ixy="0.0" ixz="0.0" iyz="0.0"/>
             </inertial>
         </link>
         <link name="small_link_2_4">
             <inertial>
-                <mass value="0.0005"/>
-                <inertia ixx="0.0005" iyy="0.0005" izz="0.0005" ixy="0.0" ixz="0.0" iyz="0.0"/>
+                <mass value="1e-05"/>
+                <inertia ixx="1e-05" iyy="1e-05" izz="1e-05" ixy="0.0" ixz="0.0" iyz="0.0"/>
             </inertial>
         </link>
@@ -203,9 +194,9 @@
                     <cylinder length="0.03" radius="0.001"/>
                 </geometry>
-                <material name="black"/>
-            </visual>
-            <inertial>
-                <mass value="0.0005"/>
-                <inertia ixx="3.7625e-08" iyy="3.7625e-08" izz="2.5e-10" ixy="0.0" ixz="0.0" iyz="0.0"/>
+                <!--material name="black"/-->
+            </visual>
+            <inertial>
+                <mass value="0.0001"/>
+                <inertia ixx="7.525e-09" iyy="7.525e-09" izz="5e-11" ixy="0.0" ixz="0.0" iyz="0.0"/>
             </inertial>
         </link>
@@ -213,12 +204,12 @@
         <link name="small_link_1_5">
             <inertial>
-                <mass value="0.0005"/>
-                <inertia ixx="0.0005" iyy="0.0005" izz="0.0005" ixy="0.0" ixz="0.0" iyz="0.0"/>
+                <mass value="1e-05"/>
+                <inertia ixx="1e-05" iyy="1e-05" izz="1e-05" ixy="0.0" ixz="0.0" iyz="0.0"/>
             </inertial>
         </link>
         <link name="small_link_2_5">
             <inertial>
-                <mass value="0.0005"/>
-                <inertia ixx="0.0005" iyy="0.0005" izz="0.0005" ixy="0.0" ixz="0.0" iyz="0.0"/>
+                <mass value="1e-05"/>
+                <inertia ixx="1e-05" iyy="1e-05" izz="1e-05" ixy="0.0" ixz="0.0" iyz="0.0"/>
             </inertial>
         </link>
@@ -246,9 +237,9 @@
                     <cylinder length="0.03" radius="0.001"/>
                 </geometry>
-                <material name="black"/>
-            </visual>
-            <inertial>
-                <mass value="0.0005"/>
-                <inertia ixx="3.7625e-08" iyy="3.7625e-08" izz="2.5e-10" ixy="0.0" ixz="0.0" iyz="0.0"/>
+                <!--material name="black"/-->
+            </visual>
+            <inertial>
+                <mass value="0.0001"/>
+                <inertia ixx="7.525e-09" iyy="7.525e-09" izz="5e-11" ixy="0.0" ixz="0.0" iyz="0.0"/>
             </inertial>
         </link>
@@ -256,12 +247,12 @@
         <link name="small_link_1_6">
             <inertial>
-                <mass value="0.0005"/>
-                <inertia ixx="0.0005" iyy="0.0005" izz="0.0005" ixy="0.0" ixz="0.0" iyz="0.0"/>
+                <mass value="1e-05"/>
+                <inertia ixx="1e-05" iyy="1e-05" izz="1e-05" ixy="0.0" ixz="0.0" iyz="0.0"/>
             </inertial>
         </link>
         <link name="small_link_2_6">
             <inertial>
-                <mass value="0.0005"/>
-                <inertia ixx="0.0005" iyy="0.0005" izz="0.0005" ixy="0.0" ixz="0.0" iyz="0.0"/>
+                <mass value="1e-05"/>
+                <inertia ixx="1e-05" iyy="1e-05" izz="1e-05" ixy="0.0" ixz="0.0" iyz="0.0"/>
             </inertial>
         </link>
@@ -289,9 +280,9 @@
                     <cylinder length="0.03" radius="0.001"/>
                 </geometry>
-                <material name="black"/>
-            </visual>
-            <inertial>
-                <mass value="0.0005"/>
-                <inertia ixx="3.7625e-08" iyy="3.7625e-08" izz="2.5e-10" ixy="0.0" ixz="0.0" iyz="0.0"/>
+                <!--material name="black"/-->
+            </visual>
+            <inertial>
+                <mass value="0.0001"/>
+                <inertia ixx="7.525e-09" iyy="7.525e-09" izz="5e-11" ixy="0.0" ixz="0.0" iyz="0.0"/>
             </inertial>
         </link>
@@ -299,12 +290,12 @@
         <link name="small_link_1_7">
             <inertial>
-                <mass value="0.0005"/>
-                <inertia ixx="0.0005" iyy="0.0005" izz="0.0005" ixy="0.0" ixz="0.0" iyz="0.0"/>
+                <mass value="1e-05"/>
+                <inertia ixx="1e-05" iyy="1e-05" izz="1e-05" ixy="0.0" ixz="0.0" iyz="0.0"/>
             </inertial>
         </link>
         <link name="small_link_2_7">
             <inertial>
-                <mass value="0.0005"/>
-                <inertia ixx="0.0005" iyy="0.0005" izz="0.0005" ixy="0.0" ixz="0.0" iyz="0.0"/>
+                <mass value="1e-05"/>
+                <inertia ixx="1e-05" iyy="1e-05" izz="1e-05" ixy="0.0" ixz="0.0" iyz="0.0"/>
             </inertial>
         </link>
@@ -332,9 +323,9 @@
                     <cylinder length="0.03" radius="0.001"/>
                 </geometry>
-                <material name="black"/>
-            </visual>
-            <inertial>
-                <mass value="0.0005"/>
-                <inertia ixx="3.7625e-08" iyy="3.7625e-08" izz="2.5e-10" ixy="0.0" ixz="0.0" iyz="0.0"/>
+                <!--material name="black"/-->
+            </visual>
+            <inertial>
+                <mass value="0.0001"/>
+                <inertia ixx="7.525e-09" iyy="7.525e-09" izz="5e-11" ixy="0.0" ixz="0.0" iyz="0.0"/>
             </inertial>
         </link>
@@ -342,12 +333,12 @@
         <link name="small_link_1_8">
             <inertial>
-                <mass value="0.0005"/>
-                <inertia ixx="0.0005" iyy="0.0005" izz="0.0005" ixy="0.0" ixz="0.0" iyz="0.0"/>
+                <mass value="1e-05"/>
+                <inertia ixx="1e-05" iyy="1e-05" izz="1e-05" ixy="0.0" ixz="0.0" iyz="0.0"/>
             </inertial>
         </link>
         <link name="small_link_2_8">
             <inertial>
-                <mass value="0.0005"/>
-                <inertia ixx="0.0005" iyy="0.0005" izz="0.0005" ixy="0.0" ixz="0.0" iyz="0.0"/>
+                <mass value="1e-05"/>
+                <inertia ixx="1e-05" iyy="1e-05" izz="1e-05" ixy="0.0" ixz="0.0" iyz="0.0"/>
             </inertial>
         </link>
@@ -375,9 +366,9 @@
                     <cylinder length="0.03" radius="0.001"/>
                 </geometry>
-                <material name="black"/>
-            </visual>
-            <inertial>
-                <mass value="0.0005"/>
-                <inertia ixx="3.7625e-08" iyy="3.7625e-08" izz="2.5e-10" ixy="0.0" ixz="0.0" iyz="0.0"/>
+                <!--material name="black"/-->
+            </visual>
+            <inertial>
+                <mass value="0.0001"/>
+                <inertia ixx="7.525e-09" iyy="7.525e-09" izz="5e-11" ixy="0.0" ixz="0.0" iyz="0.0"/>
             </inertial>
         </link>
@@ -385,12 +376,12 @@
         <link name="small_link_1_9">
             <inertial>
-                <mass value="0.0005"/>
-                <inertia ixx="0.0005" iyy="0.0005" izz="0.0005" ixy="0.0" ixz="0.0" iyz="0.0"/>
+                <mass value="1e-05"/>
+                <inertia ixx="1e-05" iyy="1e-05" izz="1e-05" ixy="0.0" ixz="0.0" iyz="0.0"/>
             </inertial>
         </link>
         <link name="small_link_2_9">
             <inertial>
-                <mass value="0.0005"/>
-                <inertia ixx="0.0005" iyy="0.0005" izz="0.0005" ixy="0.0" ixz="0.0" iyz="0.0"/>
+                <mass value="1e-05"/>
+                <inertia ixx="1e-05" iyy="1e-05" izz="1e-05" ixy="0.0" ixz="0.0" iyz="0.0"/>
             </inertial>
         </link>
@@ -418,9 +409,9 @@
                     <cylinder length="0.03" radius="0.001"/>
                 </geometry>
-                <material name="black"/>
-            </visual>
-            <inertial>
-                <mass value="0.0005"/>
-                <inertia ixx="3.7625e-08" iyy="3.7625e-08" izz="2.5e-10" ixy="0.0" ixz="0.0" iyz="0.0"/>
+                <!--material name="black"/-->
+            </visual>
+            <inertial>
+                <mass value="0.0001"/>
+                <inertia ixx="7.525e-09" iyy="7.525e-09" izz="5e-11" ixy="0.0" ixz="0.0" iyz="0.0"/>
             </inertial>
         </link>
@@ -428,12 +419,12 @@
         <link name="small_link_1_10">
             <inertial>
-                <mass value="0.0005"/>
-                <inertia ixx="0.0005" iyy="0.0005" izz="0.0005" ixy="0.0" ixz="0.0" iyz="0.0"/>
+                <mass value="1e-05"/>
+                <inertia ixx="1e-05" iyy="1e-05" izz="1e-05" ixy="0.0" ixz="0.0" iyz="0.0"/>
             </inertial>
         </link>
         <link name="small_link_2_10">
             <inertial>
-                <mass value="0.0005"/>
-                <inertia ixx="0.0005" iyy="0.0005" izz="0.0005" ixy="0.0" ixz="0.0" iyz="0.0"/>
+                <mass value="1e-05"/>
+                <inertia ixx="1e-05" iyy="1e-05" izz="1e-05" ixy="0.0" ixz="0.0" iyz="0.0"/>
             </inertial>
         </link>
@@ -461,9 +452,9 @@
                     <cylinder length="0.03" radius="0.001"/>
                 </geometry>
-                <material name="black"/>
-            </visual>
-            <inertial>
-                <mass value="0.0005"/>
-                <inertia ixx="3.7625e-08" iyy="3.7625e-08" izz="2.5e-10" ixy="0.0" ixz="0.0" iyz="0.0"/>
+                <!--material name="black"/-->
+            </visual>
+            <inertial>
+                <mass value="0.0001"/>
+                <inertia ixx="7.525e-09" iyy="7.525e-09" izz="5e-11" ixy="0.0" ixz="0.0" iyz="0.0"/>
             </inertial>
         </link>
@@ -471,12 +462,12 @@
         <link name="small_link_1_11">
             <inertial>
-                <mass value="0.0005"/>
-                <inertia ixx="0.0005" iyy="0.0005" izz="0.0005" ixy="0.0" ixz="0.0" iyz="0.0"/>
+                <mass value="1e-05"/>
+                <inertia ixx="1e-05" iyy="1e-05" izz="1e-05" ixy="0.0" ixz="0.0" iyz="0.0"/>
             </inertial>
         </link>
         <link name="small_link_2_11">
             <inertial>
-                <mass value="0.0005"/>
-                <inertia ixx="0.0005" iyy="0.0005" izz="0.0005" ixy="0.0" ixz="0.0" iyz="0.0"/>
+                <mass value="1e-05"/>
+                <inertia ixx="1e-05" iyy="1e-05" izz="1e-05" ixy="0.0" ixz="0.0" iyz="0.0"/>
             </inertial>
         </link>
@@ -504,9 +495,9 @@
                     <cylinder length="0.03" radius="0.001"/>
                 </geometry>
-                <material name="black"/>
-            </visual>
-            <inertial>
-                <mass value="0.0005"/>
-                <inertia ixx="3.7625e-08" iyy="3.7625e-08" izz="2.5e-10" ixy="0.0" ixz="0.0" iyz="0.0"/>
+                <!--material name="black"/-->
+            </visual>
+            <inertial>
+                <mass value="0.0001"/>
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
File: tether_description/urdf/tether_fragment.xacro (robot description, xacro)
@@ -1,5 +1,4 @@
 <?xml version="1.0"?>
 <robot xmlns:xacro="http://ros.org/wiki/xacro">
-    <xacro:include filename="$(find world_description)/urdf/common_properties.xacro"/>
     <!--tether model-->
     <xacro:macro name="tether">
@@ -8,12 +7,12 @@
         {%- set cyl_r = 0.001 -%}
         {%- set cyl_l = 0.03 -%}
-        {%- set cyl_m = 0.0005 -%}
+        {%- set cyl_m = 0.0001 -%}
         {%- set cyl_i = 1/12*cyl_m*(3*cyl_r**2+cyl_l**2) -%}
         {%- set cyl_iz = 1/2*cyl_m*cyl_r**2 -%}
         <!--small link inatial-->
-        {%- set small_link_mass = 0.0005 -%}
-        {%- set small_link_ixx = 0.0005 -%}
-        {%- set small_link_iyy = 0.0005 -%}
-        {%- set small_link_izz = 0.0005 -%}
+        {%- set small_link_mass = 0.00001 -%}
+        {%- set small_link_ixx = 0.00001 -%}
+        {%- set small_link_iyy = 0.00001 -%}
+        {%- set small_link_izz = 0.00001 -%}
         {%- set small_link_ixy = 0.0 -%}
         {%- set small_link_ixz = 0.0 -%}
@@ -28,5 +27,5 @@
                     <cylinder length="{{cyl_l}}" radius="{{cyl_r}}"/>
                 </geometry>
-                <material name="black"/>
+                <!--material name="black"/-->
             </visual>
             <inertial>
@@ -35,15 +34,4 @@
             </inertial>
         </link>
-        {%- endmacro -%}
-        <!--tether world joint-->
-        {%- macro joint_world(n) -%}
-        <!--link between world and tether-->
-        <link name="world"/>
-        <!--world joint-->
-        <joint name="joint_world" type="fixed">
-            <parent link="world"/>
-            <child link="tether_fragment_{{n}}"/>
-            <origin rpy="0 0 0" xyz="0 0 {{cyl_l/2}}"/>
-        </joint>
         {%- endmacro -%}
         <!--tether_cylinder_joint-->
@@ -83,7 +71,5 @@
         {% for n in range(0,tether_fragments) -%}
             {{tether_fragment(n)}}
-            {% if n == 0 %}
-                {{joint_world(n)}}
-            {% else %}
+            {% if n != 0 %}
                 {{tether_joint(n)}}
             {% endif %}

File: ugv_description/urdf/pyramid_robotics_turtlebot3.urdf.xacro (robot description, xacro)
@@ -1,5 +1,4 @@
 <?xml version="1.0" ?>
 <robot name="turtlebot3_burger" xmlns:xacro="http://ros.org/wiki/xacro">
-    <xacro:include filename="$(find world_description)/urdf/common_properties.xacro"/>
     <xacro:include filename="$(find turtlebot3_description)/urdf/turtlebot3_burger.gazebo.xacro"/>
     <xacro:macro name="turtlebot3_burger">

File: ugv_description/urdf/ugv.urdf.xacro (robot description, xacro)
@@ -1,4 +1,5 @@
 <?xml version="1.0" encoding="utf-8"?>
 <robot name="tether" xmlns:xacro="http://ros.org/wiki/xacro">
+    <xacro:include filename="$(find world_description)/urdf/common_properties.xacro"/>
     <xacro:include filename="$(find ugv_description)/urdf/pyramid_robotics_turtlebot3.urdf.xacro"/>
     <xacro:turtlebot3_burger />

File: world_description/urdf/world.urdf.xacro (robot description, xacro)
@@ -1,6 +1,12 @@
 <?xml version="1.0" encoding="utf-8"?>
 <robot name="tether" xmlns:xacro="http://ros.org/wiki/xacro">
+    <xacro:include filename="$(find world_description)/urdf/common_properties.xacro"/>
     <xacro:include filename="$(find tether_description)/urdf/tether.xacro"/>
     <xacro:include filename="$(find ugv_description)/urdf/pyramid_robotics_turtlebot3.urdf.xacro"/>
+    <joint name="ugv_tether_joint" type="fixed">
+        <parent link="base_link"/>
+        <child link="tether_fragment_0"/>
+        <origin xyz="0.0 0.0 0.2" rpy="0 0 0"/>
+    </joint>
     <xacro:turtlebot3_burger />
     <xacro:tether />
