Commit message: fix bugs

File: tether_description/urdf/tether.xacro (robot description, xacro)
@@ -1,5 +1,4 @@
 <?xml version="1.0"?>
 <robot xmlns:xacro="http://ros.org/wiki/xacro">
-    <property name="pi" value="3.14159265359"/>
     <material name="red">
         <color rgba="1.0 0.0 0.0 1.0"/>
@@ -25,5 +24,5 @@
             <inertial>
                 <mass value="0.0005"/>
-                <inertia ixx="3.7625e-08" iyy="3.7625e-08" izz="2.5e-10" ixy="0" ixz="0" iyz="0"/>
+                <inertia ixx="3.7625e-08" iyy="3.7625e-08" izz="2.5e-10" ixy="0.0" ixz="0.0" iyz="0.0"/>
             </inertial>
         </link>
@@ -45,5 +44,5 @@
             <inertial>
                 <mass value="0.0005"/>
-                <inertia ixx="3.7625e-08" iyy="3.7625e-08" izz="2.5e-10" ixy="0" ixz="0" iyz="0"/>
+                <inertia ixx="3.7625e-08" iyy="3.7625e-08" izz="2.5e-10" ixy="0.0" ixz="0.0" iyz="0.0"/>
             </inertial>
         </link>
@@ -52,5 +51,5 @@
             <inertial>
                 <mass value="0.0005"/>
-                <inertia ixx="0.0005" iyy="0.0005" izz="0.0005" ixy="0.0" iyz="0.0" izz="0.0"/>
+                <inertia ixx="0.0005" iyy="0.0005" izz="0.0005" ixy="0.0" ixz="0.0" iyz="0.0"/>
             </inertial>
         </link>
@@ -58,5 +57,5 @@
             <inertial>
                 <mass value="0.0005"/>
-                <inertia ixx="0.0005" iyy="0.0005" izz="0.0005" ixy="0.0" iyz="0.0" izz="0.0"/>
+                <inertia ixx="0.0005" iyy="0.0005" izz="0.0005" ixy="0.0" ixz="0.0" iyz="0.0"/>
             </inertial>
         </link>
@@ -86,5 +85,5 @@
             <inertial>
                 <mass value="0.0005"/>
-                <inertia ixx="3.7625e-08" iyy="3.7625e-08" izz="2.5e-10" ixy="0" ixz="0" iyz="0"/>
+                <inertia ixx="3.7625e-08" iyy="3.7625e-08" izz="2.5e-10" ixy="0.0" ixz="0.0" iyz="0.0"/>
             </inertial>
         </link>
@@ -93,5 +92,5 @@
             <inertial>
                 <mass value="0.0005"/>
-                <inertia ixx="0.0005" iyy="0.0005" izz="0.0005" ixy="0.0" iyz="0.0" izz="0.0"/>
+                <inertia ixx="0.0005" iyy="0.0005" izz="0.0005" ixy="0.0" ixz="0.0" iyz="0.0"/>
             </inertial>
         </link>
@@ -99,5 +98,5 @@
             <inertial>
                 <mass value="0.0005"/>
-                <inertia ixx="0.0005" iyy="0.0005" izz="0.0005" ixy="0.0" iyz="0.0" izz="0.0"/>
+                <inertia ixx="0.0005" iyy="0.0005" izz="0.0005" ixy="0.0" ixz="0.0" iyz="0.0"/>
             </inertial>
         </link>
@@ -127,5 +126,5 @@
             <inertial>
                 <mass value="0.0005"/>
-                <inertia ixx="3.7625e-08" iyy="3.7625e-08" izz="2.5e-10" ixy="0" ixz="0" iyz="0"/>
+                <inertia ixx="3.7625e-08" iyy="3.7625e-08" izz="2.5e-10" ixy="0.0" ixz="0.0" iyz="0.0"/>
             </inertial>
         </link>
@@ -134,5 +133,5 @@
             <inertial>
                 <mass value="0.0005"/>
-                <inertia ixx="0.0005" iyy="0.0005" izz="0.0005" ixy="0.0" iyz="0.0" izz="0.0"/>
+                <inertia ixx="0.0005" iyy="0.0005" izz="0.0005" ixy="0.0" ixz="0.0" iyz="0.0"/>
             </inertial>
         </link>
@@ -140,5 +139,5 @@
             <inertial>
                 <mass value="0.0005"/>
-                <inertia ixx="0.0005" iyy="0.0005" izz="0.0005" ixy="0.0" iyz="0.0" izz="0.0"/>
+                <inertia ixx="0.0005" iyy="0.0005" izz="0.0005" ixy="0.0" ixz="0.0" iyz="0.0"/>
             </inertial>
         </link>
@@ -168,5 +167,5 @@
             <inertial>
                 <mass value="0.0005"/>
-                <inertia ixx="3.7625e-08" iyy="3.7625e-08" izz="2.5e-10" ixy="0" ixz="0" iyz="0"/>
+                <inertia ixx="3.7625e-08" iyy="3.7625e-08" izz="2.5e-10" ixy="0.0" ixz="0.0" iyz="0.0"/>
             </inertial>
         </link>
@@ -175,5 +174,5 @@
             <inertial>
                 <mass value="0.0005"/>
-                <inertia ixx="0.0005" iyy="0.0005" izz="0.0005" ixy="0.0" iyz="0.0" izz="0.0"/>
+                <inertia ixx="0.0005" iyy="0.0005" izz="0.0005" ixy="0.0" ixz="0.0" iyz="0.0"/>
             </inertial>
         </link>
@@ -181,5 +180,5 @@
             <inertial>
                 <mass value="0.0005"/>
-                <inertia ixx="0.0005" iyy="0.0005" izz="0.0005" ixy="0.0" iyz="0.0" izz="0.0"/>
+                <inertia ixx="0.0005" iyy="0.0005" izz="0.0005" ixy="0.0" ixz="0.0" iyz="0.0"/>
             </inertial>
         </link>
@@ -209,5 +208,5 @@
             <inertial>
                 <mass value="0.0005"/>
-                <inertia ixx="3.7625e-08" iyy="3.7625e-08" izz="2.5e-10" ixy="0" ixz="0" iyz="0"/>
+                <inertia ixx="3.7625e-08" iyy="3.7625e-08" izz="2.5e-10" ixy="0.0" ixz="0.0" iyz="0.0"/>
             </inertial>
         </link>
@@ -216,5 +215,5 @@
             <inertial>
                 <mass value="0.0005"/>
-                <inertia ixx="0.0005" iyy="0.0005" izz="0.0005" ixy="0.0" iyz="0.0" izz="0.0"/>
+                <inertia ixx="0.0005" iyy="0.0005" izz="0.0005" ixy="0.0" ixz="0.0" iyz="0.0"/>
             </inertial>
         </link>
@@ -222,5 +221,5 @@
             <inertial>
                 <mass value="0.0005"/>
-                <inertia ixx="0.0005" iyy="0.0005" izz="0.0005" ixy="0.0" iyz="0.0" izz="0.0"/>
+                <inertia ixx="0.0005" iyy="0.0005" izz="0.0005" ixy="0.0" ixz="0.0" iyz="0.0"/>
             </inertial>
         </link>
@@ -250,5 +249,5 @@
             <inertial>
                 <mass value="0.0005"/>
-                <inertia ixx="3.7625e-08" iyy="3.7625e-08" izz="2.5e-10" ixy="0" ixz="0" iyz="0"/>
+                <inertia ixx="3.7625e-08" iyy="3.7625e-08" izz="2.5e-10" ixy="0.0" ixz="0.0" iyz="0.0"/>
             </inertial>
         </link>
@@ -257,5 +256,5 @@
             <inertial>
                 <mass value="0.0005"/>
-                <inertia ixx="0.0005" iyy="0.0005" izz="0.0005" ixy="0.0" iyz="0.0" izz="0.0"/>
+                <inertia ixx="0.0005" iyy="0.0005" izz="0.0005" ixy="0.0" ixz="0.0" iyz="0.0"/>
             </inertial>
         </link>
@@ -263,5 +262,5 @@
             <inertial>
                 <mass value="0.0005"/>
-                <inertia ixx="0.0005" iyy="0.0005" izz="0.0005" ixy="0.0" iyz="0.0" izz="0.0"/>
+                <inertia ixx="0.0005" iyy="0.0005" izz="0.0005" ixy="0.0" ixz="0.0" iyz="0.0"/>
             </inertial>
         </link>
@@ -291,5 +290,5 @@
             <inertial>
                 <mass value="0.0005"/>
-                <inertia ixx="3.7625e-08" iyy="3.7625e-08" izz="2.5e-10" ixy="0" ixz="0" iyz="0"/>
+                <inertia ixx="3.7625e-08" iyy="3.7625e-08" izz="2.5e-10" ixy="0.0" ixz="0.0" iyz="0.0"/>
             </inertial>
         </link>
@@ -298,5 +297,5 @@
             <inertial>
                 <mass value="0.0005"/>
-                <inertia ixx="0.0005" iyy="0.0005" izz="0.0005" ixy="0.0" iyz="0.0" izz="0.0"/>
+                <inertia ixx="0.0005" iyy="0.0005" izz="0.0005" ixy="0.0" ixz="0.0" iyz="0.0"/>
             </inertial>
         </link>
@@ -304,5 +303,5 @@
             <inertial>
                 <mass value="0.0005"/>
-                <inertia ixx="0.0005" iyy="0.0005" izz="0.0005" ixy="0.0" iyz="0.0" izz="0.0"/>
+                <inertia ixx="0.0005" iyy="0.0005" izz="0.0005" ixy="0.0" ixz="0.0" iyz="0.0"/>
             </inertial>
         </link>
@@ -332,5 +331,5 @@
             <inertial>
                 <mass value="0.0005"/>
-                <inertia ixx="3.7625e-08" iyy="3.7625e-08" izz="2.5e-10" ixy="0" ixz="0" iyz="0"/>
+                <inertia ixx="3.7625e-08" iyy="3.7625e-08" izz="2.5e-10" ixy="0.0" ixz="0.0" iyz="0.0"/>
             </inertial>
         </link>
@@ -339,5 +338,5 @@
             <inertial>
                 <mass value="0.0005"/>
-                <inertia ixx="0.0005" iyy="0.0005" izz="0.0005" ixy="0.0" iyz="0.0" izz="0.0"/>
+                <inertia ixx="0.0005" iyy="0.0005" izz="0.0005" ixy="0.0" ixz="0.0" iyz="0.0"/>
             </inertial>
         </link>
@@ -345,5 +344,5 @@
             <inertial>
                 <mass value="0.0005"/>
-                <inertia ixx="0.0005" iyy="0.0005" izz="0.0005" ixy="0.0" iyz="0.0" izz="0.0"/>
+                <inertia ixx="0.0005" iyy="0.0005" izz="0.0005" ixy="0.0" ixz="0.0" iyz="0.0"/>
             </inertial>
         </link>
@@ -373,5 +372,5 @@
             <inertial>
                 <mass value="0.0005"/>
-                <inertia ixx="3.7625e-08" iyy="3.7625e-08" izz="2.5e-10" ixy="0" ixz="0" iyz="0"/>
+                <inertia ixx="3.7625e-08" iyy="3.7625e-08" izz="2.5e-10" ixy="0.0" ixz="0.0" iyz="0.0"/>
             </inertial>
         </link>
@@ -380,5 +379,5 @@
             <inertial>
                 <mass value="0.0005"/>
-                <inertia ixx="0.0005" iyy="0.0005" izz="0.0005" ixy="0.0" iyz="0.0" izz="0.0"/>
+                <inertia ixx="0.0005" iyy="0.0005" izz="0.0005" ixy="0.0" ixz="0.0" iyz="0.0"/>
             </inertial>
         </link>
@@ -386,5 +385,5 @@
             <inertial>
                 <mass value="0.0005"/>
-                <inertia ixx="0.0005" iyy="0.0005" izz="0.0005" ixy="0.0" iyz="0.0" izz="0.0"/>
+                <inertia ixx="0.0005" iyy="0.0005" izz="0.0005" ixy="0.0" ixz="0.0" iyz="0.0"/>
             </inertial>
         </link>
@@ -414,5 +413,5 @@
             <inertial>
                 <mass value="0.0005"/>
-                <inertia ixx="3.7625e-08" iyy="3.7625e-08" izz="2.5e-10" ixy="0" ixz="0" iyz="0"/>
+                <inertia ixx="3.7625e-08" iyy="3.7625e-08" izz="2.5e-10" ixy="0.0" ixz="0.0" iyz="0.0"/>
             </inertial>
         </link>
@@ -421,5 +420,5 @@
             <inertial>
                 <mass value="0.0005"/>
-                <inertia ixx="0.0005" iyy="0.0005" izz="0.0005" ixy="0.0" iyz="0.0" izz="0.0"/>
+                <inertia ixx="0.0005" iyy="0.0005" izz="0.0005" ixy="0.0" ixz="0.0" iyz="0.0"/>
             </inertial>
         </link>
@@ -427,5 +426,5 @@
             <inertial>
                 <mass value="0.0005"/>
-                <inertia ixx="0.0005" iyy="0.0005" izz="0.0005" ixy="0.0" iyz="0.0" izz="0.0"/>
+                <inertia ixx="0.0005" iyy="0.0005" izz="0.0005" ixy="0.0" ixz="0.0" iyz="0.0"/>
             </inertial>
         </link>
@@ -455,5 +454,5 @@
             <inertial>
                 <mass value="0.0005"/>
-                <inertia ixx="3.7625e-08" iyy="3.7625e-08" izz="2.5e-10" ixy="0" ixz="0" iyz="0"/>
+                <inertia ixx="3.7625e-08" iyy="3.7625e-08" izz="2.5e-10" ixy="0.0" ixz="0.0" iyz="0.0"/>
             </inertial>
         </link>
@@ -462,5 +461,5 @@
             <inertial>
                 <mass value="0.0005"/>
-                <inertia ixx="0.0005" iyy="0.0005" izz="0.0005" ixy="0.0" iyz="0.0" izz="0.0"/>
+                <inertia ixx="0.0005" iyy="0.0005" izz="0.0005" ixy="0.0" ixz="0.0" iyz="0.0"/>
             </inertial>
         </link>
@@ -468,5 +467,5 @@
             <inertial>
                 <mass value="0.0005"/>
-                <inertia ixx="0.0005" iyy="0.0005" izz="0.0005" ixy="0.0" iyz="0.0" izz="0.0"/>
+                <inertia ixx="0.0005" iyy="0.0005" izz="0.0005" ixy="0.0" ixz="0.0" iyz="0.0"/>
             </inertial>
         </link>
@@ -496,5 +495,5 @@
             <inertial>
                 <mass value="0.0005"/>
-                <inertia ixx="3.7625e-08" iyy="3.7625e-08" izz="2.5e-10" ixy="0" ixz="0" iyz="0"/>
+                <inertia ixx="3.7625e-08" iyy="3.7625e-08" izz="2.5e-10" ixy="0.0" ixz="0.0" iyz="0.0"/>
             </inertial>
         </link>
@@ -503,5 +502,5 @@
             <inertial>
                 <mass value="0.0005"/>
-                <inertia ixx="0.0005" iyy="0.0005" izz="0.0005" ixy="0.0" iyz="0.0" izz="0.0"/>
+                <inertia ixx="0.0005" iyy="0.0005" izz="0.0005" ixy="0.0" ixz="0.0" iyz="0.0"/>
             </inertial>
         </link>
@@ -509,5 +508,5 @@
             <inertial>
                 <mass value="0.0005"/>
-                <inertia ixx="0.0005" iyy="0.0005" izz="0.0005" ixy="0.0" iyz="0.0" izz="0.0"/>
+                <inertia ixx="0.0005" iyy="0.0005" izz="0.0005" ixy="0.0" ixz="0.0" iyz="0.0"/>
             </inertial>
         </link>
@@ -537,5 +536,5 @@
             <inertial>
                 <mass value="0.0005"/>
-                <inertia ixx="3.7625e-08" iyy="3.7625e-08" izz="2.5e-10" ixy="0" ixz="0" iyz="0"/>
+                <inertia ixx="3.7625e-08" iyy="3.7625e-08" izz="2.5e-10" ixy="0.0" ixz="0.0" iyz="0.0"/>
             </inertial>
         </link>
@@ -544,5 +543,5 @@
             <inertial>
                 <mass value="0.0005"/>
-                <inertia ixx="0.0005" iyy="0.0005" izz="0.0005" ixy="0.0" iyz="0.0" izz="0.0"/>
+                <inertia ixx="0.0005" iyy="0.0005" izz="0.0005" ixy="0.0" ixz="0.0" iyz="0.0"/>
             </inertial>
         </link>
@@ -550,5 +549,5 @@
             <inertial>
                 <mass value="0.0005"/>
-                <inertia ixx="0.0005" iyy="0.0005" izz="0.0005" ixy="0.0" iyz="0.0" izz="0.0"/>
+                <inertia ixx="0.0005" iyy="0.0005" izz="0.0005" ixy="0.0" ixz="0.0" iyz="0.0"/>
             </inertial>
         </link>
@@ -578,5 +577,5 @@
             <inertial>
                 <mass value="0.0005"/>
-                <inertia ixx="3.7625e-08" iyy="3.7625e-08" izz="2.5e-10" ixy="0" ixz="0" iyz="0"/>
+                <inertia ixx="3.7625e-08" iyy="3.7625e-08" izz="2.5e-10" ixy="0.0" ixz="0.0" iyz="0.0"/>
             </inertial>
         </link>
@@ -585,5 +584,5 @@
             <inertial>
                 <mass value="0.0005"/>
-                <inertia ixx="0.0005" iyy="0.0005" izz="0.0005" ixy="0.0" iyz="0.0" izz="0.0"/>
+                <inertia ixx="0.0005" iyy="0.0005" izz="0.0005" ixy="0.0" ixz="0.0" iyz="0.0"/>
             </inertial>
         </link>
@@ -591,5 +590,5 @@
             <inertial>
                 <mass value="0.0005"/>
-                <inertia ixx="0.0005" iyy="0.0005" izz="0.0005" ixy="0.0" iyz="0.0" izz="0.0"/>
+                <inertia ixx="0.0005" iyy="0.0005" izz="0.0005" ixy="0.0" ixz="0.0" iyz="0.0"/>
             </inertial>
         </link>
@@ -619,5 +618,5 @@
             <inertial>
                 <mass value="0.0005"/>
-                <inertia ixx="3.7625e-08" iyy="3.7625e-08" izz="2.5e-10" ixy="0" ixz="0" iyz="0"/>
+                <inertia ixx="3.7625e-08" iyy="3.7625e-08" izz="2.5e-10" ixy="0.0" ixz="0.0" iyz="0.0"/>
             </inertial>
         </link>
@@ -626,5 +625,5 @@
             <inertial>
                 <mass value="0.0005"/>
-                <inertia ixx="0.0005" iyy="0.0005" izz="0.0005" ixy="0.0" iyz="0.0" izz="0.0"/>
+                <inertia ixx="0.0005" iyy="0.0005" izz="0.0005" ixy="0.0" ixz="0.0" iyz="0.0"/>
             </inertial>
         </link>
@@ -632,5 +631,5 @@
             <inertial>
                 <mass value="0.0005"/>
-                <inertia ixx="0.0005" iyy="0.0005" izz="0.0005" ixy="0.0" iyz="0.0" izz="0.0"/>
+                <inertia ixx="0.0005" iyy="0.0005" izz="0.0005" ixy="0.0" ixz="0.0" iyz="0.0"/>
             </inertial>
         </link>
@@ -660,5 +659,5 @@
             <inertial>
                 <mass value="0.0005"/>
-                <inertia ixx="3.7625e-08" iyy="3.7625e-08" izz="2.5e-10" ixy="0" ixz="0" iyz="0"/>
+                <inertia ixx="3.7625e-08" iyy="3.7625e-08" izz="2.5e-10" ixy="0.0" ixz="0.0" iyz="0.0"/>
             </inertial>
         </link>
@@ -667,5 +666,5 @@
             <inertial>
                 <mass value="0.0005"/>
-                <inertia ixx="0.0005" iyy="0.0005" izz="0.0005" ixy="0.0" iyz="0.0" izz="0.0"/>
+                <inertia ixx="0.0005" iyy="0.0005" izz="0.0005" ixy="0.0" ixz="0.0" iyz="0.0"/>
             </inertial>
         </link>
@@ -673,5 +672,5 @@
             <inertial>
                 <mass value="0.0005"/>
-                <inertia ixx="0.0005" iyy="0.0005" izz="0.0005" ixy="0.0" iyz="0.0" izz="0.0"/>
+                <inertia ixx="0.0005" iyy="0.0005" izz="0.0005" ixy="0.0" ixz="0.0" iyz="0.0"/>
             </inertial>
         </link>
@@ -701,5 +700,5 @@
             <inertial>
                 <mass value="0.0005"/>
-                <inertia ixx="3.7625e-08" iyy="3.7625e-08" izz="2.5e-10" ixy="0" ixz="0" iyz="0"/>
+                <inertia ixx="3.7625e-08" iyy="3.7625e-08" izz="2.5e-10" ixy="0.0" ixz="0.0" iyz="0.0"/>
             </inertial>
         </link>
@@ -708,5 +707,5 @@
             <inertial>
                 <mass value="0.0005"/>
-                <inertia ixx="0.0005" iyy="0.0005" izz="0.0005" ixy="0.0" iyz="0.0" izz="0.0"/>
+                <inertia ixx="0.0005" iyy="0.0005" izz="0.0005" ixy="0.0" ixz="0.0" iyz="0.0"/>
             </inertial>
         </link>
@@ -714,5 +713,5 @@
             <inertial>
                 <mass value="0.0005"/>
-                <inertia ixx="0.0005" iyy="0.0005" izz="0.0005" ixy="0.0" iyz="0.0" izz="0.0"/>
+                <inertia ixx="0.0005" iyy="0.0005" izz="0.0005" ixy="0.0" ixz="0.0" iyz="0.0"/>
             </inertial>
         </link>
@@ -742,5 +741,5 @@
             <inertial>
                 <mass value="0.0005"/>
-                <inertia ixx="3.7625e-08" iyy="3.7625e-08" izz="2.5e-10" ixy="0" ixz="0" iyz="0"/>
+                <inertia ixx="3.7625e-08" iyy="3.7625e-08" izz="2.5e-10" ixy="0.0" ixz="0.0" iyz="0.0"/>
             </inertial>
         </link>
@@ -749,5 +748,5 @@
             <inertial>
                 <mass value="0.0005"/>
-                <inertia ixx="0.0005" iyy="0.0005" izz="0.0005" ixy="0.0" iyz="0.0" izz="0.0"/>
+                <inertia ixx="0.0005" iyy="0.0005" izz="0.0005" ixy="0.0" ixz="0.0" iyz="0.0"/>
             </inertial>
         </link>
@@ -755,5 +754,5 @@
             <inertial>
                 <mass value="0.0005"/>
-                <inertia ixx="0.0005" iyy="0.0005" izz="0.0005" ixy="0.0" iyz="0.0" izz="0.0"/>
+                <inertia ixx="0.0005" iyy="0.0005" izz="0.0005" ixy="0.0" ixz="0.0" iyz="0.0"/>
             </inertial>
         </link>
@@ -783,5 +782,5 @@
             <inertial>
                 <mass value="0.0005"/>
-                <inertia ixx="3.7625e-08" iyy="3.7625e-08" izz="2.5e-10" ixy="0" ixz="0" iyz="0"/>
+                <inertia ixx="3.7625e-08" iyy="3.7625e-08" izz="2.5e-10" ixy="0.0" ixz="0.0" iyz="0.0"/>
             </inertial>
         </link>
@@ -790,5 +789,5 @@
             <inertial>
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
File: tether_description/urdf/tether_fragment.xacro (robot description, xacro)
@@ -1,5 +1,4 @@
 <?xml version="1.0"?>
 <robot xmlns:xacro="http://ros.org/wiki/xacro">
-    <property name="pi" value="3.14159265359"/>
     <material name="red">
         <color rgba="1.0 0.0 0.0 1.0"/>
@@ -29,6 +28,6 @@
         {%- set small_link_izz = 0.0005 -%}
         {%- set small_link_ixy = 0.0 -%}
+        {%- set small_link_ixz = 0.0 -%}
         {%- set small_link_iyz = 0.0 -%}
-        {%- set small_link_izx = 0.0 -%}
         <!--link number-->
         {%- set tether_fragments = 50 -%}
@@ -43,5 +42,5 @@
             <inertial>
                 <mass value="{{cyl_m}}"/>
-                <inertia ixx="{{cyl_i}}" iyy="{{cyl_i}}" izz="{{cyl_iz}}" ixy="0" ixz="0" iyz="0"/>
+                <inertia ixx="{{cyl_i}}" iyy="{{cyl_i}}" izz="{{cyl_iz}}" ixy="0.0" ixz="0.0" iyz="0.0"/>
             </inertial>
         </link>
@@ -64,5 +63,5 @@
             <inertial>
                 <mass value="{{small_link_mass}}"/>
-                <inertia ixx="{{small_link_ixx}}" iyy="{{small_link_iyy}}" izz="{{small_link_izz}}" ixy="{{small_link_ixy}}" iyz="{{small_link_iyz}}" izz="{{small_link_izx}}"/>
+                <inertia ixx="{{small_link_ixx}}" iyy="{{small_link_iyy}}" izz="{{small_link_izz}}" ixy="{{small_link_ixy}}" ixz="{{small_link_ixz}}" iyz="{{small_link_iyz}}"/>
             </inertial>
         </link>
@@ -70,5 +69,5 @@
             <inertial>
                 <mass value="{{small_link_mass}}"/>
-                <inertia ixx="{{small_link_ixx}}" iyy="{{small_link_iyy}}" izz="{{small_link_izz}}" ixy="{{small_link_ixy}}" iyz="{{small_link_iyz}}" izz="{{small_link_izx}}"/>
+                <inertia ixx="{{small_link_ixx}}" iyy="{{small_link_iyy}}" izz="{{small_link_izz}}" ixy="{{small_link_ixy}}" ixz="{{small_link_ixz}}" iyz="{{small_link_iyz}}"/>
             </inertial>
         </link>
@@ -99,9 +98,9 @@
             {% endif %}
         {% endfor -%}
+        <gazebo>
+            <plugin name="gazebo_ros_control" filename="libgazebo_ros_control.so">
+                <robotNamespace>tether</robotNamespace>
+            </plugin>
+        </gazebo>
     </xacro:macro>
-    <gazebo>
-        <plugin name="gazebo_ros_control" filename="libgazebo_ros_control.so">
-            <robotNamespace>tether</robotNamespace>
-        </plugin>
-    </gazebo>
 </robot>
