Commit message: fix bugs & clean up

File: tether_description/urdf/tether.xacro (robot description, xacro)
@@ -17,4 +17,5 @@
         <link name="tether_fragment_0">
             <visual>
+                <origin rpy="0 0 0" xyz="0 0 0.015"/>
                 <geometry>
                     <cylinder length="0.03" radius="0.001"/>
@@ -33,8 +34,9 @@
             <parent link="world"/>
             <child link="tether_fragment_0"/>
-            <origin rpy="0 0 0" xyz="0 0 -0.015"/>
+            <origin rpy="0 0 0" xyz="0 0 0.015"/>
         </joint>
         <link name="tether_fragment_1">
             <visual>
+                <origin rpy="0 0 0" xyz="0 0 0.015"/>
                 <geometry>
                     <cylinder length="0.03" radius="0.001"/>
@@ -62,4 +64,5 @@
         <!--tether fragment joint-->
         <joint name="joint_1_1" type="continuous">
+            <origin rpy="0 0 0" xyz="0 0 0.03"/>
             <parent link="tether_fragment_0"/>
             <child link="small_link_1_1"/>
@@ -78,4 +81,5 @@
         <link name="tether_fragment_2">
             <visual>
+                <origin rpy="0 0 0" xyz="0 0 0.015"/>
                 <geometry>
                     <cylinder length="0.03" radius="0.001"/>
@@ -103,4 +107,5 @@
         <!--tether fragment joint-->
         <joint name="joint_1_2" type="continuous">
+            <origin rpy="0 0 0" xyz="0 0 0.03"/>
             <parent link="tether_fragment_1"/>
             <child link="small_link_1_2"/>
@@ -119,4 +124,5 @@
         <link name="tether_fragment_3">
             <visual>
+                <origin rpy="0 0 0" xyz="0 0 0.015"/>
                 <geometry>
                     <cylinder length="0.03" radius="0.001"/>
@@ -144,4 +150,5 @@
         <!--tether fragment joint-->
         <joint name="joint_1_3" type="continuous">
+            <origin rpy="0 0 0" xyz="0 0 0.03"/>
             <parent link="tether_fragment_2"/>
             <child link="small_link_1_3"/>
@@ -160,4 +167,5 @@
         <link name="tether_fragment_4">
             <visual>
+                <origin rpy="0 0 0" xyz="0 0 0.015"/>
                 <geometry>
                     <cylinder length="0.03" radius="0.001"/>
@@ -185,4 +193,5 @@
         <!--tether fragment joint-->
         <joint name="joint_1_4" type="continuous">
+            <origin rpy="0 0 0" xyz="0 0 0.03"/>
             <parent link="tether_fragment_3"/>
             <child link="small_link_1_4"/>
@@ -201,4 +210,5 @@
         <link name="tether_fragment_5">
             <visual>
+                <origin rpy="0 0 0" xyz="0 0 0.015"/>
                 <geometry>
                     <cylinder length="0.03" radius="0.001"/>
@@ -226,4 +236,5 @@
         <!--tether fragment joint-->
         <joint name="joint_1_5" type="continuous">
+            <origin rpy="0 0 0" xyz="0 0 0.03"/>
             <parent link="tether_fragment_4"/>
             <child link="small_link_1_5"/>
@@ -242,4 +253,5 @@
         <link name="tether_fragment_6">
             <visual>
+                <origin rpy="0 0 0" xyz="0 0 0.015"/>
                 <geometry>
                     <cylinder length="0.03" radius="0.001"/>
@@ -267,4 +279,5 @@
         <!--tether fragment joint-->
         <joint name="joint_1_6" type="continuous">
+            <origin rpy="0 0 0" xyz="0 0 0.03"/>
             <parent link="tether_fragment_5"/>
             <child link="small_link_1_6"/>
@@ -283,4 +296,5 @@
         <link name="tether_fragment_7">
             <visual>
+                <origin rpy="0 0 0" xyz="0 0 0.015"/>
                 <geometry>
                     <cylinder length="0.03" radius="0.001"/>
@@ -308,4 +322,5 @@
         <!--tether fragment joint-->
         <joint name="joint_1_7" type="continuous">
+            <origin rpy="0 0 0" xyz="0 0 0.03"/>
             <parent link="tether_fragment_6"/>
             <child link="small_link_1_7"/>
@@ -324,4 +339,5 @@
         <link name="tether_fragment_8">
             <visual>
+                <origin rpy="0 0 0" xyz="0 0 0.015"/>
                 <geometry>
                     <cylinder length="0.03" radius="0.001"/>
@@ -349,4 +365,5 @@
         <!--tether fragment joint-->
         <joint name="joint_1_8" type="continuous">
+            <origin rpy="0 0 0" xyz="0 0 0.03"/>
             <parent link="tether_fragment_7"/>
             <child link="small_link_1_8"/>
@@ -365,4 +382,5 @@
         <link name="tether_fragment_9">
             <visual>
+                <origin rpy="0 0 0" xyz="0 0 0.015"/>
                 <geometry>
                     <cylinder length="0.03" radius="0.001"/>
@@ -390,4 +408,5 @@
         <!--tether fragment joint-->
         <joint name="joint_1_9" type="continuous">
+            <origin rpy="0 0 0" xyz="0 0 0.03"/>
             <parent link="tether_fragment_8"/>
             <child link="small_link_1_9"/>
@@ -406,4 +425,5 @@
         <link name="tether_fragment_10">
             <visual>
+                <origin rpy="0 0 0" xyz="0 0 0.015"/>
                 <geometry>
                     <cylinder length="0.03" radius="0.001"/>
@@ -431,4 +451,5 @@
         <!--tether fragment joint-->
         <joint name="joint_1_10" type="continuous">
+            <origin rpy="0 0 0" xyz="0 0 0.03"/>
             <parent link="tether_fragment_9"/>
             <child link="small_link_1_10"/>
@@ -447,4 +468,5 @@
         <link name="tether_fragment_11">
             <visual>
+                <origin rpy="0 0 0" xyz="0 0 0.015"/>
                 <geometry>
                     <cylinder length="0.03" radius="0.001"/>
@@ -472,4 +494,5 @@
         <!--tether fragment joint-->
         <joint name="joint_1_11" type="continuous">
+            <origin rpy="0 0 0" xyz="0 0 0.03"/>
             <parent link="tether_fragment_10"/>
             <child link="small_link_1_11"/>
@@ -488,4 +511,5 @@
         <link name="tether_fragment_12">
             <visual>
+                <origin rpy="0 0 0" xyz="0 0 0.015"/>
                 <geometry>
                     <cylinder length="0.03" radius="0.001"/>
@@ -513,4 +537,5 @@
         <!--tether fragment joint-->
         <joint name="joint_1_12" type="continuous">
+            <origin rpy="0 0 0" xyz="0 0 0.03"/>
             <parent link="tether_fragment_11"/>
             <child link="small_link_1_12"/>
@@ -529,4 +554,5 @@
         <link name="tether_fragment_13">
             <visual>
+                <origin rpy="0 0 0" xyz="0 0 0.015"/>
                 <geometry>
                     <cylinder length="0.03" radius="0.001"/>
@@ -554,4 +580,5 @@
         <!--tether fragment joint-->
         <joint name="joint_1_13" type="continuous">
+            <origin rpy="0 0 0" xyz="0 0 0.03"/>
             <parent link="tether_fragment_12"/>
             <child link="small_link_1_13"/>
@@ -570,4 +597,5 @@
         <link name="tether_fragment_14">
             <visual>
+                <origin rpy="0 0 0" xyz="0 0 0.015"/>
                 <geometry>
                     <cylinder length="0.03" radius="0.001"/>
@@ -595,4 +623,5 @@
         <!--tether fragment joint-->
         <joint name="joint_1_14" type="continuous">
+            <origin rpy="0 0 0" xyz="0 0 0.03"/>
             <parent link="tether_fragment_13"/>
             <child link="small_link_1_14"/>
@@ -611,4 +640,5 @@
         <link name="tether_fragment_15">
             <visual>
+                <origin rpy="0 0 0" xyz="0 0 0.015"/>
                 <geometry>
                     <cylinder length="0.03" radius="0.001"/>
@@ -636,4 +666,5 @@
         <!--tether fragment joint-->
         <joint name="joint_1_15" type="continuous">
+            <origin rpy="0 0 0" xyz="0 0 0.03"/>
             <parent link="tether_fragment_14"/>
             <child link="small_link_1_15"/>
@@ -652,4 +683,5 @@
         <link name="tether_fragment_16">
             <visual>
+                <origin rpy="0 0 0" xyz="0 0 0.015"/>
                 <geometry>
                     <cylinder length="0.03" radius="0.001"/>
@@ -677,4 +709,5 @@
         <!--tether fragment joint-->
         <joint name="joint_1_16" type="continuous">
+            <origin rpy="0 0 0" xyz="0 0 0.03"/>
             <parent link="tether_fragment_15"/>
             <child link="small_link_1_16"/>
@@ -693,4 +726,5 @@
         <link name="tether_fragment_17">
             <visual>
+                <origin rpy="0 0 0" xyz="0 0 0.015"/>
                 <geometry>
                     <cylinder length="0.03" radius="0.001"/>
@@ -718,4 +752,5 @@
         <!--tether fragment joint-->
         <joint name="joint_1_17" type="continuous">
+            <origin rpy="0 0 0" xyz="0 0 0.03"/>
             <parent link="tether_fragment_16"/>
             <child link="small_link_1_17"/>
@@ -734,4 +769,5 @@
         <link name="tether_fragment_18">
             <visual>
+                <origin rpy="0 0 0" xyz="0 0 0.015"/>
                 <geometry>
                     <cylinder length="0.03" radius="0.001"/>
@@ -759,4 +795,5 @@
         <!--tether fragment joint-->
         <joint name="joint_1_18" type="continuous">
+            <origin rpy="0 0 0" xyz="0 0 0.03"/>
             <parent link="tether_fragment_17"/>
             <child link="small_link_1_18"/>
@@ -775,4 +812,5 @@
         <link name="tether_fragment_19">
             <visual>
+                <origin rpy="0 0 0" xyz="0 0 0.015"/>
                 <geometry>
                     <cylinder length="0.03" radius="0.001"/>
@@ -800,4 +838,5 @@
         <!--tether fragment joint-->
         <joint name="joint_1_19" type="continuous">
+            <origin rpy="0 0 0" xyz="0 0 0.03"/>
             <parent link="tether_fragment_18"/>
             <child link="small_link_1_19"/>
@@ -816,4 +855,5 @@
         <link name="tether_fragment_20">
             <visual>
+                <origin rpy="0 0 0" xyz="0 0 0.015"/>
                 <geometry>
                     <cylinder length="0.03" radius="0.001"/>
@@ -841,4 +881,5 @@
         <!--tether fragment joint-->
         <joint name="joint_1_20" type="continuous">
+            <origin rpy="0 0 0" xyz="0 0 0.03"/>
             <parent link="tether_fragment_19"/>
             <child link="small_link_1_20"/>
@@ -857,4 +898,5 @@
         <link name="tether_fragment_21">
             <visual>
+                <origin rpy="0 0 0" xyz="0 0 0.015"/>
                 <geometry>
                     <cylinder length="0.03" radius="0.001"/>
@@ -882,4 +924,5 @@
         <!--tether fragment joint-->
         <joint name="joint_1_21" type="continuous">
+            <origin rpy="0 0 0" xyz="0 0 0.03"/>
             <parent link="tether_fragment_20"/>
             <child link="small_link_1_21"/>
@@ -898,4 +941,5 @@
         <link name="tether_fragment_22">
             <visual>
+                <origin rpy="0 0 0" xyz="0 0 0.015"/>
                 <geometry>
                     <cylinder length="0.03" radius="0.001"/>
@@ -923,4 +967,5 @@
         <!--tether fragment joint-->
         <joint name="joint_1_22" type="continuous">
+            <origin rpy="0 0 0" xyz="0 0 0.03"/>
             <parent link="tether_fragment_21"/>
             <child link="small_link_1_22"/>
@@ -939,4 +984,5 @@
         <link name="tether_fragment_23">
             <visual>
+                <origin rpy="0 0 0" xyz="0 0 0.015"/>
                 <geometry>
                     <cylinder length="0.03" radius="0.001"/>
@@ -964,4 +1010,5 @@
         <!--tether fragment joint-->
         <joint name="joint_1_23" type="continuous">
+            <origin rpy="0 0 0" xyz="0 0 0.03"/>
             <parent link="tether_fragment_22"/>
             <child link="small_link_1_23"/>
@@ -980,4 +1027,5 @@
         <link name="tether_fragment_24">
             <visual>
+                <origin rpy="0 0 0" xyz="0 0 0.015"/>
                 <geometry>
                     <cylinder length="0.03" radius="0.001"/>
@@ -1005,4 +1053,5 @@
         <!--tether fragment joint-->
         <joint name="joint_1_24" type="continuous">
+            <origin rpy="0 0 0" xyz="0 0 0.03"/>
             <parent link="tether_fragment_23"/>
             <child link="small_link_1_24"/>
@@ -1021,4 +1070,5 @@
         <link name="tether_fragment_25">
             <visual>
+                <origin rpy="0 0 0" xyz="0 0 0.015"/>
                 <geometry>
                     <cylinder length="0.03" radius="0.001"/>
@@ -1046,4 +1096,5 @@
         <!--tether fragment joint-->
         <joint name="joint_1_25" type="continuous">
+            <origin rpy="0 0 0" xyz="0 0 0.03"/>
             <parent link="tether_fragment_24"/>
             <child link="small_link_1_25"/>
@@ -1062,4 +1113,5 @@
         <link name="tether_fragment_26">
             <visual>
+                <origin rpy="0 0 0" xyz="0 0 0.015"/>
                 <geometry>
                     <cylinder length="0.03" radius="0.001"/>
@@ -1087,4 +1139,5 @@
         <!--tether fragment joint-->
         <joint name="joint_1_26" type="continuous">
+            <origin rpy="0 0 0" xyz="0 0 0.03"/>
             <parent link="tether_fragment_25"/>
             <child link="small_link_1_26"/>
@@ -1103,4 +1156,5 @@
         <link name="tether_fragment_27">
             <visual>
+                <origin rpy="0 0 0" xyz="0 0 0.015"/>
                 <geometry>
                     <cylinder length="0.03" radius="0.001"/>
@@ -1128,4 +1182,5 @@
         <!--tether fragment joint-->
         <joint name="joint_1_27" type="continuous">
+            <origin rpy="0 0 0" xyz="0 0 0.03"/>
             <parent link="tether_fragment_26"/>
             <child link="small_link_1_27"/>
@@ -1144,4 +1199,5 @@
         <link name="tether_fragment_28">
             <visual>
+                <origin rpy="0 0 0" xyz="0 0 0.015"/>
                 <geometry>
                     <cylinder length="0.03" radius="0.001"/>
@@ -1169,4 +1225,5 @@
         <!--tether fragment joint-->
         <joint name="joint_1_28" type="continuous">
+            <origin rpy="0 0 0" xyz="0 0 0.03"/>
             <parent link="tether_fragment_27"/>
             <child link="small_link_1_28"/>
@@ -1185,4 +1242,5 @@
         <link name="tether_fragment_29">
             <visual>
+                <origin rpy="0 0 0" xyz="0 0 0.015"/>
                 <geometry>
                     <cylinder length="0.03" radius="0.001"/>
@@ -1210,4 +1268,5 @@
         <!--tether fragment joint-->
         <joint name="joint_1_29" type="continuous">
+            <origin rpy="0 0 0" xyz="0 0 0.03"/>
             <parent link="tether_fragment_28"/>
             <child link="small_link_1_29"/>
@@ -1226,4 +1285,5 @@
         <link name="tether_fragment_30">
             <visual>
+                <origin rpy="0 0 0" xyz="0 0 0.015"/>
                 <geometry>
                     <cylinder length="0.03" radius="0.001"/>
@@ -1251,4 +1311,5 @@
         <!--tether fragment joint-->
         <joint name="joint_1_30" type="continuous">
+            <origin rpy="0 0 0" xyz="0 0 0.03"/>
             <parent link="tether_fragment_29"/>
             <child link="small_link_1_30"/>
@@ -1267,4 +1328,5 @@
         <link name="tether_fragment_31">
             <visual>
+                <origin rpy="0 0 0" xyz="0 0 0.015"/>
                 <geometry>
                     <cylinder length="0.03" radius="0.001"/>
@@ -1292,4 +1354,5 @@
         <!--tether fragment joint-->
         <joint name="joint_1_31" type="continuous">
+            <origin rpy="0 0 0" xyz="0 0 0.03"/>
             <parent link="tether_fragment_30"/>
             <child link="small_link_1_31"/>
@@ -1308,4 +1371,5 @@
         <link name="tether_fragment_32">
             <visual>
+                <origin rpy="0 0 0" xyz="0 0 0.015"/>
                 <geometry>
                     <cylinder length="0.03" radius="0.001"/>
@@ -1333,4 +1397,5 @@
         <!--tether fragment joint-->
         <joint name="joint_1_32" type="continuous">
+            <origin rpy="0 0 0" xyz="0 0 0.03"/>
             <parent link="tether_fragment_31"/>
             <child link="small_link_1_32"/>
@@ -1349,4 +1414,5 @@
         <link name="tether_fragment_33">
             <visual>
+                <origin rpy="0 0 0" xyz="0 0 0.015"/>
                 <geometry>
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
File: tether_description/urdf/tether_fragment.xacro (robot description, xacro)
@@ -35,4 +35,5 @@
         <link name="tether_fragment_{{n}}">
             <visual>
+                <origin rpy="0 0 0" xyz="0 0 {{cyl_l/2}}"/>
                 <geometry>
                     <cylinder length="{{cyl_l}}" radius="{{cyl_r}}"/>
@@ -54,5 +55,5 @@
             <parent link="world"/>
             <child link="tether_fragment_{{n}}"/>
-            <origin rpy="0 0 0" xyz="0 0 -{{cyl_l/2}}"/>
+            <origin rpy="0 0 0" xyz="0 0 {{cyl_l/2}}"/>
         </joint>
         {%- endmacro -%}
@@ -74,4 +75,5 @@
         <!--tether fragment joint-->
         <joint name="joint_1_{{n}}" type="continuous">
+            <origin rpy="0 0 0" xyz="0 0 {{cyl_l}}"/>
             <parent link="tether_fragment_{{n-1}}"/>
             <child link="small_link_1_{{n}}"/>

Commit message: add descriptions

File: tether_description/urdf/tether.xacro (robot description, xacro)
@@ -1,16 +1,5 @@
 <?xml version="1.0"?>
 <robot xmlns:xacro="http://ros.org/wiki/xacro">
-    <material name="red">
-        <color rgba="1.0 0.0 0.0 1.0"/>
-    </material>
-    <material name="green">
-        <color rgba="0.0 1.0 0.0 1.0"/>
-    </material>
-    <material name="blue">
-        <color rgba="0.0 0.0 1.0 1.0"/>
-    </material>
-    <material name="black">
-        <color rgba="0 0 0 1"/>
-    </material>
+    <xacro:include filename="$(find world_description)/urdf/common_properties.xacro"/>
     <!--tether model-->
     <xacro:macro name="tether"><!--tether fragment param--><!--small link inatial--><!--link number--><!--tether world joint--><!--tether_cylinder_joint--><!-- main-->

File: tether_description/urdf/tether_fragment.xacro (robot description, xacro)
@@ -1,16 +1,5 @@
 <?xml version="1.0"?>
 <robot xmlns:xacro="http://ros.org/wiki/xacro">
-    <material name="red">
-        <color rgba="1.0 0.0 0.0 1.0"/>
-    </material>
-    <material name="green">
-        <color rgba="0.0 1.0 0.0 1.0"/>
-    </material>
-    <material name="blue">
-        <color rgba="0.0 0.0 1.0 1.0"/>
-    </material>
-    <material name="black">
-        <color rgba="0 0 0 1"/>
-    </material>
+    <xacro:include filename="$(find world_description)/urdf/common_properties.xacro"/>
     <!--tether model-->
     <xacro:macro name="tether">

File: world_description/urdf/world.urdf.xacro (robot description, xacro)
@@ -2,4 +2,6 @@
 <robot name="tether" xmlns:xacro="http://ros.org/wiki/xacro">
     <xacro:include filename="$(find tether_description)/urdf/tether.xacro"/>
+    <xacro:include filename="$(find ugv_description)/urdf/pyramid_robotics_turtlebot3.urdf.xacro"/>
+    <xacro:turtlebot3_burger />
     <xacro:tether />
 </robot>
