Commit message: fix bugs

File: tether_description/urdf/tether.xacro (robot description, xacro)
@@ -2,5 +2,6 @@
 <robot xmlns:xacro="http://ros.org/wiki/xacro">
     <!--tether model-->
-    <xacro:macro name="tether"><!--tether fragment param--><!--small link inatial--><!--link number--><!--tether_cylinder_joint--><!-- main-->
+    <xacro:macro name="tether">
+        <!--tether fragment param--><!--small link inatial--><!--link number--><!--tether_cylinder_joint--><!-- main-->
         <link name="tether_fragment_0">
             <visual>

File: tether_description/urdf/tether_fragment.xacro (robot description, xacro)
@@ -3,5 +3,4 @@
     <!--tether model-->
     <xacro:macro name="tether">
-        {%- set pi = 3.141592 -%}
         <!--tether fragment param-->
         {%- set cyl_r = 0.001 -%}

File: world_description/urdf/common_properties.xacro (robot description, xacro)
@@ -1,34 +1,35 @@
 <?xml version="1.0" ?>
 <robot name="xacro_properties" xmlns:xacro="http://ros.org/wiki/xacro">
-  <!-- Init colour -->
-  <material name="black">
-      <color rgba="0.0 0.0 0.0 1.0"/>
-  </material>
-  <material name="dark">
-    <color rgba="0.3 0.3 0.3 1.0"/>
-  </material>
-  <material name="light_black">
-    <color rgba="0.4 0.4 0.4 1.0"/>
-  </material>
-  <material name="blue">
-    <color rgba="0.0 0.0 0.8 1.0"/>
-  </material>
-  <material name="green">
-    <color rgba="0.0 0.8 0.0 1.0"/>
-  </material>
-  <material name="grey">
-    <color rgba="0.5 0.5 0.5 1.0"/>
-  </material>
-  <material name="orange">
-    <color rgba="${255/255} ${108/255} ${10/255} 1.0"/>
-  </material>
-  <material name="brown">
-    <color rgba="${222/255} ${207/255} ${195/255} 1.0"/>
-  </material>
-  <material name="red">
-    <color rgba="0.8 0.0 0.0 1.0"/>
-  </material>
-  <material name="white">
-    <color rgba="1.0 1.0 1.0 1.0"/>
-  </material>
+    <xacro:property name="pi" value="3.1415926535897931" />
+    <!-- Init colour -->
+    <material name="black">
+        <color rgba="0.0 0.0 0.0 1.0"/>
+    </material>
+    <material name="dark">
+        <color rgba="0.3 0.3 0.3 1.0"/>
+    </material>
+    <material name="light_black">
+        <color rgba="0.4 0.4 0.4 1.0"/>
+    </material>
+    <material name="blue">
+        <color rgba="0.0 0.0 0.8 1.0"/>
+    </material>
+    <material name="green">
+        <color rgba="0.0 0.8 0.0 1.0"/>
+    </material>
+    <material name="grey">
+        <color rgba="0.5 0.5 0.5 1.0"/>
+    </material>
+    <material name="orange">
+        <color rgba="${255/255} ${108/255} ${10/255} 1.0"/>
+    </material>
+    <material name="brown">
+        <color rgba="${222/255} ${207/255} ${195/255} 1.0"/>
+    </material>
+    <material name="red">
+        <color rgba="0.8 0.0 0.0 1.0"/>
+    </material>
+    <material name="white">
+        <color rgba="1.0 1.0 1.0 1.0"/>
+    </material>
 </robot>

File: world_description/urdf/world.urdf.xacro (robot description, xacro)
@@ -4,10 +4,54 @@
     <xacro:include filename="$(find tether_description)/urdf/tether.xacro"/>
     <xacro:include filename="$(find ugv_description)/urdf/pyramid_robotics_turtlebot3.urdf.xacro"/>
-    <joint name="ugv_tether_joint" type="fixed">
-        <parent link="base_link"/>
+    <link name="ugv_tether_link_1">
+        <inertial>
+            <mass value="0.00001"/>
+            <inertia ixx="0.00001" iyy="0.00001" izz="0.00001" ixy="0.00001" ixz="0.00001" iyz="0.00001"/>
+        </inertial>
+    </link>
+    <link name="ugv_tether_link_2">
+        <inertial>
+            <mass value="0.00001"/>
+            <inertia ixx="0.00001" iyy="0.00001" izz="0.00001" ixy="0.00001" ixz="0.00001" iyz="0.00001"/>
+        </inertial>
+    </link>
+    <joint name="ugv_tether_joint_1" type="continuous">
+        <parent link="base_footprint"/>
+        <child link="ugv_tether_link_1"/>
+        <axis xyz="1 0 0" />
+    </joint>
+    <joint name="ugv_tether_joint_2" type="continuous">
+        <parent link="ugv_tether_link_1"/>
+        <child link="ugv_tether_link_2"/>
+        <axis xyz="0 1 0" />
+    </joint>
+    <joint name="ugv_tether_joint_3" type="continuous">
+        <parent link="ugv_tether_link_2"/>
         <child link="tether_fragment_0"/>
-        <origin xyz="0.0 0.0 0.2" rpy="0 0 0"/>
+        <axis xyz="0 0 1" />
+        <origin xyz="0.0 0.0 0.0" rpy="0 ${pi/2} 0"/>
     </joint>
+    <joint name="uav_tether_joint_4" type="fixed">
+        <parent link="tether_fragment_49"/>
+        <child link="pesudo_uav"/>
+    </joint>
+    <link name="pesudo_uav">
+        <visual>
+            <geometry>
+                <box size="0.1 0.1 0.1"/>
+            </geometry>
+        </visual>
+        <inertial>
+            <mass value="1"/>
+            <inertia ixx="1" iyy="1" izz="1" ixy="1" ixz="1" iyz="1"/>
+        </inertial>
+        <collision>
+            <geometry>
+                <box size="0.1 0.1 0.1"/>
+            </geometry>
+        </collision>
+    </link>
     <xacro:turtlebot3_burger />
+    <!--xacro:turtlebot3_burger prefix="2nd" /-->
     <xacro:tether />
 </robot>

Commit message: add hovering_example with tether

File: tether_description/urdf/tether.xacro (robot description, xacro)
@@ -6,26 +6,26 @@
         <link name="tether_fragment_0">
             <visual>
-                <origin rpy="0 0 0" xyz="0 0 0.015"/>
-                <geometry>
-                    <cylinder length="0.03" radius="0.001"/>
-                </geometry>
-                <!--material name="black"/-->
-            </visual>
-            <inertial>
-                <mass value="0.0001"/>
-                <inertia ixx="7.525e-09" iyy="7.525e-09" izz="5e-11" ixy="0.0" ixz="0.0" iyz="0.0"/>
+                <origin rpy="0 0 0" xyz="0 0 0.05"/>
+                <geometry>
+                    <cylinder length="0.1" radius="0.001"/>
+                </geometry>
+                <!--material name="black"/-->
+            </visual>
+            <inertial>
+                <mass value="0.0001"/>
+                <inertia ixx="8.33583333333e-08" iyy="8.33583333333e-08" izz="5e-11" ixy="0.0" ixz="0.0" iyz="0.0"/>
             </inertial>
         </link>
         <link name="tether_fragment_1">
             <visual>
-                <origin rpy="0 0 0" xyz="0 0 0.015"/>
-                <geometry>
-                    <cylinder length="0.03" radius="0.001"/>
-                </geometry>
-                <!--material name="black"/-->
-            </visual>
-            <inertial>
-                <mass value="0.0001"/>
-                <inertia ixx="7.525e-09" iyy="7.525e-09" izz="5e-11" ixy="0.0" ixz="0.0" iyz="0.0"/>
+                <origin rpy="0 0 0" xyz="0 0 0.05"/>
+                <geometry>
+                    <cylinder length="0.1" radius="0.001"/>
+                </geometry>
+                <!--material name="black"/-->
+            </visual>
+            <inertial>
+                <mass value="0.0001"/>
+                <inertia ixx="8.33583333333e-08" iyy="8.33583333333e-08" izz="5e-11" ixy="0.0" ixz="0.0" iyz="0.0"/>
             </inertial>
         </link>
@@ -45,5 +45,5 @@
         <!--tether fragment joint-->
         <joint name="joint_1_1" type="continuous">
-            <origin rpy="0 0 0" xyz="0 0 0.03"/>
+            <origin rpy="0 0 0" xyz="0 0 0.1"/>
             <parent link="tether_fragment_0"/>
             <child link="small_link_1_1"/>
@@ -62,13 +62,13 @@
         <link name="tether_fragment_2">
             <visual>
-                <origin rpy="0 0 0" xyz="0 0 0.015"/>
-                <geometry>
-                    <cylinder length="0.03" radius="0.001"/>
-                </geometry>
-                <!--material name="black"/-->
-            </visual>
-            <inertial>
-                <mass value="0.0001"/>
-                <inertia ixx="7.525e-09" iyy="7.525e-09" izz="5e-11" ixy="0.0" ixz="0.0" iyz="0.0"/>
+                <origin rpy="0 0 0" xyz="0 0 0.05"/>
+                <geometry>
+                    <cylinder length="0.1" radius="0.001"/>
+                </geometry>
+                <!--material name="black"/-->
+            </visual>
+            <inertial>
+                <mass value="0.0001"/>
+                <inertia ixx="8.33583333333e-08" iyy="8.33583333333e-08" izz="5e-11" ixy="0.0" ixz="0.0" iyz="0.0"/>
             </inertial>
         </link>
@@ -88,5 +88,5 @@
         <!--tether fragment joint-->
         <joint name="joint_1_2" type="continuous">
-            <origin rpy="0 0 0" xyz="0 0 0.03"/>
+            <origin rpy="0 0 0" xyz="0 0 0.1"/>
             <parent link="tether_fragment_1"/>
             <child link="small_link_1_2"/>
@@ -105,13 +105,13 @@
         <link name="tether_fragment_3">
             <visual>
-                <origin rpy="0 0 0" xyz="0 0 0.015"/>
-                <geometry>
-                    <cylinder length="0.03" radius="0.001"/>
-                </geometry>
-                <!--material name="black"/-->
-            </visual>
-            <inertial>
-                <mass value="0.0001"/>
-                <inertia ixx="7.525e-09" iyy="7.525e-09" izz="5e-11" ixy="0.0" ixz="0.0" iyz="0.0"/>
+                <origin rpy="0 0 0" xyz="0 0 0.05"/>
+                <geometry>
+                    <cylinder length="0.1" radius="0.001"/>
+                </geometry>
+                <!--material name="black"/-->
+            </visual>
+            <inertial>
+                <mass value="0.0001"/>
+                <inertia ixx="8.33583333333e-08" iyy="8.33583333333e-08" izz="5e-11" ixy="0.0" ixz="0.0" iyz="0.0"/>
             </inertial>
         </link>
@@ -131,5 +131,5 @@
         <!--tether fragment joint-->
         <joint name="joint_1_3" type="continuous">
-            <origin rpy="0 0 0" xyz="0 0 0.03"/>
+            <origin rpy="0 0 0" xyz="0 0 0.1"/>
             <parent link="tether_fragment_2"/>
             <child link="small_link_1_3"/>
@@ -148,13 +148,13 @@
         <link name="tether_fragment_4">
             <visual>
-                <origin rpy="0 0 0" xyz="0 0 0.015"/>
-                <geometry>
-                    <cylinder length="0.03" radius="0.001"/>
-                </geometry>
-                <!--material name="black"/-->
-            </visual>
-            <inertial>
-                <mass value="0.0001"/>
-                <inertia ixx="7.525e-09" iyy="7.525e-09" izz="5e-11" ixy="0.0" ixz="0.0" iyz="0.0"/>
+                <origin rpy="0 0 0" xyz="0 0 0.05"/>
+                <geometry>
+                    <cylinder length="0.1" radius="0.001"/>
+                </geometry>
+                <!--material name="black"/-->
+            </visual>
+            <inertial>
+                <mass value="0.0001"/>
+                <inertia ixx="8.33583333333e-08" iyy="8.33583333333e-08" izz="5e-11" ixy="0.0" ixz="0.0" iyz="0.0"/>
             </inertial>
         </link>
@@ -174,5 +174,5 @@
         <!--tether fragment joint-->
         <joint name="joint_1_4" type="continuous">
-            <origin rpy="0 0 0" xyz="0 0 0.03"/>
+            <origin rpy="0 0 0" xyz="0 0 0.1"/>
             <parent link="tether_fragment_3"/>
             <child link="small_link_1_4"/>
@@ -191,13 +191,13 @@
         <link name="tether_fragment_5">
             <visual>
-                <origin rpy="0 0 0" xyz="0 0 0.015"/>
-                <geometry>
-                    <cylinder length="0.03" radius="0.001"/>
-                </geometry>
-                <!--material name="black"/-->
-            </visual>
-            <inertial>
-                <mass value="0.0001"/>
-                <inertia ixx="7.525e-09" iyy="7.525e-09" izz="5e-11" ixy="0.0" ixz="0.0" iyz="0.0"/>
+                <origin rpy="0 0 0" xyz="0 0 0.05"/>
+                <geometry>
+                    <cylinder length="0.1" radius="0.001"/>
+                </geometry>
+                <!--material name="black"/-->
+            </visual>
+            <inertial>
+                <mass value="0.0001"/>
+                <inertia ixx="8.33583333333e-08" iyy="8.33583333333e-08" izz="5e-11" ixy="0.0" ixz="0.0" iyz="0.0"/>
             </inertial>
         </link>
@@ -217,5 +217,5 @@
         <!--tether fragment joint-->
         <joint name="joint_1_5" type="continuous">
-            <origin rpy="0 0 0" xyz="0 0 0.03"/>
+            <origin rpy="0 0 0" xyz="0 0 0.1"/>
             <parent link="tether_fragment_4"/>
             <child link="small_link_1_5"/>
@@ -234,13 +234,13 @@
         <link name="tether_fragment_6">
             <visual>
-                <origin rpy="0 0 0" xyz="0 0 0.015"/>
-                <geometry>
-                    <cylinder length="0.03" radius="0.001"/>
-                </geometry>
-                <!--material name="black"/-->
-            </visual>
-            <inertial>
-                <mass value="0.0001"/>
-                <inertia ixx="7.525e-09" iyy="7.525e-09" izz="5e-11" ixy="0.0" ixz="0.0" iyz="0.0"/>
+                <origin rpy="0 0 0" xyz="0 0 0.05"/>
+                <geometry>
+                    <cylinder length="0.1" radius="0.001"/>
+                </geometry>
+                <!--material name="black"/-->
+            </visual>
+            <inertial>
+                <mass value="0.0001"/>
+                <inertia ixx="8.33583333333e-08" iyy="8.33583333333e-08" izz="5e-11" ixy="0.0" ixz="0.0" iyz="0.0"/>
             </inertial>
         </link>
@@ -260,5 +260,5 @@
         <!--tether fragment joint-->
         <joint name="joint_1_6" type="continuous">
-            <origin rpy="0 0 0" xyz="0 0 0.03"/>
+            <origin rpy="0 0 0" xyz="0 0 0.1"/>
             <parent link="tether_fragment_5"/>
             <child link="small_link_1_6"/>
@@ -277,13 +277,13 @@
         <link name="tether_fragment_7">
             <visual>
-                <origin rpy="0 0 0" xyz="0 0 0.015"/>
-                <geometry>
-                    <cylinder length="0.03" radius="0.001"/>
-                </geometry>
-                <!--material name="black"/-->
-            </visual>
-            <inertial>
-                <mass value="0.0001"/>
-                <inertia ixx="7.525e-09" iyy="7.525e-09" izz="5e-11" ixy="0.0" ixz="0.0" iyz="0.0"/>
+                <origin rpy="0 0 0" xyz="0 0 0.05"/>
+                <geometry>
+                    <cylinder length="0.1" radius="0.001"/>
+                </geometry>
+                <!--material name="black"/-->
+            </visual>
+            <inertial>
+                <mass value="0.0001"/>
+                <inertia ixx="8.33583333333e-08" iyy="8.33583333333e-08" izz="5e-11" ixy="0.0" ixz="0.0" iyz="0.0"/>
             </inertial>
         </link>
@@ -303,5 +303,5 @@
         <!--tether fragment joint-->
         <joint name="joint_1_7" type="continuous">
-            <origin rpy="0 0 0" xyz="0 0 0.03"/>
+            <origin rpy="0 0 0" xyz="0 0 0.1"/>
             <parent link="tether_fragment_6"/>
             <child link="small_link_1_7"/>
@@ -320,13 +320,13 @@
         <link name="tether_fragment_8">
             <visual>
-                <origin rpy="0 0 0" xyz="0 0 0.015"/>
-                <geometry>
-                    <cylinder length="0.03" radius="0.001"/>
-                </geometry>
-                <!--material name="black"/-->
-            </visual>
-            <inertial>
-                <mass value="0.0001"/>
-                <inertia ixx="7.525e-09" iyy="7.525e-09" izz="5e-11" ixy="0.0" ixz="0.0" iyz="0.0"/>
+                <origin rpy="0 0 0" xyz="0 0 0.05"/>
+                <geometry>
+                    <cylinder length="0.1" radius="0.001"/>
+                </geometry>
+                <!--material name="black"/-->
+            </visual>
+            <inertial>
+                <mass value="0.0001"/>
+                <inertia ixx="8.33583333333e-08" iyy="8.33583333333e-08" izz="5e-11" ixy="0.0" ixz="0.0" iyz="0.0"/>
             </inertial>
         </link>
@@ -346,5 +346,5 @@
         <!--tether fragment joint-->
         <joint name="joint_1_8" type="continuous">
-            <origin rpy="0 0 0" xyz="0 0 0.03"/>
+            <origin rpy="0 0 0" xyz="0 0 0.1"/>
             <parent link="tether_fragment_7"/>
             <child link="small_link_1_8"/>
@@ -363,13 +363,13 @@
         <link name="tether_fragment_9">
             <visual>
-                <origin rpy="0 0 0" xyz="0 0 0.015"/>
-                <geometry>
-                    <cylinder length="0.03" radius="0.001"/>
-                </geometry>
-                <!--material name="black"/-->
-            </visual>
-            <inertial>
-                <mass value="0.0001"/>
-                <inertia ixx="7.525e-09" iyy="7.525e-09" izz="5e-11" ixy="0.0" ixz="0.0" iyz="0.0"/>
+                <origin rpy="0 0 0" xyz="0 0 0.05"/>
+                <geometry>
+                    <cylinder length="0.1" radius="0.001"/>
+                </geometry>
+                <!--material name="black"/-->
+            </visual>
+            <inertial>
+                <mass value="0.0001"/>
+                <inertia ixx="8.33583333333e-08" iyy="8.33583333333e-08" izz="5e-11" ixy="0.0" ixz="0.0" iyz="0.0"/>
             </inertial>
         </link>
@@ -389,5 +389,5 @@
         <!--tether fragment joint-->
         <joint name="joint_1_9" type="continuous">
-            <origin rpy="0 0 0" xyz="0 0 0.03"/>
+            <origin rpy="0 0 0" xyz="0 0 0.1"/>
             <parent link="tether_fragment_8"/>
             <child link="small_link_1_9"/>
@@ -406,13 +406,13 @@
         <link name="tether_fragment_10">
             <visual>
-                <origin rpy="0 0 0" xyz="0 0 0.015"/>
-                <geometry>
-                    <cylinder length="0.03" radius="0.001"/>
-                </geometry>
-                <!--material name="black"/-->
-            </visual>
-            <inertial>
-                <mass value="0.0001"/>
-                <inertia ixx="7.525e-09" iyy="7.525e-09" izz="5e-11" ixy="0.0" ixz="0.0" iyz="0.0"/>
+                <origin rpy="0 0 0" xyz="0 0 0.05"/>
+                <geometry>
+                    <cylinder length="0.1" radius="0.001"/>
+                </geometry>
+                <!--material name="black"/-->
+            </visual>
+            <inertial>
+                <mass value="0.0001"/>
+                <inertia ixx="8.33583333333e-08" iyy="8.33583333333e-08" izz="5e-11" ixy="0.0" ixz="0.0" iyz="0.0"/>
             </inertial>
         </link>
@@ -432,5 +432,5 @@
         <!--tether fragment joint-->
         <joint name="joint_1_10" type="continuous">
-            <origin rpy="0 0 0" xyz="0 0 0.03"/>
+            <origin rpy="0 0 0" xyz="0 0 0.1"/>
             <parent link="tether_fragment_9"/>
             <child link="small_link_1_10"/>
@@ -449,13 +449,13 @@
         <link name="tether_fragment_11">
             <visual>
-                <origin rpy="0 0 0" xyz="0 0 0.015"/>
-                <geometry>
-                    <cylinder length="0.03" radius="0.001"/>
-                </geometry>
-                <!--material name="black"/-->
-            </visual>
-            <inertial>
-                <mass value="0.0001"/>
-                <inertia ixx="7.525e-09" iyy="7.525e-09" izz="5e-11" ixy="0.0" ixz="0.0" iyz="0.0"/>
+                <origin rpy="0 0 0" xyz="0 0 0.05"/>
+                <geometry>
+                    <cylinder length="0.1" radius="0.001"/>
+                </geometry>
+                <!--material name="black"/-->
+            </visual>
+            <inertial>
+                <mass value="0.0001"/>
+                <inertia ixx="8.33583333333e-08" iyy="8.33583333333e-08" izz="5e-11" ixy="0.0" ixz="0.0" iyz="0.0"/>
             </inertial>
         </link>
@@ -475,5 +475,5 @@
         <!--tether fragment joint-->
         <joint name="joint_1_11" type="continuous">
-            <origin rpy="0 0 0" xyz="0 0 0.03"/>
+            <origin rpy="0 0 0" xyz="0 0 0.1"/>
             <parent link="tether_fragment_10"/>
             <child link="small_link_1_11"/>
@@ -492,13 +492,13 @@
         <link name="tether_fragment_12">
             <visual>
-                <origin rpy="0 0 0" xyz="0 0 0.015"/>
-                <geometry>
-                    <cylinder length="0.03" radius="0.001"/>
-                </geometry>
-                <!--material name="black"/-->
-            </visual>
-            <inertial>
-                <mass value="0.0001"/>
-                <inertia ixx="7.525e-09" iyy="7.525e-09" izz="5e-11" ixy="0.0" ixz="0.0" iyz="0.0"/>
+                <origin rpy="0 0 0" xyz="0 0 0.05"/>
+                <geometry>
+                    <cylinder length="0.1" radius="0.001"/>
+                </geometry>
+                <!--material name="black"/-->
+            </visual>
+            <inertial>
+                <mass value="0.0001"/>
+                <inertia ixx="8.33583333333e-08" iyy="8.33583333333e-08" izz="5e-11" ixy="0.0" ixz="0.0" iyz="0.0"/>
             </inertial>
         </link>
@@ -518,5 +518,5 @@
         <!--tether fragment joint-->
         <joint name="joint_1_12" type="continuous">
-            <origin rpy="0 0 0" xyz="0 0 0.03"/>
+            <origin rpy="0 0 0" xyz="0 0 0.1"/>
             <parent link="tether_fragment_11"/>
             <child link="small_link_1_12"/>
@@ -535,13 +535,13 @@
         <link name="tether_fragment_13">
             <visual>
-                <origin rpy="0 0 0" xyz="0 0 0.015"/>
-                <geometry>
-                    <cylinder length="0.03" radius="0.001"/>
-                </geometry>
-                <!--material name="black"/-->
-            </visual>
-            <inertial>
-                <mass value="0.0001"/>
-                <inertia ixx="7.525e-09" iyy="7.525e-09" izz="5e-11" ixy="0.0" ixz="0.0" iyz="0.0"/>
+                <origin rpy="0 0 0" xyz="0 0 0.05"/>
+                <geometry>
+                    <cylinder length="0.1" radius="0.001"/>
+                </geometry>
+                <!--material name="black"/-->
+            </visual>
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
File: tether_description/urdf/tether_fragment.xacro (robot description, xacro)
@@ -5,5 +5,5 @@
         <!--tether fragment param-->
         {%- set cyl_r = 0.001 -%}
-        {%- set cyl_l = 0.03 -%}
+        {%- set cyl_l = 0.1 -%}
         {%- set cyl_m = 0.0001 -%}
         {%- set cyl_i = 1/12*cyl_m*(3*cyl_r**2+cyl_l**2) -%}
@@ -18,5 +18,5 @@
         {%- set small_link_iyz = 0.0 -%}
         <!--link number-->
-        {%- set tether_fragments = 50 -%}
+        {%- set tether_fragments = 20 -%}
         {%- macro tether_fragment(n) -%}
         <link name="tether_fragment_{{n}}">

File: uav_description/urdf/pyramid_firefly.xacro (robot description, xacro)
@@ -186,8 +186,8 @@
     <xacro:insert_block name="rotor_inertia" />
   </xacro:vertical_rotor>
-  <!--joint name="uav_tether_joint_4" type="fixed">
+  <joint name="uav_tether_joint_4" type="fixed">
       <parent link="${namespace}/base_link"/>
       <child link="tether_fragment_0"/>
   </joint>
-  <xacro:tether /-->
+  <xacro:tether />
 </robot>
