Commit message: fix bugs & could connect tether

File: tether_description/urdf/tether.xacro (robot description, xacro)
@@ -3,5 +3,10 @@
     <!--tether model-->
     <xacro:macro name="tether">
-        <!--tether fragment param--><!--small link inatial--><!--link number--><!--tether_cylinder_joint--><!-- main-->
+        <!--tether fragment param--><!--small link inatial--><!--link number--><!--tether_cylinder_joint--><joint name="uav_tether_joint" type="fixed">
+            <parent link="tether_fragment_49"/>
+            <child link="${namespace}/base_link"/>
+            <origin rpy="0 0 0" xyz="0 0 0"/>
+        </joint>
+        <!-- main-->
         <link name="tether_fragment_0">
             <visual>
@@ -832,4 +837,1294 @@
             <parent link="small_link_2_19"/>
             <child link="tether_fragment_19"/>
+            <axis xyz="0 0 1" />
+        </joint>
+        <link name="tether_fragment_20">
+            <visual>
+                <origin rpy="0 0 0" xyz="0 0 0.05"/>
+                <geometry>
+                    <cylinder length="0.1" radius="0.001"/>
+                </geometry>
+                <!--material name="black"/-->
+            </visual>
+            <inertial>
+                <mass value="0.0001"/>
+                <inertia ixx="8.33583333333e-08" iyy="8.33583333333e-08" izz="5e-11" ixy="0.0" ixz="0.0" iyz="0.0"/>
+            </inertial>
+        </link>
+                <!--link between two tether fragments-->
+        <link name="small_link_1_20">
+            <inertial>
+                <mass value="1e-05"/>
+                <inertia ixx="1e-05" iyy="1e-05" izz="1e-05" ixy="0.0" ixz="0.0" iyz="0.0"/>
+            </inertial>
+        </link>
+        <link name="small_link_2_20">
+            <inertial>
+                <mass value="1e-05"/>
+                <inertia ixx="1e-05" iyy="1e-05" izz="1e-05" ixy="0.0" ixz="0.0" iyz="0.0"/>
+            </inertial>
+        </link>
+        <!--tether fragment joint-->
+        <joint name="joint_1_20" type="continuous">
+            <origin rpy="0 0 0" xyz="0 0 0.1"/>
+            <parent link="tether_fragment_19"/>
+            <child link="small_link_1_20"/>
+            <axis xyz="1 0 0" />
+        </joint>
+        <joint name="joint_2_20" type="continuous">
+            <parent link="small_link_1_20"/>
+            <child link="small_link_2_20"/>
+            <axis xyz="0 1 0" />
+        </joint>
+        <joint name="joint_1_20_" type="continuous">
+            <parent link="small_link_2_20"/>
+            <child link="tether_fragment_20"/>
+            <axis xyz="0 0 1" />
+        </joint>
+        <link name="tether_fragment_21">
+            <visual>
+                <origin rpy="0 0 0" xyz="0 0 0.05"/>
+                <geometry>
+                    <cylinder length="0.1" radius="0.001"/>
+                </geometry>
+                <!--material name="black"/-->
+            </visual>
+            <inertial>
+                <mass value="0.0001"/>
+                <inertia ixx="8.33583333333e-08" iyy="8.33583333333e-08" izz="5e-11" ixy="0.0" ixz="0.0" iyz="0.0"/>
+            </inertial>
+        </link>
+                <!--link between two tether fragments-->
+        <link name="small_link_1_21">
+            <inertial>
+                <mass value="1e-05"/>
+                <inertia ixx="1e-05" iyy="1e-05" izz="1e-05" ixy="0.0" ixz="0.0" iyz="0.0"/>
+            </inertial>
+        </link>
+        <link name="small_link_2_21">
+            <inertial>
+                <mass value="1e-05"/>
+                <inertia ixx="1e-05" iyy="1e-05" izz="1e-05" ixy="0.0" ixz="0.0" iyz="0.0"/>
+            </inertial>
+        </link>
+        <!--tether fragment joint-->
+        <joint name="joint_1_21" type="continuous">
+            <origin rpy="0 0 0" xyz="0 0 0.1"/>
+            <parent link="tether_fragment_20"/>
+            <child link="small_link_1_21"/>
+            <axis xyz="1 0 0" />
+        </joint>
+        <joint name="joint_2_21" type="continuous">
+            <parent link="small_link_1_21"/>
+            <child link="small_link_2_21"/>
+            <axis xyz="0 1 0" />
+        </joint>
+        <joint name="joint_1_21_" type="continuous">
+            <parent link="small_link_2_21"/>
+            <child link="tether_fragment_21"/>
+            <axis xyz="0 0 1" />
+        </joint>
+        <link name="tether_fragment_22">
+            <visual>
+                <origin rpy="0 0 0" xyz="0 0 0.05"/>
+                <geometry>
+                    <cylinder length="0.1" radius="0.001"/>
+                </geometry>
+                <!--material name="black"/-->
+            </visual>
+            <inertial>
+                <mass value="0.0001"/>
+                <inertia ixx="8.33583333333e-08" iyy="8.33583333333e-08" izz="5e-11" ixy="0.0" ixz="0.0" iyz="0.0"/>
+            </inertial>
+        </link>
+                <!--link between two tether fragments-->
+        <link name="small_link_1_22">
+            <inertial>
+                <mass value="1e-05"/>
+                <inertia ixx="1e-05" iyy="1e-05" izz="1e-05" ixy="0.0" ixz="0.0" iyz="0.0"/>
+            </inertial>
+        </link>
+        <link name="small_link_2_22">
+            <inertial>
+                <mass value="1e-05"/>
+                <inertia ixx="1e-05" iyy="1e-05" izz="1e-05" ixy="0.0" ixz="0.0" iyz="0.0"/>
+            </inertial>
+        </link>
+        <!--tether fragment joint-->
+        <joint name="joint_1_22" type="continuous">
+            <origin rpy="0 0 0" xyz="0 0 0.1"/>
+            <parent link="tether_fragment_21"/>
+            <child link="small_link_1_22"/>
+            <axis xyz="1 0 0" />
+        </joint>
+        <joint name="joint_2_22" type="continuous">
+            <parent link="small_link_1_22"/>
+            <child link="small_link_2_22"/>
+            <axis xyz="0 1 0" />
+        </joint>
+        <joint name="joint_1_22_" type="continuous">
+            <parent link="small_link_2_22"/>
+            <child link="tether_fragment_22"/>
+            <axis xyz="0 0 1" />
+        </joint>
+        <link name="tether_fragment_23">
+            <visual>
+                <origin rpy="0 0 0" xyz="0 0 0.05"/>
+                <geometry>
+                    <cylinder length="0.1" radius="0.001"/>
+                </geometry>
+                <!--material name="black"/-->
+            </visual>
+            <inertial>
+                <mass value="0.0001"/>
+                <inertia ixx="8.33583333333e-08" iyy="8.33583333333e-08" izz="5e-11" ixy="0.0" ixz="0.0" iyz="0.0"/>
+            </inertial>
+        </link>
+                <!--link between two tether fragments-->
+        <link name="small_link_1_23">
+            <inertial>
+                <mass value="1e-05"/>
+                <inertia ixx="1e-05" iyy="1e-05" izz="1e-05" ixy="0.0" ixz="0.0" iyz="0.0"/>
+            </inertial>
+        </link>
+        <link name="small_link_2_23">
+            <inertial>
+                <mass value="1e-05"/>
+                <inertia ixx="1e-05" iyy="1e-05" izz="1e-05" ixy="0.0" ixz="0.0" iyz="0.0"/>
+            </inertial>
+        </link>
+        <!--tether fragment joint-->
+        <joint name="joint_1_23" type="continuous">
+            <origin rpy="0 0 0" xyz="0 0 0.1"/>
+            <parent link="tether_fragment_22"/>
+            <child link="small_link_1_23"/>
+            <axis xyz="1 0 0" />
+        </joint>
+        <joint name="joint_2_23" type="continuous">
+            <parent link="small_link_1_23"/>
+            <child link="small_link_2_23"/>
+            <axis xyz="0 1 0" />
+        </joint>
+        <joint name="joint_1_23_" type="continuous">
+            <parent link="small_link_2_23"/>
+            <child link="tether_fragment_23"/>
+            <axis xyz="0 0 1" />
+        </joint>
+        <link name="tether_fragment_24">
+            <visual>
+                <origin rpy="0 0 0" xyz="0 0 0.05"/>
+                <geometry>
+                    <cylinder length="0.1" radius="0.001"/>
+                </geometry>
+                <!--material name="black"/-->
+            </visual>
+            <inertial>
+                <mass value="0.0001"/>
+                <inertia ixx="8.33583333333e-08" iyy="8.33583333333e-08" izz="5e-11" ixy="0.0" ixz="0.0" iyz="0.0"/>
+            </inertial>
+        </link>
+                <!--link between two tether fragments-->
+        <link name="small_link_1_24">
+            <inertial>
+                <mass value="1e-05"/>
+                <inertia ixx="1e-05" iyy="1e-05" izz="1e-05" ixy="0.0" ixz="0.0" iyz="0.0"/>
+            </inertial>
+        </link>
+        <link name="small_link_2_24">
+            <inertial>
+                <mass value="1e-05"/>
+                <inertia ixx="1e-05" iyy="1e-05" izz="1e-05" ixy="0.0" ixz="0.0" iyz="0.0"/>
+            </inertial>
+        </link>
+        <!--tether fragment joint-->
+        <joint name="joint_1_24" type="continuous">
+            <origin rpy="0 0 0" xyz="0 0 0.1"/>
+            <parent link="tether_fragment_23"/>
+            <child link="small_link_1_24"/>
+            <axis xyz="1 0 0" />
+        </joint>
+        <joint name="joint_2_24" type="continuous">
+            <parent link="small_link_1_24"/>
+            <child link="small_link_2_24"/>
+            <axis xyz="0 1 0" />
+        </joint>
+        <joint name="joint_1_24_" type="continuous">
+            <parent link="small_link_2_24"/>
+            <child link="tether_fragment_24"/>
+            <axis xyz="0 0 1" />
+        </joint>
+        <link name="tether_fragment_25">
+            <visual>
+                <origin rpy="0 0 0" xyz="0 0 0.05"/>
+                <geometry>
+                    <cylinder length="0.1" radius="0.001"/>
+                </geometry>
+                <!--material name="black"/-->
+            </visual>
+            <inertial>
+                <mass value="0.0001"/>
+                <inertia ixx="8.33583333333e-08" iyy="8.33583333333e-08" izz="5e-11" ixy="0.0" ixz="0.0" iyz="0.0"/>
+            </inertial>
+        </link>
+                <!--link between two tether fragments-->
+        <link name="small_link_1_25">
+            <inertial>
+                <mass value="1e-05"/>
+                <inertia ixx="1e-05" iyy="1e-05" izz="1e-05" ixy="0.0" ixz="0.0" iyz="0.0"/>
+            </inertial>
+        </link>
+        <link name="small_link_2_25">
+            <inertial>
+                <mass value="1e-05"/>
+                <inertia ixx="1e-05" iyy="1e-05" izz="1e-05" ixy="0.0" ixz="0.0" iyz="0.0"/>
+            </inertial>
+        </link>
+        <!--tether fragment joint-->
+        <joint name="joint_1_25" type="continuous">
+            <origin rpy="0 0 0" xyz="0 0 0.1"/>
+            <parent link="tether_fragment_24"/>
+            <child link="small_link_1_25"/>
+            <axis xyz="1 0 0" />
+        </joint>
+        <joint name="joint_2_25" type="continuous">
+            <parent link="small_link_1_25"/>
+            <child link="small_link_2_25"/>
+            <axis xyz="0 1 0" />
+        </joint>
+        <joint name="joint_1_25_" type="continuous">
+            <parent link="small_link_2_25"/>
+            <child link="tether_fragment_25"/>
+            <axis xyz="0 0 1" />
+        </joint>
+        <link name="tether_fragment_26">
+            <visual>
+                <origin rpy="0 0 0" xyz="0 0 0.05"/>
+                <geometry>
+                    <cylinder length="0.1" radius="0.001"/>
+                </geometry>
+                <!--material name="black"/-->
+            </visual>
+            <inertial>
+                <mass value="0.0001"/>
+                <inertia ixx="8.33583333333e-08" iyy="8.33583333333e-08" izz="5e-11" ixy="0.0" ixz="0.0" iyz="0.0"/>
+            </inertial>
+        </link>
+                <!--link between two tether fragments-->
+        <link name="small_link_1_26">
+            <inertial>
+                <mass value="1e-05"/>
+                <inertia ixx="1e-05" iyy="1e-05" izz="1e-05" ixy="0.0" ixz="0.0" iyz="0.0"/>
+            </inertial>
+        </link>
+        <link name="small_link_2_26">
+            <inertial>
+                <mass value="1e-05"/>
+                <inertia ixx="1e-05" iyy="1e-05" izz="1e-05" ixy="0.0" ixz="0.0" iyz="0.0"/>
+            </inertial>
+        </link>
+        <!--tether fragment joint-->
+        <joint name="joint_1_26" type="continuous">
+            <origin rpy="0 0 0" xyz="0 0 0.1"/>
+            <parent link="tether_fragment_25"/>
+            <child link="small_link_1_26"/>
+            <axis xyz="1 0 0" />
+        </joint>
+        <joint name="joint_2_26" type="continuous">
+            <parent link="small_link_1_26"/>
+            <child link="small_link_2_26"/>
+            <axis xyz="0 1 0" />
+        </joint>
+        <joint name="joint_1_26_" type="continuous">
+            <parent link="small_link_2_26"/>
+            <child link="tether_fragment_26"/>
+            <axis xyz="0 0 1" />
+        </joint>
+        <link name="tether_fragment_27">
+            <visual>
+                <origin rpy="0 0 0" xyz="0 0 0.05"/>
+                <geometry>
+                    <cylinder length="0.1" radius="0.001"/>
+                </geometry>
+                <!--material name="black"/-->
+            </visual>
+            <inertial>
+                <mass value="0.0001"/>
+                <inertia ixx="8.33583333333e-08" iyy="8.33583333333e-08" izz="5e-11" ixy="0.0" ixz="0.0" iyz="0.0"/>
+            </inertial>
+        </link>
+                <!--link between two tether fragments-->
+        <link name="small_link_1_27">
+            <inertial>
+                <mass value="1e-05"/>
+                <inertia ixx="1e-05" iyy="1e-05" izz="1e-05" ixy="0.0" ixz="0.0" iyz="0.0"/>
+            </inertial>
+        </link>
+        <link name="small_link_2_27">
+            <inertial>
+                <mass value="1e-05"/>
+                <inertia ixx="1e-05" iyy="1e-05" izz="1e-05" ixy="0.0" ixz="0.0" iyz="0.0"/>
+            </inertial>
+        </link>
+        <!--tether fragment joint-->
+        <joint name="joint_1_27" type="continuous">
+            <origin rpy="0 0 0" xyz="0 0 0.1"/>
+            <parent link="tether_fragment_26"/>
+            <child link="small_link_1_27"/>
+            <axis xyz="1 0 0" />
+        </joint>
+        <joint name="joint_2_27" type="continuous">
+            <parent link="small_link_1_27"/>
+            <child link="small_link_2_27"/>
+            <axis xyz="0 1 0" />
+        </joint>
+        <joint name="joint_1_27_" type="continuous">
+            <parent link="small_link_2_27"/>
+            <child link="tether_fragment_27"/>
+            <axis xyz="0 0 1" />
+        </joint>
+        <link name="tether_fragment_28">
+            <visual>
+                <origin rpy="0 0 0" xyz="0 0 0.05"/>
+                <geometry>
+                    <cylinder length="0.1" radius="0.001"/>
+                </geometry>
+                <!--material name="black"/-->
+            </visual>
+            <inertial>
+                <mass value="0.0001"/>
+                <inertia ixx="8.33583333333e-08" iyy="8.33583333333e-08" izz="5e-11" ixy="0.0" ixz="0.0" iyz="0.0"/>
+            </inertial>
+        </link>
+                <!--link between two tether fragments-->
+        <link name="small_link_1_28">
+            <inertial>
+                <mass value="1e-05"/>
+                <inertia ixx="1e-05" iyy="1e-05" izz="1e-05" ixy="0.0" ixz="0.0" iyz="0.0"/>
+            </inertial>
+        </link>
+        <link name="small_link_2_28">
+            <inertial>
+                <mass value="1e-05"/>
+                <inertia ixx="1e-05" iyy="1e-05" izz="1e-05" ixy="0.0" ixz="0.0" iyz="0.0"/>
+            </inertial>
+        </link>
+        <!--tether fragment joint-->
+        <joint name="joint_1_28" type="continuous">
+            <origin rpy="0 0 0" xyz="0 0 0.1"/>
+            <parent link="tether_fragment_27"/>
+            <child link="small_link_1_28"/>
+            <axis xyz="1 0 0" />
+        </joint>
+        <joint name="joint_2_28" type="continuous">
+            <parent link="small_link_1_28"/>
+            <child link="small_link_2_28"/>
+            <axis xyz="0 1 0" />
+        </joint>
+        <joint name="joint_1_28_" type="continuous">
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
File: tether_description/urdf/tether_fragment.xacro (robot description, xacro)
@@ -18,5 +18,5 @@
         {%- set small_link_iyz = 0.0 -%}
         <!--link number-->
-        {%- set tether_fragments = 20 -%}
+        {%- set tether_fragments = 50 -%}
         {%- macro tether_fragment(n) -%}
         <link name="tether_fragment_{{n}}">
@@ -67,4 +67,9 @@
         </joint>
         {%- endmacro -%}
+        <joint name="uav_tether_joint" type="fixed">
+            <parent link="tether_fragment_{{tether_fragments-1}}"/>
+            <child link="${namespace}/base_link"/>
+            <origin rpy="0 0 0" xyz="0 0 0"/>
+        </joint>
         <!-- main-->
         {% for n in range(0,tether_fragments) -%}

File: uav_description/urdf/pyramid_firefly.xacro (robot description, xacro)
@@ -186,8 +186,4 @@
     <xacro:insert_block name="rotor_inertia" />
   </xacro:vertical_rotor>
-  <joint name="uav_tether_joint_4" type="fixed">
-      <parent link="${namespace}/base_link"/>
-      <child link="tether_fragment_0"/>
-  </joint>
   <xacro:tether />
 </robot>

Commit message: fix bugs & could control uav with tether in my own environment

File: tether_description/urdf/tether.xacro (robot description, xacro)
@@ -2129,9 +2129,4 @@
             <axis xyz="0 0 1" />
         </joint>
-        <gazebo>
-            <plugin name="gazebo_ros_control" filename="libgazebo_ros_control.so">
-                <robotNamespace>tether</robotNamespace>
-            </plugin>
-        </gazebo>
-    </xacro:macro>
+        </xacro:macro>
 </robot>

File: tether_description/urdf/tether_fragment.xacro (robot description, xacro)
@@ -79,9 +79,4 @@
             {% endif %}
         {% endfor -%}
-        <gazebo>
-            <plugin name="gazebo_ros_control" filename="libgazebo_ros_control.so">
-                <robotNamespace>tether</robotNamespace>
-            </plugin>
-        </gazebo>
     </xacro:macro>
 </robot>

File: uav_description/urdf/pyramid_firefly.xacro (robot description, xacro)
@@ -186,4 +186,4 @@
     <xacro:insert_block name="rotor_inertia" />
   </xacro:vertical_rotor>
-  <!--xacro:tether /-->
+  <xacro:tether />
 </robot>
