Commit message: clean up & could connect tether and box by four directions

File: tether_description/urdf/tether.xacro (robot description, xacro)
@@ -3,2129 +3,8596 @@
     <!--tether model-->
     <xacro:macro name="tether">
-        <!--tether fragment param--><!--small link inatial--><!--link number--><!--tether_cylinder_joint--><joint name="uav_tether_joint" type="fixed">
-            <parent link="tether_fragment_49"/>
-            <child link="${namespace}/base_link"/>
-            <origin rpy="0 0 0" xyz="0 0 0"/>
-        </joint>
-        <!-- main-->
-        <link name="tether_fragment_0">
-            <visual>
-                <origin rpy="0 0 0" xyz="0 0 0.05"/>
-                <geometry>
-                    <cylinder length="0.1" radius="0.001"/>
-                </geometry>
-                <!--material name="black"/-->
-            </visual>
-            <inertial>
-                <mass value="0.0001"/>
-                <inertia ixx="8.33583333333e-08" iyy="8.33583333333e-08" izz="5e-11" ixy="0.0" ixz="0.0" iyz="0.0"/>
-            </inertial>
-        </link>
-        <link name="tether_fragment_1">
-            <visual>
-                <origin rpy="0 0 0" xyz="0 0 0.05"/>
-                <geometry>
-                    <cylinder length="0.1" radius="0.001"/>
-                </geometry>
-                <!--material name="black"/-->
-            </visual>
-            <inertial>
-                <mass value="0.0001"/>
-                <inertia ixx="8.33583333333e-08" iyy="8.33583333333e-08" izz="5e-11" ixy="0.0" ixz="0.0" iyz="0.0"/>
-            </inertial>
-        </link>
-                <!--link between two tether fragments-->
-        <link name="small_link_1_1">
-            <inertial>
-                <mass value="1e-05"/>
-                <inertia ixx="1e-05" iyy="1e-05" izz="1e-05" ixy="0.0" ixz="0.0" iyz="0.0"/>
-            </inertial>
-        </link>
-        <link name="small_link_2_1">
-            <inertial>
-                <mass value="1e-05"/>
-                <inertia ixx="1e-05" iyy="1e-05" izz="1e-05" ixy="0.0" ixz="0.0" iyz="0.0"/>
-            </inertial>
-        </link>
-        <!--tether fragment joint-->
-        <joint name="joint_1_1" type="continuous">
-            <origin rpy="0 0 0" xyz="0 0 0.1"/>
-            <parent link="tether_fragment_0"/>
-            <child link="small_link_1_1"/>
-            <axis xyz="1 0 0" />
-        </joint>
-        <joint name="joint_2_1" type="continuous">
-            <parent link="small_link_1_1"/>
-            <child link="small_link_2_1"/>
-            <axis xyz="0 1 0" />
-        </joint>
-        <joint name="joint_1_1_" type="continuous">
-            <parent link="small_link_2_1"/>
-            <child link="tether_fragment_1"/>
-            <axis xyz="0 0 1" />
-        </joint>
-        <link name="tether_fragment_2">
-            <visual>
-                <origin rpy="0 0 0" xyz="0 0 0.05"/>
-                <geometry>
-                    <cylinder length="0.1" radius="0.001"/>
-                </geometry>
-                <!--material name="black"/-->
-            </visual>
-            <inertial>
-                <mass value="0.0001"/>
-                <inertia ixx="8.33583333333e-08" iyy="8.33583333333e-08" izz="5e-11" ixy="0.0" ixz="0.0" iyz="0.0"/>
-            </inertial>
-        </link>
-                <!--link between two tether fragments-->
-        <link name="small_link_1_2">
-            <inertial>
-                <mass value="1e-05"/>
-                <inertia ixx="1e-05" iyy="1e-05" izz="1e-05" ixy="0.0" ixz="0.0" iyz="0.0"/>
-            </inertial>
-        </link>
-        <link name="small_link_2_2">
-            <inertial>
-                <mass value="1e-05"/>
-                <inertia ixx="1e-05" iyy="1e-05" izz="1e-05" ixy="0.0" ixz="0.0" iyz="0.0"/>
-            </inertial>
-        </link>
-        <!--tether fragment joint-->
-        <joint name="joint_1_2" type="continuous">
-            <origin rpy="0 0 0" xyz="0 0 0.1"/>
-            <parent link="tether_fragment_1"/>
-            <child link="small_link_1_2"/>
-            <axis xyz="1 0 0" />
-        </joint>
-        <joint name="joint_2_2" type="continuous">
-            <parent link="small_link_1_2"/>
-            <child link="small_link_2_2"/>
-            <axis xyz="0 1 0" />
-        </joint>
-        <joint name="joint_1_2_" type="continuous">
-            <parent link="small_link_2_2"/>
-            <child link="tether_fragment_2"/>
-            <axis xyz="0 0 1" />
-        </joint>
-        <link name="tether_fragment_3">
-            <visual>
-                <origin rpy="0 0 0" xyz="0 0 0.05"/>
-                <geometry>
-                    <cylinder length="0.1" radius="0.001"/>
-                </geometry>
-                <!--material name="black"/-->
-            </visual>
-            <inertial>
-                <mass value="0.0001"/>
-                <inertia ixx="8.33583333333e-08" iyy="8.33583333333e-08" izz="5e-11" ixy="0.0" ixz="0.0" iyz="0.0"/>
-            </inertial>
-        </link>
-                <!--link between two tether fragments-->
-        <link name="small_link_1_3">
-            <inertial>
-                <mass value="1e-05"/>
-                <inertia ixx="1e-05" iyy="1e-05" izz="1e-05" ixy="0.0" ixz="0.0" iyz="0.0"/>
-            </inertial>
-        </link>
-        <link name="small_link_2_3">
-            <inertial>
-                <mass value="1e-05"/>
-                <inertia ixx="1e-05" iyy="1e-05" izz="1e-05" ixy="0.0" ixz="0.0" iyz="0.0"/>
-            </inertial>
-        </link>
-        <!--tether fragment joint-->
-        <joint name="joint_1_3" type="continuous">
-            <origin rpy="0 0 0" xyz="0 0 0.1"/>
-            <parent link="tether_fragment_2"/>
-            <child link="small_link_1_3"/>
-            <axis xyz="1 0 0" />
-        </joint>
-        <joint name="joint_2_3" type="continuous">
-            <parent link="small_link_1_3"/>
-            <child link="small_link_2_3"/>
-            <axis xyz="0 1 0" />
-        </joint>
-        <joint name="joint_1_3_" type="continuous">
-            <parent link="small_link_2_3"/>
-            <child link="tether_fragment_3"/>
-            <axis xyz="0 0 1" />
-        </joint>
-        <link name="tether_fragment_4">
-            <visual>
-                <origin rpy="0 0 0" xyz="0 0 0.05"/>
-                <geometry>
-                    <cylinder length="0.1" radius="0.001"/>
-                </geometry>
-                <!--material name="black"/-->
-            </visual>
-            <inertial>
-                <mass value="0.0001"/>
-                <inertia ixx="8.33583333333e-08" iyy="8.33583333333e-08" izz="5e-11" ixy="0.0" ixz="0.0" iyz="0.0"/>
-            </inertial>
-        </link>
-                <!--link between two tether fragments-->
-        <link name="small_link_1_4">
-            <inertial>
-                <mass value="1e-05"/>
-                <inertia ixx="1e-05" iyy="1e-05" izz="1e-05" ixy="0.0" ixz="0.0" iyz="0.0"/>
-            </inertial>
-        </link>
-        <link name="small_link_2_4">
-            <inertial>
-                <mass value="1e-05"/>
-                <inertia ixx="1e-05" iyy="1e-05" izz="1e-05" ixy="0.0" ixz="0.0" iyz="0.0"/>
-            </inertial>
-        </link>
-        <!--tether fragment joint-->
-        <joint name="joint_1_4" type="continuous">
-            <origin rpy="0 0 0" xyz="0 0 0.1"/>
-            <parent link="tether_fragment_3"/>
-            <child link="small_link_1_4"/>
-            <axis xyz="1 0 0" />
-        </joint>
-        <joint name="joint_2_4" type="continuous">
-            <parent link="small_link_1_4"/>
-            <child link="small_link_2_4"/>
-            <axis xyz="0 1 0" />
-        </joint>
-        <joint name="joint_1_4_" type="continuous">
-            <parent link="small_link_2_4"/>
-            <child link="tether_fragment_4"/>
-            <axis xyz="0 0 1" />
-        </joint>
-        <link name="tether_fragment_5">
-            <visual>
-                <origin rpy="0 0 0" xyz="0 0 0.05"/>
-                <geometry>
-                    <cylinder length="0.1" radius="0.001"/>
-                </geometry>
-                <!--material name="black"/-->
-            </visual>
-            <inertial>
-                <mass value="0.0001"/>
-                <inertia ixx="8.33583333333e-08" iyy="8.33583333333e-08" izz="5e-11" ixy="0.0" ixz="0.0" iyz="0.0"/>
-            </inertial>
-        </link>
-                <!--link between two tether fragments-->
-        <link name="small_link_1_5">
-            <inertial>
-                <mass value="1e-05"/>
-                <inertia ixx="1e-05" iyy="1e-05" izz="1e-05" ixy="0.0" ixz="0.0" iyz="0.0"/>
-            </inertial>
-        </link>
-        <link name="small_link_2_5">
-            <inertial>
-                <mass value="1e-05"/>
-                <inertia ixx="1e-05" iyy="1e-05" izz="1e-05" ixy="0.0" ixz="0.0" iyz="0.0"/>
-            </inertial>
-        </link>
-        <!--tether fragment joint-->
-        <joint name="joint_1_5" type="continuous">
-            <origin rpy="0 0 0" xyz="0 0 0.1"/>
-            <parent link="tether_fragment_4"/>
-            <child link="small_link_1_5"/>
-            <axis xyz="1 0 0" />
-        </joint>
-        <joint name="joint_2_5" type="continuous">
-            <parent link="small_link_1_5"/>
-            <child link="small_link_2_5"/>
-            <axis xyz="0 1 0" />
-        </joint>
-        <joint name="joint_1_5_" type="continuous">
-            <parent link="small_link_2_5"/>
-            <child link="tether_fragment_5"/>
-            <axis xyz="0 0 1" />
-        </joint>
-        <link name="tether_fragment_6">
-            <visual>
-                <origin rpy="0 0 0" xyz="0 0 0.05"/>
-                <geometry>
-                    <cylinder length="0.1" radius="0.001"/>
-                </geometry>
-                <!--material name="black"/-->
-            </visual>
-            <inertial>
-                <mass value="0.0001"/>
-                <inertia ixx="8.33583333333e-08" iyy="8.33583333333e-08" izz="5e-11" ixy="0.0" ixz="0.0" iyz="0.0"/>
-            </inertial>
-        </link>
-                <!--link between two tether fragments-->
-        <link name="small_link_1_6">
-            <inertial>
-                <mass value="1e-05"/>
-                <inertia ixx="1e-05" iyy="1e-05" izz="1e-05" ixy="0.0" ixz="0.0" iyz="0.0"/>
-            </inertial>
-        </link>
-        <link name="small_link_2_6">
-            <inertial>
-                <mass value="1e-05"/>
-                <inertia ixx="1e-05" iyy="1e-05" izz="1e-05" ixy="0.0" ixz="0.0" iyz="0.0"/>
-            </inertial>
-        </link>
-        <!--tether fragment joint-->
-        <joint name="joint_1_6" type="continuous">
-            <origin rpy="0 0 0" xyz="0 0 0.1"/>
-            <parent link="tether_fragment_5"/>
-            <child link="small_link_1_6"/>
-            <axis xyz="1 0 0" />
-        </joint>
-        <joint name="joint_2_6" type="continuous">
-            <parent link="small_link_1_6"/>
-            <child link="small_link_2_6"/>
-            <axis xyz="0 1 0" />
-        </joint>
-        <joint name="joint_1_6_" type="continuous">
-            <parent link="small_link_2_6"/>
-            <child link="tether_fragment_6"/>
-            <axis xyz="0 0 1" />
-        </joint>
-        <link name="tether_fragment_7">
-            <visual>
-                <origin rpy="0 0 0" xyz="0 0 0.05"/>
-                <geometry>
-                    <cylinder length="0.1" radius="0.001"/>
-                </geometry>
-                <!--material name="black"/-->
-            </visual>
-            <inertial>
-                <mass value="0.0001"/>
-                <inertia ixx="8.33583333333e-08" iyy="8.33583333333e-08" izz="5e-11" ixy="0.0" ixz="0.0" iyz="0.0"/>
-            </inertial>
-        </link>
-                <!--link between two tether fragments-->
-        <link name="small_link_1_7">
-            <inertial>
-                <mass value="1e-05"/>
-                <inertia ixx="1e-05" iyy="1e-05" izz="1e-05" ixy="0.0" ixz="0.0" iyz="0.0"/>
-            </inertial>
-        </link>
-        <link name="small_link_2_7">
-            <inertial>
-                <mass value="1e-05"/>
-                <inertia ixx="1e-05" iyy="1e-05" izz="1e-05" ixy="0.0" ixz="0.0" iyz="0.0"/>
-            </inertial>
-        </link>
-        <!--tether fragment joint-->
-        <joint name="joint_1_7" type="continuous">
-            <origin rpy="0 0 0" xyz="0 0 0.1"/>
-            <parent link="tether_fragment_6"/>
-            <child link="small_link_1_7"/>
-            <axis xyz="1 0 0" />
-        </joint>
-        <joint name="joint_2_7" type="continuous">
-            <parent link="small_link_1_7"/>
-            <child link="small_link_2_7"/>
-            <axis xyz="0 1 0" />
-        </joint>
-        <joint name="joint_1_7_" type="continuous">
-            <parent link="small_link_2_7"/>
-            <child link="tether_fragment_7"/>
-            <axis xyz="0 0 1" />
-        </joint>
-        <link name="tether_fragment_8">
-            <visual>
-                <origin rpy="0 0 0" xyz="0 0 0.05"/>
-                <geometry>
-                    <cylinder length="0.1" radius="0.001"/>
-                </geometry>
-                <!--material name="black"/-->
-            </visual>
-            <inertial>
-                <mass value="0.0001"/>
-                <inertia ixx="8.33583333333e-08" iyy="8.33583333333e-08" izz="5e-11" ixy="0.0" ixz="0.0" iyz="0.0"/>
-            </inertial>
-        </link>
-                <!--link between two tether fragments-->
-        <link name="small_link_1_8">
-            <inertial>
-                <mass value="1e-05"/>
-                <inertia ixx="1e-05" iyy="1e-05" izz="1e-05" ixy="0.0" ixz="0.0" iyz="0.0"/>
-            </inertial>
-        </link>
-        <link name="small_link_2_8">
-            <inertial>
-                <mass value="1e-05"/>
-                <inertia ixx="1e-05" iyy="1e-05" izz="1e-05" ixy="0.0" ixz="0.0" iyz="0.0"/>
-            </inertial>
-        </link>
-        <!--tether fragment joint-->
-        <joint name="joint_1_8" type="continuous">
-            <origin rpy="0 0 0" xyz="0 0 0.1"/>
-            <parent link="tether_fragment_7"/>
-            <child link="small_link_1_8"/>
-            <axis xyz="1 0 0" />
-        </joint>
-        <joint name="joint_2_8" type="continuous">
-            <parent link="small_link_1_8"/>
-            <child link="small_link_2_8"/>
-            <axis xyz="0 1 0" />
-        </joint>
-        <joint name="joint_1_8_" type="continuous">
-            <parent link="small_link_2_8"/>
-            <child link="tether_fragment_8"/>
-            <axis xyz="0 0 1" />
-        </joint>
-        <link name="tether_fragment_9">
-            <visual>
-                <origin rpy="0 0 0" xyz="0 0 0.05"/>
-                <geometry>
-                    <cylinder length="0.1" radius="0.001"/>
-                </geometry>
-                <!--material name="black"/-->
-            </visual>
-            <inertial>
-                <mass value="0.0001"/>
-                <inertia ixx="8.33583333333e-08" iyy="8.33583333333e-08" izz="5e-11" ixy="0.0" ixz="0.0" iyz="0.0"/>
-            </inertial>
-        </link>
-                <!--link between two tether fragments-->
-        <link name="small_link_1_9">
-            <inertial>
-                <mass value="1e-05"/>
-                <inertia ixx="1e-05" iyy="1e-05" izz="1e-05" ixy="0.0" ixz="0.0" iyz="0.0"/>
-            </inertial>
-        </link>
-        <link name="small_link_2_9">
-            <inertial>
-                <mass value="1e-05"/>
-                <inertia ixx="1e-05" iyy="1e-05" izz="1e-05" ixy="0.0" ixz="0.0" iyz="0.0"/>
-            </inertial>
-        </link>
-        <!--tether fragment joint-->
-        <joint name="joint_1_9" type="continuous">
-            <origin rpy="0 0 0" xyz="0 0 0.1"/>
-            <parent link="tether_fragment_8"/>
-            <child link="small_link_1_9"/>
-            <axis xyz="1 0 0" />
-        </joint>
-        <joint name="joint_2_9" type="continuous">
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
File: tether_description/urdf/tether_fragment.xacro (robot description, xacro)
@@ -19,6 +19,12 @@
         <!--link number-->
         {%- set tether_fragments = 50 -%}
-        {%- macro tether_fragment(n) -%}
-        <link name="tether_fragment_{{n}}">
+        {%- set tether_number = 4 -%}
+        <!--box inertial-->
+        {%- set box_m = 0.5 -%}
+        {%- set box_x = 0.1 -%}
+        {%- set box_y = 0.1 -%}
+        {%- set box_z = 0.1 -%}
+        {%- macro tether_fragment(dirc, n) -%}
+        <link name="tether_{{dirc}}/fragment_{{n}}">
             <visual>
                 <origin rpy="0 0 0" xyz="0 0 {{cyl_l/2}}"/>
@@ -35,7 +41,7 @@
         {%- endmacro -%}
         <!--tether_cylinder_joint-->
-        {%- macro tether_joint(n) -%}
+        {%- macro tether_joint(dirc, n) -%}
         <!--link between two tether fragments-->
-        <link name="small_link_1_{{n}}">
+        <link name="tether_{{dirc}}/small_link_1_{{n}}">
             <inertial>
                 <mass value="{{small_link_mass}}"/>
@@ -43,5 +49,5 @@
             </inertial>
         </link>
-        <link name="small_link_2_{{n}}">
+        <link name="tether_{{dirc}}/small_link_2_{{n}}">
             <inertial>
                 <mass value="{{small_link_mass}}"/>
@@ -50,32 +56,75 @@
         </link>
         <!--tether fragment joint-->
-        <joint name="joint_1_{{n}}" type="continuous">
+        <joint name="tether_{{dirc}}/joint_1_{{n}}" type="continuous">
             <origin rpy="0 0 0" xyz="0 0 {{cyl_l}}"/>
-            <parent link="tether_fragment_{{n-1}}"/>
-            <child link="small_link_1_{{n}}"/>
+            <parent link="tether_{{dirc}}/fragment_{{n-1}}"/>
+            <child link="tether_{{dirc}}/small_link_1_{{n}}"/>
             <axis xyz="1 0 0" />
         </joint>
-        <joint name="joint_2_{{n}}" type="continuous">
-            <parent link="small_link_1_{{n}}"/>
-            <child link="small_link_2_{{n}}"/>
+        <joint name="tether_{{dirc}}/joint_2_{{n}}" type="continuous">
+            <parent link="tether_{{dirc}}/small_link_1_{{n}}"/>
+            <child link="tether_{{dirc}}/small_link_2_{{n}}"/>
             <axis xyz="0 1 0" />
         </joint>
-        <joint name="joint_1_{{n}}_" type="continuous">
-            <parent link="small_link_2_{{n}}"/>
-            <child link="tether_fragment_{{n}}"/>
+        <joint name="tether_{{dirc}}/joint_1_{{n}}_" type="continuous">
+            <parent link="tether_{{dirc}}/small_link_2_{{n}}"/>
+            <child link="tether_{{dirc}}/fragment_{{n}}"/>
             <axis xyz="0 0 1" />
         </joint>
         {%- endmacro -%}
-        <joint name="uav_tether_joint" type="fixed">
-            <parent link="tether_fragment_{{tether_fragments-1}}"/>
-            <child link="${namespace}/base_link"/>
-            <origin rpy="0 0 0" xyz="0 0 0"/>
+        {%- macro uav_joint(dirc) -%}
+        <!--uav => tether joint-->
+        <joint name="tether_{{dirc}}/uav_joint" type="fixed">
+            <parent link="${namespace}/base_link"/>
+            <child link="tether_{{dirc}}/fragment_0"/>
+            {% if dirc == 0 %}
+                <origin rpy="0 ${pi/2} 0" xyz="0 0 0"/>
+            {% elif dirc == 1 %}
+                <origin rpy="${pi/2} 0 0" xyz="0 0 0"/>
+            {% elif dirc == 2 %}
+                <origin rpy="0 ${-pi/2} 0" xyz="0 0 0"/>
+            {% elif dirc == 3 %}
+                <origin rpy="${-pi/2} 0 0" xyz="0 0 0"/>
+            {% endif %}
         </joint>
+        {%- endmacro -%}
+        {%- macro pesudo_ugv(dirc) -%}
+        <link name="pesudo_ugv_{{dirc}}">
+            <visual>
+                <geometry>
+                    <box size="{{box_x}} {{box_y}} {{box_z}}"/>
+                </geometry>
+                <material name="silver">
+                    <color rgba="0.75 0.75 0.75 1"/>
+                </material>
+            </visual>
+            <collision>
+                <geometry>
+                    <box size="{{box_x}} {{box_y}} {{box_z}}"/>
+                </geometry>
+            </collision>
+            <inertial>
+                <mass value="{{box_m}}"/>
+                {%- set box_ix = 1/12*box_m*(box_y**2+box_z**2) -%}
+                {%- set box_iy = 1/12*box_m*(box_x**2+box_z**2) -%}
+                {%- set box_iz = 1/12*box_m*(box_x**2+box_y**2) -%}
+                <inertia ixx="{{box_ix}}" iyy="{{box_iy}}" izz="{{box_iz}}" ixy="0" ixz="0" iyz="0"/>
+            </inertial>
+        </link>
+        <joint name="tether_{{dirc}}/pesudo_ugv_joint" type="fixed">
+            <parent link="tether_{{dirc}}/fragment_{{tether_fragments-1}}"/>
+            <child link="pesudo_ugv_{{dirc}}"/>
+        </joint>
+        {%- endmacro -%}
         <!-- main-->
-        {% for n in range(0,tether_fragments) -%}
-            {{tether_fragment(n)}}
-            {% if n != 0 %}
-                {{tether_joint(n)}}
-            {% endif %}
+        {% for dirc in range(0,tether_number) %}
+            {% for n in range(0,tether_fragments) -%}
+                {{tether_fragment(dirc, n)}}
+                {% if n != 0 %}
+                    {{tether_joint(dirc, n)}}
+                {% endif %}
+            {% endfor -%}
+            {{uav_joint(dirc)}}
+            {{pesudo_ugv(dirc)}}
         {% endfor -%}
     </xacro:macro>
