Commit message: add wind gust & simulate terher connected uav

File: tether_description/urdf/tether.xacro (robot description, xacro)
@@ -2145,5 +2145,5 @@
             </collision>
             <inertial>
-                <mass value="0.5"/><inertia ixx="0.000833333333333" iyy="0.000833333333333" izz="0.000833333333333" ixy="0" ixz="0" iyz="0"/>
+                <mass value="50"/><inertia ixx="0.0833333333333" iyy="0.0833333333333" izz="0.0833333333333" ixy="0" ixz="0" iyz="0"/>
             </inertial>
         </link>
@@ -4293,5 +4293,5 @@
             </collision>
             <inertial>
-                <mass value="0.5"/><inertia ixx="0.000833333333333" iyy="0.000833333333333" izz="0.000833333333333" ixy="0" ixz="0" iyz="0"/>
+                <mass value="50"/><inertia ixx="0.0833333333333" iyy="0.0833333333333" izz="0.0833333333333" ixy="0" ixz="0" iyz="0"/>
             </inertial>
         </link>
@@ -6441,5 +6441,5 @@
             </collision>
             <inertial>
-                <mass value="0.5"/><inertia ixx="0.000833333333333" iyy="0.000833333333333" izz="0.000833333333333" ixy="0" ixz="0" iyz="0"/>
+                <mass value="50"/><inertia ixx="0.0833333333333" iyy="0.0833333333333" izz="0.0833333333333" ixy="0" ixz="0" iyz="0"/>
             </inertial>
         </link>
@@ -8589,5 +8589,5 @@
             </collision>
             <inertial>
-                <mass value="0.5"/><inertia ixx="0.000833333333333" iyy="0.000833333333333" izz="0.000833333333333" ixy="0" ixz="0" iyz="0"/>
+                <mass value="50"/><inertia ixx="0.0833333333333" iyy="0.0833333333333" izz="0.0833333333333" ixy="0" ixz="0" iyz="0"/>
             </inertial>
         </link>

File: tether_description/urdf/tether_fragment.xacro (robot description, xacro)
@@ -21,5 +21,5 @@
         {%- set tether_number = 4 -%}
         <!--box inertial-->
-        {%- set box_m = 0.5 -%}
+        {%- set box_m = 50 -%}
         {%- set box_x = 0.1 -%}
         {%- set box_y = 0.1 -%}

File: uav_description/urdf/pyramid_firefly.xacro (robot description, xacro)
@@ -187,4 +187,4 @@
   </xacro:vertical_rotor>
   <!--tether model-->
-  <!--xacro:tether /-->
+  <xacro:tether />
 </robot>

Commit message: clean up

File: tether_description/urdf/tether.xacro (robot description, xacro)
@@ -1264,864 +1264,4 @@
             <axis xyz="0 0 1" />
         </joint>
-            <link name="tether_0/fragment_30">
-            <visual>
-                <origin rpy="0 0 0" xyz="0 0 0.05"/>
-                <geometry>
-                    <cylinder length="0.1" radius="0.001"/>
-                </geometry>
-                <!--material name="black"/-->
-            </visual>
-            <inertial>
-                <mass value="0.0001"/>
-                <inertia ixx="8.33583333333e-08" iyy="8.33583333333e-08" izz="5e-11" ixy="0.0" ixz="0.0" iyz="0.0"/>
-            </inertial>
-        </link>
-                    <!--link between two tether fragments-->
-        <link name="tether_0/small_link_1_30">
-            <inertial>
-                <mass value="1e-05"/>
-                <inertia ixx="1e-05" iyy="1e-05" izz="1e-05" ixy="0.0" ixz="0.0" iyz="0.0"/>
-            </inertial>
-        </link>
-        <link name="tether_0/small_link_2_30">
-            <inertial>
-                <mass value="1e-05"/>
-                <inertia ixx="1e-05" iyy="1e-05" izz="1e-05" ixy="0.0" ixz="0.0" iyz="0.0"/>
-            </inertial>
-        </link>
-        <!--tether fragment joint-->
-        <joint name="tether_0/joint_1_30" type="continuous">
-            <origin rpy="0 0 0" xyz="0 0 0.1"/>
-            <parent link="tether_0/fragment_29"/>
-            <child link="tether_0/small_link_1_30"/>
-            <axis xyz="1 0 0" />
-        </joint>
-        <joint name="tether_0/joint_2_30" type="continuous">
-            <parent link="tether_0/small_link_1_30"/>
-            <child link="tether_0/small_link_2_30"/>
-            <axis xyz="0 1 0" />
-        </joint>
-        <joint name="tether_0/joint_1_30_" type="continuous">
-            <parent link="tether_0/small_link_2_30"/>
-            <child link="tether_0/fragment_30"/>
-            <axis xyz="0 0 1" />
-        </joint>
-            <link name="tether_0/fragment_31">
-            <visual>
-                <origin rpy="0 0 0" xyz="0 0 0.05"/>
-                <geometry>
-                    <cylinder length="0.1" radius="0.001"/>
-                </geometry>
-                <!--material name="black"/-->
-            </visual>
-            <inertial>
-                <mass value="0.0001"/>
-                <inertia ixx="8.33583333333e-08" iyy="8.33583333333e-08" izz="5e-11" ixy="0.0" ixz="0.0" iyz="0.0"/>
-            </inertial>
-        </link>
-                    <!--link between two tether fragments-->
-        <link name="tether_0/small_link_1_31">
-            <inertial>
-                <mass value="1e-05"/>
-                <inertia ixx="1e-05" iyy="1e-05" izz="1e-05" ixy="0.0" ixz="0.0" iyz="0.0"/>
-            </inertial>
-        </link>
-        <link name="tether_0/small_link_2_31">
-            <inertial>
-                <mass value="1e-05"/>
-                <inertia ixx="1e-05" iyy="1e-05" izz="1e-05" ixy="0.0" ixz="0.0" iyz="0.0"/>
-            </inertial>
-        </link>
-        <!--tether fragment joint-->
-        <joint name="tether_0/joint_1_31" type="continuous">
-            <origin rpy="0 0 0" xyz="0 0 0.1"/>
-            <parent link="tether_0/fragment_30"/>
-            <child link="tether_0/small_link_1_31"/>
-            <axis xyz="1 0 0" />
-        </joint>
-        <joint name="tether_0/joint_2_31" type="continuous">
-            <parent link="tether_0/small_link_1_31"/>
-            <child link="tether_0/small_link_2_31"/>
-            <axis xyz="0 1 0" />
-        </joint>
-        <joint name="tether_0/joint_1_31_" type="continuous">
-            <parent link="tether_0/small_link_2_31"/>
-            <child link="tether_0/fragment_31"/>
-            <axis xyz="0 0 1" />
-        </joint>
-            <link name="tether_0/fragment_32">
-            <visual>
-                <origin rpy="0 0 0" xyz="0 0 0.05"/>
-                <geometry>
-                    <cylinder length="0.1" radius="0.001"/>
-                </geometry>
-                <!--material name="black"/-->
-            </visual>
-            <inertial>
-                <mass value="0.0001"/>
-                <inertia ixx="8.33583333333e-08" iyy="8.33583333333e-08" izz="5e-11" ixy="0.0" ixz="0.0" iyz="0.0"/>
-            </inertial>
-        </link>
-                    <!--link between two tether fragments-->
-        <link name="tether_0/small_link_1_32">
-            <inertial>
-                <mass value="1e-05"/>
-                <inertia ixx="1e-05" iyy="1e-05" izz="1e-05" ixy="0.0" ixz="0.0" iyz="0.0"/>
-            </inertial>
-        </link>
-        <link name="tether_0/small_link_2_32">
-            <inertial>
-                <mass value="1e-05"/>
-                <inertia ixx="1e-05" iyy="1e-05" izz="1e-05" ixy="0.0" ixz="0.0" iyz="0.0"/>
-            </inertial>
-        </link>
-        <!--tether fragment joint-->
-        <joint name="tether_0/joint_1_32" type="continuous">
-            <origin rpy="0 0 0" xyz="0 0 0.1"/>
-            <parent link="tether_0/fragment_31"/>
-            <child link="tether_0/small_link_1_32"/>
-            <axis xyz="1 0 0" />
-        </joint>
-        <joint name="tether_0/joint_2_32" type="continuous">
-            <parent link="tether_0/small_link_1_32"/>
-            <child link="tether_0/small_link_2_32"/>
-            <axis xyz="0 1 0" />
-        </joint>
-        <joint name="tether_0/joint_1_32_" type="continuous">
-            <parent link="tether_0/small_link_2_32"/>
-            <child link="tether_0/fragment_32"/>
-            <axis xyz="0 0 1" />
-        </joint>
-            <link name="tether_0/fragment_33">
-            <visual>
-                <origin rpy="0 0 0" xyz="0 0 0.05"/>
-                <geometry>
-                    <cylinder length="0.1" radius="0.001"/>
-                </geometry>
-                <!--material name="black"/-->
-            </visual>
-            <inertial>
-                <mass value="0.0001"/>
-                <inertia ixx="8.33583333333e-08" iyy="8.33583333333e-08" izz="5e-11" ixy="0.0" ixz="0.0" iyz="0.0"/>
-            </inertial>
-        </link>
-                    <!--link between two tether fragments-->
-        <link name="tether_0/small_link_1_33">
-            <inertial>
-                <mass value="1e-05"/>
-                <inertia ixx="1e-05" iyy="1e-05" izz="1e-05" ixy="0.0" ixz="0.0" iyz="0.0"/>
-            </inertial>
-        </link>
-        <link name="tether_0/small_link_2_33">
-            <inertial>
-                <mass value="1e-05"/>
-                <inertia ixx="1e-05" iyy="1e-05" izz="1e-05" ixy="0.0" ixz="0.0" iyz="0.0"/>
-            </inertial>
-        </link>
-        <!--tether fragment joint-->
-        <joint name="tether_0/joint_1_33" type="continuous">
-            <origin rpy="0 0 0" xyz="0 0 0.1"/>
-            <parent link="tether_0/fragment_32"/>
-            <child link="tether_0/small_link_1_33"/>
-            <axis xyz="1 0 0" />
-        </joint>
-        <joint name="tether_0/joint_2_33" type="continuous">
-            <parent link="tether_0/small_link_1_33"/>
-            <child link="tether_0/small_link_2_33"/>
-            <axis xyz="0 1 0" />
-        </joint>
-        <joint name="tether_0/joint_1_33_" type="continuous">
-            <parent link="tether_0/small_link_2_33"/>
-            <child link="tether_0/fragment_33"/>
-            <axis xyz="0 0 1" />
-        </joint>
-            <link name="tether_0/fragment_34">
-            <visual>
-                <origin rpy="0 0 0" xyz="0 0 0.05"/>
-                <geometry>
-                    <cylinder length="0.1" radius="0.001"/>
-                </geometry>
-                <!--material name="black"/-->
-            </visual>
-            <inertial>
-                <mass value="0.0001"/>
-                <inertia ixx="8.33583333333e-08" iyy="8.33583333333e-08" izz="5e-11" ixy="0.0" ixz="0.0" iyz="0.0"/>
-            </inertial>
-        </link>
-                    <!--link between two tether fragments-->
-        <link name="tether_0/small_link_1_34">
-            <inertial>
-                <mass value="1e-05"/>
-                <inertia ixx="1e-05" iyy="1e-05" izz="1e-05" ixy="0.0" ixz="0.0" iyz="0.0"/>
-            </inertial>
-        </link>
-        <link name="tether_0/small_link_2_34">
-            <inertial>
-                <mass value="1e-05"/>
-                <inertia ixx="1e-05" iyy="1e-05" izz="1e-05" ixy="0.0" ixz="0.0" iyz="0.0"/>
-            </inertial>
-        </link>
-        <!--tether fragment joint-->
-        <joint name="tether_0/joint_1_34" type="continuous">
-            <origin rpy="0 0 0" xyz="0 0 0.1"/>
-            <parent link="tether_0/fragment_33"/>
-            <child link="tether_0/small_link_1_34"/>
-            <axis xyz="1 0 0" />
-        </joint>
-        <joint name="tether_0/joint_2_34" type="continuous">
-            <parent link="tether_0/small_link_1_34"/>
-            <child link="tether_0/small_link_2_34"/>
-            <axis xyz="0 1 0" />
-        </joint>
-        <joint name="tether_0/joint_1_34_" type="continuous">
-            <parent link="tether_0/small_link_2_34"/>
-            <child link="tether_0/fragment_34"/>
-            <axis xyz="0 0 1" />
-        </joint>
-            <link name="tether_0/fragment_35">
-            <visual>
-                <origin rpy="0 0 0" xyz="0 0 0.05"/>
-                <geometry>
-                    <cylinder length="0.1" radius="0.001"/>
-                </geometry>
-                <!--material name="black"/-->
-            </visual>
-            <inertial>
-                <mass value="0.0001"/>
-                <inertia ixx="8.33583333333e-08" iyy="8.33583333333e-08" izz="5e-11" ixy="0.0" ixz="0.0" iyz="0.0"/>
-            </inertial>
-        </link>
-                    <!--link between two tether fragments-->
-        <link name="tether_0/small_link_1_35">
-            <inertial>
-                <mass value="1e-05"/>
-                <inertia ixx="1e-05" iyy="1e-05" izz="1e-05" ixy="0.0" ixz="0.0" iyz="0.0"/>
-            </inertial>
-        </link>
-        <link name="tether_0/small_link_2_35">
-            <inertial>
-                <mass value="1e-05"/>
-                <inertia ixx="1e-05" iyy="1e-05" izz="1e-05" ixy="0.0" ixz="0.0" iyz="0.0"/>
-            </inertial>
-        </link>
-        <!--tether fragment joint-->
-        <joint name="tether_0/joint_1_35" type="continuous">
-            <origin rpy="0 0 0" xyz="0 0 0.1"/>
-            <parent link="tether_0/fragment_34"/>
-            <child link="tether_0/small_link_1_35"/>
-            <axis xyz="1 0 0" />
-        </joint>
-        <joint name="tether_0/joint_2_35" type="continuous">
-            <parent link="tether_0/small_link_1_35"/>
-            <child link="tether_0/small_link_2_35"/>
-            <axis xyz="0 1 0" />
-        </joint>
-        <joint name="tether_0/joint_1_35_" type="continuous">
-            <parent link="tether_0/small_link_2_35"/>
-            <child link="tether_0/fragment_35"/>
-            <axis xyz="0 0 1" />
-        </joint>
-            <link name="tether_0/fragment_36">
-            <visual>
-                <origin rpy="0 0 0" xyz="0 0 0.05"/>
-                <geometry>
-                    <cylinder length="0.1" radius="0.001"/>
-                </geometry>
-                <!--material name="black"/-->
-            </visual>
-            <inertial>
-                <mass value="0.0001"/>
-                <inertia ixx="8.33583333333e-08" iyy="8.33583333333e-08" izz="5e-11" ixy="0.0" ixz="0.0" iyz="0.0"/>
-            </inertial>
-        </link>
-                    <!--link between two tether fragments-->
-        <link name="tether_0/small_link_1_36">
-            <inertial>
-                <mass value="1e-05"/>
-                <inertia ixx="1e-05" iyy="1e-05" izz="1e-05" ixy="0.0" ixz="0.0" iyz="0.0"/>
-            </inertial>
-        </link>
-        <link name="tether_0/small_link_2_36">
-            <inertial>
-                <mass value="1e-05"/>
-                <inertia ixx="1e-05" iyy="1e-05" izz="1e-05" ixy="0.0" ixz="0.0" iyz="0.0"/>
-            </inertial>
-        </link>
-        <!--tether fragment joint-->
-        <joint name="tether_0/joint_1_36" type="continuous">
-            <origin rpy="0 0 0" xyz="0 0 0.1"/>
-            <parent link="tether_0/fragment_35"/>
-            <child link="tether_0/small_link_1_36"/>
-            <axis xyz="1 0 0" />
-        </joint>
-        <joint name="tether_0/joint_2_36" type="continuous">
-            <parent link="tether_0/small_link_1_36"/>
-            <child link="tether_0/small_link_2_36"/>
-            <axis xyz="0 1 0" />
-        </joint>
-        <joint name="tether_0/joint_1_36_" type="continuous">
-            <parent link="tether_0/small_link_2_36"/>
-            <child link="tether_0/fragment_36"/>
-            <axis xyz="0 0 1" />
-        </joint>
-            <link name="tether_0/fragment_37">
-            <visual>
-                <origin rpy="0 0 0" xyz="0 0 0.05"/>
-                <geometry>
-                    <cylinder length="0.1" radius="0.001"/>
-                </geometry>
-                <!--material name="black"/-->
-            </visual>
-            <inertial>
-                <mass value="0.0001"/>
-                <inertia ixx="8.33583333333e-08" iyy="8.33583333333e-08" izz="5e-11" ixy="0.0" ixz="0.0" iyz="0.0"/>
-            </inertial>
-        </link>
-                    <!--link between two tether fragments-->
-        <link name="tether_0/small_link_1_37">
-            <inertial>
-                <mass value="1e-05"/>
-                <inertia ixx="1e-05" iyy="1e-05" izz="1e-05" ixy="0.0" ixz="0.0" iyz="0.0"/>
-            </inertial>
-        </link>
-        <link name="tether_0/small_link_2_37">
-            <inertial>
-                <mass value="1e-05"/>
-                <inertia ixx="1e-05" iyy="1e-05" izz="1e-05" ixy="0.0" ixz="0.0" iyz="0.0"/>
-            </inertial>
-        </link>
-        <!--tether fragment joint-->
-        <joint name="tether_0/joint_1_37" type="continuous">
-            <origin rpy="0 0 0" xyz="0 0 0.1"/>
-            <parent link="tether_0/fragment_36"/>
-            <child link="tether_0/small_link_1_37"/>
-            <axis xyz="1 0 0" />
-        </joint>
-        <joint name="tether_0/joint_2_37" type="continuous">
-            <parent link="tether_0/small_link_1_37"/>
-            <child link="tether_0/small_link_2_37"/>
-            <axis xyz="0 1 0" />
-        </joint>
-        <joint name="tether_0/joint_1_37_" type="continuous">
-            <parent link="tether_0/small_link_2_37"/>
-            <child link="tether_0/fragment_37"/>
-            <axis xyz="0 0 1" />
-        </joint>
-            <link name="tether_0/fragment_38">
-            <visual>
-                <origin rpy="0 0 0" xyz="0 0 0.05"/>
-                <geometry>
-                    <cylinder length="0.1" radius="0.001"/>
-                </geometry>
-                <!--material name="black"/-->
-            </visual>
-            <inertial>
-                <mass value="0.0001"/>
-                <inertia ixx="8.33583333333e-08" iyy="8.33583333333e-08" izz="5e-11" ixy="0.0" ixz="0.0" iyz="0.0"/>
-            </inertial>
-        </link>
-                    <!--link between two tether fragments-->
-        <link name="tether_0/small_link_1_38">
-            <inertial>
-                <mass value="1e-05"/>
-                <inertia ixx="1e-05" iyy="1e-05" izz="1e-05" ixy="0.0" ixz="0.0" iyz="0.0"/>
-            </inertial>
-        </link>
-        <link name="tether_0/small_link_2_38">
-            <inertial>
-                <mass value="1e-05"/>
-                <inertia ixx="1e-05" iyy="1e-05" izz="1e-05" ixy="0.0" ixz="0.0" iyz="0.0"/>
-            </inertial>
-        </link>
-        <!--tether fragment joint-->
-        <joint name="tether_0/joint_1_38" type="continuous">
-            <origin rpy="0 0 0" xyz="0 0 0.1"/>
-            <parent link="tether_0/fragment_37"/>
-            <child link="tether_0/small_link_1_38"/>
-            <axis xyz="1 0 0" />
-        </joint>
-        <joint name="tether_0/joint_2_38" type="continuous">
-            <parent link="tether_0/small_link_1_38"/>
-            <child link="tether_0/small_link_2_38"/>
-            <axis xyz="0 1 0" />
-        </joint>
-        <joint name="tether_0/joint_1_38_" type="continuous">
-            <parent link="tether_0/small_link_2_38"/>
-            <child link="tether_0/fragment_38"/>
-            <axis xyz="0 0 1" />
-        </joint>
-            <link name="tether_0/fragment_39">
-            <visual>
-                <origin rpy="0 0 0" xyz="0 0 0.05"/>
-                <geometry>
-                    <cylinder length="0.1" radius="0.001"/>
-                </geometry>
-                <!--material name="black"/-->
-            </visual>
-            <inertial>
-                <mass value="0.0001"/>
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
File: tether_description/urdf/tether_fragment.xacro (robot description, xacro)
@@ -18,8 +18,8 @@
         {%- set small_link_iyz = 0.0 -%}
         <!--link number-->
-        {%- set tether_fragments = 50 -%}
+        {%- set tether_fragments = 30 -%}
         {%- set tether_number = 4 -%}
         <!--box inertial-->
-        {%- set box_m = 50 -%}
+        {%- set box_m = 0.50 -%}
         {%- set box_x = 0.1 -%}
         {%- set box_y = 0.1 -%}
