Commit message: fix bugs & add collision and dynamics to tether model

File: tether_description/urdf/tether.xacro (robot description, xacro)
@@ -3,17 +3,22 @@
     <!--tether model-->
     <xacro:macro name="tether">
-        <!--tether fragment param--><!--small link inatial--><!--link number--><!--box inertial--><!--tether_cylinder_joint--><!-- main-->
+        <!--tether fragment param--><!--small link inatial--><!--joint dynamics--><!--link number--><!--box inertial--><!--tether_cylinder_joint--><!-- main-->
             <link name="tether_0/fragment_0">
             <visual>
                 <origin rpy="0 0 0" xyz="0 0 0.05"/>
                 <geometry>
-                    <cylinder length="0.1" radius="0.001"/>
-                </geometry>
-                <!--material name="black"/-->
-            </visual>
-            <inertial>
-                <mass value="0.0001"/>
-                <inertia ixx="8.33583333333e-08" iyy="8.33583333333e-08" izz="5e-11" ixy="0.0" ixz="0.0" iyz="0.0"/>
-            </inertial>
+                    <cylinder length="0.1" radius="0.0033"/>
+                </geometry>
+                <!--material name="black"/-->
+            </visual>
+            <inertial>
+                <mass value="0.012"/>
+                <inertia ixx="1.003267e-05" iyy="1.003267e-05" izz="6.534e-08" ixy="0.0" ixz="0.0" iyz="0.0"/>
+            </inertial>
+            <collision>
+                <geometry>
+                    <cylinder length="0.1" radius="0.0033"/>
+                </geometry>
+            </collision>
         </link>
             <link name="tether_0/fragment_1">
@@ -21,24 +26,29 @@
                 <origin rpy="0 0 0" xyz="0 0 0.05"/>
                 <geometry>
-                    <cylinder length="0.1" radius="0.001"/>
-                </geometry>
-                <!--material name="black"/-->
-            </visual>
-            <inertial>
-                <mass value="0.0001"/>
-                <inertia ixx="8.33583333333e-08" iyy="8.33583333333e-08" izz="5e-11" ixy="0.0" ixz="0.0" iyz="0.0"/>
-            </inertial>
+                    <cylinder length="0.1" radius="0.0033"/>
+                </geometry>
+                <!--material name="black"/-->
+            </visual>
+            <inertial>
+                <mass value="0.012"/>
+                <inertia ixx="1.003267e-05" iyy="1.003267e-05" izz="6.534e-08" ixy="0.0" ixz="0.0" iyz="0.0"/>
+            </inertial>
+            <collision>
+                <geometry>
+                    <cylinder length="0.1" radius="0.0033"/>
+                </geometry>
+            </collision>
         </link>
                     <!--link between two tether fragments-->
         <link name="tether_0/small_link_1_1">
             <inertial>
-                <mass value="1e-05"/>
-                <inertia ixx="1e-05" iyy="1e-05" izz="1e-05" ixy="0.0" ixz="0.0" iyz="0.0"/>
+                <mass value="0.001"/>
+                <inertia ixx="0.001" iyy="0.001" izz="0.001" ixy="0.0" ixz="0.0" iyz="0.0"/>
             </inertial>
         </link>
         <link name="tether_0/small_link_2_1">
             <inertial>
-                <mass value="1e-05"/>
-                <inertia ixx="1e-05" iyy="1e-05" izz="1e-05" ixy="0.0" ixz="0.0" iyz="0.0"/>
+                <mass value="0.001"/>
+                <inertia ixx="0.001" iyy="0.001" izz="0.001" ixy="0.0" ixz="0.0" iyz="0.0"/>
             </inertial>
         </link>
@@ -49,4 +59,5 @@
             <child link="tether_0/small_link_1_1"/>
             <axis xyz="1 0 0" />
+            <dynamics damping="0.01" friction="0.15"/>
         </joint>
         <joint name="tether_0/joint_2_1" type="continuous">
@@ -54,4 +65,5 @@
             <child link="tether_0/small_link_2_1"/>
             <axis xyz="0 1 0" />
+            <dynamics damping="0.01" friction="0.15"/>
         </joint>
         <joint name="tether_0/joint_1_1_" type="continuous">
@@ -59,4 +71,5 @@
             <child link="tether_0/fragment_1"/>
             <axis xyz="0 0 1" />
+            <dynamics damping="0.01" friction="0.15"/>
         </joint>
             <link name="tether_0/fragment_2">
@@ -64,24 +77,29 @@
                 <origin rpy="0 0 0" xyz="0 0 0.05"/>
                 <geometry>
-                    <cylinder length="0.1" radius="0.001"/>
-                </geometry>
-                <!--material name="black"/-->
-            </visual>
-            <inertial>
-                <mass value="0.0001"/>
-                <inertia ixx="8.33583333333e-08" iyy="8.33583333333e-08" izz="5e-11" ixy="0.0" ixz="0.0" iyz="0.0"/>
-            </inertial>
+                    <cylinder length="0.1" radius="0.0033"/>
+                </geometry>
+                <!--material name="black"/-->
+            </visual>
+            <inertial>
+                <mass value="0.012"/>
+                <inertia ixx="1.003267e-05" iyy="1.003267e-05" izz="6.534e-08" ixy="0.0" ixz="0.0" iyz="0.0"/>
+            </inertial>
+            <collision>
+                <geometry>
+                    <cylinder length="0.1" radius="0.0033"/>
+                </geometry>
+            </collision>
         </link>
                     <!--link between two tether fragments-->
         <link name="tether_0/small_link_1_2">
             <inertial>
-                <mass value="1e-05"/>
-                <inertia ixx="1e-05" iyy="1e-05" izz="1e-05" ixy="0.0" ixz="0.0" iyz="0.0"/>
+                <mass value="0.001"/>
+                <inertia ixx="0.001" iyy="0.001" izz="0.001" ixy="0.0" ixz="0.0" iyz="0.0"/>
             </inertial>
         </link>
         <link name="tether_0/small_link_2_2">
             <inertial>
-                <mass value="1e-05"/>
-                <inertia ixx="1e-05" iyy="1e-05" izz="1e-05" ixy="0.0" ixz="0.0" iyz="0.0"/>
+                <mass value="0.001"/>
+                <inertia ixx="0.001" iyy="0.001" izz="0.001" ixy="0.0" ixz="0.0" iyz="0.0"/>
             </inertial>
         </link>
@@ -92,4 +110,5 @@
             <child link="tether_0/small_link_1_2"/>
             <axis xyz="1 0 0" />
+            <dynamics damping="0.01" friction="0.15"/>
         </joint>
         <joint name="tether_0/joint_2_2" type="continuous">
@@ -97,4 +116,5 @@
             <child link="tether_0/small_link_2_2"/>
             <axis xyz="0 1 0" />
+            <dynamics damping="0.01" friction="0.15"/>
         </joint>
         <joint name="tether_0/joint_1_2_" type="continuous">
@@ -102,4 +122,5 @@
             <child link="tether_0/fragment_2"/>
             <axis xyz="0 0 1" />
+            <dynamics damping="0.01" friction="0.15"/>
         </joint>
             <link name="tether_0/fragment_3">
@@ -107,24 +128,29 @@
                 <origin rpy="0 0 0" xyz="0 0 0.05"/>
                 <geometry>
-                    <cylinder length="0.1" radius="0.001"/>
-                </geometry>
-                <!--material name="black"/-->
-            </visual>
-            <inertial>
-                <mass value="0.0001"/>
-                <inertia ixx="8.33583333333e-08" iyy="8.33583333333e-08" izz="5e-11" ixy="0.0" ixz="0.0" iyz="0.0"/>
-            </inertial>
+                    <cylinder length="0.1" radius="0.0033"/>
+                </geometry>
+                <!--material name="black"/-->
+            </visual>
+            <inertial>
+                <mass value="0.012"/>
+                <inertia ixx="1.003267e-05" iyy="1.003267e-05" izz="6.534e-08" ixy="0.0" ixz="0.0" iyz="0.0"/>
+            </inertial>
+            <collision>
+                <geometry>
+                    <cylinder length="0.1" radius="0.0033"/>
+                </geometry>
+            </collision>
         </link>
                     <!--link between two tether fragments-->
         <link name="tether_0/small_link_1_3">
             <inertial>
-                <mass value="1e-05"/>
-                <inertia ixx="1e-05" iyy="1e-05" izz="1e-05" ixy="0.0" ixz="0.0" iyz="0.0"/>
+                <mass value="0.001"/>
+                <inertia ixx="0.001" iyy="0.001" izz="0.001" ixy="0.0" ixz="0.0" iyz="0.0"/>
             </inertial>
         </link>
         <link name="tether_0/small_link_2_3">
             <inertial>
-                <mass value="1e-05"/>
-                <inertia ixx="1e-05" iyy="1e-05" izz="1e-05" ixy="0.0" ixz="0.0" iyz="0.0"/>
+                <mass value="0.001"/>
+                <inertia ixx="0.001" iyy="0.001" izz="0.001" ixy="0.0" ixz="0.0" iyz="0.0"/>
             </inertial>
         </link>
@@ -135,4 +161,5 @@
             <child link="tether_0/small_link_1_3"/>
             <axis xyz="1 0 0" />
+            <dynamics damping="0.01" friction="0.15"/>
         </joint>
         <joint name="tether_0/joint_2_3" type="continuous">
@@ -140,4 +167,5 @@
             <child link="tether_0/small_link_2_3"/>
             <axis xyz="0 1 0" />
+            <dynamics damping="0.01" friction="0.15"/>
         </joint>
         <joint name="tether_0/joint_1_3_" type="continuous">
@@ -145,4 +173,5 @@
             <child link="tether_0/fragment_3"/>
             <axis xyz="0 0 1" />
+            <dynamics damping="0.01" friction="0.15"/>
         </joint>
             <link name="tether_0/fragment_4">
@@ -150,24 +179,29 @@
                 <origin rpy="0 0 0" xyz="0 0 0.05"/>
                 <geometry>
-                    <cylinder length="0.1" radius="0.001"/>
-                </geometry>
-                <!--material name="black"/-->
-            </visual>
-            <inertial>
-                <mass value="0.0001"/>
-                <inertia ixx="8.33583333333e-08" iyy="8.33583333333e-08" izz="5e-11" ixy="0.0" ixz="0.0" iyz="0.0"/>
-            </inertial>
+                    <cylinder length="0.1" radius="0.0033"/>
+                </geometry>
+                <!--material name="black"/-->
+            </visual>
+            <inertial>
+                <mass value="0.012"/>
+                <inertia ixx="1.003267e-05" iyy="1.003267e-05" izz="6.534e-08" ixy="0.0" ixz="0.0" iyz="0.0"/>
+            </inertial>
+            <collision>
+                <geometry>
+                    <cylinder length="0.1" radius="0.0033"/>
+                </geometry>
+            </collision>
         </link>
                     <!--link between two tether fragments-->
         <link name="tether_0/small_link_1_4">
             <inertial>
-                <mass value="1e-05"/>
-                <inertia ixx="1e-05" iyy="1e-05" izz="1e-05" ixy="0.0" ixz="0.0" iyz="0.0"/>
+                <mass value="0.001"/>
+                <inertia ixx="0.001" iyy="0.001" izz="0.001" ixy="0.0" ixz="0.0" iyz="0.0"/>
             </inertial>
         </link>
         <link name="tether_0/small_link_2_4">
             <inertial>
-                <mass value="1e-05"/>
-                <inertia ixx="1e-05" iyy="1e-05" izz="1e-05" ixy="0.0" ixz="0.0" iyz="0.0"/>
+                <mass value="0.001"/>
+                <inertia ixx="0.001" iyy="0.001" izz="0.001" ixy="0.0" ixz="0.0" iyz="0.0"/>
             </inertial>
         </link>
@@ -178,4 +212,5 @@
             <child link="tether_0/small_link_1_4"/>
             <axis xyz="1 0 0" />
+            <dynamics damping="0.01" friction="0.15"/>
         </joint>
         <joint name="tether_0/joint_2_4" type="continuous">
@@ -183,4 +218,5 @@
             <child link="tether_0/small_link_2_4"/>
             <axis xyz="0 1 0" />
+            <dynamics damping="0.01" friction="0.15"/>
         </joint>
         <joint name="tether_0/joint_1_4_" type="continuous">
@@ -188,4 +224,5 @@
             <child link="tether_0/fragment_4"/>
             <axis xyz="0 0 1" />
+            <dynamics damping="0.01" friction="0.15"/>
         </joint>
             <link name="tether_0/fragment_5">
@@ -193,24 +230,29 @@
                 <origin rpy="0 0 0" xyz="0 0 0.05"/>
                 <geometry>
-                    <cylinder length="0.1" radius="0.001"/>
-                </geometry>
-                <!--material name="black"/-->
-            </visual>
-            <inertial>
-                <mass value="0.0001"/>
-                <inertia ixx="8.33583333333e-08" iyy="8.33583333333e-08" izz="5e-11" ixy="0.0" ixz="0.0" iyz="0.0"/>
-            </inertial>
+                    <cylinder length="0.1" radius="0.0033"/>
+                </geometry>
+                <!--material name="black"/-->
+            </visual>
+            <inertial>
+                <mass value="0.012"/>
+                <inertia ixx="1.003267e-05" iyy="1.003267e-05" izz="6.534e-08" ixy="0.0" ixz="0.0" iyz="0.0"/>
+            </inertial>
+            <collision>
+                <geometry>
+                    <cylinder length="0.1" radius="0.0033"/>
+                </geometry>
+            </collision>
         </link>
                     <!--link between two tether fragments-->
         <link name="tether_0/small_link_1_5">
             <inertial>
-                <mass value="1e-05"/>
-                <inertia ixx="1e-05" iyy="1e-05" izz="1e-05" ixy="0.0" ixz="0.0" iyz="0.0"/>
+                <mass value="0.001"/>
+                <inertia ixx="0.001" iyy="0.001" izz="0.001" ixy="0.0" ixz="0.0" iyz="0.0"/>
             </inertial>
         </link>
         <link name="tether_0/small_link_2_5">
             <inertial>
-                <mass value="1e-05"/>
-                <inertia ixx="1e-05" iyy="1e-05" izz="1e-05" ixy="0.0" ixz="0.0" iyz="0.0"/>
+                <mass value="0.001"/>
+                <inertia ixx="0.001" iyy="0.001" izz="0.001" ixy="0.0" ixz="0.0" iyz="0.0"/>
             </inertial>
         </link>
@@ -221,4 +263,5 @@
             <child link="tether_0/small_link_1_5"/>
             <axis xyz="1 0 0" />
+            <dynamics damping="0.01" friction="0.15"/>
         </joint>
         <joint name="tether_0/joint_2_5" type="continuous">
@@ -226,4 +269,5 @@
             <child link="tether_0/small_link_2_5"/>
             <axis xyz="0 1 0" />
+            <dynamics damping="0.01" friction="0.15"/>
         </joint>
         <joint name="tether_0/joint_1_5_" type="continuous">
@@ -231,4 +275,5 @@
             <child link="tether_0/fragment_5"/>
             <axis xyz="0 0 1" />
+            <dynamics damping="0.01" friction="0.15"/>
         </joint>
             <link name="tether_0/fragment_6">
@@ -236,24 +281,29 @@
                 <origin rpy="0 0 0" xyz="0 0 0.05"/>
                 <geometry>
-                    <cylinder length="0.1" radius="0.001"/>
-                </geometry>
-                <!--material name="black"/-->
-            </visual>
-            <inertial>
-                <mass value="0.0001"/>
-                <inertia ixx="8.33583333333e-08" iyy="8.33583333333e-08" izz="5e-11" ixy="0.0" ixz="0.0" iyz="0.0"/>
-            </inertial>
+                    <cylinder length="0.1" radius="0.0033"/>
+                </geometry>
+                <!--material name="black"/-->
+            </visual>
+            <inertial>
+                <mass value="0.012"/>
+                <inertia ixx="1.003267e-05" iyy="1.003267e-05" izz="6.534e-08" ixy="0.0" ixz="0.0" iyz="0.0"/>
+            </inertial>
+            <collision>
+                <geometry>
+                    <cylinder length="0.1" radius="0.0033"/>
+                </geometry>
+            </collision>
         </link>
                     <!--link between two tether fragments-->
         <link name="tether_0/small_link_1_6">
             <inertial>
-                <mass value="1e-05"/>
-                <inertia ixx="1e-05" iyy="1e-05" izz="1e-05" ixy="0.0" ixz="0.0" iyz="0.0"/>
+                <mass value="0.001"/>
+                <inertia ixx="0.001" iyy="0.001" izz="0.001" ixy="0.0" ixz="0.0" iyz="0.0"/>
             </inertial>
         </link>
         <link name="tether_0/small_link_2_6">
             <inertial>
-                <mass value="1e-05"/>
-                <inertia ixx="1e-05" iyy="1e-05" izz="1e-05" ixy="0.0" ixz="0.0" iyz="0.0"/>
+                <mass value="0.001"/>
+                <inertia ixx="0.001" iyy="0.001" izz="0.001" ixy="0.0" ixz="0.0" iyz="0.0"/>
             </inertial>
         </link>
@@ -264,4 +314,5 @@
             <child link="tether_0/small_link_1_6"/>
             <axis xyz="1 0 0" />
+            <dynamics damping="0.01" friction="0.15"/>
         </joint>
         <joint name="tether_0/joint_2_6" type="continuous">
@@ -269,4 +320,5 @@
             <child link="tether_0/small_link_2_6"/>
             <axis xyz="0 1 0" />
+            <dynamics damping="0.01" friction="0.15"/>
         </joint>
         <joint name="tether_0/joint_1_6_" type="continuous">
@@ -274,4 +326,5 @@
             <child link="tether_0/fragment_6"/>
             <axis xyz="0 0 1" />
+            <dynamics damping="0.01" friction="0.15"/>
         </joint>
             <link name="tether_0/fragment_7">
@@ -279,24 +332,29 @@
                 <origin rpy="0 0 0" xyz="0 0 0.05"/>
                 <geometry>
-                    <cylinder length="0.1" radius="0.001"/>
-                </geometry>
-                <!--material name="black"/-->
-            </visual>
-            <inertial>
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
File: tether_description/urdf/tether_fragment.xacro (robot description, xacro)
@@ -4,22 +4,25 @@
     <xacro:macro name="tether">
         <!--tether fragment param-->
-        {%- set cyl_r = 0.001 -%}
+        {%- set cyl_r = 0.0033 -%}
         {%- set cyl_l = 0.1 -%}
-        {%- set cyl_m = 0.0001 -%}
+        {%- set cyl_m = 0.012 -%}
         {%- set cyl_i = 1/12*cyl_m*(3*cyl_r**2+cyl_l**2) -%}
         {%- set cyl_iz = 1/2*cyl_m*cyl_r**2 -%}
         <!--small link inatial-->
-        {%- set small_link_mass = 0.00001 -%}
-        {%- set small_link_ixx = 0.00001 -%}
-        {%- set small_link_iyy = 0.00001 -%}
-        {%- set small_link_izz = 0.00001 -%}
+        {%- set small_link_mass = 0.001 -%}
+        {%- set small_link_ixx = 0.001 -%}
+        {%- set small_link_iyy = 0.001 -%}
+        {%- set small_link_izz = 0.001 -%}
         {%- set small_link_ixy = 0.0 -%}
         {%- set small_link_ixz = 0.0 -%}
         {%- set small_link_iyz = 0.0 -%}
+        <!--joint dynamics-->
+        {%- set damping = 0.01 -%}
+        {%- set friction = 0.15 -%}
         <!--link number-->
         {%- set tether_fragments = 30 -%}
         {%- set tether_number = 4 -%}
         <!--box inertial-->
-        {%- set box_m = 0.50 -%}
+        {%- set box_m = 50 -%}
         {%- set box_x = 0.1 -%}
         {%- set box_y = 0.1 -%}
@@ -38,4 +41,9 @@
                 <inertia ixx="{{cyl_i}}" iyy="{{cyl_i}}" izz="{{cyl_iz}}" ixy="0.0" ixz="0.0" iyz="0.0"/>
             </inertial>
+            <collision>
+                <geometry>
+                    <cylinder length="{{cyl_l}}" radius="{{cyl_r}}"/>
+                </geometry>
+            </collision>
         </link>
         {%- endmacro -%}
@@ -61,4 +69,5 @@
             <child link="tether_{{dirc}}/small_link_1_{{n}}"/>
             <axis xyz="1 0 0" />
+            <dynamics damping="{{damping}}" friction="{{friction}}"/>
         </joint>
         <joint name="tether_{{dirc}}/joint_2_{{n}}" type="continuous">
@@ -66,4 +75,5 @@
             <child link="tether_{{dirc}}/small_link_2_{{n}}"/>
             <axis xyz="0 1 0" />
+            <dynamics damping="{{damping}}" friction="{{friction}}"/>
         </joint>
         <joint name="tether_{{dirc}}/joint_1_{{n}}_" type="continuous">
@@ -71,4 +81,5 @@
             <child link="tether_{{dirc}}/fragment_{{n}}"/>
             <axis xyz="0 0 1" />
+            <dynamics damping="{{damping}}" friction="{{friction}}"/>
         </joint>
         {%- endmacro -%}
