Commit message: connect uav and ugv

File: tether_description/urdf/tether.xacro (robot description, xacro)
@@ -1507,25 +1507,36 @@
                 <origin rpy="0 ${pi/2} 0" xyz="0 0 0"/>
         </joint>
-            <link name="pesudo_ugv_0">
-            <visual>
-                <geometry>
-                    <box size="0.1 0.1 0.1"/>
-                </geometry>
-                <material name="silver">
-                    <color rgba="0.75 0.75 0.75 1"/>
-                </material>
-            </visual>
-            <collision>
-                <geometry>
-                    <box size="0.1 0.1 0.1"/>
-                </geometry>
-            </collision>
-            <inertial>
-                <mass value="50"/><inertia ixx="0.0833333333333" iyy="0.0833333333333" izz="0.0833333333333" ixy="0" ixz="0" iyz="0"/>
-            </inertial>
-        </link>
-        <joint name="tether_0/pesudo_ugv_joint" type="fixed">
+            <!--link between tether and ugv-->
+        <link name="tether_0/end_link_1">
+            <inertial>
+                <mass value="0.001"/>
+                <inertia ixx="0.001" iyy="0.001" izz="0.001" ixy="0.0" ixz="0.0" iyz="0.0"/>
+            </inertial>
+        </link>
+        <link name="tether_0/end_link_2">
+            <inertial>
+                <mass value="0.001"/>
+                <inertia ixx="0.001" iyy="0.001" izz="0.001" ixy="0.0" ixz="0.0" iyz="0.0"/>
+            </inertial>
+        </link>
+        <!--tether end joint-->
+        <joint name="tether_0/ugv_joint_1" type="continuous">
+            <origin rpy="0 ${-pi/2} 0" xyz="0 0 0"/>
             <parent link="tether_0/fragment_29"/>
-            <child link="pesudo_ugv_0"/>
+            <child link="tether_0/end_link_1"/>
+            <axis xyz="1 0 0" />
+            <dynamics damping="0.01" friction="0.15"/>
+        </joint>
+        <joint name="tether_0/ugv_joint_2" type="continuous">
+            <parent link="tether_0/end_link_1"/>
+            <child link="tether_0/end_link_2"/>
+            <axis xyz="0 1 0" />
+            <dynamics damping="0.01" friction="0.15"/>
+        </joint>
+        <joint name="tether_0/ugv_joint_3" type="continuous">
+            <parent link="tether_0/end_link_2"/>
+            <child link="mp_500_0/tether_end"/>
+            <axis xyz="0 0 1" />
+            <dynamics damping="0.01" friction="0.15"/>
         </joint>
             <link name="tether_1/fragment_0">
@@ -3032,25 +3043,36 @@
                 <origin rpy="${pi/2} 0 0" xyz="0 0 0"/>
         </joint>
-            <link name="pesudo_ugv_1">
-            <visual>
-                <geometry>
-                    <box size="0.1 0.1 0.1"/>
-                </geometry>
-                <material name="silver">
-                    <color rgba="0.75 0.75 0.75 1"/>
-                </material>
-            </visual>
-            <collision>
-                <geometry>
-                    <box size="0.1 0.1 0.1"/>
-                </geometry>
-            </collision>
-            <inertial>
-                <mass value="50"/><inertia ixx="0.0833333333333" iyy="0.0833333333333" izz="0.0833333333333" ixy="0" ixz="0" iyz="0"/>
-            </inertial>
-        </link>
-        <joint name="tether_1/pesudo_ugv_joint" type="fixed">
+            <!--link between tether and ugv-->
+        <link name="tether_1/end_link_1">
+            <inertial>
+                <mass value="0.001"/>
+                <inertia ixx="0.001" iyy="0.001" izz="0.001" ixy="0.0" ixz="0.0" iyz="0.0"/>
+            </inertial>
+        </link>
+        <link name="tether_1/end_link_2">
+            <inertial>
+                <mass value="0.001"/>
+                <inertia ixx="0.001" iyy="0.001" izz="0.001" ixy="0.0" ixz="0.0" iyz="0.0"/>
+            </inertial>
+        </link>
+        <!--tether end joint-->
+        <joint name="tether_1/ugv_joint_1" type="continuous">
+            <origin rpy="0 ${-pi/2} 0" xyz="0 0 0"/>
             <parent link="tether_1/fragment_29"/>
-            <child link="pesudo_ugv_1"/>
+            <child link="tether_1/end_link_1"/>
+            <axis xyz="1 0 0" />
+            <dynamics damping="0.01" friction="0.15"/>
+        </joint>
+        <joint name="tether_1/ugv_joint_2" type="continuous">
+            <parent link="tether_1/end_link_1"/>
+            <child link="tether_1/end_link_2"/>
+            <axis xyz="0 1 0" />
+            <dynamics damping="0.01" friction="0.15"/>
+        </joint>
+        <joint name="tether_1/ugv_joint_3" type="continuous">
+            <parent link="tether_1/end_link_2"/>
+            <child link="mp_500_1/tether_end"/>
+            <axis xyz="0 0 1" />
+            <dynamics damping="0.01" friction="0.15"/>
         </joint>
             <link name="tether_2/fragment_0">
@@ -4557,25 +4579,36 @@
                 <origin rpy="0 ${-pi/2} 0" xyz="0 0 0"/>
         </joint>
-            <link name="pesudo_ugv_2">
-            <visual>
-                <geometry>
-                    <box size="0.1 0.1 0.1"/>
-                </geometry>
-                <material name="silver">
-                    <color rgba="0.75 0.75 0.75 1"/>
-                </material>
-            </visual>
-            <collision>
-                <geometry>
-                    <box size="0.1 0.1 0.1"/>
-                </geometry>
-            </collision>
-            <inertial>
-                <mass value="50"/><inertia ixx="0.0833333333333" iyy="0.0833333333333" izz="0.0833333333333" ixy="0" ixz="0" iyz="0"/>
-            </inertial>
-        </link>
-        <joint name="tether_2/pesudo_ugv_joint" type="fixed">
+            <!--link between tether and ugv-->
+        <link name="tether_2/end_link_1">
+            <inertial>
+                <mass value="0.001"/>
+                <inertia ixx="0.001" iyy="0.001" izz="0.001" ixy="0.0" ixz="0.0" iyz="0.0"/>
+            </inertial>
+        </link>
+        <link name="tether_2/end_link_2">
+            <inertial>
+                <mass value="0.001"/>
+                <inertia ixx="0.001" iyy="0.001" izz="0.001" ixy="0.0" ixz="0.0" iyz="0.0"/>
+            </inertial>
+        </link>
+        <!--tether end joint-->
+        <joint name="tether_2/ugv_joint_1" type="continuous">
+            <origin rpy="0 ${-pi/2} 0" xyz="0 0 0"/>
             <parent link="tether_2/fragment_29"/>
-            <child link="pesudo_ugv_2"/>
+            <child link="tether_2/end_link_1"/>
+            <axis xyz="1 0 0" />
+            <dynamics damping="0.01" friction="0.15"/>
+        </joint>
+        <joint name="tether_2/ugv_joint_2" type="continuous">
+            <parent link="tether_2/end_link_1"/>
+            <child link="tether_2/end_link_2"/>
+            <axis xyz="0 1 0" />
+            <dynamics damping="0.01" friction="0.15"/>
+        </joint>
+        <joint name="tether_2/ugv_joint_3" type="continuous">
+            <parent link="tether_2/end_link_2"/>
+            <child link="mp_500_2/tether_end"/>
+            <axis xyz="0 0 1" />
+            <dynamics damping="0.01" friction="0.15"/>
         </joint>
             <link name="tether_3/fragment_0">
@@ -6082,25 +6115,36 @@
                 <origin rpy="${-pi/2} 0 0" xyz="0 0 0"/>
         </joint>
-            <link name="pesudo_ugv_3">
-            <visual>
-                <geometry>
-                    <box size="0.1 0.1 0.1"/>
-                </geometry>
-                <material name="silver">
-                    <color rgba="0.75 0.75 0.75 1"/>
-                </material>
-            </visual>
-            <collision>
-                <geometry>
-                    <box size="0.1 0.1 0.1"/>
-                </geometry>
-            </collision>
-            <inertial>
-                <mass value="50"/><inertia ixx="0.0833333333333" iyy="0.0833333333333" izz="0.0833333333333" ixy="0" ixz="0" iyz="0"/>
-            </inertial>
-        </link>
-        <joint name="tether_3/pesudo_ugv_joint" type="fixed">
+            <!--link between tether and ugv-->
+        <link name="tether_3/end_link_1">
+            <inertial>
+                <mass value="0.001"/>
+                <inertia ixx="0.001" iyy="0.001" izz="0.001" ixy="0.0" ixz="0.0" iyz="0.0"/>
+            </inertial>
+        </link>
+        <link name="tether_3/end_link_2">
+            <inertial>
+                <mass value="0.001"/>
+                <inertia ixx="0.001" iyy="0.001" izz="0.001" ixy="0.0" ixz="0.0" iyz="0.0"/>
+            </inertial>
+        </link>
+        <!--tether end joint-->
+        <joint name="tether_3/ugv_joint_1" type="continuous">
+            <origin rpy="0 ${-pi/2} 0" xyz="0 0 0"/>
             <parent link="tether_3/fragment_29"/>
-            <child link="pesudo_ugv_3"/>
+            <child link="tether_3/end_link_1"/>
+            <axis xyz="1 0 0" />
+            <dynamics damping="0.01" friction="0.15"/>
+        </joint>
+        <joint name="tether_3/ugv_joint_2" type="continuous">
+            <parent link="tether_3/end_link_1"/>
+            <child link="tether_3/end_link_2"/>
+            <axis xyz="0 1 0" />
+            <dynamics damping="0.01" friction="0.15"/>
+        </joint>
+        <joint name="tether_3/ugv_joint_3" type="continuous">
+            <parent link="tether_3/end_link_2"/>
+            <child link="mp_500_3/tether_end"/>
+            <axis xyz="0 0 1" />
+            <dynamics damping="0.01" friction="0.15"/>
         </joint>
         </xacro:macro>

File: tether_description/urdf/tether_fragment_pseudo.xacro (robot description, xacro)
@@ -100,37 +100,30 @@
         </joint>
         {%- endmacro -%}
-        {%- macro ugv_joint(dirc) -%}
-        <!--link between tether and ugv-->
-        <link name="tether_{{dirc}}/end_link_1">
+        {%- macro pesudo_ugv(dirc) -%}
+        <link name="pesudo_ugv_{{dirc}}">
+            <visual>
+                <geometry>
+                    <box size="{{box_x}} {{box_y}} {{box_z}}"/>
+                </geometry>
+                <material name="silver">
+                    <color rgba="0.75 0.75 0.75 1"/>
+                </material>
+            </visual>
+            <collision>
+                <geometry>
+                    <box size="{{box_x}} {{box_y}} {{box_z}}"/>
+                </geometry>
+            </collision>
             <inertial>
-                <mass value="{{small_link_mass}}"/>
-                <inertia ixx="{{small_link_ixx}}" iyy="{{small_link_iyy}}" izz="{{small_link_izz}}" ixy="{{small_link_ixy}}" ixz="{{small_link_ixz}}" iyz="{{small_link_iyz}}"/>
+                <mass value="{{box_m}}"/>
+                {%- set box_ix = 1/12*box_m*(box_y**2+box_z**2) -%}
+                {%- set box_iy = 1/12*box_m*(box_x**2+box_z**2) -%}
+                {%- set box_iz = 1/12*box_m*(box_x**2+box_y**2) -%}
+                <inertia ixx="{{box_ix}}" iyy="{{box_iy}}" izz="{{box_iz}}" ixy="0" ixz="0" iyz="0"/>
             </inertial>
         </link>
-        <link name="tether_{{dirc}}/end_link_2">
-            <inertial>
-                <mass value="{{small_link_mass}}"/>
-                <inertia ixx="{{small_link_ixx}}" iyy="{{small_link_iyy}}" izz="{{small_link_izz}}" ixy="{{small_link_ixy}}" ixz="{{small_link_ixz}}" iyz="{{small_link_iyz}}"/>
-            </inertial>
-        </link>
-        <!--tether end joint-->
-        <joint name="tether_{{dirc}}/ugv_joint_1" type="continuous">
-            <origin rpy="0 ${-pi/2} 0" xyz="0 0 0"/>
+        <joint name="tether_{{dirc}}/pesudo_ugv_joint" type="fixed">
             <parent link="tether_{{dirc}}/fragment_{{tether_fragments-1}}"/>
-            <child link="tether_{{dirc}}/end_link_1"/>
-            <axis xyz="1 0 0" />
-            <dynamics damping="{{damping}}" friction="{{friction}}"/>
-        </joint>
-        <joint name="tether_{{dirc}}/ugv_joint_2" type="continuous">
-            <parent link="tether_{{dirc}}/end_link_1"/>
-            <child link="tether_{{dirc}}/end_link_2"/>
-            <axis xyz="0 1 0" />
-            <dynamics damping="{{damping}}" friction="{{friction}}"/>
-        </joint>
-        <joint name="tether_{{dirc}}/ugv_joint_3" type="continuous">
-            <parent link="tether_{{dirc}}/end_link_2"/>
-            <child link="mp_500_{{dirc}}/tether_end"/>
-            <axis xyz="0 0 1" />
-            <dynamics damping="{{damping}}" friction="{{friction}}"/>
+            <child link="pesudo_ugv_{{dirc}}"/>
         </joint>
         {%- endmacro -%}
@@ -144,5 +137,5 @@
             {% endfor -%}
             {{uav_joint(dirc)}}
-            {{ugv_joint(dirc)}}
+            {{pesudo_ugv(dirc)}}
         {% endfor -%}
     </xacro:macro>

File: world_description/urdf/uav_2_ugv_ex.xacro (robot description, xacro)
@@ -14,8 +14,3 @@
         <xacro:tether />
     </xacro:if>
-    <xacro:include filename="$(find ugv_description)/urdf/mp_500/mp_500_tether.urdf.xacro"/>
-    <xacro:mp_500_tether namespace="mp_500_0"/>
-    <xacro:mp_500_tether namespace="mp_500_1"/>
-    <xacro:mp_500_tether namespace="mp_500_2"/>
-    <xacro:mp_500_tether namespace="mp_500_3"/>
 </robot>

Commit message: fix bugs & could control uav and ugv with tether

File: tether_description/urdf/tether.xacro (robot description, xacro)
@@ -1522,5 +1522,5 @@
         <!--tether end joint-->
         <joint name="tether_0/ugv_joint_1" type="continuous">
-            <origin rpy="0 ${-pi/2} 0" xyz="0 0 0"/>
+                <origin rpy="0 ${-pi/2} 0" xyz="0 0 0"/>
             <parent link="tether_0/fragment_29"/>
             <child link="tether_0/end_link_1"/>
@@ -3058,5 +3058,5 @@
         <!--tether end joint-->
         <joint name="tether_1/ugv_joint_1" type="continuous">
-            <origin rpy="0 ${-pi/2} 0" xyz="0 0 0"/>
+                <origin rpy="${-pi/2} 0 0" xyz="0 0 0"/>
             <parent link="tether_1/fragment_29"/>
             <child link="tether_1/end_link_1"/>
@@ -4594,5 +4594,5 @@
         <!--tether end joint-->
         <joint name="tether_2/ugv_joint_1" type="continuous">
-            <origin rpy="0 ${-pi/2} 0" xyz="0 0 0"/>
+                <origin rpy="0 ${pi/2} 0" xyz="0 0 0"/>
             <parent link="tether_2/fragment_29"/>
             <child link="tether_2/end_link_1"/>
@@ -6130,5 +6130,5 @@
         <!--tether end joint-->
         <joint name="tether_3/ugv_joint_1" type="continuous">
-            <origin rpy="0 ${-pi/2} 0" xyz="0 0 0"/>
+                <origin rpy="${pi/2} 0 0" xyz="0 0 0"/>
             <parent link="tether_3/fragment_29"/>
             <child link="tether_3/end_link_1"/>

File: tether_description/urdf/tether_fragment.xacro (robot description, xacro)
@@ -116,5 +116,13 @@
         <!--tether end joint-->
         <joint name="tether_{{dirc}}/ugv_joint_1" type="continuous">
-            <origin rpy="0 ${-pi/2} 0" xyz="0 0 0"/>
+            {% if dirc == 0 %}
+                <origin rpy="0 ${-pi/2} 0" xyz="0 0 0"/>
+            {% elif dirc == 1 %}
+                <origin rpy="${-pi/2} 0 0" xyz="0 0 0"/>
+            {% elif dirc == 2 %}
+                <origin rpy="0 ${pi/2} 0" xyz="0 0 0"/>
+            {% elif dirc == 3 %}
+                <origin rpy="${pi/2} 0 0" xyz="0 0 0"/>
+            {% endif %}
             <parent link="tether_{{dirc}}/fragment_{{tether_fragments-1}}"/>
             <child link="tether_{{dirc}}/end_link_1"/>
