Commit message: clean up

File: tether_description/urdf/tether.xacro (robot description, xacro)
@@ -59,5 +59,5 @@
             <child link="tether_0/small_link_1_1"/>
             <axis xyz="1 0 0" />
-            <dynamics damping="0.01" friction="0.15"/>
+            <dynamics damping="0.01" friction="0.01"/>
         </joint>
         <joint name="tether_0/joint_2_1" type="continuous">
@@ -65,5 +65,5 @@
             <child link="tether_0/small_link_2_1"/>
             <axis xyz="0 1 0" />
-            <dynamics damping="0.01" friction="0.15"/>
+            <dynamics damping="0.01" friction="0.01"/>
         </joint>
         <joint name="tether_0/joint_1_1_" type="continuous">
@@ -71,5 +71,5 @@
             <child link="tether_0/fragment_1"/>
             <axis xyz="0 0 1" />
-            <dynamics damping="0.01" friction="0.15"/>
+            <dynamics damping="0.01" friction="0.01"/>
         </joint>
             <link name="tether_0/fragment_2">
@@ -110,5 +110,5 @@
             <child link="tether_0/small_link_1_2"/>
             <axis xyz="1 0 0" />
-            <dynamics damping="0.01" friction="0.15"/>
+            <dynamics damping="0.01" friction="0.01"/>
         </joint>
         <joint name="tether_0/joint_2_2" type="continuous">
@@ -116,5 +116,5 @@
             <child link="tether_0/small_link_2_2"/>
             <axis xyz="0 1 0" />
-            <dynamics damping="0.01" friction="0.15"/>
+            <dynamics damping="0.01" friction="0.01"/>
         </joint>
         <joint name="tether_0/joint_1_2_" type="continuous">
@@ -122,5 +122,5 @@
             <child link="tether_0/fragment_2"/>
             <axis xyz="0 0 1" />
-            <dynamics damping="0.01" friction="0.15"/>
+            <dynamics damping="0.01" friction="0.01"/>
         </joint>
             <link name="tether_0/fragment_3">
@@ -161,5 +161,5 @@
             <child link="tether_0/small_link_1_3"/>
             <axis xyz="1 0 0" />
-            <dynamics damping="0.01" friction="0.15"/>
+            <dynamics damping="0.01" friction="0.01"/>
         </joint>
         <joint name="tether_0/joint_2_3" type="continuous">
@@ -167,5 +167,5 @@
             <child link="tether_0/small_link_2_3"/>
             <axis xyz="0 1 0" />
-            <dynamics damping="0.01" friction="0.15"/>
+            <dynamics damping="0.01" friction="0.01"/>
         </joint>
         <joint name="tether_0/joint_1_3_" type="continuous">
@@ -173,5 +173,5 @@
             <child link="tether_0/fragment_3"/>
             <axis xyz="0 0 1" />
-            <dynamics damping="0.01" friction="0.15"/>
+            <dynamics damping="0.01" friction="0.01"/>
         </joint>
             <link name="tether_0/fragment_4">
@@ -212,5 +212,5 @@
             <child link="tether_0/small_link_1_4"/>
             <axis xyz="1 0 0" />
-            <dynamics damping="0.01" friction="0.15"/>
+            <dynamics damping="0.01" friction="0.01"/>
         </joint>
         <joint name="tether_0/joint_2_4" type="continuous">
@@ -218,5 +218,5 @@
             <child link="tether_0/small_link_2_4"/>
             <axis xyz="0 1 0" />
-            <dynamics damping="0.01" friction="0.15"/>
+            <dynamics damping="0.01" friction="0.01"/>
         </joint>
         <joint name="tether_0/joint_1_4_" type="continuous">
@@ -224,5 +224,5 @@
             <child link="tether_0/fragment_4"/>
             <axis xyz="0 0 1" />
-            <dynamics damping="0.01" friction="0.15"/>
+            <dynamics damping="0.01" friction="0.01"/>
         </joint>
             <link name="tether_0/fragment_5">
@@ -263,5 +263,5 @@
             <child link="tether_0/small_link_1_5"/>
             <axis xyz="1 0 0" />
-            <dynamics damping="0.01" friction="0.15"/>
+            <dynamics damping="0.01" friction="0.01"/>
         </joint>
         <joint name="tether_0/joint_2_5" type="continuous">
@@ -269,5 +269,5 @@
             <child link="tether_0/small_link_2_5"/>
             <axis xyz="0 1 0" />
-            <dynamics damping="0.01" friction="0.15"/>
+            <dynamics damping="0.01" friction="0.01"/>
         </joint>
         <joint name="tether_0/joint_1_5_" type="continuous">
@@ -275,5 +275,5 @@
             <child link="tether_0/fragment_5"/>
             <axis xyz="0 0 1" />
-            <dynamics damping="0.01" friction="0.15"/>
+            <dynamics damping="0.01" friction="0.01"/>
         </joint>
             <link name="tether_0/fragment_6">
@@ -314,5 +314,5 @@
             <child link="tether_0/small_link_1_6"/>
             <axis xyz="1 0 0" />
-            <dynamics damping="0.01" friction="0.15"/>
+            <dynamics damping="0.01" friction="0.01"/>
         </joint>
         <joint name="tether_0/joint_2_6" type="continuous">
@@ -320,5 +320,5 @@
             <child link="tether_0/small_link_2_6"/>
             <axis xyz="0 1 0" />
-            <dynamics damping="0.01" friction="0.15"/>
+            <dynamics damping="0.01" friction="0.01"/>
         </joint>
         <joint name="tether_0/joint_1_6_" type="continuous">
@@ -326,5 +326,5 @@
             <child link="tether_0/fragment_6"/>
             <axis xyz="0 0 1" />
-            <dynamics damping="0.01" friction="0.15"/>
+            <dynamics damping="0.01" friction="0.01"/>
         </joint>
             <link name="tether_0/fragment_7">
@@ -365,5 +365,5 @@
             <child link="tether_0/small_link_1_7"/>
             <axis xyz="1 0 0" />
-            <dynamics damping="0.01" friction="0.15"/>
+            <dynamics damping="0.01" friction="0.01"/>
         </joint>
         <joint name="tether_0/joint_2_7" type="continuous">
@@ -371,5 +371,5 @@
             <child link="tether_0/small_link_2_7"/>
             <axis xyz="0 1 0" />
-            <dynamics damping="0.01" friction="0.15"/>
+            <dynamics damping="0.01" friction="0.01"/>
         </joint>
         <joint name="tether_0/joint_1_7_" type="continuous">
@@ -377,5 +377,5 @@
             <child link="tether_0/fragment_7"/>
             <axis xyz="0 0 1" />
-            <dynamics damping="0.01" friction="0.15"/>
+            <dynamics damping="0.01" friction="0.01"/>
         </joint>
             <link name="tether_0/fragment_8">
@@ -416,5 +416,5 @@
             <child link="tether_0/small_link_1_8"/>
             <axis xyz="1 0 0" />
-            <dynamics damping="0.01" friction="0.15"/>
+            <dynamics damping="0.01" friction="0.01"/>
         </joint>
         <joint name="tether_0/joint_2_8" type="continuous">
@@ -422,5 +422,5 @@
             <child link="tether_0/small_link_2_8"/>
             <axis xyz="0 1 0" />
-            <dynamics damping="0.01" friction="0.15"/>
+            <dynamics damping="0.01" friction="0.01"/>
         </joint>
         <joint name="tether_0/joint_1_8_" type="continuous">
@@ -428,5 +428,5 @@
             <child link="tether_0/fragment_8"/>
             <axis xyz="0 0 1" />
-            <dynamics damping="0.01" friction="0.15"/>
+            <dynamics damping="0.01" friction="0.01"/>
         </joint>
             <link name="tether_0/fragment_9">
@@ -467,5 +467,5 @@
             <child link="tether_0/small_link_1_9"/>
             <axis xyz="1 0 0" />
-            <dynamics damping="0.01" friction="0.15"/>
+            <dynamics damping="0.01" friction="0.01"/>
         </joint>
         <joint name="tether_0/joint_2_9" type="continuous">
@@ -473,5 +473,5 @@
             <child link="tether_0/small_link_2_9"/>
             <axis xyz="0 1 0" />
-            <dynamics damping="0.01" friction="0.15"/>
+            <dynamics damping="0.01" friction="0.01"/>
         </joint>
         <joint name="tether_0/joint_1_9_" type="continuous">
@@ -479,5 +479,5 @@
             <child link="tether_0/fragment_9"/>
             <axis xyz="0 0 1" />
-            <dynamics damping="0.01" friction="0.15"/>
+            <dynamics damping="0.01" friction="0.01"/>
         </joint>
             <link name="tether_0/fragment_10">
@@ -518,5 +518,5 @@
             <child link="tether_0/small_link_1_10"/>
             <axis xyz="1 0 0" />
-            <dynamics damping="0.01" friction="0.15"/>
+            <dynamics damping="0.01" friction="0.01"/>
         </joint>
         <joint name="tether_0/joint_2_10" type="continuous">
@@ -524,5 +524,5 @@
             <child link="tether_0/small_link_2_10"/>
             <axis xyz="0 1 0" />
-            <dynamics damping="0.01" friction="0.15"/>
+            <dynamics damping="0.01" friction="0.01"/>
         </joint>
         <joint name="tether_0/joint_1_10_" type="continuous">
@@ -530,5 +530,5 @@
             <child link="tether_0/fragment_10"/>
             <axis xyz="0 0 1" />
-            <dynamics damping="0.01" friction="0.15"/>
+            <dynamics damping="0.01" friction="0.01"/>
         </joint>
             <link name="tether_0/fragment_11">
@@ -569,5 +569,5 @@
             <child link="tether_0/small_link_1_11"/>
             <axis xyz="1 0 0" />
-            <dynamics damping="0.01" friction="0.15"/>
+            <dynamics damping="0.01" friction="0.01"/>
         </joint>
         <joint name="tether_0/joint_2_11" type="continuous">
@@ -575,5 +575,5 @@
             <child link="tether_0/small_link_2_11"/>
             <axis xyz="0 1 0" />
-            <dynamics damping="0.01" friction="0.15"/>
+            <dynamics damping="0.01" friction="0.01"/>
         </joint>
         <joint name="tether_0/joint_1_11_" type="continuous">
@@ -581,5 +581,5 @@
             <child link="tether_0/fragment_11"/>
             <axis xyz="0 0 1" />
-            <dynamics damping="0.01" friction="0.15"/>
+            <dynamics damping="0.01" friction="0.01"/>
         </joint>
             <link name="tether_0/fragment_12">
@@ -620,5 +620,5 @@
             <child link="tether_0/small_link_1_12"/>
             <axis xyz="1 0 0" />
-            <dynamics damping="0.01" friction="0.15"/>
+            <dynamics damping="0.01" friction="0.01"/>
         </joint>
         <joint name="tether_0/joint_2_12" type="continuous">
@@ -626,5 +626,5 @@
             <child link="tether_0/small_link_2_12"/>
             <axis xyz="0 1 0" />
-            <dynamics damping="0.01" friction="0.15"/>
+            <dynamics damping="0.01" friction="0.01"/>
         </joint>
         <joint name="tether_0/joint_1_12_" type="continuous">
@@ -632,5 +632,5 @@
             <child link="tether_0/fragment_12"/>
             <axis xyz="0 0 1" />
-            <dynamics damping="0.01" friction="0.15"/>
+            <dynamics damping="0.01" friction="0.01"/>
         </joint>
             <link name="tether_0/fragment_13">
@@ -671,5 +671,5 @@
             <child link="tether_0/small_link_1_13"/>
             <axis xyz="1 0 0" />
-            <dynamics damping="0.01" friction="0.15"/>
+            <dynamics damping="0.01" friction="0.01"/>
         </joint>
         <joint name="tether_0/joint_2_13" type="continuous">
@@ -677,5 +677,5 @@
             <child link="tether_0/small_link_2_13"/>
             <axis xyz="0 1 0" />
-            <dynamics damping="0.01" friction="0.15"/>
+            <dynamics damping="0.01" friction="0.01"/>
         </joint>
         <joint name="tether_0/joint_1_13_" type="continuous">
@@ -683,5 +683,5 @@
             <child link="tether_0/fragment_13"/>
             <axis xyz="0 0 1" />
-            <dynamics damping="0.01" friction="0.15"/>
+            <dynamics damping="0.01" friction="0.01"/>
         </joint>
             <link name="tether_0/fragment_14">
@@ -722,5 +722,5 @@
             <child link="tether_0/small_link_1_14"/>
             <axis xyz="1 0 0" />
-            <dynamics damping="0.01" friction="0.15"/>
+            <dynamics damping="0.01" friction="0.01"/>
         </joint>
         <joint name="tether_0/joint_2_14" type="continuous">
@@ -728,5 +728,5 @@
             <child link="tether_0/small_link_2_14"/>
             <axis xyz="0 1 0" />
-            <dynamics damping="0.01" friction="0.15"/>
+            <dynamics damping="0.01" friction="0.01"/>
         </joint>
         <joint name="tether_0/joint_1_14_" type="continuous">
@@ -734,5 +734,5 @@
             <child link="tether_0/fragment_14"/>
             <axis xyz="0 0 1" />
-            <dynamics damping="0.01" friction="0.15"/>
+            <dynamics damping="0.01" friction="0.01"/>
         </joint>
             <link name="tether_0/fragment_15">
@@ -773,5 +773,5 @@
             <child link="tether_0/small_link_1_15"/>
             <axis xyz="1 0 0" />
-            <dynamics damping="0.01" friction="0.15"/>
+            <dynamics damping="0.01" friction="0.01"/>
         </joint>
         <joint name="tether_0/joint_2_15" type="continuous">
@@ -779,5 +779,5 @@
             <child link="tether_0/small_link_2_15"/>
             <axis xyz="0 1 0" />
-            <dynamics damping="0.01" friction="0.15"/>
+            <dynamics damping="0.01" friction="0.01"/>
         </joint>
         <joint name="tether_0/joint_1_15_" type="continuous">
@@ -785,5 +785,5 @@
             <child link="tether_0/fragment_15"/>
             <axis xyz="0 0 1" />
-            <dynamics damping="0.01" friction="0.15"/>
+            <dynamics damping="0.01" friction="0.01"/>
         </joint>
             <link name="tether_0/fragment_16">
@@ -824,5 +824,5 @@
             <child link="tether_0/small_link_1_16"/>
             <axis xyz="1 0 0" />
-            <dynamics damping="0.01" friction="0.15"/>
+            <dynamics damping="0.01" friction="0.01"/>
         </joint>
         <joint name="tether_0/joint_2_16" type="continuous">
@@ -830,5 +830,5 @@
             <child link="tether_0/small_link_2_16"/>
             <axis xyz="0 1 0" />
-            <dynamics damping="0.01" friction="0.15"/>
+            <dynamics damping="0.01" friction="0.01"/>
         </joint>
         <joint name="tether_0/joint_1_16_" type="continuous">
@@ -836,5 +836,5 @@
             <child link="tether_0/fragment_16"/>
             <axis xyz="0 0 1" />
-            <dynamics damping="0.01" friction="0.15"/>
+            <dynamics damping="0.01" friction="0.01"/>
         </joint>
             <link name="tether_0/fragment_17">
@@ -875,5 +875,5 @@
             <child link="tether_0/small_link_1_17"/>
             <axis xyz="1 0 0" />
-            <dynamics damping="0.01" friction="0.15"/>
+            <dynamics damping="0.01" friction="0.01"/>
         </joint>
         <joint name="tether_0/joint_2_17" type="continuous">
@@ -881,5 +881,5 @@
             <child link="tether_0/small_link_2_17"/>
             <axis xyz="0 1 0" />
-            <dynamics damping="0.01" friction="0.15"/>
+            <dynamics damping="0.01" friction="0.01"/>
         </joint>
         <joint name="tether_0/joint_1_17_" type="continuous">
@@ -887,5 +887,5 @@
             <child link="tether_0/fragment_17"/>
             <axis xyz="0 0 1" />
-            <dynamics damping="0.01" friction="0.15"/>
+            <dynamics damping="0.01" friction="0.01"/>
         </joint>
             <link name="tether_0/fragment_18">
@@ -926,5 +926,5 @@
             <child link="tether_0/small_link_1_18"/>
             <axis xyz="1 0 0" />
-            <dynamics damping="0.01" friction="0.15"/>
+            <dynamics damping="0.01" friction="0.01"/>
         </joint>
         <joint name="tether_0/joint_2_18" type="continuous">
@@ -932,5 +932,5 @@
             <child link="tether_0/small_link_2_18"/>
             <axis xyz="0 1 0" />
-            <dynamics damping="0.01" friction="0.15"/>
+            <dynamics damping="0.01" friction="0.01"/>
         </joint>
         <joint name="tether_0/joint_1_18_" type="continuous">
@@ -938,5 +938,5 @@
             <child link="tether_0/fragment_18"/>
             <axis xyz="0 0 1" />
-            <dynamics damping="0.01" friction="0.15"/>
+            <dynamics damping="0.01" friction="0.01"/>
         </joint>
             <link name="tether_0/fragment_19">
@@ -977,5 +977,5 @@
             <child link="tether_0/small_link_1_19"/>
             <axis xyz="1 0 0" />
-            <dynamics damping="0.01" friction="0.15"/>
+            <dynamics damping="0.01" friction="0.01"/>
         </joint>
         <joint name="tether_0/joint_2_19" type="continuous">
@@ -983,5 +983,5 @@
             <child link="tether_0/small_link_2_19"/>
             <axis xyz="0 1 0" />
-            <dynamics damping="0.01" friction="0.15"/>
+            <dynamics damping="0.01" friction="0.01"/>
         </joint>
         <joint name="tether_0/joint_1_19_" type="continuous">
@@ -989,5 +989,5 @@
             <child link="tether_0/fragment_19"/>
             <axis xyz="0 0 1" />
-            <dynamics damping="0.01" friction="0.15"/>
+            <dynamics damping="0.01" friction="0.01"/>
         </joint>
             <link name="tether_0/fragment_20">
@@ -1028,5 +1028,5 @@
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
File: tether_description/urdf/tether_fragment.xacro (robot description, xacro)
@@ -19,5 +19,5 @@
         <!--joint dynamics-->
         {%- set damping = 0.01 -%}
-        {%- set friction = 0.15 -%}
+        {%- set friction = 0.01 -%}
         <!--link number-->
         {%- set tether_fragments = 30 -%}

File: ugv_description/urdf/mp_500/xacros/mp_500_tether_end.xacro (robot description, xacro)
@@ -22,5 +22,5 @@
                 </geometry>
             </collision>
-            </link>
+        </link>
         </xacro:macro>
 </robot>
