Commit message: Update tether fragment length 0.10[m] -> 0.15[m]

File: tether_description/urdf/tether.xacro (robot description, xacro)
@@ -6,17 +6,17 @@
             <link name="tether_0/fragment_0">
             <visual>
-                <origin rpy="0 0 0" xyz="0 0 0.05"/>
-                <geometry>
-                    <cylinder length="0.1" radius="0.0033"/>
-                </geometry>
-                <!--material name="black"/-->
-            </visual>
-            <inertial>
-                <mass value="0.012"/>
-                <inertia ixx="1.003267e-05" iyy="1.003267e-05" izz="6.534e-08" ixy="0.0" ixz="0.0" iyz="0.0"/>
-            </inertial>
-            <collision>
-                <geometry>
-                    <cylinder length="0.1" radius="0.0033"/>
+                <origin rpy="0 0 0" xyz="0 0 0.075"/>
+                <geometry>
+                    <cylinder length="0.15" radius="0.0033"/>
+                </geometry>
+                <!--material name="black"/-->
+            </visual>
+            <inertial>
+                <mass value="0.012"/>
+                <inertia ixx="2.253267e-05" iyy="2.253267e-05" izz="6.534e-08" ixy="0.0" ixz="0.0" iyz="0.0"/>
+            </inertial>
+            <collision>
+                <geometry>
+                    <cylinder length="0.15" radius="0.0033"/>
                 </geometry>
             </collision>
@@ -24,17 +24,17 @@
             <link name="tether_0/fragment_1">
             <visual>
-                <origin rpy="0 0 0" xyz="0 0 0.05"/>
-                <geometry>
-                    <cylinder length="0.1" radius="0.0033"/>
-                </geometry>
-                <!--material name="black"/-->
-            </visual>
-            <inertial>
-                <mass value="0.012"/>
-                <inertia ixx="1.003267e-05" iyy="1.003267e-05" izz="6.534e-08" ixy="0.0" ixz="0.0" iyz="0.0"/>
-            </inertial>
-            <collision>
-                <geometry>
-                    <cylinder length="0.1" radius="0.0033"/>
+                <origin rpy="0 0 0" xyz="0 0 0.075"/>
+                <geometry>
+                    <cylinder length="0.15" radius="0.0033"/>
+                </geometry>
+                <!--material name="black"/-->
+            </visual>
+            <inertial>
+                <mass value="0.012"/>
+                <inertia ixx="2.253267e-05" iyy="2.253267e-05" izz="6.534e-08" ixy="0.0" ixz="0.0" iyz="0.0"/>
+            </inertial>
+            <collision>
+                <geometry>
+                    <cylinder length="0.15" radius="0.0033"/>
                 </geometry>
             </collision>
@@ -55,5 +55,5 @@
         <!--tether fragment joint-->
         <joint name="tether_0/joint_1_1" type="continuous">
-            <origin rpy="0 0 0" xyz="0 0 0.1"/>
+            <origin rpy="0 0 0" xyz="0 0 0.15"/>
             <parent link="tether_0/fragment_0"/>
             <child link="tether_0/small_link_1_1"/>
@@ -75,17 +75,17 @@
             <link name="tether_0/fragment_2">
             <visual>
-                <origin rpy="0 0 0" xyz="0 0 0.05"/>
-                <geometry>
-                    <cylinder length="0.1" radius="0.0033"/>
-                </geometry>
-                <!--material name="black"/-->
-            </visual>
-            <inertial>
-                <mass value="0.012"/>
-                <inertia ixx="1.003267e-05" iyy="1.003267e-05" izz="6.534e-08" ixy="0.0" ixz="0.0" iyz="0.0"/>
-            </inertial>
-            <collision>
-                <geometry>
-                    <cylinder length="0.1" radius="0.0033"/>
+                <origin rpy="0 0 0" xyz="0 0 0.075"/>
+                <geometry>
+                    <cylinder length="0.15" radius="0.0033"/>
+                </geometry>
+                <!--material name="black"/-->
+            </visual>
+            <inertial>
+                <mass value="0.012"/>
+                <inertia ixx="2.253267e-05" iyy="2.253267e-05" izz="6.534e-08" ixy="0.0" ixz="0.0" iyz="0.0"/>
+            </inertial>
+            <collision>
+                <geometry>
+                    <cylinder length="0.15" radius="0.0033"/>
                 </geometry>
             </collision>
@@ -106,5 +106,5 @@
         <!--tether fragment joint-->
         <joint name="tether_0/joint_1_2" type="continuous">
-            <origin rpy="0 0 0" xyz="0 0 0.1"/>
+            <origin rpy="0 0 0" xyz="0 0 0.15"/>
             <parent link="tether_0/fragment_1"/>
             <child link="tether_0/small_link_1_2"/>
@@ -126,17 +126,17 @@
             <link name="tether_0/fragment_3">
             <visual>
-                <origin rpy="0 0 0" xyz="0 0 0.05"/>
-                <geometry>
-                    <cylinder length="0.1" radius="0.0033"/>
-                </geometry>
-                <!--material name="black"/-->
-            </visual>
-            <inertial>
-                <mass value="0.012"/>
-                <inertia ixx="1.003267e-05" iyy="1.003267e-05" izz="6.534e-08" ixy="0.0" ixz="0.0" iyz="0.0"/>
-            </inertial>
-            <collision>
-                <geometry>
-                    <cylinder length="0.1" radius="0.0033"/>
+                <origin rpy="0 0 0" xyz="0 0 0.075"/>
+                <geometry>
+                    <cylinder length="0.15" radius="0.0033"/>
+                </geometry>
+                <!--material name="black"/-->
+            </visual>
+            <inertial>
+                <mass value="0.012"/>
+                <inertia ixx="2.253267e-05" iyy="2.253267e-05" izz="6.534e-08" ixy="0.0" ixz="0.0" iyz="0.0"/>
+            </inertial>
+            <collision>
+                <geometry>
+                    <cylinder length="0.15" radius="0.0033"/>
                 </geometry>
             </collision>
@@ -157,5 +157,5 @@
         <!--tether fragment joint-->
         <joint name="tether_0/joint_1_3" type="continuous">
-            <origin rpy="0 0 0" xyz="0 0 0.1"/>
+            <origin rpy="0 0 0" xyz="0 0 0.15"/>
             <parent link="tether_0/fragment_2"/>
             <child link="tether_0/small_link_1_3"/>
@@ -177,17 +177,17 @@
             <link name="tether_0/fragment_4">
             <visual>
-                <origin rpy="0 0 0" xyz="0 0 0.05"/>
-                <geometry>
-                    <cylinder length="0.1" radius="0.0033"/>
-                </geometry>
-                <!--material name="black"/-->
-            </visual>
-            <inertial>
-                <mass value="0.012"/>
-                <inertia ixx="1.003267e-05" iyy="1.003267e-05" izz="6.534e-08" ixy="0.0" ixz="0.0" iyz="0.0"/>
-            </inertial>
-            <collision>
-                <geometry>
-                    <cylinder length="0.1" radius="0.0033"/>
+                <origin rpy="0 0 0" xyz="0 0 0.075"/>
+                <geometry>
+                    <cylinder length="0.15" radius="0.0033"/>
+                </geometry>
+                <!--material name="black"/-->
+            </visual>
+            <inertial>
+                <mass value="0.012"/>
+                <inertia ixx="2.253267e-05" iyy="2.253267e-05" izz="6.534e-08" ixy="0.0" ixz="0.0" iyz="0.0"/>
+            </inertial>
+            <collision>
+                <geometry>
+                    <cylinder length="0.15" radius="0.0033"/>
                 </geometry>
             </collision>
@@ -208,5 +208,5 @@
         <!--tether fragment joint-->
         <joint name="tether_0/joint_1_4" type="continuous">
-            <origin rpy="0 0 0" xyz="0 0 0.1"/>
+            <origin rpy="0 0 0" xyz="0 0 0.15"/>
             <parent link="tether_0/fragment_3"/>
             <child link="tether_0/small_link_1_4"/>
@@ -228,17 +228,17 @@
             <link name="tether_0/fragment_5">
             <visual>
-                <origin rpy="0 0 0" xyz="0 0 0.05"/>
-                <geometry>
-                    <cylinder length="0.1" radius="0.0033"/>
-                </geometry>
-                <!--material name="black"/-->
-            </visual>
-            <inertial>
-                <mass value="0.012"/>
-                <inertia ixx="1.003267e-05" iyy="1.003267e-05" izz="6.534e-08" ixy="0.0" ixz="0.0" iyz="0.0"/>
-            </inertial>
-            <collision>
-                <geometry>
-                    <cylinder length="0.1" radius="0.0033"/>
+                <origin rpy="0 0 0" xyz="0 0 0.075"/>
+                <geometry>
+                    <cylinder length="0.15" radius="0.0033"/>
+                </geometry>
+                <!--material name="black"/-->
+            </visual>
+            <inertial>
+                <mass value="0.012"/>
+                <inertia ixx="2.253267e-05" iyy="2.253267e-05" izz="6.534e-08" ixy="0.0" ixz="0.0" iyz="0.0"/>
+            </inertial>
+            <collision>
+                <geometry>
+                    <cylinder length="0.15" radius="0.0033"/>
                 </geometry>
             </collision>
@@ -259,5 +259,5 @@
         <!--tether fragment joint-->
         <joint name="tether_0/joint_1_5" type="continuous">
-            <origin rpy="0 0 0" xyz="0 0 0.1"/>
+            <origin rpy="0 0 0" xyz="0 0 0.15"/>
             <parent link="tether_0/fragment_4"/>
             <child link="tether_0/small_link_1_5"/>
@@ -279,17 +279,17 @@
             <link name="tether_0/fragment_6">
             <visual>
-                <origin rpy="0 0 0" xyz="0 0 0.05"/>
-                <geometry>
-                    <cylinder length="0.1" radius="0.0033"/>
-                </geometry>
-                <!--material name="black"/-->
-            </visual>
-            <inertial>
-                <mass value="0.012"/>
-                <inertia ixx="1.003267e-05" iyy="1.003267e-05" izz="6.534e-08" ixy="0.0" ixz="0.0" iyz="0.0"/>
-            </inertial>
-            <collision>
-                <geometry>
-                    <cylinder length="0.1" radius="0.0033"/>
+                <origin rpy="0 0 0" xyz="0 0 0.075"/>
+                <geometry>
+                    <cylinder length="0.15" radius="0.0033"/>
+                </geometry>
+                <!--material name="black"/-->
+            </visual>
+            <inertial>
+                <mass value="0.012"/>
+                <inertia ixx="2.253267e-05" iyy="2.253267e-05" izz="6.534e-08" ixy="0.0" ixz="0.0" iyz="0.0"/>
+            </inertial>
+            <collision>
+                <geometry>
+                    <cylinder length="0.15" radius="0.0033"/>
                 </geometry>
             </collision>
@@ -310,5 +310,5 @@
         <!--tether fragment joint-->
         <joint name="tether_0/joint_1_6" type="continuous">
-            <origin rpy="0 0 0" xyz="0 0 0.1"/>
+            <origin rpy="0 0 0" xyz="0 0 0.15"/>
             <parent link="tether_0/fragment_5"/>
             <child link="tether_0/small_link_1_6"/>
@@ -330,17 +330,17 @@
             <link name="tether_0/fragment_7">
             <visual>
-                <origin rpy="0 0 0" xyz="0 0 0.05"/>
-                <geometry>
-                    <cylinder length="0.1" radius="0.0033"/>
-                </geometry>
-                <!--material name="black"/-->
-            </visual>
-            <inertial>
-                <mass value="0.012"/>
-                <inertia ixx="1.003267e-05" iyy="1.003267e-05" izz="6.534e-08" ixy="0.0" ixz="0.0" iyz="0.0"/>
-            </inertial>
-            <collision>
-                <geometry>
-                    <cylinder length="0.1" radius="0.0033"/>
+                <origin rpy="0 0 0" xyz="0 0 0.075"/>
+                <geometry>
+                    <cylinder length="0.15" radius="0.0033"/>
+                </geometry>
+                <!--material name="black"/-->
+            </visual>
+            <inertial>
+                <mass value="0.012"/>
+                <inertia ixx="2.253267e-05" iyy="2.253267e-05" izz="6.534e-08" ixy="0.0" ixz="0.0" iyz="0.0"/>
+            </inertial>
+            <collision>
+                <geometry>
+                    <cylinder length="0.15" radius="0.0033"/>
                 </geometry>
             </collision>
@@ -361,5 +361,5 @@
         <!--tether fragment joint-->
         <joint name="tether_0/joint_1_7" type="continuous">
-            <origin rpy="0 0 0" xyz="0 0 0.1"/>
+            <origin rpy="0 0 0" xyz="0 0 0.15"/>
             <parent link="tether_0/fragment_6"/>
             <child link="tether_0/small_link_1_7"/>
@@ -381,17 +381,17 @@
             <link name="tether_0/fragment_8">
             <visual>
-                <origin rpy="0 0 0" xyz="0 0 0.05"/>
-                <geometry>
-                    <cylinder length="0.1" radius="0.0033"/>
-                </geometry>
-                <!--material name="black"/-->
-            </visual>
-            <inertial>
-                <mass value="0.012"/>
-                <inertia ixx="1.003267e-05" iyy="1.003267e-05" izz="6.534e-08" ixy="0.0" ixz="0.0" iyz="0.0"/>
-            </inertial>
-            <collision>
-                <geometry>
-                    <cylinder length="0.1" radius="0.0033"/>
+                <origin rpy="0 0 0" xyz="0 0 0.075"/>
+                <geometry>
+                    <cylinder length="0.15" radius="0.0033"/>
+                </geometry>
+                <!--material name="black"/-->
+            </visual>
+            <inertial>
+                <mass value="0.012"/>
+                <inertia ixx="2.253267e-05" iyy="2.253267e-05" izz="6.534e-08" ixy="0.0" ixz="0.0" iyz="0.0"/>
+            </inertial>
+            <collision>
+                <geometry>
+                    <cylinder length="0.15" radius="0.0033"/>
                 </geometry>
             </collision>
@@ -412,5 +412,5 @@
         <!--tether fragment joint-->
         <joint name="tether_0/joint_1_8" type="continuous">
-            <origin rpy="0 0 0" xyz="0 0 0.1"/>
+            <origin rpy="0 0 0" xyz="0 0 0.15"/>
             <parent link="tether_0/fragment_7"/>
             <child link="tether_0/small_link_1_8"/>
@@ -432,17 +432,17 @@
             <link name="tether_0/fragment_9">
             <visual>
-                <origin rpy="0 0 0" xyz="0 0 0.05"/>
-                <geometry>
-                    <cylinder length="0.1" radius="0.0033"/>
-                </geometry>
-                <!--material name="black"/-->
-            </visual>
-            <inertial>
-                <mass value="0.012"/>
-                <inertia ixx="1.003267e-05" iyy="1.003267e-05" izz="6.534e-08" ixy="0.0" ixz="0.0" iyz="0.0"/>
-            </inertial>
-            <collision>
-                <geometry>
-                    <cylinder length="0.1" radius="0.0033"/>
+                <origin rpy="0 0 0" xyz="0 0 0.075"/>
+                <geometry>
+                    <cylinder length="0.15" radius="0.0033"/>
+                </geometry>
+                <!--material name="black"/-->
+            </visual>
+            <inertial>
+                <mass value="0.012"/>
+                <inertia ixx="2.253267e-05" iyy="2.253267e-05" izz="6.534e-08" ixy="0.0" ixz="0.0" iyz="0.0"/>
+            </inertial>
+            <collision>
+                <geometry>
+                    <cylinder length="0.15" radius="0.0033"/>
                 </geometry>
             </collision>
@@ -463,5 +463,5 @@
         <!--tether fragment joint-->
         <joint name="tether_0/joint_1_9" type="continuous">
-            <origin rpy="0 0 0" xyz="0 0 0.1"/>
+            <origin rpy="0 0 0" xyz="0 0 0.15"/>
             <parent link="tether_0/fragment_8"/>
             <child link="tether_0/small_link_1_9"/>
@@ -483,17 +483,17 @@
             <link name="tether_0/fragment_10">
             <visual>
-                <origin rpy="0 0 0" xyz="0 0 0.05"/>
-                <geometry>
-                    <cylinder length="0.1" radius="0.0033"/>
-                </geometry>
-                <!--material name="black"/-->
-            </visual>
-            <inertial>
-                <mass value="0.012"/>
-                <inertia ixx="1.003267e-05" iyy="1.003267e-05" izz="6.534e-08" ixy="0.0" ixz="0.0" iyz="0.0"/>
-            </inertial>
-            <collision>
-                <geometry>
-                    <cylinder length="0.1" radius="0.0033"/>
+                <origin rpy="0 0 0" xyz="0 0 0.075"/>
+                <geometry>
+                    <cylinder length="0.15" radius="0.0033"/>
+                </geometry>
+                <!--material name="black"/-->
+            </visual>
+            <inertial>
+                <mass value="0.012"/>
+                <inertia ixx="2.253267e-05" iyy="2.253267e-05" izz="6.534e-08" ixy="0.0" ixz="0.0" iyz="0.0"/>
+            </inertial>
+            <collision>
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
File: tether_description/urdf/tether_fragment.xacro (robot description, xacro)
@@ -5,5 +5,5 @@
         <!--tether fragment param-->
         {%- set cyl_r = 0.0033 -%}
-        {%- set cyl_l = 0.1 -%}
+        {%- set cyl_l = 0.15 -%}
         {%- set cyl_m = 0.012 -%}
         {%- set cyl_i = 1/12*cyl_m*(3*cyl_r**2+cyl_l**2) -%}
@@ -24,5 +24,5 @@
         {%- set tether_number = 4 -%}
         <!--box inertial-->
-        {%- set box_m = 50 -%}
+        {%- set box_m = 100 -%}
         {%- set box_x = 0.1 -%}
         {%- set box_y = 0.1 -%}
