Commit message: Update lumped-mass tether model

File: tether_description/urdf/lumped_mass_tether_fragment.xacro (robot description, xacro)
@@ -4,18 +4,18 @@
     <xacro:macro name="tether">
         <!--tether fragment param-->
-        {%- set lump_mass = 0.0033 -%}
-        {%- set lump_radius = 0.1 -%}
-        {%- set lump_inertia = 2/5*lump_mass*lump_radius**2 -%}
-        {%- set element_length = 0.1 -%}
+        {%- set lump_mass = 0.1 -%}
+        {%- set lump_radius = 0.01 -%}
+        {%- set lump_inertia = 3*lump_mass*lump_radius**2 -%}
+        {%- set element_length = 1.0 -%}
         <!--joint dynamics-->
-        {%- set damping = 0.01 -%}
-        {%- set friction = 0.01 -%}
+        {%- set damping = 0.1 -%}
+        {%- set friction = 0.1 -%}
         <!--link number-->
-        {%- set tether_fragments = 30 -%}
+        {%- set tether_fragments = 5 -%}
         {%- set tether_number = 4 -%}
         {%- macro tether_fragment(dirc, n) -%}
         <link name="tether_{{dirc}}/fragment_{{n}}">
             <visual>
-                <origin rpy="0 0 0" xyz="0 0 {{cyl_l/2}}"/>
+                <origin rpy="0 0 0" xyz="0 0 0"/>
                 <geometry>
                     <sphere radius="{{lump_radius}}"/>
@@ -31,8 +31,8 @@
                 </geometry>
             </collision>
-            <gazebo reference="tether_{{dirc}}/fragment_{{n}}">
-                <material>Gazebo/Red</material>
-            </gazebo>
         </link>
+        <gazebo reference="tether_{{dirc}}/fragment_{{n}}">
+            <material>Gazebo/Red</material>
+        </gazebo>
         {%- endmacro -%}
         <!--tether_cylinder_joint-->
@@ -64,43 +64,18 @@
         {%- endmacro -%}
         {%- macro ugv_joint(dirc) -%}
-        <!--link between tether and ugv-->
-        <link name="tether_{{dirc}}/end_link_1">
-            <inertial>
-                <mass value="{{small_link_mass}}"/>
-                <inertia ixx="{{small_link_ixx}}" iyy="{{small_link_iyy}}" izz="{{small_link_izz}}" ixy="{{small_link_ixy}}" ixz="{{small_link_ixz}}" iyz="{{small_link_iyz}}"/>
-            </inertial>
-        </link>
-        <link name="tether_{{dirc}}/end_link_2">
-            <inertial>
-                <mass value="{{small_link_mass}}"/>
-                <inertia ixx="{{small_link_ixx}}" iyy="{{small_link_iyy}}" izz="{{small_link_izz}}" ixy="{{small_link_ixy}}" ixz="{{small_link_ixz}}" iyz="{{small_link_iyz}}"/>
-            </inertial>
-        </link>
         <!--tether end joint-->
         <joint name="tether_{{dirc}}/ugv_joint_1" type="continuous">
             {% if dirc == 0 %}
-                <origin rpy="0 ${-pi/2} 0" xyz="0 0 0"/>
+                <origin rpy="0 ${-pi/2} 0" xyz="0 0 {{element_length}}"/>
             {% elif dirc == 1 %}
-                <origin rpy="${-pi/2} 0 0" xyz="0 0 0"/>
+                <origin rpy="${-pi/2} 0 0" xyz="0 0 {{element_length}}"/>
             {% elif dirc == 2 %}
-                <origin rpy="0 ${pi/2} 0" xyz="0 0 0"/>
+                <origin rpy="0 ${pi/2} 0" xyz="0 0 {{element_length}}"/>
             {% elif dirc == 3 %}
-                <origin rpy="${pi/2} 0 0" xyz="0 0 0"/>
+                <origin rpy="${pi/2} 0 0" xyz="0 0 {{element_length}}"/>
             {% endif %}
             <parent link="tether_{{dirc}}/fragment_{{tether_fragments-1}}"/>
-            <child link="tether_{{dirc}}/end_link_1"/>
+            <child link="mp_500_{{dirc}}/tether_end"/>
             <axis xyz="1 0 0" />
-            <dynamics damping="{{damping}}" friction="{{friction}}"/>
-        </joint>
-        <joint name="tether_{{dirc}}/ugv_joint_2" type="continuous">
-            <parent link="tether_{{dirc}}/end_link_1"/>
-            <child link="tether_{{dirc}}/end_link_2"/>
-            <axis xyz="0 1 0" />
-            <dynamics damping="{{damping}}" friction="{{friction}}"/>
-        </joint>
-        <joint name="tether_{{dirc}}/ugv_joint_3" type="continuous">
-            <parent link="tether_{{dirc}}/end_link_2"/>
-            <child link="mp_500_{{dirc}}/tether_end"/>
-            <axis xyz="0 0 1" />
             <dynamics damping="{{damping}}" friction="{{friction}}"/>
         </joint>

File: tether_description/urdf/tether.xacro (robot description, xacro)
@@ -3,1501 +3,136 @@
     <!--tether model-->
     <xacro:macro name="tether">
-        <!--tether fragment param--><!--small link inatial--><!--joint dynamics--><!--link number--><!--box inertial--><!--tether_cylinder_joint--><!-- main-->
+        <!--tether fragment param--><!--joint dynamics--><!--link number--><!--tether_cylinder_joint--><!-- main-->
             <link name="tether_0/fragment_0">
             <visual>
-                <origin rpy="0 0 0" xyz="0 0 0.075"/>
-                <geometry>
-                    <cylinder length="0.15" radius="0.0033"/>
-                </geometry>
-                <!--material name="black"/-->
-            </visual>
-            <inertial>
-                <mass value="0.012"/>
-                <inertia ixx="2.253267e-05" iyy="2.253267e-05" izz="6.534e-08" ixy="0.0" ixz="0.0" iyz="0.0"/>
-            </inertial>
-            <collision>
-                <geometry>
-                    <cylinder length="0.15" radius="0.0033"/>
-                </geometry>
-            </collision>
-        </link>
+                <origin rpy="0 0 0" xyz="0 0 0"/>
+                <geometry>
+                    <sphere radius="0.01"/>
+                </geometry>
+            </visual>
+            <inertial>
+                <mass value="0.1"/>
+                <inertia ixx="3e-05" iyy="3e-05" izz="3e-05" ixy="0.0" ixz="0.0" iyz="0.0"/>
+            </inertial>
+            <collision>
+                <geometry>
+                    <sphere radius="0.01"/>
+                </geometry>
+            </collision>
+        </link>
+        <gazebo reference="tether_0/fragment_0">
+            <material>Gazebo/Red</material>
+        </gazebo>
             <link name="tether_0/fragment_1">
             <visual>
-                <origin rpy="0 0 0" xyz="0 0 0.075"/>
-                <geometry>
-                    <cylinder length="0.15" radius="0.0033"/>
-                </geometry>
-                <!--material name="black"/-->
-            </visual>
-            <inertial>
-                <mass value="0.012"/>
-                <inertia ixx="2.253267e-05" iyy="2.253267e-05" izz="6.534e-08" ixy="0.0" ixz="0.0" iyz="0.0"/>
-            </inertial>
-            <collision>
-                <geometry>
-                    <cylinder length="0.15" radius="0.0033"/>
-                </geometry>
-            </collision>
-        </link>
-                    <!--link between two tether fragments-->
-        <link name="tether_0/small_link_1_1">
-            <inertial>
-                <mass value="0.001"/>
-                <inertia ixx="0.001" iyy="0.001" izz="0.001" ixy="0.0" ixz="0.0" iyz="0.0"/>
-            </inertial>
-        </link>
-        <link name="tether_0/small_link_2_1">
-            <inertial>
-                <mass value="0.001"/>
-                <inertia ixx="0.001" iyy="0.001" izz="0.001" ixy="0.0" ixz="0.0" iyz="0.0"/>
-            </inertial>
-        </link>
-        <!--tether fragment joint-->
-        <joint name="tether_0/joint_1_1" type="continuous">
-            <origin rpy="0 0 0" xyz="0 0 0.15"/>
+                <origin rpy="0 0 0" xyz="0 0 0"/>
+                <geometry>
+                    <sphere radius="0.01"/>
+                </geometry>
+            </visual>
+            <inertial>
+                <mass value="0.1"/>
+                <inertia ixx="3e-05" iyy="3e-05" izz="3e-05" ixy="0.0" ixz="0.0" iyz="0.0"/>
+            </inertial>
+            <collision>
+                <geometry>
+                    <sphere radius="0.01"/>
+                </geometry>
+            </collision>
+        </link>
+        <gazebo reference="tether_0/fragment_1">
+            <material>Gazebo/Red</material>
+        </gazebo>
+                    <!--tether fragment joint-->
+        <joint name="tether_0/joint_1" type="continuous">
+            <origin rpy="0 0 0" xyz="0 0 1.0"/>
             <parent link="tether_0/fragment_0"/>
-            <child link="tether_0/small_link_1_1"/>
-            <axis xyz="1 0 0" />
-            <dynamics damping="0.01" friction="0.01"/>
-        </joint>
-        <joint name="tether_0/joint_2_1" type="continuous">
-            <parent link="tether_0/small_link_1_1"/>
-            <child link="tether_0/small_link_2_1"/>
-            <axis xyz="0 1 0" />
-            <dynamics damping="0.01" friction="0.01"/>
-        </joint>
-        <joint name="tether_0/joint_1_1_" type="continuous">
-            <parent link="tether_0/small_link_2_1"/>
             <child link="tether_0/fragment_1"/>
-            <axis xyz="0 0 1" />
-            <dynamics damping="0.01" friction="0.01"/>
+            <axis xyz="1 0 0" />
+            <dynamics damping="0.1" friction="0.1"/>
         </joint>
             <link name="tether_0/fragment_2">
             <visual>
-                <origin rpy="0 0 0" xyz="0 0 0.075"/>
-                <geometry>
-                    <cylinder length="0.15" radius="0.0033"/>
-                </geometry>
-                <!--material name="black"/-->
-            </visual>
-            <inertial>
-                <mass value="0.012"/>
-                <inertia ixx="2.253267e-05" iyy="2.253267e-05" izz="6.534e-08" ixy="0.0" ixz="0.0" iyz="0.0"/>
-            </inertial>
-            <collision>
-                <geometry>
-                    <cylinder length="0.15" radius="0.0033"/>
-                </geometry>
-            </collision>
-        </link>
-                    <!--link between two tether fragments-->
-        <link name="tether_0/small_link_1_2">
-            <inertial>
-                <mass value="0.001"/>
-                <inertia ixx="0.001" iyy="0.001" izz="0.001" ixy="0.0" ixz="0.0" iyz="0.0"/>
-            </inertial>
-        </link>
-        <link name="tether_0/small_link_2_2">
-            <inertial>
-                <mass value="0.001"/>
-                <inertia ixx="0.001" iyy="0.001" izz="0.001" ixy="0.0" ixz="0.0" iyz="0.0"/>
-            </inertial>
-        </link>
-        <!--tether fragment joint-->
-        <joint name="tether_0/joint_1_2" type="continuous">
-            <origin rpy="0 0 0" xyz="0 0 0.15"/>
+                <origin rpy="0 0 0" xyz="0 0 0"/>
+                <geometry>
+                    <sphere radius="0.01"/>
+                </geometry>
+            </visual>
+            <inertial>
+                <mass value="0.1"/>
+                <inertia ixx="3e-05" iyy="3e-05" izz="3e-05" ixy="0.0" ixz="0.0" iyz="0.0"/>
+            </inertial>
+            <collision>
+                <geometry>
+                    <sphere radius="0.01"/>
+                </geometry>
+            </collision>
+        </link>
+        <gazebo reference="tether_0/fragment_2">
+            <material>Gazebo/Red</material>
+        </gazebo>
+                    <!--tether fragment joint-->
+        <joint name="tether_0/joint_2" type="continuous">
+            <origin rpy="0 0 0" xyz="0 0 1.0"/>
             <parent link="tether_0/fragment_1"/>
-            <child link="tether_0/small_link_1_2"/>
-            <axis xyz="1 0 0" />
-            <dynamics damping="0.01" friction="0.01"/>
-        </joint>
-        <joint name="tether_0/joint_2_2" type="continuous">
-            <parent link="tether_0/small_link_1_2"/>
-            <child link="tether_0/small_link_2_2"/>
-            <axis xyz="0 1 0" />
-            <dynamics damping="0.01" friction="0.01"/>
-        </joint>
-        <joint name="tether_0/joint_1_2_" type="continuous">
-            <parent link="tether_0/small_link_2_2"/>
             <child link="tether_0/fragment_2"/>
-            <axis xyz="0 0 1" />
-            <dynamics damping="0.01" friction="0.01"/>
+            <axis xyz="1 0 0" />
+            <dynamics damping="0.1" friction="0.1"/>
         </joint>
             <link name="tether_0/fragment_3">
             <visual>
-                <origin rpy="0 0 0" xyz="0 0 0.075"/>
-                <geometry>
-                    <cylinder length="0.15" radius="0.0033"/>
-                </geometry>
-                <!--material name="black"/-->
-            </visual>
-            <inertial>
-                <mass value="0.012"/>
-                <inertia ixx="2.253267e-05" iyy="2.253267e-05" izz="6.534e-08" ixy="0.0" ixz="0.0" iyz="0.0"/>
-            </inertial>
-            <collision>
-                <geometry>
-                    <cylinder length="0.15" radius="0.0033"/>
-                </geometry>
-            </collision>
-        </link>
-                    <!--link between two tether fragments-->
-        <link name="tether_0/small_link_1_3">
-            <inertial>
-                <mass value="0.001"/>
-                <inertia ixx="0.001" iyy="0.001" izz="0.001" ixy="0.0" ixz="0.0" iyz="0.0"/>
-            </inertial>
-        </link>
-        <link name="tether_0/small_link_2_3">
-            <inertial>
-                <mass value="0.001"/>
-                <inertia ixx="0.001" iyy="0.001" izz="0.001" ixy="0.0" ixz="0.0" iyz="0.0"/>
-            </inertial>
-        </link>
-        <!--tether fragment joint-->
-        <joint name="tether_0/joint_1_3" type="continuous">
-            <origin rpy="0 0 0" xyz="0 0 0.15"/>
+                <origin rpy="0 0 0" xyz="0 0 0"/>
+                <geometry>
+                    <sphere radius="0.01"/>
+                </geometry>
+            </visual>
+            <inertial>
+                <mass value="0.1"/>
+                <inertia ixx="3e-05" iyy="3e-05" izz="3e-05" ixy="0.0" ixz="0.0" iyz="0.0"/>
+            </inertial>
+            <collision>
+                <geometry>
+                    <sphere radius="0.01"/>
+                </geometry>
+            </collision>
+        </link>
+        <gazebo reference="tether_0/fragment_3">
+            <material>Gazebo/Red</material>
+        </gazebo>
+                    <!--tether fragment joint-->
+        <joint name="tether_0/joint_3" type="continuous">
+            <origin rpy="0 0 0" xyz="0 0 1.0"/>
             <parent link="tether_0/fragment_2"/>
-            <child link="tether_0/small_link_1_3"/>
-            <axis xyz="1 0 0" />
-            <dynamics damping="0.01" friction="0.01"/>
-        </joint>
-        <joint name="tether_0/joint_2_3" type="continuous">
-            <parent link="tether_0/small_link_1_3"/>
-            <child link="tether_0/small_link_2_3"/>
-            <axis xyz="0 1 0" />
-            <dynamics damping="0.01" friction="0.01"/>
-        </joint>
-        <joint name="tether_0/joint_1_3_" type="continuous">
-            <parent link="tether_0/small_link_2_3"/>
             <child link="tether_0/fragment_3"/>
-            <axis xyz="0 0 1" />
-            <dynamics damping="0.01" friction="0.01"/>
+            <axis xyz="1 0 0" />
+            <dynamics damping="0.1" friction="0.1"/>
         </joint>
             <link name="tether_0/fragment_4">
             <visual>
-                <origin rpy="0 0 0" xyz="0 0 0.075"/>
-                <geometry>
-                    <cylinder length="0.15" radius="0.0033"/>
-                </geometry>
-                <!--material name="black"/-->
-            </visual>
-            <inertial>
-                <mass value="0.012"/>
-                <inertia ixx="2.253267e-05" iyy="2.253267e-05" izz="6.534e-08" ixy="0.0" ixz="0.0" iyz="0.0"/>
-            </inertial>
-            <collision>
-                <geometry>
-                    <cylinder length="0.15" radius="0.0033"/>
-                </geometry>
-            </collision>
-        </link>
-                    <!--link between two tether fragments-->
-        <link name="tether_0/small_link_1_4">
-            <inertial>
-                <mass value="0.001"/>
-                <inertia ixx="0.001" iyy="0.001" izz="0.001" ixy="0.0" ixz="0.0" iyz="0.0"/>
-            </inertial>
-        </link>
-        <link name="tether_0/small_link_2_4">
-            <inertial>
-                <mass value="0.001"/>
-                <inertia ixx="0.001" iyy="0.001" izz="0.001" ixy="0.0" ixz="0.0" iyz="0.0"/>
-            </inertial>
-        </link>
-        <!--tether fragment joint-->
-        <joint name="tether_0/joint_1_4" type="continuous">
-            <origin rpy="0 0 0" xyz="0 0 0.15"/>
+                <origin rpy="0 0 0" xyz="0 0 0"/>
+                <geometry>
+                    <sphere radius="0.01"/>
+                </geometry>
+            </visual>
+            <inertial>
+                <mass value="0.1"/>
+                <inertia ixx="3e-05" iyy="3e-05" izz="3e-05" ixy="0.0" ixz="0.0" iyz="0.0"/>
+            </inertial>
+            <collision>
+                <geometry>
+                    <sphere radius="0.01"/>
+                </geometry>
+            </collision>
+        </link>
+        <gazebo reference="tether_0/fragment_4">
+            <material>Gazebo/Red</material>
+        </gazebo>
+                    <!--tether fragment joint-->
+        <joint name="tether_0/joint_4" type="continuous">
+            <origin rpy="0 0 0" xyz="0 0 1.0"/>
             <parent link="tether_0/fragment_3"/>
-            <child link="tether_0/small_link_1_4"/>
-            <axis xyz="1 0 0" />
-            <dynamics damping="0.01" friction="0.01"/>
-        </joint>
-        <joint name="tether_0/joint_2_4" type="continuous">
-            <parent link="tether_0/small_link_1_4"/>
-            <child link="tether_0/small_link_2_4"/>
-            <axis xyz="0 1 0" />
-            <dynamics damping="0.01" friction="0.01"/>
-        </joint>
-        <joint name="tether_0/joint_1_4_" type="continuous">
-            <parent link="tether_0/small_link_2_4"/>
             <child link="tether_0/fragment_4"/>
-            <axis xyz="0 0 1" />
-            <dynamics damping="0.01" friction="0.01"/>
-        </joint>
-            <link name="tether_0/fragment_5">
-            <visual>
-                <origin rpy="0 0 0" xyz="0 0 0.075"/>
-                <geometry>
-                    <cylinder length="0.15" radius="0.0033"/>
-                </geometry>
-                <!--material name="black"/-->
-            </visual>
-            <inertial>
-                <mass value="0.012"/>
-                <inertia ixx="2.253267e-05" iyy="2.253267e-05" izz="6.534e-08" ixy="0.0" ixz="0.0" iyz="0.0"/>
-            </inertial>
-            <collision>
-                <geometry>
-                    <cylinder length="0.15" radius="0.0033"/>
-                </geometry>
-            </collision>
-        </link>
-                    <!--link between two tether fragments-->
-        <link name="tether_0/small_link_1_5">
-            <inertial>
-                <mass value="0.001"/>
-                <inertia ixx="0.001" iyy="0.001" izz="0.001" ixy="0.0" ixz="0.0" iyz="0.0"/>
-            </inertial>
-        </link>
-        <link name="tether_0/small_link_2_5">
-            <inertial>
-                <mass value="0.001"/>
-                <inertia ixx="0.001" iyy="0.001" izz="0.001" ixy="0.0" ixz="0.0" iyz="0.0"/>
-            </inertial>
-        </link>
-        <!--tether fragment joint-->
-        <joint name="tether_0/joint_1_5" type="continuous">
-            <origin rpy="0 0 0" xyz="0 0 0.15"/>
-            <parent link="tether_0/fragment_4"/>
-            <child link="tether_0/small_link_1_5"/>
-            <axis xyz="1 0 0" />
-            <dynamics damping="0.01" friction="0.01"/>
-        </joint>
-        <joint name="tether_0/joint_2_5" type="continuous">
-            <parent link="tether_0/small_link_1_5"/>
-            <child link="tether_0/small_link_2_5"/>
-            <axis xyz="0 1 0" />
-            <dynamics damping="0.01" friction="0.01"/>
-        </joint>
-        <joint name="tether_0/joint_1_5_" type="continuous">
-            <parent link="tether_0/small_link_2_5"/>
-            <child link="tether_0/fragment_5"/>
-            <axis xyz="0 0 1" />
-            <dynamics damping="0.01" friction="0.01"/>
-        </joint>
-            <link name="tether_0/fragment_6">
-            <visual>
-                <origin rpy="0 0 0" xyz="0 0 0.075"/>
-                <geometry>
-                    <cylinder length="0.15" radius="0.0033"/>
-                </geometry>
-                <!--material name="black"/-->
-            </visual>
-            <inertial>
-                <mass value="0.012"/>
-                <inertia ixx="2.253267e-05" iyy="2.253267e-05" izz="6.534e-08" ixy="0.0" ixz="0.0" iyz="0.0"/>
-            </inertial>
-            <collision>
-                <geometry>
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