Commit message: FIx bugs

File: tether_description/urdf/lumped_mass_tether_fragment.xacro (robot description, xacro)
@@ -4,7 +4,7 @@
     <xacro:macro name="tether">
         <!--tether fragment param-->
-        {%- set lump_mass = 0.1 -%}
+        {%- set lump_mass = 0.10 -%}
         {%- set lump_radius = 0.01 -%}
-        {%- set lump_inertia = 3*lump_mass*lump_radius**2 -%}
+        {%- set lump_inertia = 2*lump_mass*lump_radius**2 -%}
         {%- set element_length = 1.0 -%}
         <!--joint dynamics-->
@@ -12,5 +12,5 @@
         {%- set friction = 0.1 -%}
         <!--link number-->
-        {%- set tether_fragments = 5 -%}
+        {%- set tether_fragments = 10 -%}
         {%- set tether_number = 4 -%}
         {%- macro tether_fragment(dirc, n) -%}
@@ -43,13 +43,41 @@
             <parent link="tether_{{dirc}}/fragment_{{n-1}}"/>
             <child link="tether_{{dirc}}/fragment_{{n}}"/>
-            <axis xyz="1 0 0" />
+            {% if dirc == 0 %}
+                <axis xyz="0 1 0" />
+            {% elif dirc == 1 %}
+                <axis xyz="1 0 0" />
+            {% elif dirc == 2 %}
+                <axis xyz="0 1 0" />
+            {% elif dirc == 3 %}
+                <axis xyz="1 0 0" />
+            {% endif %}
             <dynamics damping="{{damping}}" friction="{{friction}}"/>
         </joint>
         {%- endmacro -%}
         {%- macro uav_joint(dirc) -%}
+        <link name="tether_{{dirc}}/rod">
+            <visual>
+                <origin rpy="0 0 0" xyz="0 0 0.1"/>
+                <geometry>
+                    <cylinder length="0.2" radius="0.01"/>
+                </geometry>
+            </visual>
+            <inertial>
+                <mass value="0.01"/>
+                <inertia ixx="0.01" iyy="0.01" izz="0.01" ixy="0.0" ixz="0.0" iyz="0.0"/>
+            </inertial>
+            <collision>
+                <geometry>
+                    <cylinder length="0.2" radius="0.01"/>
+                </geometry>
+            </collision>
+        </link>
+        <gazebo reference="tether_{{dirc}}/rod">
+            <material>Gazebo/Orange</material>
+        </gazebo>
         <!--uav => tether joint-->
-        <joint name="tether_{{dirc}}/uav_joint" type="fixed">
+        <joint name="tether_{{dirc}}/rod_joint" type="fixed">
             <parent link="${namespace}/base_link"/>
-            <child link="tether_{{dirc}}/fragment_0"/>
+            <child link="tether_{{dirc}}/rod"/>
             {% if dirc == 0 %}
                 <origin rpy="0 ${pi/2} 0" xyz="0 0 0"/>
@@ -60,4 +88,17 @@
             {% elif dirc == 3 %}
                 <origin rpy="${-pi/2} 0 0" xyz="0 0 0"/>
+            {% endif %}
+        </joint>
+        <joint name="tether_{{dirc}}/uav_joint" type="continuous">
+            <parent link="tether_{{dirc}}/rod"/>
+            <child link="tether_{{dirc}}/fragment_0"/>
+            {% if dirc == 0 %}
+                <axis xyz="0 1 0" />
+            {% elif dirc == 1 %}
+                <axis xyz="1 0 0" />
+            {% elif dirc == 2 %}
+                <axis xyz="0 1 0" />
+            {% elif dirc == 3 %}
+                <axis xyz="1 0 0" />
             {% endif %}
         </joint>

File: tether_description/urdf/tether.xacro (robot description, xacro)
@@ -13,5 +13,5 @@
             <inertial>
                 <mass value="0.1"/>
-                <inertia ixx="3e-05" iyy="3e-05" izz="3e-05" ixy="0.0" ixz="0.0" iyz="0.0"/>
+                <inertia ixx="2e-05" iyy="2e-05" izz="2e-05" ixy="0.0" ixz="0.0" iyz="0.0"/>
             </inertial>
             <collision>
@@ -33,5 +33,5 @@
             <inertial>
                 <mass value="0.1"/>
-                <inertia ixx="3e-05" iyy="3e-05" izz="3e-05" ixy="0.0" ixz="0.0" iyz="0.0"/>
+                <inertia ixx="2e-05" iyy="2e-05" izz="2e-05" ixy="0.0" ixz="0.0" iyz="0.0"/>
             </inertial>
             <collision>
@@ -49,5 +49,5 @@
             <parent link="tether_0/fragment_0"/>
             <child link="tether_0/fragment_1"/>
-            <axis xyz="1 0 0" />
+                <axis xyz="0 1 0" />
             <dynamics damping="0.1" friction="0.1"/>
         </joint>
@@ -61,5 +61,5 @@
             <inertial>
                 <mass value="0.1"/>
-                <inertia ixx="3e-05" iyy="3e-05" izz="3e-05" ixy="0.0" ixz="0.0" iyz="0.0"/>
+                <inertia ixx="2e-05" iyy="2e-05" izz="2e-05" ixy="0.0" ixz="0.0" iyz="0.0"/>
             </inertial>
             <collision>
@@ -77,5 +77,5 @@
             <parent link="tether_0/fragment_1"/>
             <child link="tether_0/fragment_2"/>
-            <axis xyz="1 0 0" />
+                <axis xyz="0 1 0" />
             <dynamics damping="0.1" friction="0.1"/>
         </joint>
@@ -89,5 +89,5 @@
             <inertial>
                 <mass value="0.1"/>
-                <inertia ixx="3e-05" iyy="3e-05" izz="3e-05" ixy="0.0" ixz="0.0" iyz="0.0"/>
+                <inertia ixx="2e-05" iyy="2e-05" izz="2e-05" ixy="0.0" ixz="0.0" iyz="0.0"/>
             </inertial>
             <collision>
@@ -105,5 +105,5 @@
             <parent link="tether_0/fragment_2"/>
             <child link="tether_0/fragment_3"/>
-            <axis xyz="1 0 0" />
+                <axis xyz="0 1 0" />
             <dynamics damping="0.1" friction="0.1"/>
         </joint>
@@ -117,5 +117,5 @@
             <inertial>
                 <mass value="0.1"/>
-                <inertia ixx="3e-05" iyy="3e-05" izz="3e-05" ixy="0.0" ixz="0.0" iyz="0.0"/>
+                <inertia ixx="2e-05" iyy="2e-05" izz="2e-05" ixy="0.0" ixz="0.0" iyz="0.0"/>
             </inertial>
             <collision>
@@ -133,17 +133,182 @@
             <parent link="tether_0/fragment_3"/>
             <child link="tether_0/fragment_4"/>
-            <axis xyz="1 0 0" />
-            <dynamics damping="0.1" friction="0.1"/>
-        </joint>
-            <!--uav => tether joint-->
-        <joint name="tether_0/uav_joint" type="fixed">
+                <axis xyz="0 1 0" />
+            <dynamics damping="0.1" friction="0.1"/>
+        </joint>
+            <link name="tether_0/fragment_5">
+            <visual>
+                <origin rpy="0 0 0" xyz="0 0 0"/>
+                <geometry>
+                    <sphere radius="0.01"/>
+                </geometry>
+            </visual>
+            <inertial>
+                <mass value="0.1"/>
+                <inertia ixx="2e-05" iyy="2e-05" izz="2e-05" ixy="0.0" ixz="0.0" iyz="0.0"/>
+            </inertial>
+            <collision>
+                <geometry>
+                    <sphere radius="0.01"/>
+                </geometry>
+            </collision>
+        </link>
+        <gazebo reference="tether_0/fragment_5">
+            <material>Gazebo/Red</material>
+        </gazebo>
+                    <!--tether fragment joint-->
+        <joint name="tether_0/joint_5" type="continuous">
+            <origin rpy="0 0 0" xyz="0 0 1.0"/>
+            <parent link="tether_0/fragment_4"/>
+            <child link="tether_0/fragment_5"/>
+                <axis xyz="0 1 0" />
+            <dynamics damping="0.1" friction="0.1"/>
+        </joint>
+            <link name="tether_0/fragment_6">
+            <visual>
+                <origin rpy="0 0 0" xyz="0 0 0"/>
+                <geometry>
+                    <sphere radius="0.01"/>
+                </geometry>
+            </visual>
+            <inertial>
+                <mass value="0.1"/>
+                <inertia ixx="2e-05" iyy="2e-05" izz="2e-05" ixy="0.0" ixz="0.0" iyz="0.0"/>
+            </inertial>
+            <collision>
+                <geometry>
+                    <sphere radius="0.01"/>
+                </geometry>
+            </collision>
+        </link>
+        <gazebo reference="tether_0/fragment_6">
+            <material>Gazebo/Red</material>
+        </gazebo>
+                    <!--tether fragment joint-->
+        <joint name="tether_0/joint_6" type="continuous">
+            <origin rpy="0 0 0" xyz="0 0 1.0"/>
+            <parent link="tether_0/fragment_5"/>
+            <child link="tether_0/fragment_6"/>
+                <axis xyz="0 1 0" />
+            <dynamics damping="0.1" friction="0.1"/>
+        </joint>
+            <link name="tether_0/fragment_7">
+            <visual>
+                <origin rpy="0 0 0" xyz="0 0 0"/>
+                <geometry>
+                    <sphere radius="0.01"/>
+                </geometry>
+            </visual>
+            <inertial>
+                <mass value="0.1"/>
+                <inertia ixx="2e-05" iyy="2e-05" izz="2e-05" ixy="0.0" ixz="0.0" iyz="0.0"/>
+            </inertial>
+            <collision>
+                <geometry>
+                    <sphere radius="0.01"/>
+                </geometry>
+            </collision>
+        </link>
+        <gazebo reference="tether_0/fragment_7">
+            <material>Gazebo/Red</material>
+        </gazebo>
+                    <!--tether fragment joint-->
+        <joint name="tether_0/joint_7" type="continuous">
+            <origin rpy="0 0 0" xyz="0 0 1.0"/>
+            <parent link="tether_0/fragment_6"/>
+            <child link="tether_0/fragment_7"/>
+                <axis xyz="0 1 0" />
+            <dynamics damping="0.1" friction="0.1"/>
+        </joint>
+            <link name="tether_0/fragment_8">
+            <visual>
+                <origin rpy="0 0 0" xyz="0 0 0"/>
+                <geometry>
+                    <sphere radius="0.01"/>
+                </geometry>
+            </visual>
+            <inertial>
+                <mass value="0.1"/>
+                <inertia ixx="2e-05" iyy="2e-05" izz="2e-05" ixy="0.0" ixz="0.0" iyz="0.0"/>
+            </inertial>
+            <collision>
+                <geometry>
+                    <sphere radius="0.01"/>
+                </geometry>
+            </collision>
+        </link>
+        <gazebo reference="tether_0/fragment_8">
+            <material>Gazebo/Red</material>
+        </gazebo>
+                    <!--tether fragment joint-->
+        <joint name="tether_0/joint_8" type="continuous">
+            <origin rpy="0 0 0" xyz="0 0 1.0"/>
+            <parent link="tether_0/fragment_7"/>
+            <child link="tether_0/fragment_8"/>
+                <axis xyz="0 1 0" />
+            <dynamics damping="0.1" friction="0.1"/>
+        </joint>
+            <link name="tether_0/fragment_9">
+            <visual>
+                <origin rpy="0 0 0" xyz="0 0 0"/>
+                <geometry>
+                    <sphere radius="0.01"/>
+                </geometry>
+            </visual>
+            <inertial>
+                <mass value="0.1"/>
+                <inertia ixx="2e-05" iyy="2e-05" izz="2e-05" ixy="0.0" ixz="0.0" iyz="0.0"/>
+            </inertial>
+            <collision>
+                <geometry>
+                    <sphere radius="0.01"/>
+                </geometry>
+            </collision>
+        </link>
+        <gazebo reference="tether_0/fragment_9">
+            <material>Gazebo/Red</material>
+        </gazebo>
+                    <!--tether fragment joint-->
+        <joint name="tether_0/joint_9" type="continuous">
+            <origin rpy="0 0 0" xyz="0 0 1.0"/>
+            <parent link="tether_0/fragment_8"/>
+            <child link="tether_0/fragment_9"/>
+                <axis xyz="0 1 0" />
+            <dynamics damping="0.1" friction="0.1"/>
+        </joint>
+            <link name="tether_0/rod">
+            <visual>
+                <origin rpy="0 0 0" xyz="0 0 0.1"/>
+                <geometry>
+                    <cylinder length="0.2" radius="0.01"/>
+                </geometry>
+            </visual>
+            <inertial>
+                <mass value="0.01"/>
+                <inertia ixx="0.01" iyy="0.01" izz="0.01" ixy="0.0" ixz="0.0" iyz="0.0"/>
+            </inertial>
+            <collision>
+                <geometry>
+                    <cylinder length="0.2" radius="0.01"/>
+                </geometry>
+            </collision>
+        </link>
+        <gazebo reference="tether_0/rod">
+            <material>Gazebo/Orange</material>
+        </gazebo>
+        <!--uav => tether joint-->
+        <joint name="tether_0/rod_joint" type="fixed">
             <parent link="${namespace}/base_link"/>
+            <child link="tether_0/rod"/>
+                <origin rpy="0 ${pi/2} 0" xyz="0 0 0"/>
+        </joint>
+        <joint name="tether_0/uav_joint" type="continuous">
+            <parent link="tether_0/rod"/>
             <child link="tether_0/fragment_0"/>
-                <origin rpy="0 ${pi/2} 0" xyz="0 0 0"/>
+                <axis xyz="0 1 0" />
         </joint>
             <!--tether end joint-->
         <joint name="tether_0/ugv_joint_1" type="continuous">
                 <origin rpy="0 ${-pi/2} 0" xyz="0 0 1.0"/>
-            <parent link="tether_0/fragment_4"/>
+            <parent link="tether_0/fragment_9"/>
             <child link="mp_500_0/tether_end"/>
             <axis xyz="1 0 0" />
@@ -159,5 +324,5 @@
             <inertial>
                 <mass value="0.1"/>
-                <inertia ixx="3e-05" iyy="3e-05" izz="3e-05" ixy="0.0" ixz="0.0" iyz="0.0"/>
+                <inertia ixx="2e-05" iyy="2e-05" izz="2e-05" ixy="0.0" ixz="0.0" iyz="0.0"/>
             </inertial>
             <collision>
@@ -179,5 +344,5 @@
             <inertial>
                 <mass value="0.1"/>
-                <inertia ixx="3e-05" iyy="3e-05" izz="3e-05" ixy="0.0" ixz="0.0" iyz="0.0"/>
+                <inertia ixx="2e-05" iyy="2e-05" izz="2e-05" ixy="0.0" ixz="0.0" iyz="0.0"/>
             </inertial>
             <collision>
@@ -195,5 +360,5 @@
             <parent link="tether_1/fragment_0"/>
             <child link="tether_1/fragment_1"/>
-            <axis xyz="1 0 0" />
+                <axis xyz="1 0 0" />
             <dynamics damping="0.1" friction="0.1"/>
         </joint>
@@ -207,5 +372,5 @@
             <inertial>
                 <mass value="0.1"/>
-                <inertia ixx="3e-05" iyy="3e-05" izz="3e-05" ixy="0.0" ixz="0.0" iyz="0.0"/>
+                <inertia ixx="2e-05" iyy="2e-05" izz="2e-05" ixy="0.0" ixz="0.0" iyz="0.0"/>
             </inertial>
             <collision>
@@ -223,5 +388,5 @@
             <parent link="tether_1/fragment_1"/>
             <child link="tether_1/fragment_2"/>
-            <axis xyz="1 0 0" />
+                <axis xyz="1 0 0" />
             <dynamics damping="0.1" friction="0.1"/>
         </joint>
@@ -235,5 +400,5 @@
             <inertial>
                 <mass value="0.1"/>
-                <inertia ixx="3e-05" iyy="3e-05" izz="3e-05" ixy="0.0" ixz="0.0" iyz="0.0"/>
+                <inertia ixx="2e-05" iyy="2e-05" izz="2e-05" ixy="0.0" ixz="0.0" iyz="0.0"/>
             </inertial>
             <collision>
@@ -251,5 +416,5 @@
             <parent link="tether_1/fragment_2"/>
             <child link="tether_1/fragment_3"/>
-            <axis xyz="1 0 0" />
+                <axis xyz="1 0 0" />
             <dynamics damping="0.1" friction="0.1"/>
         </joint>
@@ -263,5 +428,5 @@
             <inertial>
                 <mass value="0.1"/>
-                <inertia ixx="3e-05" iyy="3e-05" izz="3e-05" ixy="0.0" ixz="0.0" iyz="0.0"/>
+                <inertia ixx="2e-05" iyy="2e-05" izz="2e-05" ixy="0.0" ixz="0.0" iyz="0.0"/>
             </inertial>
             <collision>
@@ -279,17 +444,182 @@
             <parent link="tether_1/fragment_3"/>
             <child link="tether_1/fragment_4"/>
-            <axis xyz="1 0 0" />
-            <dynamics damping="0.1" friction="0.1"/>
-        </joint>
-            <!--uav => tether joint-->
-        <joint name="tether_1/uav_joint" type="fixed">
+                <axis xyz="1 0 0" />
+            <dynamics damping="0.1" friction="0.1"/>
+        </joint>
+            <link name="tether_1/fragment_5">
+            <visual>
+                <origin rpy="0 0 0" xyz="0 0 0"/>
+                <geometry>
+                    <sphere radius="0.01"/>
+                </geometry>
+            </visual>
+            <inertial>
+                <mass value="0.1"/>
+                <inertia ixx="2e-05" iyy="2e-05" izz="2e-05" ixy="0.0" ixz="0.0" iyz="0.0"/>
+            </inertial>
+            <collision>
+                <geometry>
+                    <sphere radius="0.01"/>
+                </geometry>
+            </collision>
+        </link>
+        <gazebo reference="tether_1/fragment_5">
+            <material>Gazebo/Red</material>
+        </gazebo>
+                    <!--tether fragment joint-->
+        <joint name="tether_1/joint_5" type="continuous">
+            <origin rpy="0 0 0" xyz="0 0 1.0"/>
+            <parent link="tether_1/fragment_4"/>
+            <child link="tether_1/fragment_5"/>
+                <axis xyz="1 0 0" />
+            <dynamics damping="0.1" friction="0.1"/>
+        </joint>
+            <link name="tether_1/fragment_6">
+            <visual>
+                <origin rpy="0 0 0" xyz="0 0 0"/>
+                <geometry>
+                    <sphere radius="0.01"/>
+                </geometry>
+            </visual>
+            <inertial>
+                <mass value="0.1"/>
+                <inertia ixx="2e-05" iyy="2e-05" izz="2e-05" ixy="0.0" ixz="0.0" iyz="0.0"/>
+            </inertial>
+            <collision>
+                <geometry>
+                    <sphere radius="0.01"/>
+                </geometry>
+            </collision>
+        </link>
+        <gazebo reference="tether_1/fragment_6">
+            <material>Gazebo/Red</material>
+        </gazebo>
+                    <!--tether fragment joint-->
+        <joint name="tether_1/joint_6" type="continuous">
+            <origin rpy="0 0 0" xyz="0 0 1.0"/>
+            <parent link="tether_1/fragment_5"/>
+            <child link="tether_1/fragment_6"/>
+                <axis xyz="1 0 0" />
+            <dynamics damping="0.1" friction="0.1"/>
+        </joint>
+            <link name="tether_1/fragment_7">
+            <visual>
+                <origin rpy="0 0 0" xyz="0 0 0"/>
+                <geometry>
+                    <sphere radius="0.01"/>
+                </geometry>
+            </visual>
+            <inertial>
+                <mass value="0.1"/>
+                <inertia ixx="2e-05" iyy="2e-05" izz="2e-05" ixy="0.0" ixz="0.0" iyz="0.0"/>
+            </inertial>
+            <collision>
+                <geometry>
+                    <sphere radius="0.01"/>
+                </geometry>
+            </collision>
+        </link>
+        <gazebo reference="tether_1/fragment_7">
+            <material>Gazebo/Red</material>
+        </gazebo>
+                    <!--tether fragment joint-->
+        <joint name="tether_1/joint_7" type="continuous">
+            <origin rpy="0 0 0" xyz="0 0 1.0"/>
+            <parent link="tether_1/fragment_6"/>
+            <child link="tether_1/fragment_7"/>
+                <axis xyz="1 0 0" />
+            <dynamics damping="0.1" friction="0.1"/>
+        </joint>
+            <link name="tether_1/fragment_8">
+            <visual>
+                <origin rpy="0 0 0" xyz="0 0 0"/>
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
File: ugv_description/urdf/mp_500/xacros/mp_500_tether_end.xacro (robot description, xacro)
@@ -2,8 +2,9 @@
 <robot xmlns:xacro="http://www.ros.org/wiki/xacro" name="mp_500">
     <xacro:macro name="mp_500_tether_end" params="name">
-        <joint name="${name}_joint" type="fixed">
+        <joint name="${name}_joint" type="continuous">
             <parent link="${name}" />
             <child link="${namespace}/base_link" />
             <origin xyz="0.0 0.0 -0.4" rpy="0 0 0" />
+            <axis xyz="0 0 1" />
         </joint>
         <link name="${name}">
