Commit message: Update params

File: tether_description/urdf/lumped_mass_tether_fragment.xacro (robot description, xacro)
@@ -6,5 +6,5 @@
         {%- set lump_mass = 0.10 -%}
         {%- set lump_radius = 0.01 -%}
-        {%- set lump_inertia = 2*lump_mass*lump_radius**2 -%}
+        {%- set lump_inertia = 5*lump_mass*lump_radius**2 -%}
         {%- set element_length = 1.0 -%}
         <!--joint dynamics-->

File: tether_description/urdf/tether.xacro (robot description, xacro)
@@ -13,5 +13,5 @@
             <inertial>
                 <mass value="0.1"/>
-                <inertia ixx="2e-05" iyy="2e-05" izz="2e-05" ixy="0.0" ixz="0.0" iyz="0.0"/>
+                <inertia ixx="5e-05" iyy="5e-05" izz="5e-05" ixy="0.0" ixz="0.0" iyz="0.0"/>
             </inertial>
             <collision>
@@ -33,5 +33,5 @@
             <inertial>
                 <mass value="0.1"/>
-                <inertia ixx="2e-05" iyy="2e-05" izz="2e-05" ixy="0.0" ixz="0.0" iyz="0.0"/>
+                <inertia ixx="5e-05" iyy="5e-05" izz="5e-05" ixy="0.0" ixz="0.0" iyz="0.0"/>
             </inertial>
             <collision>
@@ -61,5 +61,5 @@
             <inertial>
                 <mass value="0.1"/>
-                <inertia ixx="2e-05" iyy="2e-05" izz="2e-05" ixy="0.0" ixz="0.0" iyz="0.0"/>
+                <inertia ixx="5e-05" iyy="5e-05" izz="5e-05" ixy="0.0" ixz="0.0" iyz="0.0"/>
             </inertial>
             <collision>
@@ -89,5 +89,5 @@
             <inertial>
                 <mass value="0.1"/>
-                <inertia ixx="2e-05" iyy="2e-05" izz="2e-05" ixy="0.0" ixz="0.0" iyz="0.0"/>
+                <inertia ixx="5e-05" iyy="5e-05" izz="5e-05" ixy="0.0" ixz="0.0" iyz="0.0"/>
             </inertial>
             <collision>
@@ -117,5 +117,5 @@
             <inertial>
                 <mass value="0.1"/>
-                <inertia ixx="2e-05" iyy="2e-05" izz="2e-05" ixy="0.0" ixz="0.0" iyz="0.0"/>
+                <inertia ixx="5e-05" iyy="5e-05" izz="5e-05" ixy="0.0" ixz="0.0" iyz="0.0"/>
             </inertial>
             <collision>
@@ -145,5 +145,5 @@
             <inertial>
                 <mass value="0.1"/>
-                <inertia ixx="2e-05" iyy="2e-05" izz="2e-05" ixy="0.0" ixz="0.0" iyz="0.0"/>
+                <inertia ixx="5e-05" iyy="5e-05" izz="5e-05" ixy="0.0" ixz="0.0" iyz="0.0"/>
             </inertial>
             <collision>
@@ -173,5 +173,5 @@
             <inertial>
                 <mass value="0.1"/>
-                <inertia ixx="2e-05" iyy="2e-05" izz="2e-05" ixy="0.0" ixz="0.0" iyz="0.0"/>
+                <inertia ixx="5e-05" iyy="5e-05" izz="5e-05" ixy="0.0" ixz="0.0" iyz="0.0"/>
             </inertial>
             <collision>
@@ -201,5 +201,5 @@
             <inertial>
                 <mass value="0.1"/>
-                <inertia ixx="2e-05" iyy="2e-05" izz="2e-05" ixy="0.0" ixz="0.0" iyz="0.0"/>
+                <inertia ixx="5e-05" iyy="5e-05" izz="5e-05" ixy="0.0" ixz="0.0" iyz="0.0"/>
             </inertial>
             <collision>
@@ -229,5 +229,5 @@
             <inertial>
                 <mass value="0.1"/>
-                <inertia ixx="2e-05" iyy="2e-05" izz="2e-05" ixy="0.0" ixz="0.0" iyz="0.0"/>
+                <inertia ixx="5e-05" iyy="5e-05" izz="5e-05" ixy="0.0" ixz="0.0" iyz="0.0"/>
             </inertial>
             <collision>
@@ -257,5 +257,5 @@
             <inertial>
                 <mass value="0.1"/>
-                <inertia ixx="2e-05" iyy="2e-05" izz="2e-05" ixy="0.0" ixz="0.0" iyz="0.0"/>
+                <inertia ixx="5e-05" iyy="5e-05" izz="5e-05" ixy="0.0" ixz="0.0" iyz="0.0"/>
             </inertial>
             <collision>
@@ -324,5 +324,5 @@
             <inertial>
                 <mass value="0.1"/>
-                <inertia ixx="2e-05" iyy="2e-05" izz="2e-05" ixy="0.0" ixz="0.0" iyz="0.0"/>
+                <inertia ixx="5e-05" iyy="5e-05" izz="5e-05" ixy="0.0" ixz="0.0" iyz="0.0"/>
             </inertial>
             <collision>
@@ -344,5 +344,5 @@
             <inertial>
                 <mass value="0.1"/>
-                <inertia ixx="2e-05" iyy="2e-05" izz="2e-05" ixy="0.0" ixz="0.0" iyz="0.0"/>
+                <inertia ixx="5e-05" iyy="5e-05" izz="5e-05" ixy="0.0" ixz="0.0" iyz="0.0"/>
             </inertial>
             <collision>
@@ -372,5 +372,5 @@
             <inertial>
                 <mass value="0.1"/>
-                <inertia ixx="2e-05" iyy="2e-05" izz="2e-05" ixy="0.0" ixz="0.0" iyz="0.0"/>
+                <inertia ixx="5e-05" iyy="5e-05" izz="5e-05" ixy="0.0" ixz="0.0" iyz="0.0"/>
             </inertial>
             <collision>
@@ -400,5 +400,5 @@
             <inertial>
                 <mass value="0.1"/>
-                <inertia ixx="2e-05" iyy="2e-05" izz="2e-05" ixy="0.0" ixz="0.0" iyz="0.0"/>
+                <inertia ixx="5e-05" iyy="5e-05" izz="5e-05" ixy="0.0" ixz="0.0" iyz="0.0"/>
             </inertial>
             <collision>
@@ -428,5 +428,5 @@
             <inertial>
                 <mass value="0.1"/>
-                <inertia ixx="2e-05" iyy="2e-05" izz="2e-05" ixy="0.0" ixz="0.0" iyz="0.0"/>
+                <inertia ixx="5e-05" iyy="5e-05" izz="5e-05" ixy="0.0" ixz="0.0" iyz="0.0"/>
             </inertial>
             <collision>
@@ -456,5 +456,5 @@
             <inertial>
                 <mass value="0.1"/>
-                <inertia ixx="2e-05" iyy="2e-05" izz="2e-05" ixy="0.0" ixz="0.0" iyz="0.0"/>
+                <inertia ixx="5e-05" iyy="5e-05" izz="5e-05" ixy="0.0" ixz="0.0" iyz="0.0"/>
             </inertial>
             <collision>
@@ -484,5 +484,5 @@
             <inertial>
                 <mass value="0.1"/>
-                <inertia ixx="2e-05" iyy="2e-05" izz="2e-05" ixy="0.0" ixz="0.0" iyz="0.0"/>
+                <inertia ixx="5e-05" iyy="5e-05" izz="5e-05" ixy="0.0" ixz="0.0" iyz="0.0"/>
             </inertial>
             <collision>
@@ -512,5 +512,5 @@
             <inertial>
                 <mass value="0.1"/>
-                <inertia ixx="2e-05" iyy="2e-05" izz="2e-05" ixy="0.0" ixz="0.0" iyz="0.0"/>
+                <inertia ixx="5e-05" iyy="5e-05" izz="5e-05" ixy="0.0" ixz="0.0" iyz="0.0"/>
             </inertial>
             <collision>
@@ -540,5 +540,5 @@
             <inertial>
                 <mass value="0.1"/>
-                <inertia ixx="2e-05" iyy="2e-05" izz="2e-05" ixy="0.0" ixz="0.0" iyz="0.0"/>
+                <inertia ixx="5e-05" iyy="5e-05" izz="5e-05" ixy="0.0" ixz="0.0" iyz="0.0"/>
             </inertial>
             <collision>
@@ -568,5 +568,5 @@
             <inertial>
                 <mass value="0.1"/>
-                <inertia ixx="2e-05" iyy="2e-05" izz="2e-05" ixy="0.0" ixz="0.0" iyz="0.0"/>
+                <inertia ixx="5e-05" iyy="5e-05" izz="5e-05" ixy="0.0" ixz="0.0" iyz="0.0"/>
             </inertial>
             <collision>
@@ -635,5 +635,5 @@
             <inertial>
                 <mass value="0.1"/>
-                <inertia ixx="2e-05" iyy="2e-05" izz="2e-05" ixy="0.0" ixz="0.0" iyz="0.0"/>
+                <inertia ixx="5e-05" iyy="5e-05" izz="5e-05" ixy="0.0" ixz="0.0" iyz="0.0"/>
             </inertial>
             <collision>
@@ -655,5 +655,5 @@
             <inertial>
                 <mass value="0.1"/>
-                <inertia ixx="2e-05" iyy="2e-05" izz="2e-05" ixy="0.0" ixz="0.0" iyz="0.0"/>
+                <inertia ixx="5e-05" iyy="5e-05" izz="5e-05" ixy="0.0" ixz="0.0" iyz="0.0"/>
             </inertial>
             <collision>
@@ -683,5 +683,5 @@
             <inertial>
                 <mass value="0.1"/>
-                <inertia ixx="2e-05" iyy="2e-05" izz="2e-05" ixy="0.0" ixz="0.0" iyz="0.0"/>
+                <inertia ixx="5e-05" iyy="5e-05" izz="5e-05" ixy="0.0" ixz="0.0" iyz="0.0"/>
             </inertial>
             <collision>
@@ -711,5 +711,5 @@
             <inertial>
                 <mass value="0.1"/>
-                <inertia ixx="2e-05" iyy="2e-05" izz="2e-05" ixy="0.0" ixz="0.0" iyz="0.0"/>
+                <inertia ixx="5e-05" iyy="5e-05" izz="5e-05" ixy="0.0" ixz="0.0" iyz="0.0"/>
             </inertial>
             <collision>
@@ -739,5 +739,5 @@
             <inertial>
                 <mass value="0.1"/>
-                <inertia ixx="2e-05" iyy="2e-05" izz="2e-05" ixy="0.0" ixz="0.0" iyz="0.0"/>
+                <inertia ixx="5e-05" iyy="5e-05" izz="5e-05" ixy="0.0" ixz="0.0" iyz="0.0"/>
             </inertial>
             <collision>
@@ -767,5 +767,5 @@
             <inertial>
                 <mass value="0.1"/>
-                <inertia ixx="2e-05" iyy="2e-05" izz="2e-05" ixy="0.0" ixz="0.0" iyz="0.0"/>
+                <inertia ixx="5e-05" iyy="5e-05" izz="5e-05" ixy="0.0" ixz="0.0" iyz="0.0"/>
             </inertial>
             <collision>
@@ -795,5 +795,5 @@
             <inertial>
                 <mass value="0.1"/>
-                <inertia ixx="2e-05" iyy="2e-05" izz="2e-05" ixy="0.0" ixz="0.0" iyz="0.0"/>
+                <inertia ixx="5e-05" iyy="5e-05" izz="5e-05" ixy="0.0" ixz="0.0" iyz="0.0"/>
             </inertial>
             <collision>
@@ -823,5 +823,5 @@
             <inertial>
                 <mass value="0.1"/>
-                <inertia ixx="2e-05" iyy="2e-05" izz="2e-05" ixy="0.0" ixz="0.0" iyz="0.0"/>
+                <inertia ixx="5e-05" iyy="5e-05" izz="5e-05" ixy="0.0" ixz="0.0" iyz="0.0"/>
             </inertial>
             <collision>
@@ -851,5 +851,5 @@
             <inertial>
                 <mass value="0.1"/>
-                <inertia ixx="2e-05" iyy="2e-05" izz="2e-05" ixy="0.0" ixz="0.0" iyz="0.0"/>
+                <inertia ixx="5e-05" iyy="5e-05" izz="5e-05" ixy="0.0" ixz="0.0" iyz="0.0"/>
             </inertial>
             <collision>
@@ -879,5 +879,5 @@
             <inertial>
                 <mass value="0.1"/>
-                <inertia ixx="2e-05" iyy="2e-05" izz="2e-05" ixy="0.0" ixz="0.0" iyz="0.0"/>
+                <inertia ixx="5e-05" iyy="5e-05" izz="5e-05" ixy="0.0" ixz="0.0" iyz="0.0"/>
             </inertial>
             <collision>
@@ -946,5 +946,5 @@
             <inertial>
                 <mass value="0.1"/>
-                <inertia ixx="2e-05" iyy="2e-05" izz="2e-05" ixy="0.0" ixz="0.0" iyz="0.0"/>
+                <inertia ixx="5e-05" iyy="5e-05" izz="5e-05" ixy="0.0" ixz="0.0" iyz="0.0"/>
             </inertial>
             <collision>
@@ -966,5 +966,5 @@
             <inertial>
                 <mass value="0.1"/>
-                <inertia ixx="2e-05" iyy="2e-05" izz="2e-05" ixy="0.0" ixz="0.0" iyz="0.0"/>
+                <inertia ixx="5e-05" iyy="5e-05" izz="5e-05" ixy="0.0" ixz="0.0" iyz="0.0"/>
             </inertial>
             <collision>
@@ -994,5 +994,5 @@
             <inertial>
                 <mass value="0.1"/>
-                <inertia ixx="2e-05" iyy="2e-05" izz="2e-05" ixy="0.0" ixz="0.0" iyz="0.0"/>
+                <inertia ixx="5e-05" iyy="5e-05" izz="5e-05" ixy="0.0" ixz="0.0" iyz="0.0"/>
             </inertial>
             <collision>
@@ -1022,5 +1022,5 @@
             <inertial>
                 <mass value="0.1"/>
-                <inertia ixx="2e-05" iyy="2e-05" izz="2e-05" ixy="0.0" ixz="0.0" iyz="0.0"/>
+                <inertia ixx="5e-05" iyy="5e-05" izz="5e-05" ixy="0.0" ixz="0.0" iyz="0.0"/>
             </inertial>
             <collision>
@@ -1050,5 +1050,5 @@
             <inertial>
                 <mass value="0.1"/>
-                <inertia ixx="2e-05" iyy="2e-05" izz="2e-05" ixy="0.0" ixz="0.0" iyz="0.0"/>
+                <inertia ixx="5e-05" iyy="5e-05" izz="5e-05" ixy="0.0" ixz="0.0" iyz="0.0"/>
             </inertial>
             <collision>
@@ -1078,5 +1078,5 @@
             <inertial>
                 <mass value="0.1"/>
-                <inertia ixx="2e-05" iyy="2e-05" izz="2e-05" ixy="0.0" ixz="0.0" iyz="0.0"/>
+                <inertia ixx="5e-05" iyy="5e-05" izz="5e-05" ixy="0.0" ixz="0.0" iyz="0.0"/>
             </inertial>
             <collision>
@@ -1106,5 +1106,5 @@
             <inertial>
                 <mass value="0.1"/>
-                <inertia ixx="2e-05" iyy="2e-05" izz="2e-05" ixy="0.0" ixz="0.0" iyz="0.0"/>
+                <inertia ixx="5e-05" iyy="5e-05" izz="5e-05" ixy="0.0" ixz="0.0" iyz="0.0"/>
             </inertial>
             <collision>
@@ -1134,5 +1134,5 @@
             <inertial>
                 <mass value="0.1"/>
-                <inertia ixx="2e-05" iyy="2e-05" izz="2e-05" ixy="0.0" ixz="0.0" iyz="0.0"/>
+                <inertia ixx="5e-05" iyy="5e-05" izz="5e-05" ixy="0.0" ixz="0.0" iyz="0.0"/>
             </inertial>
             <collision>
@@ -1162,5 +1162,5 @@
             <inertial>
                 <mass value="0.1"/>
-                <inertia ixx="2e-05" iyy="2e-05" izz="2e-05" ixy="0.0" ixz="0.0" iyz="0.0"/>
+                <inertia ixx="5e-05" iyy="5e-05" izz="5e-05" ixy="0.0" ixz="0.0" iyz="0.0"/>
             </inertial>
             <collision>
@@ -1190,5 +1190,5 @@
             <inertial>
                 <mass value="0.1"/>
-                <inertia ixx="2e-05" iyy="2e-05" izz="2e-05" ixy="0.0" ixz="0.0" iyz="0.0"/>
+                <inertia ixx="5e-05" iyy="5e-05" izz="5e-05" ixy="0.0" ixz="0.0" iyz="0.0"/>
             </inertial>
             <collision>

File: ugv_description/urdf/mp_500/mp_500_tether.urdf.xacro (robot description, xacro)
@@ -22,4 +22,6 @@
         <xacro:mp_500_tether_end name="${namespace}/tether_end">
         </xacro:mp_500_tether_end>
+        <xacro:counter_weight name="${namespace}/counter_weight">
+        </xacro:counter_weight>
         <!--+++++++++++++++++++laserscanner_front_link++++++++++++++++++++++++-->
         <!-- SENSORS -->

File: ugv_description/urdf/mp_500/xacros/mp_500_tether_end.xacro (robot description, xacro)
@@ -1,9 +1,13 @@
 <?xml version="1.0"?>
 <robot xmlns:xacro="http://www.ros.org/wiki/xacro" name="mp_500">
+    <xacro:property name="counter_weight_mass" value="5.0" />
+    <xacro:property name="counter_weight_x" value="0.1" />
+    <xacro:property name="counter_weight_y" value="0.1" />
+    <xacro:property name="counter_weight_z" value="0.1" />
     <xacro:macro name="mp_500_tether_end" params="name">
         <joint name="${name}_joint" type="continuous">
             <parent link="${name}" />
             <child link="${namespace}/base_link" />
-            <origin xyz="0.0 0.0 -0.4" rpy="0 0 0" />
+            <origin xyz="0.0 0.0 -0.2" rpy="0 0 0" />
             <axis xyz="0 0 1" />
         </joint>
@@ -24,4 +28,27 @@
             </collision>
         </link>
-        </xacro:macro>
+    </xacro:macro>
+    <xacro:macro name="counter_weight" params="name">
+        <joint name="${name}_joint" type="fixed">
+            <parent link="${namespace}/base_link" />
+            <child link="${name}" />
+            <origin xyz="-0.4 0.0 0.4" rpy="0 0 0" />
+        </joint>
+        <link name="${name}">
+            <visual>
+                <geometry>
+                    <box size="${counter_weight_x} ${counter_weight_y} ${counter_weight_z}"/>
+                </geometry>
+            </visual>
+            <collision>
+                <geometry>
+                    <box size="${counter_weight_x} ${counter_weight_y} ${counter_weight_z}"/>
+                </geometry>
+            </collision>
+            <inertial>
+                <mass value="${counter_weight_mass}"/>
+                <inertia ixx="1/12*${counter_weight_mass}*(${counter_weight_y}**2+${counter_weight_z}**2)" iyy="1/12*${counter_weight_mass}*(${counter_weight_z}**2+${counter_weight_x}**2)" izz="1/12*${counter_weight_mass}*(${counter_weight_x}**2+${counter_weight_y}**2)" ixy="0" ixz="0" iyz="0"/>
+            </inertial>
+        </link>
+    </xacro:macro>
 </robot>
