Commit message: Update params

File: tether_description/urdf/lumped_mass_tether_fragment.xacro (robot description, xacro)
@@ -4,13 +4,13 @@
     <xacro:macro name="tether">
         <!--tether fragment param-->
-        {%- set lump_mass = 0.10 -%}
-        {%- set lump_radius = 0.01 -%}
-        {%- set lump_inertia = 5*lump_mass*lump_radius**2 -%}
-        {%- set element_length = 1.0 -%}
+        {%- set lump_mass = 0.05 -%}
+        {%- set lump_radius = 0.03 -%}
+        {%- set lump_inertia = 3*lump_mass*lump_radius**2 -%}
+        {%- set element_length = 5.0 -%}
         <!--joint dynamics-->
         {%- set damping = 0.1 -%}
         {%- set friction = 0.1 -%}
         <!--link number-->
-        {%- set tether_fragments = 10 -%}
+        {%- set tether_fragments = 4 -%}
         {%- set tether_number = 4 -%}
         {%- macro tether_fragment(dirc, n) -%}

File: tether_description/urdf/tether.xacro (robot description, xacro)
@@ -8,14 +8,14 @@
                 <origin rpy="0 0 0" xyz="0 0 0"/>
                 <geometry>
-                    <sphere radius="0.01"/>
-                </geometry>
-            </visual>
-            <inertial>
-                <mass value="0.1"/>
-                <inertia ixx="5e-05" iyy="5e-05" izz="5e-05" ixy="0.0" ixz="0.0" iyz="0.0"/>
-            </inertial>
-            <collision>
-                <geometry>
-                    <sphere radius="0.01"/>
+                    <sphere radius="0.03"/>
+                </geometry>
+            </visual>
+            <inertial>
+                <mass value="0.05"/>
+                <inertia ixx="0.000135" iyy="0.000135" izz="0.000135" ixy="0.0" ixz="0.0" iyz="0.0"/>
+            </inertial>
+            <collision>
+                <geometry>
+                    <sphere radius="0.03"/>
                 </geometry>
             </collision>
@@ -28,14 +28,14 @@
                 <origin rpy="0 0 0" xyz="0 0 0"/>
                 <geometry>
-                    <sphere radius="0.01"/>
-                </geometry>
-            </visual>
-            <inertial>
-                <mass value="0.1"/>
-                <inertia ixx="5e-05" iyy="5e-05" izz="5e-05" ixy="0.0" ixz="0.0" iyz="0.0"/>
-            </inertial>
-            <collision>
-                <geometry>
-                    <sphere radius="0.01"/>
+                    <sphere radius="0.03"/>
+                </geometry>
+            </visual>
+            <inertial>
+                <mass value="0.05"/>
+                <inertia ixx="0.000135" iyy="0.000135" izz="0.000135" ixy="0.0" ixz="0.0" iyz="0.0"/>
+            </inertial>
+            <collision>
+                <geometry>
+                    <sphere radius="0.03"/>
                 </geometry>
             </collision>
@@ -46,5 +46,5 @@
                     <!--tether fragment joint-->
         <joint name="tether_0/joint_1" type="continuous">
-            <origin rpy="0 0 0" xyz="0 0 1.0"/>
+            <origin rpy="0 0 0" xyz="0 0 5.0"/>
             <parent link="tether_0/fragment_0"/>
             <child link="tether_0/fragment_1"/>
@@ -56,14 +56,14 @@
                 <origin rpy="0 0 0" xyz="0 0 0"/>
                 <geometry>
-                    <sphere radius="0.01"/>
-                </geometry>
-            </visual>
-            <inertial>
-                <mass value="0.1"/>
-                <inertia ixx="5e-05" iyy="5e-05" izz="5e-05" ixy="0.0" ixz="0.0" iyz="0.0"/>
-            </inertial>
-            <collision>
-                <geometry>
-                    <sphere radius="0.01"/>
+                    <sphere radius="0.03"/>
+                </geometry>
+            </visual>
+            <inertial>
+                <mass value="0.05"/>
+                <inertia ixx="0.000135" iyy="0.000135" izz="0.000135" ixy="0.0" ixz="0.0" iyz="0.0"/>
+            </inertial>
+            <collision>
+                <geometry>
+                    <sphere radius="0.03"/>
                 </geometry>
             </collision>
@@ -74,5 +74,5 @@
                     <!--tether fragment joint-->
         <joint name="tether_0/joint_2" type="continuous">
-            <origin rpy="0 0 0" xyz="0 0 1.0"/>
+            <origin rpy="0 0 0" xyz="0 0 5.0"/>
             <parent link="tether_0/fragment_1"/>
             <child link="tether_0/fragment_2"/>
@@ -84,14 +84,14 @@
                 <origin rpy="0 0 0" xyz="0 0 0"/>
                 <geometry>
-                    <sphere radius="0.01"/>
-                </geometry>
-            </visual>
-            <inertial>
-                <mass value="0.1"/>
-                <inertia ixx="5e-05" iyy="5e-05" izz="5e-05" ixy="0.0" ixz="0.0" iyz="0.0"/>
-            </inertial>
-            <collision>
-                <geometry>
-                    <sphere radius="0.01"/>
+                    <sphere radius="0.03"/>
+                </geometry>
+            </visual>
+            <inertial>
+                <mass value="0.05"/>
+                <inertia ixx="0.000135" iyy="0.000135" izz="0.000135" ixy="0.0" ixz="0.0" iyz="0.0"/>
+            </inertial>
+            <collision>
+                <geometry>
+                    <sphere radius="0.03"/>
                 </geometry>
             </collision>
@@ -102,175 +102,7 @@
                     <!--tether fragment joint-->
         <joint name="tether_0/joint_3" type="continuous">
-            <origin rpy="0 0 0" xyz="0 0 1.0"/>
+            <origin rpy="0 0 0" xyz="0 0 5.0"/>
             <parent link="tether_0/fragment_2"/>
             <child link="tether_0/fragment_3"/>
-                <axis xyz="0 1 0" />
-            <dynamics damping="0.1" friction="0.1"/>
-        </joint>
-            <link name="tether_0/fragment_4">
-            <visual>
-                <origin rpy="0 0 0" xyz="0 0 0"/>
-                <geometry>
-                    <sphere radius="0.01"/>
-                </geometry>
-            </visual>
-            <inertial>
-                <mass value="0.1"/>
-                <inertia ixx="5e-05" iyy="5e-05" izz="5e-05" ixy="0.0" ixz="0.0" iyz="0.0"/>
-            </inertial>
-            <collision>
-                <geometry>
-                    <sphere radius="0.01"/>
-                </geometry>
-            </collision>
-        </link>
-        <gazebo reference="tether_0/fragment_4">
-            <material>Gazebo/Red</material>
-        </gazebo>
-                    <!--tether fragment joint-->
-        <joint name="tether_0/joint_4" type="continuous">
-            <origin rpy="0 0 0" xyz="0 0 1.0"/>
-            <parent link="tether_0/fragment_3"/>
-            <child link="tether_0/fragment_4"/>
-                <axis xyz="0 1 0" />
-            <dynamics damping="0.1" friction="0.1"/>
-        </joint>
-            <link name="tether_0/fragment_5">
-            <visual>
-                <origin rpy="0 0 0" xyz="0 0 0"/>
-                <geometry>
-                    <sphere radius="0.01"/>
-                </geometry>
-            </visual>
-            <inertial>
-                <mass value="0.1"/>
-                <inertia ixx="5e-05" iyy="5e-05" izz="5e-05" ixy="0.0" ixz="0.0" iyz="0.0"/>
-            </inertial>
-            <collision>
-                <geometry>
-                    <sphere radius="0.01"/>
-                </geometry>
-            </collision>
-        </link>
-        <gazebo reference="tether_0/fragment_5">
-            <material>Gazebo/Red</material>
-        </gazebo>
-                    <!--tether fragment joint-->
-        <joint name="tether_0/joint_5" type="continuous">
-            <origin rpy="0 0 0" xyz="0 0 1.0"/>
-            <parent link="tether_0/fragment_4"/>
-            <child link="tether_0/fragment_5"/>
-                <axis xyz="0 1 0" />
-            <dynamics damping="0.1" friction="0.1"/>
-        </joint>
-            <link name="tether_0/fragment_6">
-            <visual>
-                <origin rpy="0 0 0" xyz="0 0 0"/>
-                <geometry>
-                    <sphere radius="0.01"/>
-                </geometry>
-            </visual>
-            <inertial>
-                <mass value="0.1"/>
-                <inertia ixx="5e-05" iyy="5e-05" izz="5e-05" ixy="0.0" ixz="0.0" iyz="0.0"/>
-            </inertial>
-            <collision>
-                <geometry>
-                    <sphere radius="0.01"/>
-                </geometry>
-            </collision>
-        </link>
-        <gazebo reference="tether_0/fragment_6">
-            <material>Gazebo/Red</material>
-        </gazebo>
-                    <!--tether fragment joint-->
-        <joint name="tether_0/joint_6" type="continuous">
-            <origin rpy="0 0 0" xyz="0 0 1.0"/>
-            <parent link="tether_0/fragment_5"/>
-            <child link="tether_0/fragment_6"/>
-                <axis xyz="0 1 0" />
-            <dynamics damping="0.1" friction="0.1"/>
-        </joint>
-            <link name="tether_0/fragment_7">
-            <visual>
-                <origin rpy="0 0 0" xyz="0 0 0"/>
-                <geometry>
-                    <sphere radius="0.01"/>
-                </geometry>
-            </visual>
-            <inertial>
-                <mass value="0.1"/>
-                <inertia ixx="5e-05" iyy="5e-05" izz="5e-05" ixy="0.0" ixz="0.0" iyz="0.0"/>
-            </inertial>
-            <collision>
-                <geometry>
-                    <sphere radius="0.01"/>
-                </geometry>
-            </collision>
-        </link>
-        <gazebo reference="tether_0/fragment_7">
-            <material>Gazebo/Red</material>
-        </gazebo>
-                    <!--tether fragment joint-->
-        <joint name="tether_0/joint_7" type="continuous">
-            <origin rpy="0 0 0" xyz="0 0 1.0"/>
-            <parent link="tether_0/fragment_6"/>
-            <child link="tether_0/fragment_7"/>
-                <axis xyz="0 1 0" />
-            <dynamics damping="0.1" friction="0.1"/>
-        </joint>
-            <link name="tether_0/fragment_8">
-            <visual>
-                <origin rpy="0 0 0" xyz="0 0 0"/>
-                <geometry>
-                    <sphere radius="0.01"/>
-                </geometry>
-            </visual>
-            <inertial>
-                <mass value="0.1"/>
-                <inertia ixx="5e-05" iyy="5e-05" izz="5e-05" ixy="0.0" ixz="0.0" iyz="0.0"/>
-            </inertial>
-            <collision>
-                <geometry>
-                    <sphere radius="0.01"/>
-                </geometry>
-            </collision>
-        </link>
-        <gazebo reference="tether_0/fragment_8">
-            <material>Gazebo/Red</material>
-        </gazebo>
-                    <!--tether fragment joint-->
-        <joint name="tether_0/joint_8" type="continuous">
-            <origin rpy="0 0 0" xyz="0 0 1.0"/>
-            <parent link="tether_0/fragment_7"/>
-            <child link="tether_0/fragment_8"/>
-                <axis xyz="0 1 0" />
-            <dynamics damping="0.1" friction="0.1"/>
-        </joint>
-            <link name="tether_0/fragment_9">
-            <visual>
-                <origin rpy="0 0 0" xyz="0 0 0"/>
-                <geometry>
-                    <sphere radius="0.01"/>
-                </geometry>
-            </visual>
-            <inertial>
-                <mass value="0.1"/>
-                <inertia ixx="5e-05" iyy="5e-05" izz="5e-05" ixy="0.0" ixz="0.0" iyz="0.0"/>
-            </inertial>
-            <collision>
-                <geometry>
-                    <sphere radius="0.01"/>
-                </geometry>
-            </collision>
-        </link>
-        <gazebo reference="tether_0/fragment_9">
-            <material>Gazebo/Red</material>
-        </gazebo>
-                    <!--tether fragment joint-->
-        <joint name="tether_0/joint_9" type="continuous">
-            <origin rpy="0 0 0" xyz="0 0 1.0"/>
-            <parent link="tether_0/fragment_8"/>
-            <child link="tether_0/fragment_9"/>
                 <axis xyz="0 1 0" />
             <dynamics damping="0.1" friction="0.1"/>
@@ -309,6 +141,6 @@
             <!--tether end joint-->
         <joint name="tether_0/ugv_joint_1" type="continuous">
-                <origin rpy="0 ${-pi/2} 0" xyz="0 0 1.0"/>
-            <parent link="tether_0/fragment_9"/>
+                <origin rpy="0 ${-pi/2} 0" xyz="0 0 5.0"/>
+            <parent link="tether_0/fragment_3"/>
             <child link="mp_500_0/tether_end"/>
             <axis xyz="1 0 0" />
@@ -319,14 +151,14 @@
                 <origin rpy="0 0 0" xyz="0 0 0"/>
                 <geometry>
-                    <sphere radius="0.01"/>
-                </geometry>
-            </visual>
-            <inertial>
-                <mass value="0.1"/>
-                <inertia ixx="5e-05" iyy="5e-05" izz="5e-05" ixy="0.0" ixz="0.0" iyz="0.0"/>
-            </inertial>
-            <collision>
-                <geometry>
-                    <sphere radius="0.01"/>
+                    <sphere radius="0.03"/>
+                </geometry>
+            </visual>
+            <inertial>
+                <mass value="0.05"/>
+                <inertia ixx="0.000135" iyy="0.000135" izz="0.000135" ixy="0.0" ixz="0.0" iyz="0.0"/>
+            </inertial>
+            <collision>
+                <geometry>
+                    <sphere radius="0.03"/>
                 </geometry>
             </collision>
@@ -339,14 +171,14 @@
                 <origin rpy="0 0 0" xyz="0 0 0"/>
                 <geometry>
-                    <sphere radius="0.01"/>
-                </geometry>
-            </visual>
-            <inertial>
-                <mass value="0.1"/>
-                <inertia ixx="5e-05" iyy="5e-05" izz="5e-05" ixy="0.0" ixz="0.0" iyz="0.0"/>
-            </inertial>
-            <collision>
-                <geometry>
-                    <sphere radius="0.01"/>
+                    <sphere radius="0.03"/>
+                </geometry>
+            </visual>
+            <inertial>
+                <mass value="0.05"/>
+                <inertia ixx="0.000135" iyy="0.000135" izz="0.000135" ixy="0.0" ixz="0.0" iyz="0.0"/>
+            </inertial>
+            <collision>
+                <geometry>
+                    <sphere radius="0.03"/>
                 </geometry>
             </collision>
@@ -357,5 +189,5 @@
                     <!--tether fragment joint-->
         <joint name="tether_1/joint_1" type="continuous">
-            <origin rpy="0 0 0" xyz="0 0 1.0"/>
+            <origin rpy="0 0 0" xyz="0 0 5.0"/>
             <parent link="tether_1/fragment_0"/>
             <child link="tether_1/fragment_1"/>
@@ -367,14 +199,14 @@
                 <origin rpy="0 0 0" xyz="0 0 0"/>
                 <geometry>
-                    <sphere radius="0.01"/>
-                </geometry>
-            </visual>
-            <inertial>
-                <mass value="0.1"/>
-                <inertia ixx="5e-05" iyy="5e-05" izz="5e-05" ixy="0.0" ixz="0.0" iyz="0.0"/>
-            </inertial>
-            <collision>
-                <geometry>
-                    <sphere radius="0.01"/>
+                    <sphere radius="0.03"/>
+                </geometry>
+            </visual>
+            <inertial>
+                <mass value="0.05"/>
+                <inertia ixx="0.000135" iyy="0.000135" izz="0.000135" ixy="0.0" ixz="0.0" iyz="0.0"/>
+            </inertial>
+            <collision>
+                <geometry>
+                    <sphere radius="0.03"/>
                 </geometry>
             </collision>
@@ -385,5 +217,5 @@
                     <!--tether fragment joint-->
         <joint name="tether_1/joint_2" type="continuous">
-            <origin rpy="0 0 0" xyz="0 0 1.0"/>
+            <origin rpy="0 0 0" xyz="0 0 5.0"/>
             <parent link="tether_1/fragment_1"/>
             <child link="tether_1/fragment_2"/>
@@ -395,14 +227,14 @@
                 <origin rpy="0 0 0" xyz="0 0 0"/>
                 <geometry>
-                    <sphere radius="0.01"/>
-                </geometry>
-            </visual>
-            <inertial>
-                <mass value="0.1"/>
-                <inertia ixx="5e-05" iyy="5e-05" izz="5e-05" ixy="0.0" ixz="0.0" iyz="0.0"/>
-            </inertial>
-            <collision>
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
File: ugv_description/urdf/mp_500/xacros/mp_500_tether_end.xacro (robot description, xacro)
@@ -9,5 +9,5 @@
             <parent link="${name}" />
             <child link="${namespace}/base_link" />
-            <origin xyz="0.0 0.0 -0.2" rpy="0 0 0" />
+            <origin xyz="0.0 0.0 -0.03" rpy="0 0 0" />
             <axis xyz="0 0 1" />
         </joint>
@@ -15,5 +15,5 @@
             <visual>
                 <geometry>
-                    <cylinder length="0.2" radius="0.02"/>
+                    <cylinder length="0.05" radius="0.02"/>
                 </geometry>
             </visual>
@@ -24,5 +24,5 @@
             <collision>
                 <geometry>
-                    <cylinder length="0.2" radius="0.02"/>
+                    <cylinder length="0.05" radius="0.02"/>
                 </geometry>
             </collision>
