Commit message: Update tether model 4DoF to 6DoF

File: tether_description/urdf/lumped_mass_tether_fragment.xacro (robot description, xacro)
@@ -4,16 +4,16 @@
     <xacro:macro name="tether">
         <!--tether fragment param-->
-        {%- set lump_mass = 0.05 -%}
+        {%- set lump_mass = 0.01 -%}
         {%- set lump_radius = 0.03 -%}
         {%- set lump_inertia = 3*lump_mass*lump_radius**2 -%}
         {%- set element_length = 5.0 -%}
         <!--joint dynamics-->
-        {%- set damping = 0.1 -%}
-        {%- set friction = 0.1 -%}
+        {%- set damping = 1 -%}
+        {%- set friction = 1 -%}
         <!--link number-->
-        {%- set tether_fragments = 4 -%}
+        {%- set tether_fragments = 5 -%}
         {%- set tether_number = 4 -%}
         {%- macro tether_fragment(dirc, n) -%}
-        <link name="tether_{{dirc}}/fragment_{{n}}">
+        <link name="tether_{{dirc}}/fragment_{{n}}_1">
             <visual>
                 <origin rpy="0 0 0" xyz="0 0 0"/>
@@ -26,11 +26,36 @@
                 <inertia ixx="{{lump_inertia}}" iyy="{{lump_inertia}}" izz="{{lump_inertia}}" ixy="0.0" ixz="0.0" iyz="0.0"/>
             </inertial>
-            <collision>
+        </link>
+        <gazebo reference="tether_{{dirc}}/fragment_{{n}}_1">
+            <material>Gazebo/Red</material>
+        </gazebo>
+        <link name="tether_{{dirc}}/fragment_{{n}}_2">
+            <visual>
+                <origin rpy="0 0 0" xyz="0 0 0"/>
                 <geometry>
                     <sphere radius="{{lump_radius}}"/>
                 </geometry>
-            </collision>
+            </visual>
+            <inertial>
+                <mass value="{{lump_mass}}"/>
+                <inertia ixx="{{lump_inertia}}" iyy="{{lump_inertia}}" izz="{{lump_inertia}}" ixy="0.0" ixz="0.0" iyz="0.0"/>
+            </inertial>
         </link>
-        <gazebo reference="tether_{{dirc}}/fragment_{{n}}">
+        <gazebo reference="tether_{{dirc}}/fragment_{{n}}_2">
+            <material>Gazebo/Red</material>
+        </gazebo>
+        <link name="tether_{{dirc}}/fragment_{{n}}_3">
+            <visual>
+                <origin rpy="0 0 0" xyz="0 0 0"/>
+                <geometry>
+                    <sphere radius="{{lump_radius}}"/>
+                </geometry>
+            </visual>
+            <inertial>
+                <mass value="{{lump_mass}}"/>
+                <inertia ixx="{{lump_inertia}}" iyy="{{lump_inertia}}" izz="{{lump_inertia}}" ixy="0.0" ixz="0.0" iyz="0.0"/>
+            </inertial>
+        </link>
+        <gazebo reference="tether_{{dirc}}/fragment_{{n}}_3">
             <material>Gazebo/Red</material>
         </gazebo>
@@ -39,17 +64,23 @@
         {%- macro tether_joint(dirc, n) -%}
         <!--tether fragment joint-->
-        <joint name="tether_{{dirc}}/joint_{{n}}" type="continuous">
+        <joint name="tether_{{dirc}}/joint_roll_{{n}}" type="continuous">
             <origin rpy="0 0 0" xyz="0 0 {{element_length}}"/>
-            <parent link="tether_{{dirc}}/fragment_{{n-1}}"/>
-            <child link="tether_{{dirc}}/fragment_{{n}}"/>
-            {% if dirc == 0 %}
-                <axis xyz="0 1 0" />
-            {% elif dirc == 1 %}
-                <axis xyz="1 0 0" />
-            {% elif dirc == 2 %}
-                <axis xyz="0 1 0" />
-            {% elif dirc == 3 %}
-                <axis xyz="1 0 0" />
-            {% endif %}
+            <parent link="tether_{{dirc}}/fragment_{{n-1}}_3"/>
+            <child link="tether_{{dirc}}/fragment_{{n}}_1"/>
+            <axis xyz="1 0 0" />
+            <dynamics damping="{{damping}}" friction="{{friction}}"/>
+        </joint>
+        <joint name="tether_{{dirc}}/joint_pitch_{{n}}" type="continuous">
+            <origin rpy="0 0 0" xyz="0 0 0"/>
+            <parent link="tether_{{dirc}}/fragment_{{n}}_1"/>
+            <child link="tether_{{dirc}}/fragment_{{n}}_2"/>
+            <axis xyz="0 1 0" />
+            <dynamics damping="{{damping}}" friction="{{friction}}"/>
+        </joint>
+        <joint name="tether_{{dirc}}/joint_yaw_{{n}}" type="continuous">
+            <origin rpy="0 0 0" xyz="0 0 0"/>
+            <parent link="tether_{{dirc}}/fragment_{{n}}_2"/>
+            <child link="tether_{{dirc}}/fragment_{{n}}_3"/>
+            <axis xyz="0 0 1" />
             <dynamics damping="{{damping}}" friction="{{friction}}"/>
         </joint>
@@ -90,16 +121,24 @@
             {% endif %}
         </joint>
-        <joint name="tether_{{dirc}}/uav_joint" type="continuous">
+        <joint name="tether_{{dirc}}/uav_roll_joint" type="continuous">
+            <origin rpy="0 0 0" xyz="0 0 0.2"/>
             <parent link="tether_{{dirc}}/rod"/>
-            <child link="tether_{{dirc}}/fragment_0"/>
-            {% if dirc == 0 %}
-                <axis xyz="0 1 0" />
-            {% elif dirc == 1 %}
-                <axis xyz="1 0 0" />
-            {% elif dirc == 2 %}
-                <axis xyz="0 1 0" />
-            {% elif dirc == 3 %}
-                <axis xyz="1 0 0" />
-            {% endif %}
+            <child link="tether_{{dirc}}/fragment_0_1"/>
+            <axis xyz="1 0 0" />
+            <dynamics damping="{{damping}}" friction="{{friction}}"/>
+        </joint>
+        <joint name="tether_{{dirc}}/uav_pitch_joint" type="continuous">
+            <origin rpy="0 0 0" xyz="0 0 0"/>
+            <parent link="tether_{{dirc}}/fragment_0_1"/>
+            <child link="tether_{{dirc}}/fragment_0_2"/>
+            <axis xyz="0 1 0" />
+            <dynamics damping="{{damping}}" friction="{{friction}}"/>
+        </joint>
+        <joint name="tether_{{dirc}}/joint_yaw_joint" type="continuous">
+            <origin rpy="0 0 0" xyz="0 0 0"/>
+            <parent link="tether_{{dirc}}/fragment_0_2"/>
+            <child link="tether_{{dirc}}/fragment_0_3"/>
+            <axis xyz="0 0 1" />
+            <dynamics damping="{{damping}}" friction="{{friction}}"/>
         </joint>
         {%- endmacro -%}
@@ -116,5 +155,5 @@
                 <origin rpy="${pi/2} 0 0" xyz="0 0 {{element_length}}"/>
             {% endif %}
-            <parent link="tether_{{dirc}}/fragment_{{tether_fragments-1}}"/>
+            <parent link="tether_{{dirc}}/fragment_{{tether_fragments-1}}_3"/>
             <child link="mp_500_{{dirc}}/tether_end"/>
             <axis xyz="1 0 0" />

File: tether_description/urdf/tether.xacro (robot description, xacro)
@@ -4,107 +4,316 @@
     <xacro:macro name="tether">
         <!--tether fragment param--><!--joint dynamics--><!--link number--><!--tether_cylinder_joint--><!-- main-->
-            <link name="tether_0/fragment_0">
-            <visual>
-                <origin rpy="0 0 0" xyz="0 0 0"/>
-                <geometry>
-                    <sphere radius="0.03"/>
-                </geometry>
-            </visual>
-            <inertial>
-                <mass value="0.05"/>
-                <inertia ixx="0.000135" iyy="0.000135" izz="0.000135" ixy="0.0" ixz="0.0" iyz="0.0"/>
-            </inertial>
-            <collision>
-                <geometry>
-                    <sphere radius="0.03"/>
-                </geometry>
-            </collision>
-        </link>
-        <gazebo reference="tether_0/fragment_0">
-            <material>Gazebo/Red</material>
-        </gazebo>
-            <link name="tether_0/fragment_1">
-            <visual>
-                <origin rpy="0 0 0" xyz="0 0 0"/>
-                <geometry>
-                    <sphere radius="0.03"/>
-                </geometry>
-            </visual>
-            <inertial>
-                <mass value="0.05"/>
-                <inertia ixx="0.000135" iyy="0.000135" izz="0.000135" ixy="0.0" ixz="0.0" iyz="0.0"/>
-            </inertial>
-            <collision>
-                <geometry>
-                    <sphere radius="0.03"/>
-                </geometry>
-            </collision>
-        </link>
-        <gazebo reference="tether_0/fragment_1">
-            <material>Gazebo/Red</material>
-        </gazebo>
-                    <!--tether fragment joint-->
-        <joint name="tether_0/joint_1" type="continuous">
-            <origin rpy="0 0 0" xyz="0 0 5.0"/>
-            <parent link="tether_0/fragment_0"/>
-            <child link="tether_0/fragment_1"/>
-                <axis xyz="0 1 0" />
-            <dynamics damping="0.1" friction="0.1"/>
-        </joint>
-            <link name="tether_0/fragment_2">
-            <visual>
-                <origin rpy="0 0 0" xyz="0 0 0"/>
-                <geometry>
-                    <sphere radius="0.03"/>
-                </geometry>
-            </visual>
-            <inertial>
-                <mass value="0.05"/>
-                <inertia ixx="0.000135" iyy="0.000135" izz="0.000135" ixy="0.0" ixz="0.0" iyz="0.0"/>
-            </inertial>
-            <collision>
-                <geometry>
-                    <sphere radius="0.03"/>
-                </geometry>
-            </collision>
-        </link>
-        <gazebo reference="tether_0/fragment_2">
-            <material>Gazebo/Red</material>
-        </gazebo>
-                    <!--tether fragment joint-->
-        <joint name="tether_0/joint_2" type="continuous">
-            <origin rpy="0 0 0" xyz="0 0 5.0"/>
-            <parent link="tether_0/fragment_1"/>
-            <child link="tether_0/fragment_2"/>
-                <axis xyz="0 1 0" />
-            <dynamics damping="0.1" friction="0.1"/>
-        </joint>
-            <link name="tether_0/fragment_3">
-            <visual>
-                <origin rpy="0 0 0" xyz="0 0 0"/>
-                <geometry>
-                    <sphere radius="0.03"/>
-                </geometry>
-            </visual>
-            <inertial>
-                <mass value="0.05"/>
-                <inertia ixx="0.000135" iyy="0.000135" izz="0.000135" ixy="0.0" ixz="0.0" iyz="0.0"/>
-            </inertial>
-            <collision>
-                <geometry>
-                    <sphere radius="0.03"/>
-                </geometry>
-            </collision>
-        </link>
-        <gazebo reference="tether_0/fragment_3">
-            <material>Gazebo/Red</material>
-        </gazebo>
-                    <!--tether fragment joint-->
-        <joint name="tether_0/joint_3" type="continuous">
-            <origin rpy="0 0 0" xyz="0 0 5.0"/>
-            <parent link="tether_0/fragment_2"/>
-            <child link="tether_0/fragment_3"/>
-                <axis xyz="0 1 0" />
-            <dynamics damping="0.1" friction="0.1"/>
+            <link name="tether_0/fragment_0_1">
+            <visual>
+                <origin rpy="0 0 0" xyz="0 0 0"/>
+                <geometry>
+                    <sphere radius="0.03"/>
+                </geometry>
+            </visual>
+            <inertial>
+                <mass value="0.01"/>
+                <inertia ixx="2.7e-05" iyy="2.7e-05" izz="2.7e-05" ixy="0.0" ixz="0.0" iyz="0.0"/>
+            </inertial>
+        </link>
+        <gazebo reference="tether_0/fragment_0_1">
+            <material>Gazebo/Red</material>
+        </gazebo>
+        <link name="tether_0/fragment_0_2">
+            <visual>
+                <origin rpy="0 0 0" xyz="0 0 0"/>
+                <geometry>
+                    <sphere radius="0.03"/>
+                </geometry>
+            </visual>
+            <inertial>
+                <mass value="0.01"/>
+                <inertia ixx="2.7e-05" iyy="2.7e-05" izz="2.7e-05" ixy="0.0" ixz="0.0" iyz="0.0"/>
+            </inertial>
+        </link>
+        <gazebo reference="tether_0/fragment_0_2">
+            <material>Gazebo/Red</material>
+        </gazebo>
+        <link name="tether_0/fragment_0_3">
+            <visual>
+                <origin rpy="0 0 0" xyz="0 0 0"/>
+                <geometry>
+                    <sphere radius="0.03"/>
+                </geometry>
+            </visual>
+            <inertial>
+                <mass value="0.01"/>
+                <inertia ixx="2.7e-05" iyy="2.7e-05" izz="2.7e-05" ixy="0.0" ixz="0.0" iyz="0.0"/>
+            </inertial>
+        </link>
+        <gazebo reference="tether_0/fragment_0_3">
+            <material>Gazebo/Red</material>
+        </gazebo>
+            <link name="tether_0/fragment_1_1">
+            <visual>
+                <origin rpy="0 0 0" xyz="0 0 0"/>
+                <geometry>
+                    <sphere radius="0.03"/>
+                </geometry>
+            </visual>
+            <inertial>
+                <mass value="0.01"/>
+                <inertia ixx="2.7e-05" iyy="2.7e-05" izz="2.7e-05" ixy="0.0" ixz="0.0" iyz="0.0"/>
+            </inertial>
+        </link>
+        <gazebo reference="tether_0/fragment_1_1">
+            <material>Gazebo/Red</material>
+        </gazebo>
+        <link name="tether_0/fragment_1_2">
+            <visual>
+                <origin rpy="0 0 0" xyz="0 0 0"/>
+                <geometry>
+                    <sphere radius="0.03"/>
+                </geometry>
+            </visual>
+            <inertial>
+                <mass value="0.01"/>
+                <inertia ixx="2.7e-05" iyy="2.7e-05" izz="2.7e-05" ixy="0.0" ixz="0.0" iyz="0.0"/>
+            </inertial>
+        </link>
+        <gazebo reference="tether_0/fragment_1_2">
+            <material>Gazebo/Red</material>
+        </gazebo>
+        <link name="tether_0/fragment_1_3">
+            <visual>
+                <origin rpy="0 0 0" xyz="0 0 0"/>
+                <geometry>
+                    <sphere radius="0.03"/>
+                </geometry>
+            </visual>
+            <inertial>
+                <mass value="0.01"/>
+                <inertia ixx="2.7e-05" iyy="2.7e-05" izz="2.7e-05" ixy="0.0" ixz="0.0" iyz="0.0"/>
+            </inertial>
+        </link>
+        <gazebo reference="tether_0/fragment_1_3">
+            <material>Gazebo/Red</material>
+        </gazebo>
+                    <!--tether fragment joint-->
+        <joint name="tether_0/joint_roll_1" type="continuous">
+            <origin rpy="0 0 0" xyz="0 0 5.0"/>
+            <parent link="tether_0/fragment_0_3"/>
+            <child link="tether_0/fragment_1_1"/>
+            <axis xyz="1 0 0" />
+            <dynamics damping="1" friction="1"/>
+        </joint>
+        <joint name="tether_0/joint_pitch_1" type="continuous">
+            <origin rpy="0 0 0" xyz="0 0 0"/>
+            <parent link="tether_0/fragment_1_1"/>
+            <child link="tether_0/fragment_1_2"/>
+            <axis xyz="0 1 0" />
+            <dynamics damping="1" friction="1"/>
+        </joint>
+        <joint name="tether_0/joint_yaw_1" type="continuous">
+            <origin rpy="0 0 0" xyz="0 0 0"/>
+            <parent link="tether_0/fragment_1_2"/>
+            <child link="tether_0/fragment_1_3"/>
+            <axis xyz="0 0 1" />
+            <dynamics damping="1" friction="1"/>
+        </joint>
+            <link name="tether_0/fragment_2_1">
+            <visual>
+                <origin rpy="0 0 0" xyz="0 0 0"/>
+                <geometry>
+                    <sphere radius="0.03"/>
+                </geometry>
+            </visual>
+            <inertial>
+                <mass value="0.01"/>
+                <inertia ixx="2.7e-05" iyy="2.7e-05" izz="2.7e-05" ixy="0.0" ixz="0.0" iyz="0.0"/>
+            </inertial>
+        </link>
+        <gazebo reference="tether_0/fragment_2_1">
+            <material>Gazebo/Red</material>
+        </gazebo>
+        <link name="tether_0/fragment_2_2">
+            <visual>
+                <origin rpy="0 0 0" xyz="0 0 0"/>
+                <geometry>
+                    <sphere radius="0.03"/>
+                </geometry>
+            </visual>
+            <inertial>
+                <mass value="0.01"/>
+                <inertia ixx="2.7e-05" iyy="2.7e-05" izz="2.7e-05" ixy="0.0" ixz="0.0" iyz="0.0"/>
+            </inertial>
+        </link>
+        <gazebo reference="tether_0/fragment_2_2">
+            <material>Gazebo/Red</material>
+        </gazebo>
+        <link name="tether_0/fragment_2_3">
+            <visual>
+                <origin rpy="0 0 0" xyz="0 0 0"/>
+                <geometry>
+                    <sphere radius="0.03"/>
+                </geometry>
+            </visual>
+            <inertial>
+                <mass value="0.01"/>
+                <inertia ixx="2.7e-05" iyy="2.7e-05" izz="2.7e-05" ixy="0.0" ixz="0.0" iyz="0.0"/>
+            </inertial>
+        </link>
+        <gazebo reference="tether_0/fragment_2_3">
+            <material>Gazebo/Red</material>
+        </gazebo>
+                    <!--tether fragment joint-->
+        <joint name="tether_0/joint_roll_2" type="continuous">
+            <origin rpy="0 0 0" xyz="0 0 5.0"/>
+            <parent link="tether_0/fragment_1_3"/>
+            <child link="tether_0/fragment_2_1"/>
+            <axis xyz="1 0 0" />
+            <dynamics damping="1" friction="1"/>
+        </joint>
+        <joint name="tether_0/joint_pitch_2" type="continuous">
+            <origin rpy="0 0 0" xyz="0 0 0"/>
+            <parent link="tether_0/fragment_2_1"/>
+            <child link="tether_0/fragment_2_2"/>
+            <axis xyz="0 1 0" />
+            <dynamics damping="1" friction="1"/>
+        </joint>
+        <joint name="tether_0/joint_yaw_2" type="continuous">
+            <origin rpy="0 0 0" xyz="0 0 0"/>
+            <parent link="tether_0/fragment_2_2"/>
+            <child link="tether_0/fragment_2_3"/>
+            <axis xyz="0 0 1" />
+            <dynamics damping="1" friction="1"/>
+        </joint>
+            <link name="tether_0/fragment_3_1">
+            <visual>
+                <origin rpy="0 0 0" xyz="0 0 0"/>
+                <geometry>
+                    <sphere radius="0.03"/>
+                </geometry>
+            </visual>
+            <inertial>
+                <mass value="0.01"/>
+                <inertia ixx="2.7e-05" iyy="2.7e-05" izz="2.7e-05" ixy="0.0" ixz="0.0" iyz="0.0"/>
+            </inertial>
+        </link>
+        <gazebo reference="tether_0/fragment_3_1">
+            <material>Gazebo/Red</material>
+        </gazebo>
+        <link name="tether_0/fragment_3_2">
+            <visual>
+                <origin rpy="0 0 0" xyz="0 0 0"/>
+                <geometry>
+                    <sphere radius="0.03"/>
+                </geometry>
+            </visual>
+            <inertial>
+                <mass value="0.01"/>
+                <inertia ixx="2.7e-05" iyy="2.7e-05" izz="2.7e-05" ixy="0.0" ixz="0.0" iyz="0.0"/>
+            </inertial>
+        </link>
+        <gazebo reference="tether_0/fragment_3_2">
+            <material>Gazebo/Red</material>
+        </gazebo>
+        <link name="tether_0/fragment_3_3">
+            <visual>
+                <origin rpy="0 0 0" xyz="0 0 0"/>
+                <geometry>
+                    <sphere radius="0.03"/>
+                </geometry>
+            </visual>
+            <inertial>
+                <mass value="0.01"/>
+                <inertia ixx="2.7e-05" iyy="2.7e-05" izz="2.7e-05" ixy="0.0" ixz="0.0" iyz="0.0"/>
+            </inertial>
+        </link>
+        <gazebo reference="tether_0/fragment_3_3">
+            <material>Gazebo/Red</material>
+        </gazebo>
+                    <!--tether fragment joint-->
+        <joint name="tether_0/joint_roll_3" type="continuous">
+            <origin rpy="0 0 0" xyz="0 0 5.0"/>
+            <parent link="tether_0/fragment_2_3"/>
+            <child link="tether_0/fragment_3_1"/>
+            <axis xyz="1 0 0" />
+            <dynamics damping="1" friction="1"/>
+        </joint>
+        <joint name="tether_0/joint_pitch_3" type="continuous">
+            <origin rpy="0 0 0" xyz="0 0 0"/>
+            <parent link="tether_0/fragment_3_1"/>
+            <child link="tether_0/fragment_3_2"/>
+            <axis xyz="0 1 0" />
+            <dynamics damping="1" friction="1"/>
+        </joint>
+        <joint name="tether_0/joint_yaw_3" type="continuous">
+            <origin rpy="0 0 0" xyz="0 0 0"/>
+            <parent link="tether_0/fragment_3_2"/>
+            <child link="tether_0/fragment_3_3"/>
+            <axis xyz="0 0 1" />
+            <dynamics damping="1" friction="1"/>
+        </joint>
+            <link name="tether_0/fragment_4_1">
+            <visual>
+                <origin rpy="0 0 0" xyz="0 0 0"/>
+                <geometry>
+                    <sphere radius="0.03"/>
+                </geometry>
+            </visual>
+            <inertial>
+                <mass value="0.01"/>
+                <inertia ixx="2.7e-05" iyy="2.7e-05" izz="2.7e-05" ixy="0.0" ixz="0.0" iyz="0.0"/>
+            </inertial>
+        </link>
+        <gazebo reference="tether_0/fragment_4_1">
+            <material>Gazebo/Red</material>
+        </gazebo>
+        <link name="tether_0/fragment_4_2">
+            <visual>
+                <origin rpy="0 0 0" xyz="0 0 0"/>
+                <geometry>
+                    <sphere radius="0.03"/>
+                </geometry>
+            </visual>
+            <inertial>
+                <mass value="0.01"/>
+                <inertia ixx="2.7e-05" iyy="2.7e-05" izz="2.7e-05" ixy="0.0" ixz="0.0" iyz="0.0"/>
+            </inertial>
+        </link>
+        <gazebo reference="tether_0/fragment_4_2">
+            <material>Gazebo/Red</material>
+        </gazebo>
+        <link name="tether_0/fragment_4_3">
+            <visual>
+                <origin rpy="0 0 0" xyz="0 0 0"/>
+                <geometry>
+                    <sphere radius="0.03"/>
+                </geometry>
+            </visual>
+            <inertial>
+                <mass value="0.01"/>
+                <inertia ixx="2.7e-05" iyy="2.7e-05" izz="2.7e-05" ixy="0.0" ixz="0.0" iyz="0.0"/>
+            </inertial>
+        </link>
+        <gazebo reference="tether_0/fragment_4_3">
+            <material>Gazebo/Red</material>
+        </gazebo>
+                    <!--tether fragment joint-->
+        <joint name="tether_0/joint_roll_4" type="continuous">
+            <origin rpy="0 0 0" xyz="0 0 5.0"/>
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