Commit message: Update params

File: tether_description/urdf/lumped_mass_tether_fragment.xacro (robot description, xacro)
@@ -4,13 +4,13 @@
     <xacro:macro name="tether">
         <!--tether fragment param-->
-        {%- set lump_mass = 0.01 -%}
+        {%- set lump_mass = 0.05 -%}
         {%- set lump_radius = 0.03 -%}
         {%- set lump_inertia = 3*lump_mass*lump_radius**2 -%}
-        {%- set element_length = 5.0 -%}
+        {%- set element_length = 10.0 -%}
         <!--joint dynamics-->
         {%- set damping = 1 -%}
         {%- set friction = 1 -%}
         <!--link number-->
-        {%- set tether_fragments = 5 -%}
+        {%- set tether_fragments = 2 -%}
         {%- set tether_number = 4 -%}
         {%- macro tether_fragment(dirc, n) -%}
@@ -148,14 +148,17 @@
             {% if dirc == 0 %}
                 <origin rpy="0 ${-pi/2} 0" xyz="0 0 {{element_length}}"/>
+                <axis xyz="0 1 0" />
             {% elif dirc == 1 %}
                 <origin rpy="${-pi/2} 0 0" xyz="0 0 {{element_length}}"/>
+                <axis xyz="1 0 0" />
             {% elif dirc == 2 %}
                 <origin rpy="0 ${pi/2} 0" xyz="0 0 {{element_length}}"/>
+                <axis xyz="0 1 0" />
             {% elif dirc == 3 %}
                 <origin rpy="${pi/2} 0 0" xyz="0 0 {{element_length}}"/>
+                <axis xyz="1 0 0" />
             {% endif %}
             <parent link="tether_{{dirc}}/fragment_{{tether_fragments-1}}_3"/>
             <child link="mp_500_{{dirc}}/tether_end"/>
-            <axis xyz="1 0 0" />
             <dynamics damping="{{damping}}" friction="{{friction}}"/>
         </joint>

File: tether_description/urdf/tether.xacro (robot description, xacro)
@@ -12,6 +12,6 @@
             </visual>
             <inertial>
-                <mass value="0.01"/>
-                <inertia ixx="2.7e-05" iyy="2.7e-05" izz="2.7e-05" ixy="0.0" ixz="0.0" iyz="0.0"/>
+                <mass value="0.05"/>
+                <inertia ixx="0.000135" iyy="0.000135" izz="0.000135" ixy="0.0" ixz="0.0" iyz="0.0"/>
             </inertial>
         </link>
@@ -27,6 +27,6 @@
             </visual>
             <inertial>
-                <mass value="0.01"/>
-                <inertia ixx="2.7e-05" iyy="2.7e-05" izz="2.7e-05" ixy="0.0" ixz="0.0" iyz="0.0"/>
+                <mass value="0.05"/>
+                <inertia ixx="0.000135" iyy="0.000135" izz="0.000135" ixy="0.0" ixz="0.0" iyz="0.0"/>
             </inertial>
         </link>
@@ -42,6 +42,6 @@
             </visual>
             <inertial>
-                <mass value="0.01"/>
-                <inertia ixx="2.7e-05" iyy="2.7e-05" izz="2.7e-05" ixy="0.0" ixz="0.0" iyz="0.0"/>
+                <mass value="0.05"/>
+                <inertia ixx="0.000135" iyy="0.000135" izz="0.000135" ixy="0.0" ixz="0.0" iyz="0.0"/>
             </inertial>
         </link>
@@ -57,6 +57,6 @@
             </visual>
             <inertial>
-                <mass value="0.01"/>
-                <inertia ixx="2.7e-05" iyy="2.7e-05" izz="2.7e-05" ixy="0.0" ixz="0.0" iyz="0.0"/>
+                <mass value="0.05"/>
+                <inertia ixx="0.000135" iyy="0.000135" izz="0.000135" ixy="0.0" ixz="0.0" iyz="0.0"/>
             </inertial>
         </link>
@@ -72,6 +72,6 @@
             </visual>
             <inertial>
-                <mass value="0.01"/>
-                <inertia ixx="2.7e-05" iyy="2.7e-05" izz="2.7e-05" ixy="0.0" ixz="0.0" iyz="0.0"/>
+                <mass value="0.05"/>
+                <inertia ixx="0.000135" iyy="0.000135" izz="0.000135" ixy="0.0" ixz="0.0" iyz="0.0"/>
             </inertial>
         </link>
@@ -87,6 +87,6 @@
             </visual>
             <inertial>
-                <mass value="0.01"/>
-                <inertia ixx="2.7e-05" iyy="2.7e-05" izz="2.7e-05" ixy="0.0" ixz="0.0" iyz="0.0"/>
+                <mass value="0.05"/>
+                <inertia ixx="0.000135" iyy="0.000135" izz="0.000135" ixy="0.0" ixz="0.0" iyz="0.0"/>
             </inertial>
         </link>
@@ -96,5 +96,5 @@
                     <!--tether fragment joint-->
         <joint name="tether_0/joint_roll_1" type="continuous">
-            <origin rpy="0 0 0" xyz="0 0 5.0"/>
+            <origin rpy="0 0 0" xyz="0 0 10.0"/>
             <parent link="tether_0/fragment_0_3"/>
             <child link="tether_0/fragment_1_1"/>
@@ -113,205 +113,4 @@
             <parent link="tether_0/fragment_1_2"/>
             <child link="tether_0/fragment_1_3"/>
-            <axis xyz="0 0 1" />
-            <dynamics damping="1" friction="1"/>
-        </joint>
-            <link name="tether_0/fragment_2_1">
-            <visual>
-                <origin rpy="0 0 0" xyz="0 0 0"/>
-                <geometry>
-                    <sphere radius="0.03"/>
-                </geometry>
-            </visual>
-            <inertial>
-                <mass value="0.01"/>
-                <inertia ixx="2.7e-05" iyy="2.7e-05" izz="2.7e-05" ixy="0.0" ixz="0.0" iyz="0.0"/>
-            </inertial>
-        </link>
-        <gazebo reference="tether_0/fragment_2_1">
-            <material>Gazebo/Red</material>
-        </gazebo>
-        <link name="tether_0/fragment_2_2">
-            <visual>
-                <origin rpy="0 0 0" xyz="0 0 0"/>
-                <geometry>
-                    <sphere radius="0.03"/>
-                </geometry>
-            </visual>
-            <inertial>
-                <mass value="0.01"/>
-                <inertia ixx="2.7e-05" iyy="2.7e-05" izz="2.7e-05" ixy="0.0" ixz="0.0" iyz="0.0"/>
-            </inertial>
-        </link>
-        <gazebo reference="tether_0/fragment_2_2">
-            <material>Gazebo/Red</material>
-        </gazebo>
-        <link name="tether_0/fragment_2_3">
-            <visual>
-                <origin rpy="0 0 0" xyz="0 0 0"/>
-                <geometry>
-                    <sphere radius="0.03"/>
-                </geometry>
-            </visual>
-            <inertial>
-                <mass value="0.01"/>
-                <inertia ixx="2.7e-05" iyy="2.7e-05" izz="2.7e-05" ixy="0.0" ixz="0.0" iyz="0.0"/>
-            </inertial>
-        </link>
-        <gazebo reference="tether_0/fragment_2_3">
-            <material>Gazebo/Red</material>
-        </gazebo>
-                    <!--tether fragment joint-->
-        <joint name="tether_0/joint_roll_2" type="continuous">
-            <origin rpy="0 0 0" xyz="0 0 5.0"/>
-            <parent link="tether_0/fragment_1_3"/>
-            <child link="tether_0/fragment_2_1"/>
-            <axis xyz="1 0 0" />
-            <dynamics damping="1" friction="1"/>
-        </joint>
-        <joint name="tether_0/joint_pitch_2" type="continuous">
-            <origin rpy="0 0 0" xyz="0 0 0"/>
-            <parent link="tether_0/fragment_2_1"/>
-            <child link="tether_0/fragment_2_2"/>
-            <axis xyz="0 1 0" />
-            <dynamics damping="1" friction="1"/>
-        </joint>
-        <joint name="tether_0/joint_yaw_2" type="continuous">
-            <origin rpy="0 0 0" xyz="0 0 0"/>
-            <parent link="tether_0/fragment_2_2"/>
-            <child link="tether_0/fragment_2_3"/>
-            <axis xyz="0 0 1" />
-            <dynamics damping="1" friction="1"/>
-        </joint>
-            <link name="tether_0/fragment_3_1">
-            <visual>
-                <origin rpy="0 0 0" xyz="0 0 0"/>
-                <geometry>
-                    <sphere radius="0.03"/>
-                </geometry>
-            </visual>
-            <inertial>
-                <mass value="0.01"/>
-                <inertia ixx="2.7e-05" iyy="2.7e-05" izz="2.7e-05" ixy="0.0" ixz="0.0" iyz="0.0"/>
-            </inertial>
-        </link>
-        <gazebo reference="tether_0/fragment_3_1">
-            <material>Gazebo/Red</material>
-        </gazebo>
-        <link name="tether_0/fragment_3_2">
-            <visual>
-                <origin rpy="0 0 0" xyz="0 0 0"/>
-                <geometry>
-                    <sphere radius="0.03"/>
-                </geometry>
-            </visual>
-            <inertial>
-                <mass value="0.01"/>
-                <inertia ixx="2.7e-05" iyy="2.7e-05" izz="2.7e-05" ixy="0.0" ixz="0.0" iyz="0.0"/>
-            </inertial>
-        </link>
-        <gazebo reference="tether_0/fragment_3_2">
-            <material>Gazebo/Red</material>
-        </gazebo>
-        <link name="tether_0/fragment_3_3">
-            <visual>
-                <origin rpy="0 0 0" xyz="0 0 0"/>
-                <geometry>
-                    <sphere radius="0.03"/>
-                </geometry>
-            </visual>
-            <inertial>
-                <mass value="0.01"/>
-                <inertia ixx="2.7e-05" iyy="2.7e-05" izz="2.7e-05" ixy="0.0" ixz="0.0" iyz="0.0"/>
-            </inertial>
-        </link>
-        <gazebo reference="tether_0/fragment_3_3">
-            <material>Gazebo/Red</material>
-        </gazebo>
-                    <!--tether fragment joint-->
-        <joint name="tether_0/joint_roll_3" type="continuous">
-            <origin rpy="0 0 0" xyz="0 0 5.0"/>
-            <parent link="tether_0/fragment_2_3"/>
-            <child link="tether_0/fragment_3_1"/>
-            <axis xyz="1 0 0" />
-            <dynamics damping="1" friction="1"/>
-        </joint>
-        <joint name="tether_0/joint_pitch_3" type="continuous">
-            <origin rpy="0 0 0" xyz="0 0 0"/>
-            <parent link="tether_0/fragment_3_1"/>
-            <child link="tether_0/fragment_3_2"/>
-            <axis xyz="0 1 0" />
-            <dynamics damping="1" friction="1"/>
-        </joint>
-        <joint name="tether_0/joint_yaw_3" type="continuous">
-            <origin rpy="0 0 0" xyz="0 0 0"/>
-            <parent link="tether_0/fragment_3_2"/>
-            <child link="tether_0/fragment_3_3"/>
-            <axis xyz="0 0 1" />
-            <dynamics damping="1" friction="1"/>
-        </joint>
-            <link name="tether_0/fragment_4_1">
-            <visual>
-                <origin rpy="0 0 0" xyz="0 0 0"/>
-                <geometry>
-                    <sphere radius="0.03"/>
-                </geometry>
-            </visual>
-            <inertial>
-                <mass value="0.01"/>
-                <inertia ixx="2.7e-05" iyy="2.7e-05" izz="2.7e-05" ixy="0.0" ixz="0.0" iyz="0.0"/>
-            </inertial>
-        </link>
-        <gazebo reference="tether_0/fragment_4_1">
-            <material>Gazebo/Red</material>
-        </gazebo>
-        <link name="tether_0/fragment_4_2">
-            <visual>
-                <origin rpy="0 0 0" xyz="0 0 0"/>
-                <geometry>
-                    <sphere radius="0.03"/>
-                </geometry>
-            </visual>
-            <inertial>
-                <mass value="0.01"/>
-                <inertia ixx="2.7e-05" iyy="2.7e-05" izz="2.7e-05" ixy="0.0" ixz="0.0" iyz="0.0"/>
-            </inertial>
-        </link>
-        <gazebo reference="tether_0/fragment_4_2">
-            <material>Gazebo/Red</material>
-        </gazebo>
-        <link name="tether_0/fragment_4_3">
-            <visual>
-                <origin rpy="0 0 0" xyz="0 0 0"/>
-                <geometry>
-                    <sphere radius="0.03"/>
-                </geometry>
-            </visual>
-            <inertial>
-                <mass value="0.01"/>
-                <inertia ixx="2.7e-05" iyy="2.7e-05" izz="2.7e-05" ixy="0.0" ixz="0.0" iyz="0.0"/>
-            </inertial>
-        </link>
-        <gazebo reference="tether_0/fragment_4_3">
-            <material>Gazebo/Red</material>
-        </gazebo>
-                    <!--tether fragment joint-->
-        <joint name="tether_0/joint_roll_4" type="continuous">
-            <origin rpy="0 0 0" xyz="0 0 5.0"/>
-            <parent link="tether_0/fragment_3_3"/>
-            <child link="tether_0/fragment_4_1"/>
-            <axis xyz="1 0 0" />
-            <dynamics damping="1" friction="1"/>
-        </joint>
-        <joint name="tether_0/joint_pitch_4" type="continuous">
-            <origin rpy="0 0 0" xyz="0 0 0"/>
-            <parent link="tether_0/fragment_4_1"/>
-            <child link="tether_0/fragment_4_2"/>
-            <axis xyz="0 1 0" />
-            <dynamics damping="1" friction="1"/>
-        </joint>
-        <joint name="tether_0/joint_yaw_4" type="continuous">
-            <origin rpy="0 0 0" xyz="0 0 0"/>
-            <parent link="tether_0/fragment_4_2"/>
-            <child link="tether_0/fragment_4_3"/>
             <axis xyz="0 0 1" />
             <dynamics damping="1" friction="1"/>
@@ -366,8 +165,8 @@
             <!--tether end joint-->
         <joint name="tether_0/ugv_joint_1" type="continuous">
-                <origin rpy="0 ${-pi/2} 0" xyz="0 0 5.0"/>
-            <parent link="tether_0/fragment_4_3"/>
+                <origin rpy="0 ${-pi/2} 0" xyz="0 0 10.0"/>
+                <axis xyz="0 1 0" />
+            <parent link="tether_0/fragment_1_3"/>
             <child link="mp_500_0/tether_end"/>
-            <axis xyz="1 0 0" />
             <dynamics damping="1" friction="1"/>
         </joint>
@@ -380,6 +179,6 @@
             </visual>
             <inertial>
-                <mass value="0.01"/>
-                <inertia ixx="2.7e-05" iyy="2.7e-05" izz="2.7e-05" ixy="0.0" ixz="0.0" iyz="0.0"/>
+                <mass value="0.05"/>
+                <inertia ixx="0.000135" iyy="0.000135" izz="0.000135" ixy="0.0" ixz="0.0" iyz="0.0"/>
             </inertial>
         </link>
@@ -395,6 +194,6 @@
             </visual>
             <inertial>
-                <mass value="0.01"/>
-                <inertia ixx="2.7e-05" iyy="2.7e-05" izz="2.7e-05" ixy="0.0" ixz="0.0" iyz="0.0"/>
+                <mass value="0.05"/>
+                <inertia ixx="0.000135" iyy="0.000135" izz="0.000135" ixy="0.0" ixz="0.0" iyz="0.0"/>
             </inertial>
         </link>
@@ -410,6 +209,6 @@
             </visual>
             <inertial>
-                <mass value="0.01"/>
-                <inertia ixx="2.7e-05" iyy="2.7e-05" izz="2.7e-05" ixy="0.0" ixz="0.0" iyz="0.0"/>
+                <mass value="0.05"/>
+                <inertia ixx="0.000135" iyy="0.000135" izz="0.000135" ixy="0.0" ixz="0.0" iyz="0.0"/>
             </inertial>
         </link>
@@ -425,6 +224,6 @@
             </visual>
             <inertial>
-                <mass value="0.01"/>
-                <inertia ixx="2.7e-05" iyy="2.7e-05" izz="2.7e-05" ixy="0.0" ixz="0.0" iyz="0.0"/>
+                <mass value="0.05"/>
+                <inertia ixx="0.000135" iyy="0.000135" izz="0.000135" ixy="0.0" ixz="0.0" iyz="0.0"/>
             </inertial>
         </link>
@@ -440,6 +239,6 @@
             </visual>
             <inertial>
-                <mass value="0.01"/>
-                <inertia ixx="2.7e-05" iyy="2.7e-05" izz="2.7e-05" ixy="0.0" ixz="0.0" iyz="0.0"/>
+                <mass value="0.05"/>
+                <inertia ixx="0.000135" iyy="0.000135" izz="0.000135" ixy="0.0" ixz="0.0" iyz="0.0"/>
             </inertial>
         </link>
@@ -455,6 +254,6 @@
             </visual>
             <inertial>
-                <mass value="0.01"/>
-                <inertia ixx="2.7e-05" iyy="2.7e-05" izz="2.7e-05" ixy="0.0" ixz="0.0" iyz="0.0"/>
+                <mass value="0.05"/>
+                <inertia ixx="0.000135" iyy="0.000135" izz="0.000135" ixy="0.0" ixz="0.0" iyz="0.0"/>
             </inertial>
         </link>
@@ -464,5 +263,5 @@
                     <!--tether fragment joint-->
         <joint name="tether_1/joint_roll_1" type="continuous">
-            <origin rpy="0 0 0" xyz="0 0 5.0"/>
+            <origin rpy="0 0 0" xyz="0 0 10.0"/>
             <parent link="tether_1/fragment_0_3"/>
             <child link="tether_1/fragment_1_1"/>
@@ -481,205 +280,4 @@
             <parent link="tether_1/fragment_1_2"/>
             <child link="tether_1/fragment_1_3"/>
-            <axis xyz="0 0 1" />
-            <dynamics damping="1" friction="1"/>
-        </joint>
-            <link name="tether_1/fragment_2_1">
-            <visual>
-                <origin rpy="0 0 0" xyz="0 0 0"/>
-                <geometry>
-                    <sphere radius="0.03"/>
-                </geometry>
-            </visual>
-            <inertial>
-                <mass value="0.01"/>
-                <inertia ixx="2.7e-05" iyy="2.7e-05" izz="2.7e-05" ixy="0.0" ixz="0.0" iyz="0.0"/>
-            </inertial>
-        </link>
-        <gazebo reference="tether_1/fragment_2_1">
-            <material>Gazebo/Red</material>
-        </gazebo>
-        <link name="tether_1/fragment_2_2">
-            <visual>
-                <origin rpy="0 0 0" xyz="0 0 0"/>
-                <geometry>
-                    <sphere radius="0.03"/>
-                </geometry>
-            </visual>
-            <inertial>
-                <mass value="0.01"/>
-                <inertia ixx="2.7e-05" iyy="2.7e-05" izz="2.7e-05" ixy="0.0" ixz="0.0" iyz="0.0"/>
-            </inertial>
-        </link>
-        <gazebo reference="tether_1/fragment_2_2">
-            <material>Gazebo/Red</material>
-        </gazebo>
-        <link name="tether_1/fragment_2_3">
-            <visual>
-                <origin rpy="0 0 0" xyz="0 0 0"/>
-                <geometry>
-                    <sphere radius="0.03"/>
-                </geometry>
-            </visual>
-            <inertial>
-                <mass value="0.01"/>
-                <inertia ixx="2.7e-05" iyy="2.7e-05" izz="2.7e-05" ixy="0.0" ixz="0.0" iyz="0.0"/>
-            </inertial>
-        </link>
-        <gazebo reference="tether_1/fragment_2_3">
-            <material>Gazebo/Red</material>
-        </gazebo>
-                    <!--tether fragment joint-->
-        <joint name="tether_1/joint_roll_2" type="continuous">
-            <origin rpy="0 0 0" xyz="0 0 5.0"/>
-            <parent link="tether_1/fragment_1_3"/>
-            <child link="tether_1/fragment_2_1"/>
-            <axis xyz="1 0 0" />
-            <dynamics damping="1" friction="1"/>
-        </joint>
-        <joint name="tether_1/joint_pitch_2" type="continuous">
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