Commit message: Update params

File: tether_description/urdf/lumped_mass_tether_fragment.xacro (robot description, xacro)
@@ -4,14 +4,65 @@
     <xacro:macro name="tether">
         <!--tether fragment param-->
+        {%- set uav_link_mass = 0.005 -%}
+        {%- set uav_link_radius = 0.02 -%}
+        {%- set uav_link_inertia = 3*uav_link_mass*uav_link_radius**2 -%}
+        <!--tether fragment param-->
         {%- set lump_mass = 0.05 -%}
-        {%- set lump_radius = 0.03 -%}
-        {%- set lump_inertia = 3*lump_mass*lump_radius**2 -%}
-        {%- set element_length = 10.0 -%}
+        {%- set lump_radius = 0.02 -%}
+        {%- set lump_inertia = lump_mass*lump_radius**2 -%}
+        {%- set element_length = 1.0 -%}
         <!--joint dynamics-->
         {%- set damping = 1 -%}
         {%- set friction = 1 -%}
         <!--link number-->
-        {%- set tether_fragments = 2 -%}
+        {%- set tether_fragments = 4 -%}
         {%- set tether_number = 4 -%}
+        {%- macro uav_link(dirc, n) -%}
+        <link name="tether_{{dirc}}/fragment_{{n}}_1">
+            <visual>
+                <origin rpy="0 0 0" xyz="0 0 0"/>
+                <geometry>
+                    <sphere radius="{{uav_link_radius}}"/>
+                </geometry>
+            </visual>
+            <inertial>
+                <mass value="{{uav_link_mass}}"/>
+                <inertia ixx="{{uav_link_inertia}}" iyy="{{uav_link_inertia}}" izz="{{uav_link_inertia}}" ixy="0.0" ixz="0.0" iyz="0.0"/>
+            </inertial>
+        </link>
+        <gazebo reference="tether_{{dirc}}/fragment_{{n}}_1">
+            <material>Gazebo/Black</material>
+        </gazebo>
+        <link name="tether_{{dirc}}/fragment_{{n}}_2">
+            <visual>
+                <origin rpy="0 0 0" xyz="0 0 0"/>
+                <geometry>
+                    <sphere radius="{{uav_link_radius}}"/>
+                </geometry>
+            </visual>
+            <inertial>
+                <mass value="{{uav_link_mass}}"/>
+                <inertia ixx="{{uav_link_inertia}}" iyy="{{uav_link_inertia}}" izz="{{uav_link_inertia}}" ixy="0.0" ixz="0.0" iyz="0.0"/>
+            </inertial>
+        </link>
+        <gazebo reference="tether_{{dirc}}/fragment_{{n}}_2">
+            <material>Gazebo/Black</material>
+        </gazebo>
+        <link name="tether_{{dirc}}/fragment_{{n}}_3">
+            <visual>
+                <origin rpy="0 0 0" xyz="0 0 0"/>
+                <geometry>
+                    <sphere radius="{{uav_link_radius}}"/>
+                </geometry>
+            </visual>
+            <inertial>
+                <mass value="{{uav_link_mass}}"/>
+                <inertia ixx="{{uav_link_inertia}}" iyy="{{uav_link_inertia}}" izz="{{uav_link_inertia}}" ixy="0.0" ixz="0.0" iyz="0.0"/>
+            </inertial>
+        </link>
+        <gazebo reference="tether_{{dirc}}/fragment_{{n}}_3">
+            <material>Gazebo/Black</material>
+        </gazebo>
+        {%- endmacro -%}
         {%- macro tether_fragment(dirc, n) -%}
         <link name="tether_{{dirc}}/fragment_{{n}}_1">
@@ -167,6 +218,8 @@
         {% for dirc in range(0,tether_number) %}
             {% for n in range(0,tether_fragments) -%}
-                {{tether_fragment(dirc, n)}}
-                {% if n != 0 %}
+                {% if n == 0 %}
+                    {{uav_link(dirc, n)}}
+                {% elif n != 0 %}
+                    {{tether_fragment(dirc, n)}}
                     {{tether_joint(dirc, n)}}
                 {% endif %}

File: tether_description/urdf/tether.xacro (robot description, xacro)
@@ -3,19 +3,19 @@
     <!--tether model-->
     <xacro:macro name="tether">
-        <!--tether fragment param--><!--joint dynamics--><!--link number--><!--tether_cylinder_joint--><!-- main-->
-            <link name="tether_0/fragment_0_1">
-            <visual>
-                <origin rpy="0 0 0" xyz="0 0 0"/>
-                <geometry>
-                    <sphere radius="0.03"/>
-                </geometry>
-            </visual>
-            <inertial>
-                <mass value="0.05"/>
-                <inertia ixx="0.000135" iyy="0.000135" izz="0.000135" ixy="0.0" ixz="0.0" iyz="0.0"/>
+        <!--tether fragment param--><!--tether fragment param--><!--joint dynamics--><!--link number--><!--tether_cylinder_joint--><!-- main-->
+                    <link name="tether_0/fragment_0_1">
+            <visual>
+                <origin rpy="0 0 0" xyz="0 0 0"/>
+                <geometry>
+                    <sphere radius="0.02"/>
+                </geometry>
+            </visual>
+            <inertial>
+                <mass value="0.005"/>
+                <inertia ixx="6e-06" iyy="6e-06" izz="6e-06" ixy="0.0" ixz="0.0" iyz="0.0"/>
             </inertial>
         </link>
         <gazebo reference="tether_0/fragment_0_1">
-            <material>Gazebo/Red</material>
+            <material>Gazebo/Black</material>
         </gazebo>
         <link name="tether_0/fragment_0_2">
@@ -23,14 +23,14 @@
                 <origin rpy="0 0 0" xyz="0 0 0"/>
                 <geometry>
-                    <sphere radius="0.03"/>
-                </geometry>
-            </visual>
-            <inertial>
-                <mass value="0.05"/>
-                <inertia ixx="0.000135" iyy="0.000135" izz="0.000135" ixy="0.0" ixz="0.0" iyz="0.0"/>
+                    <sphere radius="0.02"/>
+                </geometry>
+            </visual>
+            <inertial>
+                <mass value="0.005"/>
+                <inertia ixx="6e-06" iyy="6e-06" izz="6e-06" ixy="0.0" ixz="0.0" iyz="0.0"/>
             </inertial>
         </link>
         <gazebo reference="tether_0/fragment_0_2">
-            <material>Gazebo/Red</material>
+            <material>Gazebo/Black</material>
         </gazebo>
         <link name="tether_0/fragment_0_3">
@@ -38,25 +38,25 @@
                 <origin rpy="0 0 0" xyz="0 0 0"/>
                 <geometry>
-                    <sphere radius="0.03"/>
-                </geometry>
-            </visual>
-            <inertial>
-                <mass value="0.05"/>
-                <inertia ixx="0.000135" iyy="0.000135" izz="0.000135" ixy="0.0" ixz="0.0" iyz="0.0"/>
+                    <sphere radius="0.02"/>
+                </geometry>
+            </visual>
+            <inertial>
+                <mass value="0.005"/>
+                <inertia ixx="6e-06" iyy="6e-06" izz="6e-06" ixy="0.0" ixz="0.0" iyz="0.0"/>
             </inertial>
         </link>
         <gazebo reference="tether_0/fragment_0_3">
-            <material>Gazebo/Red</material>
-        </gazebo>
-            <link name="tether_0/fragment_1_1">
-            <visual>
-                <origin rpy="0 0 0" xyz="0 0 0"/>
-                <geometry>
-                    <sphere radius="0.03"/>
-                </geometry>
-            </visual>
-            <inertial>
-                <mass value="0.05"/>
-                <inertia ixx="0.000135" iyy="0.000135" izz="0.000135" ixy="0.0" ixz="0.0" iyz="0.0"/>
+            <material>Gazebo/Black</material>
+        </gazebo>
+                    <link name="tether_0/fragment_1_1">
+            <visual>
+                <origin rpy="0 0 0" xyz="0 0 0"/>
+                <geometry>
+                    <sphere radius="0.02"/>
+                </geometry>
+            </visual>
+            <inertial>
+                <mass value="0.05"/>
+                <inertia ixx="2e-05" iyy="2e-05" izz="2e-05" ixy="0.0" ixz="0.0" iyz="0.0"/>
             </inertial>
         </link>
@@ -68,10 +68,10 @@
                 <origin rpy="0 0 0" xyz="0 0 0"/>
                 <geometry>
-                    <sphere radius="0.03"/>
-                </geometry>
-            </visual>
-            <inertial>
-                <mass value="0.05"/>
-                <inertia ixx="0.000135" iyy="0.000135" izz="0.000135" ixy="0.0" ixz="0.0" iyz="0.0"/>
+                    <sphere radius="0.02"/>
+                </geometry>
+            </visual>
+            <inertial>
+                <mass value="0.05"/>
+                <inertia ixx="2e-05" iyy="2e-05" izz="2e-05" ixy="0.0" ixz="0.0" iyz="0.0"/>
             </inertial>
         </link>
@@ -83,10 +83,10 @@
                 <origin rpy="0 0 0" xyz="0 0 0"/>
                 <geometry>
-                    <sphere radius="0.03"/>
-                </geometry>
-            </visual>
-            <inertial>
-                <mass value="0.05"/>
-                <inertia ixx="0.000135" iyy="0.000135" izz="0.000135" ixy="0.0" ixz="0.0" iyz="0.0"/>
+                    <sphere radius="0.02"/>
+                </geometry>
+            </visual>
+            <inertial>
+                <mass value="0.05"/>
+                <inertia ixx="2e-05" iyy="2e-05" izz="2e-05" ixy="0.0" ixz="0.0" iyz="0.0"/>
             </inertial>
         </link>
@@ -96,5 +96,5 @@
                     <!--tether fragment joint-->
         <joint name="tether_0/joint_roll_1" type="continuous">
-            <origin rpy="0 0 0" xyz="0 0 10.0"/>
+            <origin rpy="0 0 0" xyz="0 0 1.0"/>
             <parent link="tether_0/fragment_0_3"/>
             <child link="tether_0/fragment_1_1"/>
@@ -113,4 +113,138 @@
             <parent link="tether_0/fragment_1_2"/>
             <child link="tether_0/fragment_1_3"/>
+            <axis xyz="0 0 1" />
+            <dynamics damping="1" friction="1"/>
+        </joint>
+                    <link name="tether_0/fragment_2_1">
+            <visual>
+                <origin rpy="0 0 0" xyz="0 0 0"/>
+                <geometry>
+                    <sphere radius="0.02"/>
+                </geometry>
+            </visual>
+            <inertial>
+                <mass value="0.05"/>
+                <inertia ixx="2e-05" iyy="2e-05" izz="2e-05" ixy="0.0" ixz="0.0" iyz="0.0"/>
+            </inertial>
+        </link>
+        <gazebo reference="tether_0/fragment_2_1">
+            <material>Gazebo/Red</material>
+        </gazebo>
+        <link name="tether_0/fragment_2_2">
+            <visual>
+                <origin rpy="0 0 0" xyz="0 0 0"/>
+                <geometry>
+                    <sphere radius="0.02"/>
+                </geometry>
+            </visual>
+            <inertial>
+                <mass value="0.05"/>
+                <inertia ixx="2e-05" iyy="2e-05" izz="2e-05" ixy="0.0" ixz="0.0" iyz="0.0"/>
+            </inertial>
+        </link>
+        <gazebo reference="tether_0/fragment_2_2">
+            <material>Gazebo/Red</material>
+        </gazebo>
+        <link name="tether_0/fragment_2_3">
+            <visual>
+                <origin rpy="0 0 0" xyz="0 0 0"/>
+                <geometry>
+                    <sphere radius="0.02"/>
+                </geometry>
+            </visual>
+            <inertial>
+                <mass value="0.05"/>
+                <inertia ixx="2e-05" iyy="2e-05" izz="2e-05" ixy="0.0" ixz="0.0" iyz="0.0"/>
+            </inertial>
+        </link>
+        <gazebo reference="tether_0/fragment_2_3">
+            <material>Gazebo/Red</material>
+        </gazebo>
+                    <!--tether fragment joint-->
+        <joint name="tether_0/joint_roll_2" type="continuous">
+            <origin rpy="0 0 0" xyz="0 0 1.0"/>
+            <parent link="tether_0/fragment_1_3"/>
+            <child link="tether_0/fragment_2_1"/>
+            <axis xyz="1 0 0" />
+            <dynamics damping="1" friction="1"/>
+        </joint>
+        <joint name="tether_0/joint_pitch_2" type="continuous">
+            <origin rpy="0 0 0" xyz="0 0 0"/>
+            <parent link="tether_0/fragment_2_1"/>
+            <child link="tether_0/fragment_2_2"/>
+            <axis xyz="0 1 0" />
+            <dynamics damping="1" friction="1"/>
+        </joint>
+        <joint name="tether_0/joint_yaw_2" type="continuous">
+            <origin rpy="0 0 0" xyz="0 0 0"/>
+            <parent link="tether_0/fragment_2_2"/>
+            <child link="tether_0/fragment_2_3"/>
+            <axis xyz="0 0 1" />
+            <dynamics damping="1" friction="1"/>
+        </joint>
+                    <link name="tether_0/fragment_3_1">
+            <visual>
+                <origin rpy="0 0 0" xyz="0 0 0"/>
+                <geometry>
+                    <sphere radius="0.02"/>
+                </geometry>
+            </visual>
+            <inertial>
+                <mass value="0.05"/>
+                <inertia ixx="2e-05" iyy="2e-05" izz="2e-05" ixy="0.0" ixz="0.0" iyz="0.0"/>
+            </inertial>
+        </link>
+        <gazebo reference="tether_0/fragment_3_1">
+            <material>Gazebo/Red</material>
+        </gazebo>
+        <link name="tether_0/fragment_3_2">
+            <visual>
+                <origin rpy="0 0 0" xyz="0 0 0"/>
+                <geometry>
+                    <sphere radius="0.02"/>
+                </geometry>
+            </visual>
+            <inertial>
+                <mass value="0.05"/>
+                <inertia ixx="2e-05" iyy="2e-05" izz="2e-05" ixy="0.0" ixz="0.0" iyz="0.0"/>
+            </inertial>
+        </link>
+        <gazebo reference="tether_0/fragment_3_2">
+            <material>Gazebo/Red</material>
+        </gazebo>
+        <link name="tether_0/fragment_3_3">
+            <visual>
+                <origin rpy="0 0 0" xyz="0 0 0"/>
+                <geometry>
+                    <sphere radius="0.02"/>
+                </geometry>
+            </visual>
+            <inertial>
+                <mass value="0.05"/>
+                <inertia ixx="2e-05" iyy="2e-05" izz="2e-05" ixy="0.0" ixz="0.0" iyz="0.0"/>
+            </inertial>
+        </link>
+        <gazebo reference="tether_0/fragment_3_3">
+            <material>Gazebo/Red</material>
+        </gazebo>
+                    <!--tether fragment joint-->
+        <joint name="tether_0/joint_roll_3" type="continuous">
+            <origin rpy="0 0 0" xyz="0 0 1.0"/>
+            <parent link="tether_0/fragment_2_3"/>
+            <child link="tether_0/fragment_3_1"/>
+            <axis xyz="1 0 0" />
+            <dynamics damping="1" friction="1"/>
+        </joint>
+        <joint name="tether_0/joint_pitch_3" type="continuous">
+            <origin rpy="0 0 0" xyz="0 0 0"/>
+            <parent link="tether_0/fragment_3_1"/>
+            <child link="tether_0/fragment_3_2"/>
+            <axis xyz="0 1 0" />
+            <dynamics damping="1" friction="1"/>
+        </joint>
+        <joint name="tether_0/joint_yaw_3" type="continuous">
+            <origin rpy="0 0 0" xyz="0 0 0"/>
+            <parent link="tether_0/fragment_3_2"/>
+            <child link="tether_0/fragment_3_3"/>
             <axis xyz="0 0 1" />
             <dynamics damping="1" friction="1"/>
@@ -165,24 +299,24 @@
             <!--tether end joint-->
         <joint name="tether_0/ugv_joint_1" type="continuous">
-                <origin rpy="0 ${-pi/2} 0" xyz="0 0 10.0"/>
+                <origin rpy="0 ${-pi/2} 0" xyz="0 0 1.0"/>
                 <axis xyz="0 1 0" />
-            <parent link="tether_0/fragment_1_3"/>
+            <parent link="tether_0/fragment_3_3"/>
             <child link="mp_500_0/tether_end"/>
             <dynamics damping="1" friction="1"/>
         </joint>
-            <link name="tether_1/fragment_0_1">
-            <visual>
-                <origin rpy="0 0 0" xyz="0 0 0"/>
-                <geometry>
-                    <sphere radius="0.03"/>
-                </geometry>
-            </visual>
-            <inertial>
-                <mass value="0.05"/>
-                <inertia ixx="0.000135" iyy="0.000135" izz="0.000135" ixy="0.0" ixz="0.0" iyz="0.0"/>
+                    <link name="tether_1/fragment_0_1">
+            <visual>
+                <origin rpy="0 0 0" xyz="0 0 0"/>
+                <geometry>
+                    <sphere radius="0.02"/>
+                </geometry>
+            </visual>
+            <inertial>
+                <mass value="0.005"/>
+                <inertia ixx="6e-06" iyy="6e-06" izz="6e-06" ixy="0.0" ixz="0.0" iyz="0.0"/>
             </inertial>
         </link>
         <gazebo reference="tether_1/fragment_0_1">
-            <material>Gazebo/Red</material>
+            <material>Gazebo/Black</material>
         </gazebo>
         <link name="tether_1/fragment_0_2">
@@ -190,14 +324,14 @@
                 <origin rpy="0 0 0" xyz="0 0 0"/>
                 <geometry>
-                    <sphere radius="0.03"/>
-                </geometry>
-            </visual>
-            <inertial>
-                <mass value="0.05"/>
-                <inertia ixx="0.000135" iyy="0.000135" izz="0.000135" ixy="0.0" ixz="0.0" iyz="0.0"/>
+                    <sphere radius="0.02"/>
+                </geometry>
+            </visual>
+            <inertial>
+                <mass value="0.005"/>
+                <inertia ixx="6e-06" iyy="6e-06" izz="6e-06" ixy="0.0" ixz="0.0" iyz="0.0"/>
             </inertial>
         </link>
         <gazebo reference="tether_1/fragment_0_2">
-            <material>Gazebo/Red</material>
+            <material>Gazebo/Black</material>
         </gazebo>
         <link name="tether_1/fragment_0_3">
@@ -205,25 +339,25 @@
                 <origin rpy="0 0 0" xyz="0 0 0"/>
                 <geometry>
-                    <sphere radius="0.03"/>
-                </geometry>
-            </visual>
-            <inertial>
-                <mass value="0.05"/>
-                <inertia ixx="0.000135" iyy="0.000135" izz="0.000135" ixy="0.0" ixz="0.0" iyz="0.0"/>
+                    <sphere radius="0.02"/>
+                </geometry>
+            </visual>
+            <inertial>
+                <mass value="0.005"/>
+                <inertia ixx="6e-06" iyy="6e-06" izz="6e-06" ixy="0.0" ixz="0.0" iyz="0.0"/>
             </inertial>
         </link>
         <gazebo reference="tether_1/fragment_0_3">
-            <material>Gazebo/Red</material>
-        </gazebo>
-            <link name="tether_1/fragment_1_1">
-            <visual>
-                <origin rpy="0 0 0" xyz="0 0 0"/>
-                <geometry>
-                    <sphere radius="0.03"/>
-                </geometry>
-            </visual>
-            <inertial>
-                <mass value="0.05"/>
-                <inertia ixx="0.000135" iyy="0.000135" izz="0.000135" ixy="0.0" ixz="0.0" iyz="0.0"/>
+            <material>Gazebo/Black</material>
+        </gazebo>
+                    <link name="tether_1/fragment_1_1">
+            <visual>
+                <origin rpy="0 0 0" xyz="0 0 0"/>
+                <geometry>
+                    <sphere radius="0.02"/>
+                </geometry>
+            </visual>
+            <inertial>
+                <mass value="0.05"/>
+                <inertia ixx="2e-05" iyy="2e-05" izz="2e-05" ixy="0.0" ixz="0.0" iyz="0.0"/>
             </inertial>
         </link>
@@ -235,10 +369,10 @@
                 <origin rpy="0 0 0" xyz="0 0 0"/>
                 <geometry>
-                    <sphere radius="0.03"/>
-                </geometry>
-            </visual>
-            <inertial>
-                <mass value="0.05"/>
-                <inertia ixx="0.000135" iyy="0.000135" izz="0.000135" ixy="0.0" ixz="0.0" iyz="0.0"/>
+                    <sphere radius="0.02"/>
+                </geometry>
+            </visual>
+            <inertial>
+                <mass value="0.05"/>
+                <inertia ixx="2e-05" iyy="2e-05" izz="2e-05" ixy="0.0" ixz="0.0" iyz="0.0"/>
             </inertial>
         </link>
@@ -250,10 +384,10 @@
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