Commit message: Added 4-rotor uav (pelican) urdf model

File: tether_description/urdf/lumped_mass_tether_fragment.xacro (robot description, xacro)
@@ -6,5 +6,5 @@
         {%- set uav_link_mass = 0.005 -%}
         {%- set uav_link_radius = 0.02 -%}
-        {%- set uav_link_inertia = 3*uav_link_mass*uav_link_radius**2 -%}
+        {%- set uav_link_inertia = 5*uav_link_mass*uav_link_radius**2 -%}
         <!--tether fragment param-->
         {%- set lump_mass = 0.05 -%}
@@ -142,5 +142,5 @@
                 <origin rpy="0 0 0" xyz="0 0 0.1"/>
                 <geometry>
-                    <cylinder length="0.2" radius="0.01"/>
+                    <cylinder length="0.21" radius="0.01"/>
                 </geometry>
             </visual>
@@ -149,9 +149,4 @@
                 <inertia ixx="0.01" iyy="0.01" izz="0.01" ixy="0.0" ixz="0.0" iyz="0.0"/>
             </inertial>
-            <collision>
-                <geometry>
-                    <cylinder length="0.2" radius="0.01"/>
-                </geometry>
-            </collision>
         </link>
         <gazebo reference="tether_{{dirc}}/rod">
@@ -173,5 +168,5 @@
         </joint>
         <joint name="tether_{{dirc}}/uav_roll_joint" type="continuous">
-            <origin rpy="0 0 0" xyz="0 0 0.2"/>
+            <origin rpy="0 0 0" xyz="0 0 0.21"/>
             <parent link="tether_{{dirc}}/rod"/>
             <child link="tether_{{dirc}}/fragment_0_1"/>

File: tether_description/urdf/tether.xacro (robot description, xacro)
@@ -13,5 +13,5 @@
             <inertial>
                 <mass value="0.005"/>
-                <inertia ixx="6e-06" iyy="6e-06" izz="6e-06" ixy="0.0" ixz="0.0" iyz="0.0"/>
+                <inertia ixx="1e-05" iyy="1e-05" izz="1e-05" ixy="0.0" ixz="0.0" iyz="0.0"/>
             </inertial>
         </link>
@@ -28,5 +28,5 @@
             <inertial>
                 <mass value="0.005"/>
-                <inertia ixx="6e-06" iyy="6e-06" izz="6e-06" ixy="0.0" ixz="0.0" iyz="0.0"/>
+                <inertia ixx="1e-05" iyy="1e-05" izz="1e-05" ixy="0.0" ixz="0.0" iyz="0.0"/>
             </inertial>
         </link>
@@ -43,5 +43,5 @@
             <inertial>
                 <mass value="0.005"/>
-                <inertia ixx="6e-06" iyy="6e-06" izz="6e-06" ixy="0.0" ixz="0.0" iyz="0.0"/>
+                <inertia ixx="1e-05" iyy="1e-05" izz="1e-05" ixy="0.0" ixz="0.0" iyz="0.0"/>
             </inertial>
         </link>
@@ -254,5 +254,5 @@
                 <origin rpy="0 0 0" xyz="0 0 0.1"/>
                 <geometry>
-                    <cylinder length="0.2" radius="0.01"/>
+                    <cylinder length="0.21" radius="0.01"/>
                 </geometry>
             </visual>
@@ -261,9 +261,4 @@
                 <inertia ixx="0.01" iyy="0.01" izz="0.01" ixy="0.0" ixz="0.0" iyz="0.0"/>
             </inertial>
-            <collision>
-                <geometry>
-                    <cylinder length="0.2" radius="0.01"/>
-                </geometry>
-            </collision>
         </link>
         <gazebo reference="tether_0/rod">
@@ -277,5 +272,5 @@
         </joint>
         <joint name="tether_0/uav_roll_joint" type="continuous">
-            <origin rpy="0 0 0" xyz="0 0 0.2"/>
+            <origin rpy="0 0 0" xyz="0 0 0.21"/>
             <parent link="tether_0/rod"/>
             <child link="tether_0/fragment_0_1"/>
@@ -314,5 +309,5 @@
             <inertial>
                 <mass value="0.005"/>
-                <inertia ixx="6e-06" iyy="6e-06" izz="6e-06" ixy="0.0" ixz="0.0" iyz="0.0"/>
+                <inertia ixx="1e-05" iyy="1e-05" izz="1e-05" ixy="0.0" ixz="0.0" iyz="0.0"/>
             </inertial>
         </link>
@@ -329,5 +324,5 @@
             <inertial>
                 <mass value="0.005"/>
-                <inertia ixx="6e-06" iyy="6e-06" izz="6e-06" ixy="0.0" ixz="0.0" iyz="0.0"/>
+                <inertia ixx="1e-05" iyy="1e-05" izz="1e-05" ixy="0.0" ixz="0.0" iyz="0.0"/>
             </inertial>
         </link>
@@ -344,5 +339,5 @@
             <inertial>
                 <mass value="0.005"/>
-                <inertia ixx="6e-06" iyy="6e-06" izz="6e-06" ixy="0.0" ixz="0.0" iyz="0.0"/>
+                <inertia ixx="1e-05" iyy="1e-05" izz="1e-05" ixy="0.0" ixz="0.0" iyz="0.0"/>
             </inertial>
         </link>
@@ -555,5 +550,5 @@
                 <origin rpy="0 0 0" xyz="0 0 0.1"/>
                 <geometry>
-                    <cylinder length="0.2" radius="0.01"/>
+                    <cylinder length="0.21" radius="0.01"/>
                 </geometry>
             </visual>
@@ -562,9 +557,4 @@
                 <inertia ixx="0.01" iyy="0.01" izz="0.01" ixy="0.0" ixz="0.0" iyz="0.0"/>
             </inertial>
-            <collision>
-                <geometry>
-                    <cylinder length="0.2" radius="0.01"/>
-                </geometry>
-            </collision>
         </link>
         <gazebo reference="tether_1/rod">
@@ -578,5 +568,5 @@
         </joint>
         <joint name="tether_1/uav_roll_joint" type="continuous">
-            <origin rpy="0 0 0" xyz="0 0 0.2"/>
+            <origin rpy="0 0 0" xyz="0 0 0.21"/>
             <parent link="tether_1/rod"/>
             <child link="tether_1/fragment_0_1"/>
@@ -615,5 +605,5 @@
             <inertial>
                 <mass value="0.005"/>
-                <inertia ixx="6e-06" iyy="6e-06" izz="6e-06" ixy="0.0" ixz="0.0" iyz="0.0"/>
+                <inertia ixx="1e-05" iyy="1e-05" izz="1e-05" ixy="0.0" ixz="0.0" iyz="0.0"/>
             </inertial>
         </link>
@@ -630,5 +620,5 @@
             <inertial>
                 <mass value="0.005"/>
-                <inertia ixx="6e-06" iyy="6e-06" izz="6e-06" ixy="0.0" ixz="0.0" iyz="0.0"/>
+                <inertia ixx="1e-05" iyy="1e-05" izz="1e-05" ixy="0.0" ixz="0.0" iyz="0.0"/>
             </inertial>
         </link>
@@ -645,5 +635,5 @@
             <inertial>
                 <mass value="0.005"/>
-                <inertia ixx="6e-06" iyy="6e-06" izz="6e-06" ixy="0.0" ixz="0.0" iyz="0.0"/>
+                <inertia ixx="1e-05" iyy="1e-05" izz="1e-05" ixy="0.0" ixz="0.0" iyz="0.0"/>
             </inertial>
         </link>
@@ -856,5 +846,5 @@
                 <origin rpy="0 0 0" xyz="0 0 0.1"/>
                 <geometry>
-                    <cylinder length="0.2" radius="0.01"/>
+                    <cylinder length="0.21" radius="0.01"/>
                 </geometry>
             </visual>
@@ -863,9 +853,4 @@
                 <inertia ixx="0.01" iyy="0.01" izz="0.01" ixy="0.0" ixz="0.0" iyz="0.0"/>
             </inertial>
-            <collision>
-                <geometry>
-                    <cylinder length="0.2" radius="0.01"/>
-                </geometry>
-            </collision>
         </link>
         <gazebo reference="tether_2/rod">
@@ -879,5 +864,5 @@
         </joint>
         <joint name="tether_2/uav_roll_joint" type="continuous">
-            <origin rpy="0 0 0" xyz="0 0 0.2"/>
+            <origin rpy="0 0 0" xyz="0 0 0.21"/>
             <parent link="tether_2/rod"/>
             <child link="tether_2/fragment_0_1"/>
@@ -916,5 +901,5 @@
             <inertial>
                 <mass value="0.005"/>
-                <inertia ixx="6e-06" iyy="6e-06" izz="6e-06" ixy="0.0" ixz="0.0" iyz="0.0"/>
+                <inertia ixx="1e-05" iyy="1e-05" izz="1e-05" ixy="0.0" ixz="0.0" iyz="0.0"/>
             </inertial>
         </link>
@@ -931,5 +916,5 @@
             <inertial>
                 <mass value="0.005"/>
-                <inertia ixx="6e-06" iyy="6e-06" izz="6e-06" ixy="0.0" ixz="0.0" iyz="0.0"/>
+                <inertia ixx="1e-05" iyy="1e-05" izz="1e-05" ixy="0.0" ixz="0.0" iyz="0.0"/>
             </inertial>
         </link>
@@ -946,5 +931,5 @@
             <inertial>
                 <mass value="0.005"/>
-                <inertia ixx="6e-06" iyy="6e-06" izz="6e-06" ixy="0.0" ixz="0.0" iyz="0.0"/>
+                <inertia ixx="1e-05" iyy="1e-05" izz="1e-05" ixy="0.0" ixz="0.0" iyz="0.0"/>
             </inertial>
         </link>
@@ -1157,5 +1142,5 @@
                 <origin rpy="0 0 0" xyz="0 0 0.1"/>
                 <geometry>
-                    <cylinder length="0.2" radius="0.01"/>
+                    <cylinder length="0.21" radius="0.01"/>
                 </geometry>
             </visual>
@@ -1164,9 +1149,4 @@
                 <inertia ixx="0.01" iyy="0.01" izz="0.01" ixy="0.0" ixz="0.0" iyz="0.0"/>
             </inertial>
-            <collision>
-                <geometry>
-                    <cylinder length="0.2" radius="0.01"/>
-                </geometry>
-            </collision>
         </link>
         <gazebo reference="tether_3/rod">
@@ -1180,5 +1160,5 @@
         </joint>
         <joint name="tether_3/uav_roll_joint" type="continuous">
-            <origin rpy="0 0 0" xyz="0 0 0.2"/>
+            <origin rpy="0 0 0" xyz="0 0 0.21"/>
             <parent link="tether_3/rod"/>
             <child link="tether_3/fragment_0_1"/>
