Commit message: fix launch bugs

File: uav_description/urdf/pyramid_firefly_base.xacro (robot description, xacro)
@@ -17,27 +17,29 @@
 -->
 <robot name="firefly" xmlns:xacro="http://ros.org/wiki/xacro">
-  <xacro:include filename="$(find uav_description)/urdf/pyramid_component_snippets.xacro" />
-  <!-- Instantiate firefly "mechanics" -->
-  <xacro:include filename="$(find uav_description)/urdf/pyramid_firefly.xacro" />
-  <!-- Instantiate a controller. -->
-  <xacro:controller_plugin_macro namespace="${namespace}" imu_sub_topic="imu" />
-  <!-- Instantiate a ROS message interface -->
-  <!-- <xacro:ros_interface_plugin_macro namespace="${namespace}" />-->
-  <xacro:if value="$(arg enable_mavlink_interface)">
-    <!-- Instantiate mavlink telemetry interface. -->
-    <xacro:default_mavlink_interface namespace="${namespace}" imu_sub_topic="imu" rotor_count="6" />
-  </xacro:if>
-  <!-- Mount an ADIS16448 IMU. -->
-  <xacro:default_imu namespace="${namespace}" parent_link="${namespace}/base_link" />
-  <xacro:if value="$(arg enable_ground_truth)">
-    <xacro:ground_truth_imu_and_odometry namespace="${namespace}" parent_link="${namespace}/base_link" />
-  </xacro:if>
-  <xacro:if value="$(arg enable_logging)">
-    <!-- Instantiate a logger -->
-    <xacro:bag_plugin_macro
-      namespace="${namespace}"
-      bag_file="$(arg log_file)"
-      rotor_velocity_slowdown_sim="${rotor_velocity_slowdown_sim}"
-      wait_to_record_bag="$(arg wait_to_record_bag)" />
-  </xacro:if>
+        <xacro:include filename="$(find uav_description)/urdf/pyramid_component_snippets.xacro" />
+        <!-- Instantiate firefly "mechanics" -->
+        <xacro:include filename="$(find uav_description)/urdf/pyramid_firefly.xacro" />
+    <xacro:macro name="firefly">
+        <!-- Instantiate a controller. -->
+        <xacro:controller_plugin_macro namespace="${namespace}" imu_sub_topic="imu" />
+        <!-- Instantiate a ROS message interface -->
+        <!-- <xacro:ros_interface_plugin_macro namespace="${namespace}" />-->
+        <xacro:if value="$(arg enable_mavlink_interface)">
+            <!-- Instantiate mavlink telemetry interface. -->
+            <xacro:default_mavlink_interface namespace="${namespace}" imu_sub_topic="imu" rotor_count="6" />
+        </xacro:if>
+        <!-- Mount an ADIS16448 IMU. -->
+        <xacro:default_imu namespace="${namespace}" parent_link="${namespace}/base_link" />
+        <xacro:if value="$(arg enable_ground_truth)">
+            <xacro:ground_truth_imu_and_odometry namespace="${namespace}" parent_link="${namespace}/base_link" />
+        </xacro:if>
+        <xacro:if value="$(arg enable_logging)">
+            <!-- Instantiate a logger -->
+            <xacro:bag_plugin_macro
+                namespace="${namespace}"
+                bag_file="$(arg log_file)"
+                rotor_velocity_slowdown_sim="${rotor_velocity_slowdown_sim}"
+                wait_to_record_bag="$(arg wait_to_record_bag)" />
+        </xacro:if>
+    </xacro:macro>
 </robot>
