Commit message: fix mp_500 xacros

File: ugv_description/urdf/mp_500/mp_500.urdf.xacro (robot description, xacro)
@@ -11,4 +11,5 @@
 <xacro:include filename="$(find neo_simulation)/robots/mp_500/xacros/mp_500_fixed_wheel_left.xacro" />
 <xacro:include filename="$(find neo_simulation)/robots/mp_500/xacros/mp_500_fixed_wheel_right.xacro" />
+<xacro:macro name="mp_500">
   <xacro:mp_500_base name="base_link">
   </xacro:mp_500_base>
@@ -29,3 +30,4 @@
     <origin xyz="0.244 0 0.141" rpy="3.14 0 0" />
   </xacro:sick_laser_v0>
+</xacro:macro>
 </robot>

File: ugv_description/urdf/mp_500/xacros/mp_500_body.xacro (robot description, xacro)
@@ -3,32 +3,32 @@
   <xacro:macro name="mp_500_base" params="name">
     <link name="${name}">
-  <inertial>
-        <mass value="5" />
-        <origin xyz="0 0 0" rpy="0 0 0"/>
-        <inertia ixx="1.71402" ixy="0.0" ixz="0.0"
-                 iyy="0.8856" iyz="0.0"
-                 izz="2.5725" />
-</inertial>
-  <visual name='body'>
-  <origin xyz="0.0 0.0 0" rpy="0 0 1.570796" />
-  <geometry>
-      <mesh filename="package://neo_simulation/robots/mp_500/meshes/MP-500-BODY.dae" scale="0.001 0.001 0.001"/>
-  </geometry>
-  </visual>
-  <collision name='body_collision'>
-  <origin xyz="0.0 0.0 0.0" rpy=" 0 0. 1.570796" />
-  <geometry>
-    <mesh filename="package://neo_simulation/robots/mp_500/meshes/MP-500-BODY.dae" scale="0.001 0.001 0.001"/>
-  </geometry>
-  </collision>
-  </link>
-<gazebo reference="${name}_link">
-    <kp>1000.0</kp>
-    <kd>10.0</kd>
-    <mu1>200</mu1>
-    <mu2>100</mu2>
-    <fdir1>0.5 0 0</fdir1>
-    <maxVel>10.0</maxVel>
-    <minDepth>0.0005</minDepth>
+        <inertial>
+            <mass value="5" />
+            <origin xyz="0 0 0" rpy="0 0 0"/>
+            <inertia ixx="1.71402" ixy="0.0" ixz="0.0"
+                iyy="0.8856" iyz="0.0"
+                izz="2.5725" />
+        </inertial>
+        <visual name='body'>
+            <origin xyz="0.0 0.0 0" rpy="0 0 1.570796" />
+            <geometry>
+                <mesh filename="package://neo_simulation/robots/mp_500/meshes/MP-500-BODY.dae" scale="0.001 0.001 0.001"/>
+            </geometry>
+        </visual>
+        <collision name='body_collision'>
+            <origin xyz="0.0 0.0 0.0" rpy=" 0 0. 1.570796" />
+            <geometry>
+                <mesh filename="package://neo_simulation/robots/mp_500/meshes/MP-500-BODY.dae" scale="0.001 0.001 0.001"/>
+            </geometry>
+        </collision>
+    </link>
+    <gazebo reference="${name}_link">
+        <kp>1000.0</kp>
+        <kd>10.0</kd>
+        <mu1>200</mu1>
+        <mu2>100</mu2>
+        <fdir1>0.5 0 0</fdir1>
+        <maxVel>10.0</maxVel>
+        <minDepth>0.0005</minDepth>
     </gazebo>
   </xacro:macro>

File: ugv_description/urdf/mp_500/xacros/mp_500_caster_wheel.xacro (robot description, xacro)
@@ -1,42 +1,42 @@
 <?xml version="1.0"?>
 <robot xmlns:xacro="http://www.ros.org/wiki/xacro" name="mp_500">
-  <xacro:macro name="caster_wheel" params="name parent *origin">
-   <joint name="${name}_joint" type="fixed">
-    <insert_block name="origin" />
-        <axis xyz="0 -1 0" />
-      <limit effort="1000.0" lower="-1e+16" upper="1e+16" velocity="3.5"/>
-      <parent link="${parent}" />
-      <child link="${name}_link" />
-      <joint_properties damping="1.0" friction="1.0" />
-   </joint>
-   <link name="${name}_link" type="wheel">
-    <inertial>
-        <mass value="1.82362"/>
-        <inertia ixx="0.00499743171" ixy="0.00000004464" ixz="-0.00000002245"
-                 iyy="0.00499741733" iyz="0.00000000164"
-izz="0.00839239692"/>
-</inertial>
-      <visual name='castor_wheel'>
-    <origin xyz="0 0 0" rpy="0 0 0" />
-        <geometry>
-            <mesh filename="package://neo_simulation/robots/mp_500/meshes/MP-500-WHEEL.dae" scale="0.001 0.001 0.001"/>
-        </geometry>
-      </visual>
-    <collision>
-      <origin xyz="0 0 0" rpy="0 0 0" />
-      <geometry>
-            <mesh filename="package://neo_simulation/robots/mp_500/meshes/MP-500-WHEEL.dae" scale="0.001 0.001 0.001"/>
-      </geometry>
-    </collision>
-</link>
-<gazebo reference="${name}_link">
-      <kp>8000.0</kp>
-      <kd>1460.0</kd>
-      <mu1>0.5</mu1>
-      <mu2>0.2</mu2>
-      <fdir1>1 0 0</fdir1>
-      <maxVel>3.0</maxVel>
-      <minDepth>0.00</minDepth>
-</gazebo>
-  </xacro:macro>
+    <xacro:macro name="caster_wheel" params="name parent *origin">
+        <joint name="${name}_joint" type="fixed">
+            <insert_block name="origin" />
+            <axis xyz="0 -1 0" />
+            <limit effort="1000.0" lower="-1e+16" upper="1e+16" velocity="3.5"/>
+            <parent link="${parent}" />
+            <child link="${name}_link" />
+            <joint_properties damping="1.0" friction="1.0" />
+        </joint>
+        <link name="${name}_link" type="wheel">
+            <inertial>
+                <mass value="1.82362"/>
+                <inertia ixx="0.00499743171" ixy="0.00000004464" ixz="-0.00000002245"
+                    iyy="0.00499741733" iyz="0.00000000164"
+                    izz="0.00839239692"/>
+            </inertial>
+            <visual name='castor_wheel'>
+                <origin xyz="0 0 0" rpy="0 0 0" />
+                <geometry>
+                    <mesh filename="package://neo_simulation/robots/mp_500/meshes/MP-500-WHEEL.dae" scale="0.001 0.001 0.001"/>
+                </geometry>
+            </visual>
+            <collision>
+                <origin xyz="0 0 0" rpy="0 0 0" />
+                <geometry>
+                    <mesh filename="package://neo_simulation/robots/mp_500/meshes/MP-500-WHEEL.dae" scale="0.001 0.001 0.001"/>
+                </geometry>
+            </collision>
+        </link>
+        <gazebo reference="${name}_link">
+            <kp>8000.0</kp>
+            <kd>1460.0</kd>
+            <mu1>0.5</mu1>
+            <mu2>0.2</mu2>
+            <fdir1>1 0 0</fdir1>
+            <maxVel>3.0</maxVel>
+            <minDepth>0.00</minDepth>
+        </gazebo>
+    </xacro:macro>
 </robot>

File: ugv_description/urdf/mp_500/xacros/mp_500_fixed_wheel_left.xacro (robot description, xacro)
@@ -3,49 +3,49 @@
   <xacro:macro name="fixed_wheel_left" params="name parent number *origin">
     <joint name="${name}_joint" type="revolute">
-    <insert_block name="origin" />
-    <limit effort="1000.0" lower="-1e+16" upper="1e+16" velocity="3.5"/>
-    <axis xyz="-1 0 0" />
-    <joint_properties damping="0" friction="0.0" />
-    <parent link="base_link" />
-    <child link="${name}_link" />
-   </joint>
-   <transmission name="tran_${number}">
-    <type>transmission_interface/SimpleTransmission</type>
-    <joint name="${name}_joint" type="revolute">
-      <hardwareInterface>hardware_interface/VelocityJointInterface</hardwareInterface>
+        <insert_block name="origin" />
+        <limit effort="1000.0" lower="-1e+16" upper="1e+16" velocity="3.5"/>
+        <axis xyz="-1 0 0" />
+        <joint_properties damping="0" friction="0.0" />
+        <parent link="base_link" />
+        <child link="${name}_link" />
+    </joint>
+    <transmission name="tran_${number}">
+        <type>transmission_interface/SimpleTransmission</type>
+        <joint name="${name}_joint" type="revolute">
+            <hardwareInterface>hardware_interface/VelocityJointInterface</hardwareInterface>
         </joint>
-      <actuator name="left_wheel_actuator">
-      <mechanicalReduction>7</mechanicalReduction>
+        <actuator name="left_wheel_actuator">
+            <mechanicalReduction>7</mechanicalReduction>
             <hardwareInterface>hardware_interface/VelocityJointInterface</hardwareInterface>
-      </actuator>
-  </transmission>
-   <link name="${name}_link" type="wheel">
-    <inertial>
-      <origin xyz="0 0 0" rpy="0 0 0"/>
-        <mass value="1.82362"/>
-        <inertia ixx="0.00399743171" ixy="0.00000004464" ixz="-0.00000002245"
-                 iyy="0.00399741733" iyz="-0.00000000164"
-                 izz="0.00739239692"/>
-</inertial>
-    <visual>
-    <origin xyz="0 0 0" rpy="0 0 3.14" />
-        <geometry>
-            <mesh filename="package://neo_simulation/robots/mp_500/meshes/MP-500-WHEEL-LEFT.dae" scale="0.001 0.001 0.001"/>
-        </geometry>
-      </visual>
-    <collision>
-     <origin xyz="0 0 0" rpy="0 0 0" />
-      <geometry>
-            <mesh filename="package://neo_simulation/robots/mp_500/meshes/MP-500-WHEEL-LEFT.dae" scale="0.001 0.001 0.001"/>
-      </geometry>
-    </collision>
-</link>
-  <gazebo reference="${name}_link">
-      <mu1 value = "300.0"/>
-      <mu2 value = "100.0"/>
-      <kp value="8000.0" />
-      <kd value="1460.0" />
-      <fdir1 value="0.5 0 0"/>
-</gazebo>
+        </actuator>
+    </transmission>
+    <link name="${name}_link" type="wheel">
+        <inertial>
+            <origin xyz="0 0 0" rpy="0 0 0"/>
+            <mass value="1.82362"/>
+            <inertia ixx="0.00399743171" ixy="0.00000004464" ixz="-0.00000002245"
+                iyy="0.00399741733" iyz="-0.00000000164"
+                izz="0.00739239692"/>
+        </inertial>
+        <visual>
+            <origin xyz="0 0 0" rpy="0 0 3.14" />
+            <geometry>
+                <mesh filename="package://neo_simulation/robots/mp_500/meshes/MP-500-WHEEL-LEFT.dae" scale="0.001 0.001 0.001"/>
+            </geometry>
+        </visual>
+        <collision>
+            <origin xyz="0 0 0" rpy="0 0 0" />
+            <geometry>
+                <mesh filename="package://neo_simulation/robots/mp_500/meshes/MP-500-WHEEL-LEFT.dae" scale="0.001 0.001 0.001"/>
+            </geometry>
+        </collision>
+    </link>
+    <gazebo reference="${name}_link">
+        <mu1 value = "300.0"/>
+        <mu2 value = "100.0"/>
+        <kp value="8000.0" />
+        <kd value="1460.0" />
+        <fdir1 value="0.5 0 0"/>
+    </gazebo>
   </xacro:macro>
 </robot>

Commit message: fix bugs

File: ugv_description/urdf/mp_500/mp_500.urdf.xacro (robot description, xacro)
@@ -2,24 +2,24 @@
 <!-- Materials -->
 <robot xmlns:xacro="http://www.ros.org/wiki/xacro" name="mp_500">
-<xacro:include filename="$(find neo_simulation)/robots/mp_500/xacros/mp_500_gazebo.xacro" />
+<xacro:include filename="$(find ugv_description)/urdf/mp_500/xacros/mp_500_gazebo.xacro" />
 <!--++++++++++++++++++++++++++++++base_link++++++++++++++++++++++++++++++++++++++++++++++++++++-->
 <!--++++++++++++++++++++body++++++++++++++++++++++++++++-->
-<xacro:include filename="$(find neo_simulation)/robots/mp_500/xacros/mp_500_body.xacro" />
+<xacro:include filename="$(find ugv_description)/urdf/mp_500/xacros/mp_500_body.xacro" />
 <!--+++++++++++++++++++castor_wheel_link++++++++++++++++++++++++-->
-<xacro:include filename="$(find neo_simulation)/robots/mp_500/xacros/mp_500_caster_wheel.xacro" />
+<xacro:include filename="$(find ugv_description)/urdf/mp_500/xacros/mp_500_caster_wheel.xacro" />
 <!--+++++++++++++++++++left_wheel_link++++++++++++++++++++++++-->
-<xacro:include filename="$(find neo_simulation)/robots/mp_500/xacros/mp_500_fixed_wheel_left.xacro" />
-<xacro:include filename="$(find neo_simulation)/robots/mp_500/xacros/mp_500_fixed_wheel_right.xacro" />
-<xacro:macro name="mp_500">
-  <xacro:mp_500_base name="base_link">
+<xacro:include filename="$(find ugv_description)/urdf/mp_500/xacros/mp_500_fixed_wheel_left.xacro" />
+<xacro:include filename="$(find ugv_description)/urdf/mp_500/xacros/mp_500_fixed_wheel_right.xacro" />
+<xacro:macro name="mp_500" params="namespace">
+  <xacro:mp_500_base name="${namespace}/base_link">
   </xacro:mp_500_base>
   <!-- Wheel Macro -->
-  <xacro:caster_wheel name="caster_wheel" parent="base_link">
+  <xacro:caster_wheel name="${namespace}/caster_wheel" parent="${namespace}/base_link">
     <origin xyz="-0.43 0. 0.176" rpy="-1.570796 0 1.570796 " />
   </xacro:caster_wheel>
-  <xacro:fixed_wheel_right name="wheel_right" parent="base_link" number="1">
+  <xacro:fixed_wheel_right name="${namespace}/wheel_right" parent="${namespace}/base_link" number="1">
     <origin xyz="0. -0.25 0.13" rpy="0 0 -1.570796" />
   </xacro:fixed_wheel_right>
-  <xacro:fixed_wheel_left name="wheel_left" parent="base_link" number="2">
+  <xacro:fixed_wheel_left name="${namespace}/wheel_left" parent="${namespace}/base_link" number="2">
     <origin xyz="0. 0.25 0.13" rpy="0 0 -1.570796" />
   </xacro:fixed_wheel_left>
@@ -27,5 +27,5 @@
    <!-- SENSORS -->
   <xacro:include filename="$(find neo_simulation)/robots/mp_500/xacros/sick_laser.xacro" />
-  <xacro:sick_laser_v0 name="laser_1" parent="base_link" ros_topic="/laser_1/scan">
+  <xacro:sick_laser_v0 name="${namespace}/laser_1" parent="${namespace}/base_link" ros_topic="/laser_1/scan">
     <origin xyz="0.244 0 0.141" rpy="3.14 0 0" />
   </xacro:sick_laser_v0>

File: ugv_description/urdf/mp_500/multi_mp_500.urdf.xacro (robot description, xacro)
@@ -3,4 +3,4 @@
 <robot xmlns:xacro="http://www.ros.org/wiki/xacro" name="multi_mp_500">
 <xacro:include filename="$(find ugv_description)/urdf/mp_500/mp_500.urdf.xacro" />
-<xacro:mp_500 />
+<xacro:mp_500 namespace="ugv_0"/>
 </robot>

File: ugv_description/urdf/mp_500/xacros/mp_500_fixed_wheel_left.xacro (robot description, xacro)
@@ -7,5 +7,5 @@
         <axis xyz="-1 0 0" />
         <joint_properties damping="0" friction="0.0" />
-        <parent link="base_link" />
+        <parent link="${namespace}/base_link" />
         <child link="${name}_link" />
     </joint>

File: ugv_description/urdf/mp_500/xacros/mp_500_fixed_wheel_right.xacro (robot description, xacro)
@@ -7,5 +7,5 @@
     <axis xyz="-1 0 0" />
     <joint_properties damping="0" friction="0.0" />
-    <parent link="base_link" />
+    <parent link="${namespace}/base_link" />
     <child link="${name}_link" />
    </joint>

Commit message: fix bugs

File: ugv_description/urdf/mp_500/mp_500.urdf.xacro (robot description, xacro)
@@ -1,33 +1,28 @@
 <?xml version="1.0"?>
-<!-- Materials -->
 <robot xmlns:xacro="http://www.ros.org/wiki/xacro" name="mp_500">
-<xacro:include filename="$(find ugv_description)/urdf/mp_500/xacros/mp_500_gazebo.xacro" />
-<!--++++++++++++++++++++++++++++++base_link++++++++++++++++++++++++++++++++++++++++++++++++++++-->
-<!--++++++++++++++++++++body++++++++++++++++++++++++++++-->
-<xacro:include filename="$(find ugv_description)/urdf/mp_500/xacros/mp_500_body.xacro" />
-<!--+++++++++++++++++++castor_wheel_link++++++++++++++++++++++++-->
-<xacro:include filename="$(find ugv_description)/urdf/mp_500/xacros/mp_500_caster_wheel.xacro" />
-<!--+++++++++++++++++++left_wheel_link++++++++++++++++++++++++-->
-<xacro:include filename="$(find ugv_description)/urdf/mp_500/xacros/mp_500_fixed_wheel_left.xacro" />
-<xacro:include filename="$(find ugv_description)/urdf/mp_500/xacros/mp_500_fixed_wheel_right.xacro" />
-<xacro:macro name="mp_500" params="namespace">
-  <xacro:mp_500_base name="${namespace}/base_link">
-  </xacro:mp_500_base>
-  <!-- Wheel Macro -->
-  <xacro:caster_wheel name="${namespace}/caster_wheel" parent="${namespace}/base_link">
-    <origin xyz="-0.43 0. 0.176" rpy="-1.570796 0 1.570796 " />
-  </xacro:caster_wheel>
-  <xacro:fixed_wheel_right name="${namespace}/wheel_right" parent="${namespace}/base_link" number="1">
-    <origin xyz="0. -0.25 0.13" rpy="0 0 -1.570796" />
-  </xacro:fixed_wheel_right>
-  <xacro:fixed_wheel_left name="${namespace}/wheel_left" parent="${namespace}/base_link" number="2">
-    <origin xyz="0. 0.25 0.13" rpy="0 0 -1.570796" />
-  </xacro:fixed_wheel_left>
- <!--+++++++++++++++++++laserscanner_front_link++++++++++++++++++++++++-->
-   <!-- SENSORS -->
-  <xacro:include filename="$(find neo_simulation)/robots/mp_500/xacros/sick_laser.xacro" />
-  <xacro:sick_laser_v0 name="${namespace}/laser_1" parent="${namespace}/base_link" ros_topic="/laser_1/scan">
-    <origin xyz="0.244 0 0.141" rpy="3.14 0 0" />
-  </xacro:sick_laser_v0>
-</xacro:macro>
+    <xacro:macro name="mp_500" params="namespace">
+        <xacro:include filename="$(find ugv_description)/urdf/mp_500/xacros/mp_500_gazebo.xacro" />
+        <xacro:include filename="$(find ugv_description)/urdf/mp_500/xacros/mp_500_body.xacro" />
+        <xacro:include filename="$(find ugv_description)/urdf/mp_500/xacros/mp_500_caster_wheel.xacro" />
+        <xacro:include filename="$(find ugv_description)/urdf/mp_500/xacros/mp_500_fixed_wheel_left.xacro" />
+        <xacro:include filename="$(find ugv_description)/urdf/mp_500/xacros/mp_500_fixed_wheel_right.xacro" />
+        <xacro:mp_500_base name="${namespace}/base_link">
+        </xacro:mp_500_base>
+        <!-- Wheel Macro -->
+        <xacro:caster_wheel name="${namespace}/caster_wheel" parent="${namespace}/base_link">
+            <origin xyz="-0.43 0. 0.176" rpy="-1.570796 0 1.570796 " />
+        </xacro:caster_wheel>
+        <xacro:fixed_wheel_right name="${namespace}/wheel_right" parent="${namespace}/base_link" number="1">
+            <origin xyz="0. -0.25 0.13" rpy="0 0 -1.570796" />
+        </xacro:fixed_wheel_right>
+        <xacro:fixed_wheel_left name="${namespace}/wheel_left" parent="${namespace}/base_link" number="2">
+            <origin xyz="0. 0.25 0.13" rpy="0 0 -1.570796" />
+        </xacro:fixed_wheel_left>
+        <!--+++++++++++++++++++laserscanner_front_link++++++++++++++++++++++++-->
+        <!-- SENSORS -->
+        <xacro:include filename="$(find neo_simulation)/robots/mp_500/xacros/sick_laser.xacro" />
+        <xacro:sick_laser_v0 name="${namespace}/laser_1" parent="${namespace}/base_link" ros_topic="/laser_1/scan">
+            <origin xyz="0.244 0 0.141" rpy="3.14 0 0" />
+        </xacro:sick_laser_v0>
+    </xacro:macro>
 </robot>

File: ugv_description/urdf/mp_500/multi_mp_500.urdf.xacro (robot description, xacro)
@@ -1,6 +1,5 @@
 <?xml version="1.0"?>
-<!-- Materials -->
 <robot xmlns:xacro="http://www.ros.org/wiki/xacro" name="multi_mp_500">
-<xacro:include filename="$(find ugv_description)/urdf/mp_500/mp_500.urdf.xacro" />
-<xacro:mp_500 namespace="ugv_0"/>
+    <xacro:include filename="$(find ugv_description)/urdf/mp_500/mp_500.urdf.xacro" />
+    <xacro:mp_500 namespace="ugv_0"/>
 </robot>

File: ugv_description/urdf/mp_500/xacros/mp_500_gazebo.xacro (robot description, xacro)
@@ -42,6 +42,6 @@
         <legacyMode>false</legacyMode>
         <torque>2.5</torque>
-        <leftJoint>wheel_left_joint</leftJoint>
-        <rightJoint>wheel_right_joint</rightJoint>
+        <leftJoint>${namespace}/wheel_left_joint</leftJoint>
+        <rightJoint>${namespace}/wheel_right_joint</rightJoint>
         <wheelSeparation>0.592</wheelSeparation>
         <wheelDiameter>0.260</wheelDiameter>

Commit message: added teleop_keyboard script & could control 4 ugv

File: ugv_description/urdf/mp_500/mp_500.urdf.xacro (robot description, xacro)
@@ -1,28 +1,27 @@
 <?xml version="1.0"?>
 <robot xmlns:xacro="http://www.ros.org/wiki/xacro" name="mp_500">
-    <xacro:macro name="mp_500" params="namespace">
-        <xacro:include filename="$(find ugv_description)/urdf/mp_500/xacros/mp_500_gazebo.xacro" />
-        <xacro:include filename="$(find ugv_description)/urdf/mp_500/xacros/mp_500_body.xacro" />
-        <xacro:include filename="$(find ugv_description)/urdf/mp_500/xacros/mp_500_caster_wheel.xacro" />
-        <xacro:include filename="$(find ugv_description)/urdf/mp_500/xacros/mp_500_fixed_wheel_left.xacro" />
-        <xacro:include filename="$(find ugv_description)/urdf/mp_500/xacros/mp_500_fixed_wheel_right.xacro" />
-        <xacro:mp_500_base name="${namespace}/base_link">
-        </xacro:mp_500_base>
-        <!-- Wheel Macro -->
-        <xacro:caster_wheel name="${namespace}/caster_wheel" parent="${namespace}/base_link">
-            <origin xyz="-0.43 0. 0.176" rpy="-1.570796 0 1.570796 " />
-        </xacro:caster_wheel>
-        <xacro:fixed_wheel_right name="${namespace}/wheel_right" parent="${namespace}/base_link" number="1">
-            <origin xyz="0. -0.25 0.13" rpy="0 0 -1.570796" />
-        </xacro:fixed_wheel_right>
-        <xacro:fixed_wheel_left name="${namespace}/wheel_left" parent="${namespace}/base_link" number="2">
-            <origin xyz="0. 0.25 0.13" rpy="0 0 -1.570796" />
-        </xacro:fixed_wheel_left>
-        <!--+++++++++++++++++++laserscanner_front_link++++++++++++++++++++++++-->
-        <!-- SENSORS -->
-        <xacro:include filename="$(find neo_simulation)/robots/mp_500/xacros/sick_laser.xacro" />
-        <xacro:sick_laser_v0 name="${namespace}/laser_1" parent="${namespace}/base_link" ros_topic="/laser_1/scan">
-            <origin xyz="0.244 0 0.141" rpy="3.14 0 0" />
-        </xacro:sick_laser_v0>
-    </xacro:macro>
+    <xacro:property name="namespace" value="$(arg namespace)" />
+    <xacro:include filename="$(find ugv_description)/urdf/mp_500/xacros/mp_500_gazebo.xacro" />
+    <xacro:include filename="$(find ugv_description)/urdf/mp_500/xacros/mp_500_body.xacro" />
+    <xacro:include filename="$(find ugv_description)/urdf/mp_500/xacros/mp_500_caster_wheel.xacro" />
+    <xacro:include filename="$(find ugv_description)/urdf/mp_500/xacros/mp_500_fixed_wheel_left.xacro" />
+    <xacro:include filename="$(find ugv_description)/urdf/mp_500/xacros/mp_500_fixed_wheel_right.xacro" />
+    <xacro:mp_500_base name="${namespace}/base_link">
+    </xacro:mp_500_base>
+    <!-- Wheel Macro -->
+    <xacro:caster_wheel name="${namespace}/caster_wheel" parent="${namespace}/base_link">
+        <origin xyz="-0.43 0. 0.176" rpy="-1.570796 0 1.570796 " />
+    </xacro:caster_wheel>
+    <xacro:fixed_wheel_right name="${namespace}/wheel_right" parent="${namespace}/base_link" number="1">
+        <origin xyz="0. -0.25 0.13" rpy="0 0 -1.570796" />
+    </xacro:fixed_wheel_right>
+    <xacro:fixed_wheel_left name="${namespace}/wheel_left" parent="${namespace}/base_link" number="2">
+        <origin xyz="0. 0.25 0.13" rpy="0 0 -1.570796" />
+    </xacro:fixed_wheel_left>
+    <!--+++++++++++++++++++laserscanner_front_link++++++++++++++++++++++++-->
+    <!-- SENSORS -->
+    <xacro:include filename="$(find neo_simulation)/robots/mp_500/xacros/sick_laser.xacro" />
+    <xacro:sick_laser_v0 name="${namespace}/laser_1" parent="${namespace}/base_link" ros_topic="/laser_1/scan">
+        <origin xyz="0.244 0 0.141" rpy="3.14 0 0" />
+    </xacro:sick_laser_v0>
 </robot>
