Commit message: Update

File: ugv_description/urdf/mp_500/xacros/mp_500_tether_end.xacro (robot description, xacro)
@@ -1,5 +1,5 @@
 <?xml version="1.0"?>
 <robot xmlns:xacro="http://www.ros.org/wiki/xacro" name="mp_500">
-    <xacro:property name="counter_weight_mass" value="5.0" />
+    <xacro:property name="counter_weight_mass" value="15.0" />
     <xacro:property name="counter_weight_x" value="0.1" />
     <xacro:property name="counter_weight_y" value="0.1" />
@@ -33,5 +33,5 @@
             <parent link="${namespace}/base_link" />
             <child link="${name}" />
-            <origin xyz="-0.4 0.0 0.4" rpy="0 0 0" />
+            <origin xyz="-0.2 0.0 0.4" rpy="0 0 0" />
         </joint>
         <link name="${name}">
