Commit message: Fixed tether model

File: pyramid_description/tether_description/urdf/massless_rigid_tether.xacro (robot description, xacro)
@@ -5,5 +5,5 @@
         <!--tether params-->
         {%- set tether_mass = 0.001 -%}
-        {%- set tether_length = 10.0 -%}
+        {%- set tether_length = 20.0 -%}
         {%- set tether_radius = 0.005 -%}
         {%- set tether_inertia = 0.001 -%}
@@ -11,12 +11,15 @@
         {%- set virtual_link_mass = 0.001 -%}
         {%- set virtual_link_inertia = 0.001 -%}
-        <!--joint dynamics-->
-        {%- set damping = 1 -%}
-        {%- set friction = 1 -%}
+        <!--actuated joint dynamics-->
+        {%- set actuated_damping = 0.01 -%}
+        {%- set actuated_friction = 0.0 -%}
+        <!--passive joint dynamics-->
+        {%- set passive_damping = 0.01 -%}
+        {%- set passive_friction = 0.0 -%}
         {%- set tether_number = 4 -%}
         {%- macro tether(dirc) -%}
         <link name="tether_{{dirc}}">
             <visual>
-                <origin rpy="0 0 0" xyz="0 0 0"/>
+                <origin rpy="0 0 0" xyz="0 0 {{tether_length/2}}"/>
                 <geometry>
                     <cylinder length="{{tether_length}}" radius="{{tether_radius}}"/>
@@ -101,5 +104,5 @@
             <child link="virtual_link_uav2tether_1_{{dirc}}"/>
             <axis xyz="1 0 0" />
-            <dynamics damping="{{damping}}" friction="{{friction}}"/>
+            <dynamics damping="{{passive_damping}}" friction="{{passive_friction}}"/>
         </joint>
         <joint name="rod2tether_joint_pitch_{{dirc}}" type="continuous">
@@ -108,5 +111,5 @@
             <child link="virtual_link_uav2tether_2_{{dirc}}"/>
             <axis xyz="0 1 0" />
-            <dynamics damping="{{damping}}" friction="{{friction}}"/>
+            <dynamics damping="{{passive_damping}}" friction="{{passive_friction}}"/>
         </joint>
         <joint name="rod2tether_joint_yaw_{{dirc}}" type="continuous">
@@ -115,15 +118,15 @@
             <child link="tether_{{dirc}}"/>
             <axis xyz="0 0 1" />
-            <dynamics damping="{{damping}}" friction="{{friction}}"/>
+            <dynamics damping="{{passive_damping}}" friction="{{passive_friction}}"/>
         </joint>
         {%- endmacro -%}
         {%- macro ugv2tether_joint(dirc) -%}
         <joint name="ugv2tether_joint_prismatic_{{dirc}}" type="prismatic">
-            <origin rpy="0 0 0" xyz="0 0 10"/>
+            <origin rpy="0 0 0" xyz="0 0 5"/>
             <parent link="tether_{{dirc}}"/>
             <child link="virtual_link_ugv2tether_1_{{dirc}}"/>
             <axis xyz="0 0 1" />
-            <dynamics damping="{{damping}}" friction="{{friction}}"/>
-            <limit effort="10000" lower="-5.0" upper="5.0" velocity="10.0"/>
+            <dynamics damping="{{actuated_damping}}" friction="{{actuated_friction}}"/>
+            <limit effort="10000" lower="-5.0" upper="10.0" velocity="10.0"/>
         </joint>
         <joint name="ugv2tether_joint_roll_{{dirc}}" type="continuous">
@@ -132,5 +135,5 @@
             <child link="virtual_link_ugv2tether_2_{{dirc}}"/>
             <axis xyz="1 0 0" />
-            <dynamics damping="{{damping}}" friction="{{friction}}"/>
+            <dynamics damping="{{passive_damping}}" friction="{{passive_friction}}"/>
         </joint>
         <joint name="ugv2tether_joint_pitch_{{dirc}}" type="continuous">
@@ -139,5 +142,5 @@
             <child link="virtual_link_ugv2tether_3_{{dirc}}"/>
             <axis xyz="0 1 0" />
-            <dynamics damping="{{damping}}" friction="{{friction}}"/>
+            <dynamics damping="{{passive_damping}}" friction="{{passive_friction}}"/>
         </joint>
         <joint name="ugv2tether_joint_yaw_{{dirc}}" type="continuous">
@@ -154,5 +157,5 @@
             <parent link="virtual_link_ugv2tether_3_{{dirc}}"/>
             <child link="mp_500_{{dirc}}/tether_end"/>
-            <dynamics damping="{{damping}}" friction="{{friction}}"/>
+            <dynamics damping="{{passive_damping}}" friction="{{passive_friction}}"/>
         </joint>
         {%- endmacro -%}

File: pyramid_description/tether_description/urdf/tether.xacro (robot description, xacro)
@@ -3,10 +3,10 @@
     <!--tether model-->
     <xacro:macro name="tether">
-        <!--tether params--><!--virtual link params--><!--joint dynamics--><!-- main-->
+        <!--tether params--><!--virtual link params--><!--actuated joint dynamics--><!--passive joint dynamics--><!-- main-->
             <link name="tether_0">
             <visual>
-                <origin rpy="0 0 0" xyz="0 0 0"/>
-                <geometry>
-                    <cylinder length="10.0" radius="0.005"/>
+                <origin rpy="0 0 0" xyz="0 0 10.0"/>
+                <geometry>
+                    <cylinder length="20.0" radius="0.005"/>
                 </geometry>
             </visual>
@@ -75,5 +75,5 @@
             <child link="virtual_link_uav2tether_1_0"/>
             <axis xyz="1 0 0" />
-            <dynamics damping="1" friction="1"/>
+            <dynamics damping="0.01" friction="0.0"/>
         </joint>
         <joint name="rod2tether_joint_pitch_0" type="continuous">
@@ -82,5 +82,5 @@
             <child link="virtual_link_uav2tether_2_0"/>
             <axis xyz="0 1 0" />
-            <dynamics damping="1" friction="1"/>
+            <dynamics damping="0.01" friction="0.0"/>
         </joint>
         <joint name="rod2tether_joint_yaw_0" type="continuous">
@@ -89,13 +89,13 @@
             <child link="tether_0"/>
             <axis xyz="0 0 1" />
-            <dynamics damping="1" friction="1"/>
+            <dynamics damping="0.01" friction="0.0"/>
         </joint>
             <joint name="ugv2tether_joint_prismatic_0" type="prismatic">
-            <origin rpy="0 0 0" xyz="0 0 10"/>
+            <origin rpy="0 0 0" xyz="0 0 5"/>
             <parent link="tether_0"/>
             <child link="virtual_link_ugv2tether_1_0"/>
             <axis xyz="0 0 1" />
-            <dynamics damping="1" friction="1"/>
-            <limit effort="10000" lower="-5.0" upper="5.0" velocity="10.0"/>
+            <dynamics damping="0.01" friction="0.0"/>
+            <limit effort="10000" lower="-5.0" upper="10.0" velocity="10.0"/>
         </joint>
         <joint name="ugv2tether_joint_roll_0" type="continuous">
@@ -104,5 +104,5 @@
             <child link="virtual_link_ugv2tether_2_0"/>
             <axis xyz="1 0 0" />
-            <dynamics damping="1" friction="1"/>
+            <dynamics damping="0.01" friction="0.0"/>
         </joint>
         <joint name="ugv2tether_joint_pitch_0" type="continuous">
@@ -111,5 +111,5 @@
             <child link="virtual_link_ugv2tether_3_0"/>
             <axis xyz="0 1 0" />
-            <dynamics damping="1" friction="1"/>
+            <dynamics damping="0.01" friction="0.0"/>
         </joint>
         <joint name="ugv2tether_joint_yaw_0" type="continuous">
@@ -118,11 +118,11 @@
             <parent link="virtual_link_ugv2tether_3_0"/>
             <child link="mp_500_0/tether_end"/>
-            <dynamics damping="1" friction="1"/>
+            <dynamics damping="0.01" friction="0.0"/>
         </joint>
             <link name="tether_1">
             <visual>
-                <origin rpy="0 0 0" xyz="0 0 0"/>
-                <geometry>
-                    <cylinder length="10.0" radius="0.005"/>
+                <origin rpy="0 0 0" xyz="0 0 10.0"/>
+                <geometry>
+                    <cylinder length="20.0" radius="0.005"/>
                 </geometry>
             </visual>
@@ -191,5 +191,5 @@
             <child link="virtual_link_uav2tether_1_1"/>
             <axis xyz="1 0 0" />
-            <dynamics damping="1" friction="1"/>
+            <dynamics damping="0.01" friction="0.0"/>
         </joint>
         <joint name="rod2tether_joint_pitch_1" type="continuous">
@@ -198,5 +198,5 @@
             <child link="virtual_link_uav2tether_2_1"/>
             <axis xyz="0 1 0" />
-            <dynamics damping="1" friction="1"/>
+            <dynamics damping="0.01" friction="0.0"/>
         </joint>
         <joint name="rod2tether_joint_yaw_1" type="continuous">
@@ -205,13 +205,13 @@
             <child link="tether_1"/>
             <axis xyz="0 0 1" />
-            <dynamics damping="1" friction="1"/>
+            <dynamics damping="0.01" friction="0.0"/>
         </joint>
             <joint name="ugv2tether_joint_prismatic_1" type="prismatic">
-            <origin rpy="0 0 0" xyz="0 0 10"/>
+            <origin rpy="0 0 0" xyz="0 0 5"/>
             <parent link="tether_1"/>
             <child link="virtual_link_ugv2tether_1_1"/>
             <axis xyz="0 0 1" />
-            <dynamics damping="1" friction="1"/>
-            <limit effort="10000" lower="-5.0" upper="5.0" velocity="10.0"/>
+            <dynamics damping="0.01" friction="0.0"/>
+            <limit effort="10000" lower="-5.0" upper="10.0" velocity="10.0"/>
         </joint>
         <joint name="ugv2tether_joint_roll_1" type="continuous">
@@ -220,5 +220,5 @@
             <child link="virtual_link_ugv2tether_2_1"/>
             <axis xyz="1 0 0" />
-            <dynamics damping="1" friction="1"/>
+            <dynamics damping="0.01" friction="0.0"/>
         </joint>
         <joint name="ugv2tether_joint_pitch_1" type="continuous">
@@ -227,5 +227,5 @@
             <child link="virtual_link_ugv2tether_3_1"/>
             <axis xyz="0 1 0" />
-            <dynamics damping="1" friction="1"/>
+            <dynamics damping="0.01" friction="0.0"/>
         </joint>
         <joint name="ugv2tether_joint_yaw_1" type="continuous">
@@ -234,11 +234,11 @@
             <parent link="virtual_link_ugv2tether_3_1"/>
             <child link="mp_500_1/tether_end"/>
-            <dynamics damping="1" friction="1"/>
+            <dynamics damping="0.01" friction="0.0"/>
         </joint>
             <link name="tether_2">
             <visual>
-                <origin rpy="0 0 0" xyz="0 0 0"/>
-                <geometry>
-                    <cylinder length="10.0" radius="0.005"/>
+                <origin rpy="0 0 0" xyz="0 0 10.0"/>
+                <geometry>
+                    <cylinder length="20.0" radius="0.005"/>
                 </geometry>
             </visual>
@@ -307,5 +307,5 @@
             <child link="virtual_link_uav2tether_1_2"/>
             <axis xyz="1 0 0" />
-            <dynamics damping="1" friction="1"/>
+            <dynamics damping="0.01" friction="0.0"/>
         </joint>
         <joint name="rod2tether_joint_pitch_2" type="continuous">
@@ -314,5 +314,5 @@
             <child link="virtual_link_uav2tether_2_2"/>
             <axis xyz="0 1 0" />
-            <dynamics damping="1" friction="1"/>
+            <dynamics damping="0.01" friction="0.0"/>
         </joint>
         <joint name="rod2tether_joint_yaw_2" type="continuous">
@@ -321,13 +321,13 @@
             <child link="tether_2"/>
             <axis xyz="0 0 1" />
-            <dynamics damping="1" friction="1"/>
+            <dynamics damping="0.01" friction="0.0"/>
         </joint>
             <joint name="ugv2tether_joint_prismatic_2" type="prismatic">
-            <origin rpy="0 0 0" xyz="0 0 10"/>
+            <origin rpy="0 0 0" xyz="0 0 5"/>
             <parent link="tether_2"/>
             <child link="virtual_link_ugv2tether_1_2"/>
             <axis xyz="0 0 1" />
-            <dynamics damping="1" friction="1"/>
-            <limit effort="10000" lower="-5.0" upper="5.0" velocity="10.0"/>
+            <dynamics damping="0.01" friction="0.0"/>
+            <limit effort="10000" lower="-5.0" upper="10.0" velocity="10.0"/>
         </joint>
         <joint name="ugv2tether_joint_roll_2" type="continuous">
@@ -336,5 +336,5 @@
             <child link="virtual_link_ugv2tether_2_2"/>
             <axis xyz="1 0 0" />
-            <dynamics damping="1" friction="1"/>
+            <dynamics damping="0.01" friction="0.0"/>
         </joint>
         <joint name="ugv2tether_joint_pitch_2" type="continuous">
@@ -343,5 +343,5 @@
             <child link="virtual_link_ugv2tether_3_2"/>
             <axis xyz="0 1 0" />
-            <dynamics damping="1" friction="1"/>
+            <dynamics damping="0.01" friction="0.0"/>
         </joint>
         <joint name="ugv2tether_joint_yaw_2" type="continuous">
@@ -350,11 +350,11 @@
             <parent link="virtual_link_ugv2tether_3_2"/>
             <child link="mp_500_2/tether_end"/>
-            <dynamics damping="1" friction="1"/>
+            <dynamics damping="0.01" friction="0.0"/>
         </joint>
             <link name="tether_3">
             <visual>
-                <origin rpy="0 0 0" xyz="0 0 0"/>
-                <geometry>
-                    <cylinder length="10.0" radius="0.005"/>
+                <origin rpy="0 0 0" xyz="0 0 10.0"/>
+                <geometry>
+                    <cylinder length="20.0" radius="0.005"/>
                 </geometry>
             </visual>
@@ -423,5 +423,5 @@
             <child link="virtual_link_uav2tether_1_3"/>
             <axis xyz="1 0 0" />
-            <dynamics damping="1" friction="1"/>
+            <dynamics damping="0.01" friction="0.0"/>
         </joint>
         <joint name="rod2tether_joint_pitch_3" type="continuous">
@@ -430,5 +430,5 @@
             <child link="virtual_link_uav2tether_2_3"/>
             <axis xyz="0 1 0" />
-            <dynamics damping="1" friction="1"/>
+            <dynamics damping="0.01" friction="0.0"/>
         </joint>
         <joint name="rod2tether_joint_yaw_3" type="continuous">
@@ -437,13 +437,13 @@
             <child link="tether_3"/>
             <axis xyz="0 0 1" />
-            <dynamics damping="1" friction="1"/>
+            <dynamics damping="0.01" friction="0.0"/>
         </joint>
             <joint name="ugv2tether_joint_prismatic_3" type="prismatic">
-            <origin rpy="0 0 0" xyz="0 0 10"/>
+            <origin rpy="0 0 0" xyz="0 0 5"/>
             <parent link="tether_3"/>
             <child link="virtual_link_ugv2tether_1_3"/>
             <axis xyz="0 0 1" />
-            <dynamics damping="1" friction="1"/>
-            <limit effort="10000" lower="-5.0" upper="5.0" velocity="10.0"/>
+            <dynamics damping="0.01" friction="0.0"/>
+            <limit effort="10000" lower="-5.0" upper="10.0" velocity="10.0"/>
         </joint>
         <joint name="ugv2tether_joint_roll_3" type="continuous">
@@ -452,5 +452,5 @@
             <child link="virtual_link_ugv2tether_2_3"/>
             <axis xyz="1 0 0" />
-            <dynamics damping="1" friction="1"/>
+            <dynamics damping="0.01" friction="0.0"/>
         </joint>
         <joint name="ugv2tether_joint_pitch_3" type="continuous">
@@ -459,5 +459,5 @@
             <child link="virtual_link_ugv2tether_3_3"/>
             <axis xyz="0 1 0" />
-            <dynamics damping="1" friction="1"/>
+            <dynamics damping="0.01" friction="0.0"/>
         </joint>
         <joint name="ugv2tether_joint_yaw_3" type="continuous">
@@ -466,5 +466,5 @@
             <parent link="virtual_link_ugv2tether_3_3"/>
             <child link="mp_500_3/tether_end"/>
-            <dynamics damping="1" friction="1"/>
+            <dynamics damping="0.01" friction="0.0"/>
         </joint>
         </xacro:macro>

Commit message: FIxbugs

File: pyramid_description/tether_description/urdf/massless_rigid_tether.xacro (robot description, xacro)
@@ -168,4 +168,8 @@
             {{ugv2tether_joint(dirc)}}
         {% endfor -%}
+        <gazebo>
+            <!--plugin name="rover_plugin" filename="librover_plugin.so"> </plugin-->
+            <plugin name="tensions" filename="libgazebo_tensions_plugin.so"/>
+        </gazebo>
     </xacro:macro>
 </robot>

File: pyramid_description/tether_description/urdf/tether.xacro (robot description, xacro)
@@ -468,4 +468,8 @@
             <dynamics damping="0.01" friction="0.0"/>
         </joint>
-        </xacro:macro>
+        <gazebo>
+            <!--plugin name="rover_plugin" filename="librover_plugin.so"> </plugin-->
+            <plugin name="tensions" filename="libgazebo_tensions_plugin.so"/>
+        </gazebo>
+    </xacro:macro>
 </robot>
