Commit message: Added libgazebo_ros_joint_state_publisher.so to urdf

File: pyramid_description/tether_description/urdf/massless_rigid_tether.xacro (robot description, xacro)
@@ -126,5 +126,5 @@
             <parent link="tether_{{dirc}}"/>
             <child link="virtual_link_ugv2tether_1_{{dirc}}"/>
-            <axis xyz="0 0 1" />
+            <axis xyz="0 0 -1" />
             <dynamics damping="{{actuated_damping}}" friction="{{actuated_friction}}"/>
             <limit effort="10000" lower="-5.0" upper="10.0" velocity="10.0"/>
@@ -170,4 +170,23 @@
         <gazebo>
             <plugin name="gazebo_tensions_plugin" filename="libgazebo_tensions_plugin.so"/>
+            <plugin name="joint_state_publisher" filename="libgazebo_ros_joint_state_publisher.so">
+                <robotNamespace>pelican</robotNamespace>
+                <jointName>
+                rod2tether_joint_roll_0, rod2tether_joint_pitch_0, rod2tether_joint_yaw_0,
+                rod2tether_joint_roll_1, rod2tether_joint_pitch_1, rod2tether_joint_yaw_1,
+                rod2tether_joint_roll_2, rod2tether_joint_pitch_2, rod2tether_joint_yaw_2,
+                rod2tether_joint_roll_3, rod2tether_joint_pitch_3, rod2tether_joint_yaw_3,
+                ugv2tether_joint_prismatic_0,
+                ugv2tether_joint_prismatic_1,
+                ugv2tether_joint_prismatic_2,
+                ugv2tether_joint_prismatic_3,
+                ugv2tether_joint_roll_0, ugv2tether_joint_pitch_0, ugv2tether_joint_yaw_0,
+                ugv2tether_joint_roll_1, ugv2tether_joint_pitch_1, ugv2tether_joint_yaw_1,
+                ugv2tether_joint_roll_2, ugv2tether_joint_pitch_2, ugv2tether_joint_yaw_2,
+                ugv2tether_joint_roll_3, ugv2tether_joint_pitch_3, ugv2tether_joint_yaw_3
+                </jointName>
+                <updateRate>1000</updateRate>
+                <alwaysOn>true</alwaysOn>
+            </plugin>
         </gazebo>
     </xacro:macro>

File: pyramid_description/tether_description/urdf/tether.xacro (robot description, xacro)
@@ -95,5 +95,5 @@
             <parent link="tether_0"/>
             <child link="virtual_link_ugv2tether_1_0"/>
-            <axis xyz="0 0 1" />
+            <axis xyz="0 0 -1" />
             <dynamics damping="0.01" friction="0.0"/>
             <limit effort="10000" lower="-5.0" upper="10.0" velocity="10.0"/>
@@ -211,5 +211,5 @@
             <parent link="tether_1"/>
             <child link="virtual_link_ugv2tether_1_1"/>
-            <axis xyz="0 0 1" />
+            <axis xyz="0 0 -1" />
             <dynamics damping="0.01" friction="0.0"/>
             <limit effort="10000" lower="-5.0" upper="10.0" velocity="10.0"/>
@@ -327,5 +327,5 @@
             <parent link="tether_2"/>
             <child link="virtual_link_ugv2tether_1_2"/>
-            <axis xyz="0 0 1" />
+            <axis xyz="0 0 -1" />
             <dynamics damping="0.01" friction="0.0"/>
             <limit effort="10000" lower="-5.0" upper="10.0" velocity="10.0"/>
@@ -443,5 +443,5 @@
             <parent link="tether_3"/>
             <child link="virtual_link_ugv2tether_1_3"/>
-            <axis xyz="0 0 1" />
+            <axis xyz="0 0 -1" />
             <dynamics damping="0.01" friction="0.0"/>
             <limit effort="10000" lower="-5.0" upper="10.0" velocity="10.0"/>
@@ -470,4 +470,23 @@
         <gazebo>
             <plugin name="gazebo_tensions_plugin" filename="libgazebo_tensions_plugin.so"/>
+            <plugin name="joint_state_publisher" filename="libgazebo_ros_joint_state_publisher.so">
+                <robotNamespace>pelican</robotNamespace>
+                <jointName>
+                rod2tether_joint_roll_0, rod2tether_joint_pitch_0, rod2tether_joint_yaw_0,
+                rod2tether_joint_roll_1, rod2tether_joint_pitch_1, rod2tether_joint_yaw_1,
+                rod2tether_joint_roll_2, rod2tether_joint_pitch_2, rod2tether_joint_yaw_2,
+                rod2tether_joint_roll_3, rod2tether_joint_pitch_3, rod2tether_joint_yaw_3,
+                ugv2tether_joint_prismatic_0,
+                ugv2tether_joint_prismatic_1,
+                ugv2tether_joint_prismatic_2,
+                ugv2tether_joint_prismatic_3,
+                ugv2tether_joint_roll_0, ugv2tether_joint_pitch_0, ugv2tether_joint_yaw_0,
+                ugv2tether_joint_roll_1, ugv2tether_joint_pitch_1, ugv2tether_joint_yaw_1,
+                ugv2tether_joint_roll_2, ugv2tether_joint_pitch_2, ugv2tether_joint_yaw_2,
+                ugv2tether_joint_roll_3, ugv2tether_joint_pitch_3, ugv2tether_joint_yaw_3
+                </jointName>
+                <updateRate>1000</updateRate>
+                <alwaysOn>true</alwaysOn>
+            </plugin>
         </gazebo>
     </xacro:macro>

File: pyramid_description/ugv_description/urdf/mp_500/xacros/mp_500_fixed_wheel_left.xacro (robot description, xacro)
@@ -10,4 +10,12 @@
         <child link="${name}_link" />
     </joint>
+    <gazebo>
+        <plugin name="joint_state_publisher" filename="libgazebo_ros_joint_state_publisher.so">
+            <robotNamespace>pelican</robotNamespace>
+            <jointName>${namespace}/wheel_right_joint</jointName>
+            <updateRate>1000</updateRate>
+            <alwaysOn>true</alwaysOn>
+        </plugin>
+    </gazebo>
     <transmission name="tran_${number}">
         <type>transmission_interface/SimpleTransmission</type>

File: pyramid_description/ugv_description/urdf/mp_500/xacros/mp_500_fixed_wheel_right.xacro (robot description, xacro)
@@ -10,4 +10,12 @@
     <child link="${name}_link" />
    </joint>
+   <gazebo>
+       <plugin name="joint_state_publisher" filename="libgazebo_ros_joint_state_publisher.so">
+           <robotNamespace>pelican</robotNamespace>
+           <jointName>${namespace}/wheel_left_joint</jointName>
+           <updateRate>1000</updateRate>
+           <alwaysOn>true</alwaysOn>
+       </plugin>
+   </gazebo>
    <transmission name="tran_${number}">
     <type>transmission_interface/SimpleTransmission</type>

File: pyramid_description/ugv_description/urdf/mp_500/xacros/mp_500_gazebo.xacro (robot description, xacro)
@@ -38,4 +38,5 @@
   <gazebo>
     <plugin name="diff_dirve_controller" filename="libgazebo_ros_diff_drive.so">
+        <namespace>pelican</namespace>
         <alwaysOn>true</alwaysOn>
         <updateRate>100</updateRate>
@@ -48,14 +49,14 @@
         <commandTopic>${namespace}/cmd_vel</commandTopic>
         <rosDebugLevel>na</rosDebugLevel>
-        <odometryTopic>odom</odometryTopic>
-        <odometryFrame>odom</odometryFrame>
-        <robotBaseFrame>base_link</robotBaseFrame>
+        <odometryTopic>${namespace}/odom</odometryTopic>
+        <odometryFrame>${namespace}/odom</odometryFrame>
+        <robotBaseFrame>${namespace}/base_link</robotBaseFrame>
         <publishWheelTF>true</publishWheelTF>
-        <publishWheelJointState>true</publishWheelJointState>
+        <publishWheelJointState>false</publishWheelJointState>
         <wheelAcceleration>0</wheelAcceleration>
         <wheelTorque>200</wheelTorque>
         <odometrySource>world</odometrySource>
         <publishTf>1</publishTf>
-        <publishOdomTF>true</publishOdomTF>
+        <publishOdomTF>false</publishOdomTF>
     </plugin>
   </gazebo>

File: pyramid_description/ugv_description/urdf/mp_500/xacros/mp_500_tether_end.xacro (robot description, xacro)
@@ -51,4 +51,12 @@
             </inertial>
         </link>
+        <gazebo>
+            <plugin name="joint_state_publisher" filename="libgazebo_ros_joint_state_publisher.so">
+                <robotNamespace>pelican</robotNamespace>
+                <jointName>${namespace}/tether_end_joint</jointName>
+                <updateRate>1000</updateRate>
+                <alwaysOn>true</alwaysOn>
+            </plugin>
+        </gazebo>
     </xacro:macro>
 </robot>
