Commit message: Added massless rigid tether model

File: pyramid_description/tether_description/urdf/tether.xacro (robot description, xacro)
@@ -3,252 +3,399 @@
     <!--tether model-->
     <xacro:macro name="tether">
-        <!--tether fragment param--><!--tether fragment param--><!--joint dynamics--><!--link number--><!--tether_cylinder_joint--><!-- main-->
-                    <link name="tether_0/fragment_0_1">
+        <!--tether params--><!--virtual link params--><!--joint dynamics--><!-- main-->
+            <link name="tether_0">
             <visual>
                 <origin rpy="0 0 0" xyz="0 0 0"/>
                 <geometry>
-                    <sphere radius="0.02"/>
-                </geometry>
-            </visual>
-            <inertial>
-                <mass value="0.005"/>
-                <inertia ixx="1e-05" iyy="1e-05" izz="1e-05" ixy="0.0" ixz="0.0" iyz="0.0"/>
-            </inertial>
-        </link>
-        <gazebo reference="tether_0/fragment_0_1">
+                    <cylinder length="10.0" radius="0.005"/>
+                </geometry>
+            </visual>
+            <inertial>
+                <mass value="0.001"/>
+                <inertia ixx="0.001" iyy="0.001" izz="0.001" ixy="0.0" ixz="0.0" iyz="0.0"/>
+            </inertial>
+        </link>
+        <gazebo reference="tether_0">
             <material>Gazebo/Black</material>
         </gazebo>
-        <link name="tether_0/fragment_0_2">
+            <link name="virtual_link_uav2tether_1_0">
+            <inertial>
+                <mass value="0.001"/>
+                <inertia ixx="0.001" iyy="0.001" izz="0.001" ixy="0.0" ixz="0.0" iyz="0.0"/>
+            </inertial>
+        </link>
+        <link name="virtual_link_uav2tether_2_0">
+            <inertial>
+                <mass value="0.001"/>
+                <inertia ixx="0.001" iyy="0.001" izz="0.001" ixy="0.0" ixz="0.0" iyz="0.0"/>
+            </inertial>
+        </link>
+            <link name="virtual_link_ugv2tether_1_0">
+            <inertial>
+                <mass value="0.001"/>
+                <inertia ixx="0.001" iyy="0.001" izz="0.001" ixy="0.0" ixz="0.0" iyz="0.0"/>
+            </inertial>
+        </link>
+        <link name="virtual_link_ugv2tether_2_0">
+            <inertial>
+                <mass value="0.001"/>
+                <inertia ixx="0.001" iyy="0.001" izz="0.001" ixy="0.0" ixz="0.0" iyz="0.0"/>
+            </inertial>
+        </link>
+        <link name="virtual_link_ugv2tether_3_0">
+            <inertial>
+                <mass value="0.001"/>
+                <inertia ixx="0.001" iyy="0.001" izz="0.001" ixy="0.0" ixz="0.0" iyz="0.0"/>
+            </inertial>
+        </link>
+            <link name="rod_0">
+            <visual>
+                <origin rpy="0 0 0" xyz="0 0 0.1"/>
+                <geometry>
+                    <cylinder length="0.21" radius="0.01"/>
+                </geometry>
+            </visual>
+            <inertial>
+                <mass value="0.001"/>
+                <inertia ixx="0.001" iyy="0.001" izz="0.001" ixy="0.0" ixz="0.0" iyz="0.0"/>
+            </inertial>
+        </link>
+        <gazebo reference="rod_0">
+            <material>Gazebo/Orange</material>
+        </gazebo>
+        <!--uav => tether joint-->
+        <joint name="uav2rod_joint_0" type="fixed">
+            <parent link="${namespace}/base_link"/>
+            <child link="rod_0"/>
+                <origin rpy="0 ${pi/2} 0" xyz="0 0 0"/>
+        </joint>
+        <joint name="rod2tether_joint_roll_0" type="continuous">
+            <origin rpy="0 0 0" xyz="0 0 0.21"/>
+            <parent link="rod_0"/>
+            <child link="virtual_link_uav2tether_1_0"/>
+            <axis xyz="1 0 0" />
+            <dynamics damping="1" friction="1"/>
+        </joint>
+        <joint name="rod2tether_joint_pitch_0" type="continuous">
+            <origin rpy="0 0 0" xyz="0 0 0"/>
+            <parent link="virtual_link_uav2tether_1_0"/>
+            <child link="virtual_link_uav2tether_2_0"/>
+            <axis xyz="0 1 0" />
+            <dynamics damping="1" friction="1"/>
+        </joint>
+        <joint name="rod2tether_joint_yaw_0" type="continuous">
+            <origin rpy="0 0 0" xyz="0 0 0"/>
+            <parent link="virtual_link_uav2tether_2_0"/>
+            <child link="tether_0"/>
+            <axis xyz="0 0 1" />
+            <dynamics damping="1" friction="1"/>
+        </joint>
+            <joint name="ugv2tether_joint_prismatic_0" type="prismatic">
+            <origin rpy="0 0 0" xyz="0 0 10"/>
+            <parent link="tether_0"/>
+            <child link="virtual_link_ugv2tether_1_0"/>
+            <axis xyz="0 0 1" />
+            <dynamics damping="1" friction="1"/>
+            <limit effort="10000" lower="-5.0" upper="5.0" velocity="10.0"/>
+        </joint>
+        <joint name="ugv2tether_joint_roll_0" type="continuous">
+            <origin rpy="0 0 0" xyz="0 0 0"/>
+            <parent link="virtual_link_ugv2tether_1_0"/>
+            <child link="virtual_link_ugv2tether_2_0"/>
+            <axis xyz="1 0 0" />
+            <dynamics damping="1" friction="1"/>
+        </joint>
+        <joint name="ugv2tether_joint_pitch_0" type="continuous">
+            <origin rpy="0 0 0" xyz="0 0 0"/>
+            <parent link="virtual_link_ugv2tether_2_0"/>
+            <child link="virtual_link_ugv2tether_3_0"/>
+            <axis xyz="0 1 0" />
+            <dynamics damping="1" friction="1"/>
+        </joint>
+        <joint name="ugv2tether_joint_yaw_0" type="continuous">
+                <origin rpy="0 ${-pi/2} 0" xyz="0 0 0"/>
+            <axis xyz="0 0 1" />
+            <parent link="virtual_link_ugv2tether_3_0"/>
+            <child link="mp_500_0/tether_end"/>
+            <dynamics damping="1" friction="1"/>
+        </joint>
+            <link name="tether_1">
             <visual>
                 <origin rpy="0 0 0" xyz="0 0 0"/>
                 <geometry>
-                    <sphere radius="0.02"/>
-                </geometry>
-            </visual>
-            <inertial>
-                <mass value="0.005"/>
-                <inertia ixx="1e-05" iyy="1e-05" izz="1e-05" ixy="0.0" ixz="0.0" iyz="0.0"/>
-            </inertial>
-        </link>
-        <gazebo reference="tether_0/fragment_0_2">
+                    <cylinder length="10.0" radius="0.005"/>
+                </geometry>
+            </visual>
+            <inertial>
+                <mass value="0.001"/>
+                <inertia ixx="0.001" iyy="0.001" izz="0.001" ixy="0.0" ixz="0.0" iyz="0.0"/>
+            </inertial>
+        </link>
+        <gazebo reference="tether_1">
             <material>Gazebo/Black</material>
         </gazebo>
-        <link name="tether_0/fragment_0_3">
+            <link name="virtual_link_uav2tether_1_1">
+            <inertial>
+                <mass value="0.001"/>
+                <inertia ixx="0.001" iyy="0.001" izz="0.001" ixy="0.0" ixz="0.0" iyz="0.0"/>
+            </inertial>
+        </link>
+        <link name="virtual_link_uav2tether_2_1">
+            <inertial>
+                <mass value="0.001"/>
+                <inertia ixx="0.001" iyy="0.001" izz="0.001" ixy="0.0" ixz="0.0" iyz="0.0"/>
+            </inertial>
+        </link>
+            <link name="virtual_link_ugv2tether_1_1">
+            <inertial>
+                <mass value="0.001"/>
+                <inertia ixx="0.001" iyy="0.001" izz="0.001" ixy="0.0" ixz="0.0" iyz="0.0"/>
+            </inertial>
+        </link>
+        <link name="virtual_link_ugv2tether_2_1">
+            <inertial>
+                <mass value="0.001"/>
+                <inertia ixx="0.001" iyy="0.001" izz="0.001" ixy="0.0" ixz="0.0" iyz="0.0"/>
+            </inertial>
+        </link>
+        <link name="virtual_link_ugv2tether_3_1">
+            <inertial>
+                <mass value="0.001"/>
+                <inertia ixx="0.001" iyy="0.001" izz="0.001" ixy="0.0" ixz="0.0" iyz="0.0"/>
+            </inertial>
+        </link>
+            <link name="rod_1">
+            <visual>
+                <origin rpy="0 0 0" xyz="0 0 0.1"/>
+                <geometry>
+                    <cylinder length="0.21" radius="0.01"/>
+                </geometry>
+            </visual>
+            <inertial>
+                <mass value="0.001"/>
+                <inertia ixx="0.001" iyy="0.001" izz="0.001" ixy="0.0" ixz="0.0" iyz="0.0"/>
+            </inertial>
+        </link>
+        <gazebo reference="rod_1">
+            <material>Gazebo/Orange</material>
+        </gazebo>
+        <!--uav => tether joint-->
+        <joint name="uav2rod_joint_1" type="fixed">
+            <parent link="${namespace}/base_link"/>
+            <child link="rod_1"/>
+                <origin rpy="${pi/2} 0 0" xyz="0 0 0"/>
+        </joint>
+        <joint name="rod2tether_joint_roll_1" type="continuous">
+            <origin rpy="0 0 0" xyz="0 0 0.21"/>
+            <parent link="rod_1"/>
+            <child link="virtual_link_uav2tether_1_1"/>
+            <axis xyz="1 0 0" />
+            <dynamics damping="1" friction="1"/>
+        </joint>
+        <joint name="rod2tether_joint_pitch_1" type="continuous">
+            <origin rpy="0 0 0" xyz="0 0 0"/>
+            <parent link="virtual_link_uav2tether_1_1"/>
+            <child link="virtual_link_uav2tether_2_1"/>
+            <axis xyz="0 1 0" />
+            <dynamics damping="1" friction="1"/>
+        </joint>
+        <joint name="rod2tether_joint_yaw_1" type="continuous">
+            <origin rpy="0 0 0" xyz="0 0 0"/>
+            <parent link="virtual_link_uav2tether_2_1"/>
+            <child link="tether_1"/>
+            <axis xyz="0 0 1" />
+            <dynamics damping="1" friction="1"/>
+        </joint>
+            <joint name="ugv2tether_joint_prismatic_1" type="prismatic">
+            <origin rpy="0 0 0" xyz="0 0 10"/>
+            <parent link="tether_1"/>
+            <child link="virtual_link_ugv2tether_1_1"/>
+            <axis xyz="0 0 1" />
+            <dynamics damping="1" friction="1"/>
+            <limit effort="10000" lower="-5.0" upper="5.0" velocity="10.0"/>
+        </joint>
+        <joint name="ugv2tether_joint_roll_1" type="continuous">
+            <origin rpy="0 0 0" xyz="0 0 0"/>
+            <parent link="virtual_link_ugv2tether_1_1"/>
+            <child link="virtual_link_ugv2tether_2_1"/>
+            <axis xyz="1 0 0" />
+            <dynamics damping="1" friction="1"/>
+        </joint>
+        <joint name="ugv2tether_joint_pitch_1" type="continuous">
+            <origin rpy="0 0 0" xyz="0 0 0"/>
+            <parent link="virtual_link_ugv2tether_2_1"/>
+            <child link="virtual_link_ugv2tether_3_1"/>
+            <axis xyz="0 1 0" />
+            <dynamics damping="1" friction="1"/>
+        </joint>
+        <joint name="ugv2tether_joint_yaw_1" type="continuous">
+                <origin rpy="${-pi/2} 0 0" xyz="0 0 0"/>
+            <axis xyz="0 0 1" />
+            <parent link="virtual_link_ugv2tether_3_1"/>
+            <child link="mp_500_1/tether_end"/>
+            <dynamics damping="1" friction="1"/>
+        </joint>
+            <link name="tether_2">
             <visual>
                 <origin rpy="0 0 0" xyz="0 0 0"/>
                 <geometry>
-                    <sphere radius="0.02"/>
-                </geometry>
-            </visual>
-            <inertial>
-                <mass value="0.005"/>
-                <inertia ixx="1e-05" iyy="1e-05" izz="1e-05" ixy="0.0" ixz="0.0" iyz="0.0"/>
-            </inertial>
-        </link>
-        <gazebo reference="tether_0/fragment_0_3">
+                    <cylinder length="10.0" radius="0.005"/>
+                </geometry>
+            </visual>
+            <inertial>
+                <mass value="0.001"/>
+                <inertia ixx="0.001" iyy="0.001" izz="0.001" ixy="0.0" ixz="0.0" iyz="0.0"/>
+            </inertial>
+        </link>
+        <gazebo reference="tether_2">
             <material>Gazebo/Black</material>
         </gazebo>
-                    <link name="tether_0/fragment_1_1">
+            <link name="virtual_link_uav2tether_1_2">
+            <inertial>
+                <mass value="0.001"/>
+                <inertia ixx="0.001" iyy="0.001" izz="0.001" ixy="0.0" ixz="0.0" iyz="0.0"/>
+            </inertial>
+        </link>
+        <link name="virtual_link_uav2tether_2_2">
+            <inertial>
+                <mass value="0.001"/>
+                <inertia ixx="0.001" iyy="0.001" izz="0.001" ixy="0.0" ixz="0.0" iyz="0.0"/>
+            </inertial>
+        </link>
+            <link name="virtual_link_ugv2tether_1_2">
+            <inertial>
+                <mass value="0.001"/>
+                <inertia ixx="0.001" iyy="0.001" izz="0.001" ixy="0.0" ixz="0.0" iyz="0.0"/>
+            </inertial>
+        </link>
+        <link name="virtual_link_ugv2tether_2_2">
+            <inertial>
+                <mass value="0.001"/>
+                <inertia ixx="0.001" iyy="0.001" izz="0.001" ixy="0.0" ixz="0.0" iyz="0.0"/>
+            </inertial>
+        </link>
+        <link name="virtual_link_ugv2tether_3_2">
+            <inertial>
+                <mass value="0.001"/>
+                <inertia ixx="0.001" iyy="0.001" izz="0.001" ixy="0.0" ixz="0.0" iyz="0.0"/>
+            </inertial>
+        </link>
+            <link name="rod_2">
+            <visual>
+                <origin rpy="0 0 0" xyz="0 0 0.1"/>
+                <geometry>
+                    <cylinder length="0.21" radius="0.01"/>
+                </geometry>
+            </visual>
+            <inertial>
+                <mass value="0.001"/>
+                <inertia ixx="0.001" iyy="0.001" izz="0.001" ixy="0.0" ixz="0.0" iyz="0.0"/>
+            </inertial>
+        </link>
+        <gazebo reference="rod_2">
+            <material>Gazebo/Orange</material>
+        </gazebo>
+        <!--uav => tether joint-->
+        <joint name="uav2rod_joint_2" type="fixed">
+            <parent link="${namespace}/base_link"/>
+            <child link="rod_2"/>
+                <origin rpy="0 ${-pi/2} 0" xyz="0 0 0"/>
+        </joint>
+        <joint name="rod2tether_joint_roll_2" type="continuous">
+            <origin rpy="0 0 0" xyz="0 0 0.21"/>
+            <parent link="rod_2"/>
+            <child link="virtual_link_uav2tether_1_2"/>
+            <axis xyz="1 0 0" />
+            <dynamics damping="1" friction="1"/>
+        </joint>
+        <joint name="rod2tether_joint_pitch_2" type="continuous">
+            <origin rpy="0 0 0" xyz="0 0 0"/>
+            <parent link="virtual_link_uav2tether_1_2"/>
+            <child link="virtual_link_uav2tether_2_2"/>
+            <axis xyz="0 1 0" />
+            <dynamics damping="1" friction="1"/>
+        </joint>
+        <joint name="rod2tether_joint_yaw_2" type="continuous">
+            <origin rpy="0 0 0" xyz="0 0 0"/>
+            <parent link="virtual_link_uav2tether_2_2"/>
+            <child link="tether_2"/>
+            <axis xyz="0 0 1" />
+            <dynamics damping="1" friction="1"/>
+        </joint>
+            <joint name="ugv2tether_joint_prismatic_2" type="prismatic">
+            <origin rpy="0 0 0" xyz="0 0 10"/>
+            <parent link="tether_2"/>
+            <child link="virtual_link_ugv2tether_1_2"/>
+            <axis xyz="0 0 1" />
+            <dynamics damping="1" friction="1"/>
+            <limit effort="10000" lower="-5.0" upper="5.0" velocity="10.0"/>
+        </joint>
+        <joint name="ugv2tether_joint_roll_2" type="continuous">
+            <origin rpy="0 0 0" xyz="0 0 0"/>
+            <parent link="virtual_link_ugv2tether_1_2"/>
+            <child link="virtual_link_ugv2tether_2_2"/>
+            <axis xyz="1 0 0" />
+            <dynamics damping="1" friction="1"/>
+        </joint>
+        <joint name="ugv2tether_joint_pitch_2" type="continuous">
+            <origin rpy="0 0 0" xyz="0 0 0"/>
+            <parent link="virtual_link_ugv2tether_2_2"/>
+            <child link="virtual_link_ugv2tether_3_2"/>
+            <axis xyz="0 1 0" />
+            <dynamics damping="1" friction="1"/>
+        </joint>
+        <joint name="ugv2tether_joint_yaw_2" type="continuous">
+                <origin rpy="0 ${pi/2} 0" xyz="0 0 0"/>
+            <axis xyz="0 0 1" />
+            <parent link="virtual_link_ugv2tether_3_2"/>
+            <child link="mp_500_2/tether_end"/>
+            <dynamics damping="1" friction="1"/>
+        </joint>
+            <link name="tether_3">
             <visual>
                 <origin rpy="0 0 0" xyz="0 0 0"/>
                 <geometry>
-                    <sphere radius="0.02"/>
-                </geometry>
-            </visual>
-            <inertial>
-                <mass value="0.05"/>
-                <inertia ixx="2e-05" iyy="2e-05" izz="2e-05" ixy="0.0" ixz="0.0" iyz="0.0"/>
-            </inertial>
-        </link>
-        <gazebo reference="tether_0/fragment_1_1">
-            <material>Gazebo/Red</material>
-        </gazebo>
-        <link name="tether_0/fragment_1_2">
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
Commit message: tether_end

File: pyramid_description/tether_description/urdf/tether.xacro (robot description, xacro)
@@ -4,4 +4,70 @@
     <xacro:macro name="tether">
         <!--tether params--><!--virtual link params--><!--actuated joint dynamics--><!--passive joint dynamics--><!-- main-->
+        <!-- ================================================================== -->
+  <!-- ======================== PYRAMID ROBOTICS =========================-->
+  <!-- ================================================================== -->
+    <!-- front_right -->
+    <xacro:tether_end
+        robot_namespace="${namespace}"
+        x="0.2" y="-0.2" z="0.1"
+        tether_number="0"
+        suffix="front_right_upper"
+        color="Orange">
+    </xacro:tether_end>
+    <xacro:tether_end
+        robot_namespace="${namespace}"
+        x="0.2" y="-0.2" z="-0.1"
+        tether_number="1"
+        suffix="front_right_lower"
+        color="Blue">
+    </xacro:tether_end>
+    <!-- front_left -->
+    <xacro:tether_end
+        robot_namespace="${namespace}"
+        x="0.2" y="0.2" z="0.1"
+        tether_number="2"
+        suffix="front_left_upper"
+        color="Green">
+    </xacro:tether_end>
+    <xacro:tether_end
+        robot_namespace="${namespace}"
+        x="0.2" y="0.2" z="-0.1"
+        tether_number="3"
+        suffix="front_left_lower"
+        color="Red">
+    </xacro:tether_end>
+    <!-- back right -->
+    <xacro:tether_end
+        robot_namespace="${namespace}"
+        x="-0.2" y="-0.2" z="0.1"
+        tether_number="4"
+        suffix="back_right_upper"
+        color="Red">
+    </xacro:tether_end>
+    <xacro:tether_end
+        robot_namespace="${namespace}"
+        x="-0.2" y="-0.2" z="-0.1"
+        tether_number="5"
+        suffix="back_right_lower"
+        color="Green">
+    </xacro:tether_end>
+    <!-- back left -->
+    <xacro:tether_end
+        robot_namespace="${namespace}"
+        x="-0.2" y="0.2" z="0.1"
+        tether_number="6"
+        suffix="back_left_upper"
+        color="Blue">
+    </xacro:tether_end>
+    <xacro:tether_end
+        robot_namespace="${namespace}"
+        x="-0.2" y="0.2" z="-0.1"
+        tether_number="7"
+        suffix="back_left_lower"
+        color="Orange">
+    </xacro:tether_end>
+  <!-- ================================================================== -->
+  <!-- ======================== PYRAMID ROBOTICS =========================-->
+  <!-- ================================================================== -->
             <link name="tether_0">
             <visual>

File: pyramid_description/uav_description/urdf/pyramid_multirotor_base.xacro (robot description, xacro)
@@ -134,3 +134,33 @@
     </gazebo>
   </xacro:macro>
+  <!-- ================================================================== -->
+  <!-- ======================== PYRAMID ROBOTICS =========================-->
+  <!-- ================================================================== -->
+    <!-- Tether attached point -->
+    <xacro:macro name="tether_end" params="robot_namespace x y z tether_number suffix color">
+        <joint name="${robot_namespace}/tether_joint_${tether_number}" type="fixed">
+            <origin xyz="${x} ${y} ${z}" rpy="0 0 0" />
+            <parent link="${robot_namespace}/base_link" />
+            <child link="${robot_namespace}/tether_${tether_number}" />
+        </joint>
+        <link name="${robot_namespace}/tether_${tether_number}">
+            <inertial>
+                <mass value="0.01"/>
+                <inertia ixx="0.01" iyy="0.01" izz="0.01" ixy="0.0" ixz="0.0" iyz="0.0"/>
+                <origin xyz="0 0 0" rpy="0 0 0"/>
+            </inertial>
+            <visual>
+                <origin rpy="0 0 0" xyz="0 0 0"/>
+                <geometry>
+                    <sphere radius="0.01"/>
+                </geometry>
+            </visual>
+        </link>
+        <gazebo reference="${robot_namespace}/tether_${tether_number}">
+            <material>Gazebo/${color}</material>
+        </gazebo>
+    </xacro:macro>
+    <!-- ================================================================== -->
+    <!-- ======================== PYRAMID ROBOTICS =========================-->
+    <!-- ================================================================== -->
 </robot>
