Commit message: Added material color

File: pyramid_description/urdf/pyramid_component_snippets.xacro (robot description, xacro)
@@ -18,4 +18,16 @@
 <robot xmlns:xacro="http://ros.org/wiki/xacro">
   <xacro:property name="pi" value="3.14159265359" />
+  <material name="Red">
+      <color rgba="1.0 0.0 0.0 2.0"/>
+  </material>
+  <material name="Green">
+      <color rgba="0.0 1.0 0.0 2.0"/>
+  </material>
+  <material name="Blue">
+      <color rgba="0.0 0.0 1.0 2.0"/>
+  </material>
+  <material name="Orange">
+      <color rgba="1.0 0.64 0.0 1.0"/>
+  </material>
   <!-- Macro to add logging to a bag file. -->
   <xacro:macro name="bag_plugin_macro"

File: pyramid_description/urdf/pyramid_multirotor_base.xacro (robot description, xacro)
@@ -156,4 +156,5 @@
                     <sphere radius="0.03"/>
                 </geometry>
+                <material name="${color}"/>
             </visual>
             <collision>

File: pyramid_description/urdf/pyramid_winch.xacro (robot description, xacro)
@@ -1,4 +1,16 @@
 <?xml version="1.0" encoding="utf-8"?>
 <robot name="winch" xmlns:xacro="http://ros.org/wiki/xacro">
+    <material name="Red">
+        <color rgba="1.0 0.0 0.0 2.0"/>
+    </material>
+    <material name="Green">
+        <color rgba="0.0 1.0 0.0 2.0"/>
+    </material>
+    <material name="Blue">
+        <color rgba="0.0 0.0 1.0 2.0"/>
+    </material>
+    <material name="Orange">
+        <color rgba="1.0 0.64 0.0 1.0"/>
+    </material>
     <xacro:macro name="winch" params="x y z winch_number suffix color">
         <joint name="winch_joint_${winch_number}" type="fixed">
@@ -18,4 +30,5 @@
                     <box size="0.1 0.1 0.1"/>
                 </geometry>
+                <material name="${color}"/>
             </visual>
         </link>
