Commit message: backup

File: pyramid_description/urdf/pyramid_winch.xacro (robot description, xacro)
@@ -1,4 +1,5 @@
 <?xml version="1.0" encoding="utf-8"?>
 <robot name="winch" xmlns:xacro="http://ros.org/wiki/xacro">
+    <xacro:property name="namespace" value="$(arg namespace)" />
     <material name="Red">
         <color rgba="1.0 0.0 0.0 2.0"/>
@@ -13,5 +14,5 @@
         <color rgba="1.0 0.64 0.0 1.0"/>
     </material>
-    <xacro:macro name="winch" params="x y z winch_number suffix color">
+    <xacro:macro name="winch" params="robot_namespace x y z winch_number suffix color">
         <joint name="winch_joint_${winch_number}" type="fixed">
             <origin xyz="${x} ${y} ${z}" rpy="0 0 0" />
@@ -35,5 +36,7 @@
         <gazebo>
             <plugin filename="libgazebo_winch_plugin.so" name="winch_plugin">
+                <robotNamespace>${robot_namespace}</robotNamespace>
                 <linkName>winch_${winch_number}</linkName>
+                <winchNumber>${winch_number}</winchNumber>
             </plugin>
         </gazebo>
@@ -44,16 +47,19 @@
     <link name="world"/>
     <xacro:winch
-        x="5.0" y="-5.0" z="0"
+        robot_namespace="${namespace}"
+        x="5.0" y="5.0" z="0.05"
         winch_number="0"
         suffix="front_right"
-        color="Red">
-    </xacro:winch>
-    <xacro:winch
-        x="5.0" y="5.0" z="0"
-        winch_number="1"
-        suffix="front_left"
         color="Orange">
     </xacro:winch>
     <xacro:winch
+        robot_namespace="${namespace}"
+        x="-5.0" y="5.0" z="0"
+        winch_number="1"
+        suffix="front_left"
+        color="Green">
+    </xacro:winch>
+    <xacro:winch
+        robot_namespace="${namespace}"
         x="-5.0" y="-5.0" z="0"
         winch_number="2"
@@ -62,8 +68,9 @@
     </xacro:winch>
     <xacro:winch
-        x="-5.0" y="5.0" z="0"
+        robot_namespace="${namespace}"
+        x="5.0" y="-5.0" z="0"
         winch_number="3"
         suffix="back_left"
-        color="Green">
+        color="Red">
     </xacro:winch>
 </robot>
