Commit message: modify

File: pyramid_description/urdf/pyramid_multirotor_base.xacro (robot description, xacro)
@@ -43,6 +43,6 @@
         <link name="${robot_namespace}/tether_${tether_number}">
             <inertial>
-                <mass value="0.001"/>
-                <inertia ixx="0.001" iyy="0.001" izz="0.001" ixy="0.0" ixz="0.0" iyz="0.0"/>
+                <mass value="0.01"/>
+                <inertia ixx="0.01" iyy="0.01" izz="0.01" ixy="0.0" ixz="0.0" iyz="0.0"/>
                 <origin xyz="0 0 0" rpy="0 0 0"/>
             </inertial>
@@ -53,4 +53,10 @@
                 </geometry>
             </visual>
+            <collision>
+                <origin xyz="0 0 0" rpy="0 0 0" />
+                <geometry>
+                    <sphere radius="0.01"/>
+                </geometry>
+            </collision>
         </link>
         <gazebo reference="${robot_namespace}/tether_${tether_number}">
@@ -103,4 +109,5 @@
       <!--plugin filename="libgazebo_disturbance_plugin.so" name="disturbance_plugin" /-->
       <!--plugin filename="libgazebo_external_force_plugin.so" name="external_force_plugin" /-->
+      <plugin filename="libgazebo_psuedo_tether_plugin.so" name="psuedo_tether_plugin" />
     </gazebo>
   </xacro:macro>

File: pyramid_description/urdf/pyramid_pelican.xacro (robot description, xacro)
@@ -51,5 +51,5 @@
   <!-- ================================================================== -->
     <!-- front_right -->
-    <xacro:tether_end
+    <!-- <xacro:tether_end
         robot_namespace="${namespace}"
         x="0.2" y="-0.2" z="0.1"
@@ -57,5 +57,32 @@
         suffix="front_right_upper"
         color="Orange">
-    </xacro:tether_end>
+    </xacro:tether_end> -->
+    <joint name="${namespace}/tether_joint_0" type="fixed">
+        <origin xyz="0.2 -0.2 0.1" rpy="0 0 0" />
+        <parent link="${namespace}/base_link" />
+        <child link="${namespace}/tether_0" />
+    </joint>
+    <link name="${namespace}/tether_0">
+        <inertial>
+            <mass value="0.01"/>
+            <inertia ixx="0.01" iyy="0.01" izz="0.01" ixy="0.0" ixz="0.0" iyz="0.0"/>
+            <origin xyz="0 0 0" rpy="0 0 0"/>
+        </inertial>
+        <visual>
+            <origin rpy="0 0 0" xyz="0 0 0"/>
+            <geometry>
+                <sphere radius="0.01"/>
+            </geometry>
+        </visual>
+        <collision>
+            <origin xyz="0 0 0" rpy="0 0 0" />
+            <geometry>
+                <sphere radius="0.01"/>
+            </geometry>
+        </collision>
+    </link>
+    <gazebo reference="${namespace}/tether_0">
+        <material>Gazebo/Orange</material>
+    </gazebo>
     <xacro:tether_end
         robot_namespace="${namespace}"

Commit message: add

File: pyramid_description/urdf/pyramid_multirotor_base.xacro (robot description, xacro)
@@ -31,40 +31,4 @@
     </inertial>
   </xacro:macro>
-  <!-- ================================================================== -->
-  <!-- ======================== PYRAMID ROBOTICS =========================-->
-  <!-- ================================================================== -->
-    <!-- Tether attached point -->
-    <xacro:macro name="tether_end" params="robot_namespace x y z tether_number suffix color">
-        <joint name="${robot_namespace}/tether_joint_${tether_number}" type="fixed">
-            <origin xyz="${x} ${y} ${z}" rpy="0 0 0" />
-            <parent link="${robot_namespace}/base_link" />
-            <child link="${robot_namespace}/tether_${tether_number}" />
-        </joint>
-        <link name="${robot_namespace}/tether_${tether_number}">
-            <inertial>
-                <mass value="0.01"/>
-                <inertia ixx="0.01" iyy="0.01" izz="0.01" ixy="0.0" ixz="0.0" iyz="0.0"/>
-                <origin xyz="0 0 0" rpy="0 0 0"/>
-            </inertial>
-            <visual>
-                <origin rpy="0 0 0" xyz="0 0 0"/>
-                <geometry>
-                    <sphere radius="0.01"/>
-                </geometry>
-            </visual>
-            <collision>
-                <origin xyz="0 0 0" rpy="0 0 0" />
-                <geometry>
-                    <sphere radius="0.01"/>
-                </geometry>
-            </collision>
-        </link>
-        <gazebo reference="${robot_namespace}/tether_${tether_number}">
-            <material>Gazebo/${color}</material>
-        </gazebo>
-    </xacro:macro>
-    <!-- ================================================================== -->
-    <!-- ======================== PYRAMID ROBOTICS =========================-->
-    <!-- ================================================================== -->
   <!-- Main multirotor link -->
   <xacro:macro name="multirotor_base_macro"
@@ -171,3 +135,33 @@
     </gazebo>
   </xacro:macro>
+  <!-- ================================================================== -->
+  <!-- ======================== PYRAMID ROBOTICS =========================-->
+  <!-- ================================================================== -->
+    <!-- Tether attached point -->
+    <xacro:macro name="tether_end" params="robot_namespace x y z tether_number suffix color">
+        <joint name="${robot_namespace}/tether_joint_${tether_number}" type="fixed">
+            <origin xyz="${x} ${y} ${z}" rpy="0 0 0" />
+            <parent link="${robot_namespace}/base_link" />
+            <child link="${robot_namespace}/tether_${tether_number}" />
+        </joint>
+        <link name="${robot_namespace}/tether_${tether_number}">
+            <inertial>
+                <mass value="0.01"/>
+                <inertia ixx="0.01" iyy="0.01" izz="0.01" ixy="0.0" ixz="0.0" iyz="0.0"/>
+                <origin xyz="0 0 0" rpy="0 0 0"/>
+            </inertial>
+            <visual>
+                <origin rpy="0 0 0" xyz="0 0 0"/>
+                <geometry>
+                    <sphere radius="0.01"/>
+                </geometry>
+            </visual>
+        </link>
+        <gazebo reference="${robot_namespace}/tether_${tether_number}">
+            <material>Gazebo/${color}</material>
+        </gazebo>
+    </xacro:macro>
+    <!-- ================================================================== -->
+    <!-- ======================== PYRAMID ROBOTICS =========================-->
+    <!-- ================================================================== -->
 </robot>

File: pyramid_description/urdf/pyramid_pelican.xacro (robot description, xacro)
@@ -47,98 +47,5 @@
   <!-- Included URDF Files -->
   <xacro:include filename="$(find pyramid_description)/urdf/pyramid_multirotor_base.xacro" />
-  <!-- ================================================================== -->
-  <!-- ======================== PYRAMID ROBOTICS =========================-->
-  <!-- ================================================================== -->
-    <!-- front_right -->
-    <!-- <xacro:tether_end
-        robot_namespace="${namespace}"
-        x="0.2" y="-0.2" z="0.1"
-        tether_number="0"
-        suffix="front_right_upper"
-        color="Orange">
-    </xacro:tether_end> -->
-    <joint name="${namespace}/tether_joint_0" type="fixed">
-        <origin xyz="0.2 -0.2 0.1" rpy="0 0 0" />
-        <parent link="${namespace}/base_link" />
-        <child link="${namespace}/tether_0" />
-    </joint>
-    <link name="${namespace}/tether_0">
-        <inertial>
-            <mass value="0.01"/>
-            <inertia ixx="0.01" iyy="0.01" izz="0.01" ixy="0.0" ixz="0.0" iyz="0.0"/>
-            <origin xyz="0 0 0" rpy="0 0 0"/>
-        </inertial>
-        <visual>
-            <origin rpy="0 0 0" xyz="0 0 0"/>
-            <geometry>
-                <sphere radius="0.01"/>
-            </geometry>
-        </visual>
-        <collision>
-            <origin xyz="0 0 0" rpy="0 0 0" />
-            <geometry>
-                <sphere radius="0.01"/>
-            </geometry>
-        </collision>
-    </link>
-    <gazebo reference="${namespace}/tether_0">
-        <material>Gazebo/Orange</material>
-    </gazebo>
-    <xacro:tether_end
-        robot_namespace="${namespace}"
-        x="0.2" y="-0.2" z="-0.1"
-        tether_number="1"
-        suffix="front_right_lower"
-        color="Blue">
-    </xacro:tether_end>
-    <!-- front_left -->
-    <xacro:tether_end
-        robot_namespace="${namespace}"
-        x="0.2" y="0.2" z="0.1"
-        tether_number="2"
-        suffix="front_left_upper"
-        color="Green">
-    </xacro:tether_end>
-    <xacro:tether_end
-        robot_namespace="${namespace}"
-        x="0.2" y="0.2" z="-0.1"
-        tether_number="3"
-        suffix="front_left_lower"
-        color="Red">
-    </xacro:tether_end>
-    <!-- back right -->
-    <xacro:tether_end
-        robot_namespace="${namespace}"
-        x="-0.2" y="-0.2" z="0.1"
-        tether_number="4"
-        suffix="back_right_upper"
-        color="Red">
-    </xacro:tether_end>
-    <xacro:tether_end
-        robot_namespace="${namespace}"
-        x="-0.2" y="-0.2" z="-0.1"
-        tether_number="5"
-        suffix="back_right_lower"
-        color="Green">
-    </xacro:tether_end>
-    <!-- back left -->
-    <xacro:tether_end
-        robot_namespace="${namespace}"
-        x="-0.2" y="0.2" z="0.1"
-        tether_number="6"
-        suffix="back_left_upper"
-        color="Blue">
-    </xacro:tether_end>
-    <xacro:tether_end
-        robot_namespace="${namespace}"
-        x="-0.2" y="0.2" z="-0.1"
-        tether_number="7"
-        suffix="back_left_lower"
-        color="Orange">
-    </xacro:tether_end>
-  <!-- ================================================================== -->
-  <!-- ======================== PYRAMID ROBOTICS =========================-->
-  <!-- ================================================================== -->
-  <!-- Instantiate multirotor_base_macro once -->
+    <!-- Instantiate multirotor_base_macro once -->
   <xacro:multirotor_base_macro
     robot_namespace="${namespace}"
@@ -235,3 +142,69 @@
     <xacro:insert_block name="rotor_inertia" />
   </xacro:vertical_rotor>
+  <!-- ================================================================== -->
+  <!-- ======================== PYRAMID ROBOTICS =========================-->
+  <!-- ================================================================== -->
+    <!-- front_right -->
+    <xacro:tether_end
+        robot_namespace="${namespace}"
+        x="0.2" y="-0.2" z="0.1"
+        tether_number="0"
+        suffix="front_right_upper"
+        color="Orange">
+    </xacro:tether_end>
+    <xacro:tether_end
+        robot_namespace="${namespace}"
+        x="0.2" y="-0.2" z="-0.1"
+        tether_number="1"
+        suffix="front_right_lower"
+        color="Blue">
+    </xacro:tether_end>
+    <!-- front_left -->
+    <xacro:tether_end
+        robot_namespace="${namespace}"
+        x="0.2" y="0.2" z="0.1"
+        tether_number="2"
+        suffix="front_left_upper"
+        color="Green">
+    </xacro:tether_end>
+    <xacro:tether_end
+        robot_namespace="${namespace}"
+        x="0.2" y="0.2" z="-0.1"
+        tether_number="3"
+        suffix="front_left_lower"
+        color="Red">
+    </xacro:tether_end>
+    <!-- back right -->
+    <xacro:tether_end
+        robot_namespace="${namespace}"
+        x="-0.2" y="-0.2" z="0.1"
+        tether_number="4"
+        suffix="back_right_upper"
+        color="Red">
+    </xacro:tether_end>
+    <xacro:tether_end
+        robot_namespace="${namespace}"
+        x="-0.2" y="-0.2" z="-0.1"
+        tether_number="5"
+        suffix="back_right_lower"
+        color="Green">
+    </xacro:tether_end>
+    <!-- back left -->
+    <xacro:tether_end
+        robot_namespace="${namespace}"
+        x="-0.2" y="0.2" z="0.1"
+        tether_number="6"
+        suffix="back_left_upper"
+        color="Blue">
+    </xacro:tether_end>
+    <xacro:tether_end
+        robot_namespace="${namespace}"
+        x="-0.2" y="0.2" z="-0.1"
+        tether_number="7"
+        suffix="back_left_lower"
+        color="Orange">
+    </xacro:tether_end>
+  <!-- ================================================================== -->
+  <!-- ======================== PYRAMID ROBOTICS =========================-->
+  <!-- ================================================================== -->
 </robot>

Commit message: 4 tethers -> 8 tethers & 4DoF -> 6DoF

File: pyramid_description/urdf/pyramid_multirotor_base.xacro (robot description, xacro)
@@ -72,6 +72,6 @@
       </plugin>
       <!--plugin filename="libgazebo_disturbance_plugin.so" name="disturbance_plugin" /-->
-      <!--plugin filename="libgazebo_external_force_plugin.so" name="external_force_plugin" /-->
-      <plugin filename="libgazebo_psuedo_tether_plugin.so" name="psuedo_tether_plugin" />
+      <plugin filename="libgazebo_external_force_plugin.so" name="external_force_plugin" />
+      <!-- <plugin filename="libgazebo_psuedo_tether_plugin.so" name="psuedo_tether_plugin" /> -->
     </gazebo>
   </xacro:macro>
@@ -140,10 +140,10 @@
     <!-- Tether attached point -->
     <xacro:macro name="tether_end" params="robot_namespace x y z tether_number suffix color">
-        <joint name="${robot_namespace}/tether_joint_${tether_number}" type="fixed">
+        <joint name="${robot_namespace}/tether_joint_${tether_number}" type="continuous">
             <origin xyz="${x} ${y} ${z}" rpy="0 0 0" />
             <parent link="${robot_namespace}/base_link" />
-            <child link="${robot_namespace}/tether_${tether_number}" />
+            <child link="${robot_namespace}/tether_end_${tether_number}" />
         </joint>
-        <link name="${robot_namespace}/tether_${tether_number}">
+        <link name="${robot_namespace}/tether_end_${tether_number}">
             <inertial>
                 <mass value="0.01"/>
@@ -157,6 +157,12 @@
                 </geometry>
             </visual>
+            <collision>
+                <origin xyz="0 0 0" rpy="0 0 0" />
+                <geometry>
+                    <sphere radius="0.01"/>
+                </geometry>
+            </collision>
         </link>
-        <gazebo reference="${robot_namespace}/tether_${tether_number}">
+        <gazebo reference="${robot_namespace}/tether_end_${tether_number}">
             <material>Gazebo/${color}</material>
         </gazebo>

File: pyramid_description/urdf/pyramid_pelican.xacro (robot description, xacro)
@@ -37,4 +37,6 @@
   <xacro:property name="rotor_drag_coefficient" value="8.06428e-05" />
   <xacro:property name="rolling_moment_coefficient" value="0.000001" />
+  <xacro:property name="tether_attached_pos_horizontal" value="0.4" /> <!-- [m] -->
+  <xacro:property name="tether_attached_pos_vertical" value="0.15" /> <!-- [m] -->
   <!-- Property Blocks -->
   <xacro:property name="body_inertia">
@@ -145,8 +147,9 @@
   <!-- ======================== PYRAMID ROBOTICS =========================-->
   <!-- ================================================================== -->
-    <!-- front_right -->
-    <xacro:tether_end
-        robot_namespace="${namespace}"
-        x="0.2" y="-0.2" z="0.1"
+    <!-- <xacro:tether_end
+        robot_namespace="${namespace}"
+        x="${tether_attached_pos_horizontal}"
+        y="-${tether_attached_pos_horizontal}"
+        z="${tether_attached_pos_vertical}"
         tether_number="0"
         suffix="front_right_upper"
@@ -155,13 +158,16 @@
     <xacro:tether_end
         robot_namespace="${namespace}"
-        x="0.2" y="-0.2" z="-0.1"
+        x="${tether_attached_pos_horizontal}"
+        y="-${tether_attached_pos_horizontal}"
+        z="-${tether_attached_pos_vertical}"
         tether_number="1"
         suffix="front_right_lower"
         color="Blue">
     </xacro:tether_end>
-    <!-- front_left -->
-    <xacro:tether_end
-        robot_namespace="${namespace}"
-        x="0.2" y="0.2" z="0.1"
+    <xacro:tether_end
+        robot_namespace="${namespace}"
+        x="${tether_attached_pos_horizontal}"
+        y="${tether_attached_pos_horizontal}"
+        z="${tether_attached_pos_vertical}"
         tether_number="2"
         suffix="front_left_upper"
@@ -170,13 +176,16 @@
     <xacro:tether_end
         robot_namespace="${namespace}"
-        x="0.2" y="0.2" z="-0.1"
+        x="${tether_attached_pos_horizontal}"
+        y="${tether_attached_pos_horizontal}"
+        z="-${tether_attached_pos_vertical}"
         tether_number="3"
         suffix="front_left_lower"
         color="Red">
     </xacro:tether_end>
-    <!-- back right -->
-    <xacro:tether_end
-        robot_namespace="${namespace}"
-        x="-0.2" y="-0.2" z="0.1"
+    <xacro:tether_end
+        robot_namespace="${namespace}"
+        x="-${tether_attached_pos_horizontal}"
+        y="-${tether_attached_pos_horizontal}"
+        z="${tether_attached_pos_vertical}"
         tether_number="4"
         suffix="back_right_upper"
@@ -185,13 +194,16 @@
     <xacro:tether_end
         robot_namespace="${namespace}"
-        x="-0.2" y="-0.2" z="-0.1"
+        x="-${tether_attached_pos_horizontal}"
+        y="-${tether_attached_pos_horizontal}"
+        z="-${tether_attached_pos_vertical}"
         tether_number="5"
         suffix="back_right_lower"
         color="Green">
     </xacro:tether_end>
-    <!-- back left -->
-    <xacro:tether_end
-        robot_namespace="${namespace}"
-        x="-0.2" y="0.2" z="0.1"
+    <xacro:tether_end
+        robot_namespace="${namespace}"
+        x="-${tether_attached_pos_horizontal}"
+        y="${tether_attached_pos_horizontal}"
+        z="${tether_attached_pos_vertical}"
         tether_number="6"
         suffix="back_left_upper"
@@ -200,9 +212,11 @@
     <xacro:tether_end
         robot_namespace="${namespace}"
-        x="-0.2" y="0.2" z="-0.1"
+        x="-${tether_attached_pos_horizontal}"
+        y="${tether_attached_pos_horizontal}"
+        z="-${tether_attached_pos_vertical}"
         tether_number="7"
         suffix="back_left_lower"
         color="Orange">
-    </xacro:tether_end>
+    </xacro:tether_end> -->
   <!-- ================================================================== -->
   <!-- ======================== PYRAMID ROBOTICS =========================-->

Commit message: Clean up

File: pyramid_description/urdf/pyramid_multirotor_base.xacro (robot description, xacro)
@@ -154,5 +154,5 @@
                 <origin rpy="0 0 0" xyz="0 0 0"/>
                 <geometry>
-                    <sphere radius="0.01"/>
+                    <sphere radius="0.03"/>
                 </geometry>
             </visual>
@@ -160,5 +160,5 @@
                 <origin xyz="0 0 0" rpy="0 0 0" />
                 <geometry>
-                    <sphere radius="0.01"/>
+                    <sphere radius="0.03"/>
                 </geometry>
             </collision>

File: pyramid_description/urdf/pyramid_winch.xacro (robot description, xacro)
@@ -20,4 +20,9 @@
             </visual>
         </link>
+        <gazebo>
+            <plugin filename="libgazebo_winch_plugin.so" name="winch_plugin">
+                <linkName>winch_${winch_number}</linkName>
+            </plugin>
+        </gazebo>
         <gazebo reference="winch_${winch_number}">
             <material>Gazebo/${color}</material>

Commit message: Refactoring

File: pyramid_description/urdf/pyramid_multirotor_base.xacro (robot description, xacro)
@@ -71,5 +71,5 @@
         <rotorVelocitySlowdownSim>${rotor_velocity_slowdown_sim}</rotorVelocitySlowdownSim>
       </plugin>
-      <!--plugin filename="libgazebo_disturbance_plugin.so" name="disturbance_plugin" /-->
+      <plugin filename="libgazebo_disturbance_plugin.so" name="disturbance_plugin" />
       <!-- <plugin filename="libgazebo_external_force_plugin.so" name="external_force_plugin" /> -->
       <!-- <plugin filename="libgazebo_psuedo_tether_plugin.so" name="psuedo_tether_plugin" /> -->
@@ -147,6 +147,6 @@
         <link name="${robot_namespace}/tether_end_${tether_number}">
             <inertial>
-                <mass value="0.01"/>
-                <inertia ixx="0.01" iyy="0.01" izz="0.01" ixy="0.0" ixz="0.0" iyz="0.0"/>
+                <mass value="0.0001"/>
+                <inertia ixx="0.0001" iyy="0.0001" izz="0.0001" ixy="0.0" ixz="0.0" iyz="0.0"/>
                 <origin xyz="0 0 0" rpy="0 0 0"/>
             </inertial>

Commit message: Modify

File: pyramid_description/urdf/pyramid_multirotor_base.xacro (robot description, xacro)
@@ -147,6 +147,6 @@
         <link name="${robot_namespace}/tether_end_${tether_number}">
             <inertial>
-                <mass value="0.0001"/>
-                <inertia ixx="0.0001" iyy="0.0001" izz="0.0001" ixy="0.0" ixz="0.0" iyz="0.0"/>
+                <mass value="0.00001"/>
+                <inertia ixx="0.00001" iyy="0.00001" izz="0.00001" ixy="0.0" ixz="0.0" iyz="0.0"/>
                 <origin xyz="0 0 0" rpy="0 0 0"/>
             </inertial>
